File: AMS-board-2024/CAN-transceiver.kicad_sch (KiCad schematic)
At the start: 7 parts, among them U1201 TCAN1042DQ1

Commit message: 修正
アノテーション方法の変更：最初の空き番号から使用
Parts:
- renumbered C1202 to C276, C1201 to C277, D1201 to D105, R1203 to R545, R1201 to R546, R1202 to R547, U1201 to U11
Changed lines of the file:
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@@
   (symbol (lib_id "ProjectEV:PowerProtection_NUP2105L") (at 165.1 114.3 0) (unit 1)
     (in_bom yes) (on_board yes) (dnp no) (fields_autoplaced)
-    (property "Reference" "D1201" (at 171.45 113.03 0)
+    (property "Reference" "D105" (at 171.45 113.03 0)
       (effects (font (size 1.27 1.27)) (justify left))
     )
@@
       (project "AMS-board-2024"
         (path "/3a719eb3-09ce-4343-8f6e-20cc0aaf5261/6c88c007-deae-4ed6-a37c-9d5c4c750b8f/bdebf2e5-9545-4c56-a02d-4de56fc97c11"
-          (reference "D1201") (unit 1)
+          (reference "D105") (unit 1)
         )
       )
@@
   (symbol (lib_id "power:GND") (at 104.14 78.74 0) (unit 1)
     (in_bom yes) (on_board yes) (dnp no) (fields_autoplaced)
-    (property "Reference" "#PWR01202" (at 104.14 85.09 0)
+    (property "Reference" "#PWR014" (at 104.14 85.09 0)
       (effects (font (size 1.27 1.27)) hide)
     )
@@
       (project "AMS-board-2024"
         (path "/3a719eb3-09ce-4343-8f6e-20cc0aaf5261/6c88c007-deae-4ed6-a37c-9d5c4c750b8f/bdebf2e5-9545-4c56-a02d-4de56fc97c11"
-          (reference "#PWR01202") (unit 1)
+          (reference "#PWR014") (unit 1)
         )
       )
@@
   (symbol (lib_id "Device:R") (at 152.4 82.55 0) (unit 1)
     (in_bom yes) (on_board yes) (dnp no) (fields_autoplaced)
-    (property "Reference" "R1201" (at 154.94 81.28 0)
+    (property "Reference" "R546" (at 154.94 81.28 0)
       (effects (font (size 1.27 1.27)) (justify left))
     )
@@
       (project "AMS-board-2024"
         (path "/3a719eb3-09ce-4343-8f6e-20cc0aaf5261/6c88c007-deae-4ed6-a37c-9d5c4c750b8f/bdebf2e5-9545-4c56-a02d-4de56fc97c11"
-          (reference "R1201") (unit 1)
+          (reference "R546") (unit 1)
         )
       )
@@
   (symbol (lib_id "power:VCC") (at 114.3 67.31 0) (unit 1)
     (in_bom yes) (on_board yes) (dnp no) (fields_autoplaced)
-    (property "Reference" "#PWR01201" (at 114.3 71.12 0)
+    (property "Reference" "#PWR015" (at 114.3 71.12 0)
       (effects (font (size 1.27 1.27)) hide)
     )
@@
       (project "AMS-board-2024"
         (path "/3a719eb3-09ce-4343-8f6e-20cc0aaf5261/6c88c007-deae-4ed6-a37c-9d5c4c750b8f/bdebf2e5-9545-4c56-a02d-4de56fc97c11"
-          (reference "#PWR01201") (unit 1)
+          (reference "#PWR015") (unit 1)
         )
       )
@@
   (symbol (lib_id "power:GND") (at 101.6 104.14 0) (unit 1)
     (in_bom yes) (on_board yes) (dnp no) (fields_autoplaced)
-    (property "Reference" "#PWR01204" (at 101.6 110.49 0)
+    (property "Reference" "#PWR013" (at 101.6 110.49 0)
       (effects (font (size 1.27 1.27)) hide)
     )
@@
       (project "AMS-board-2024"
         (path "/3a719eb3-09ce-4343-8f6e-20cc0aaf5261/6c88c007-deae-4ed6-a37c-9d5c4c750b8f/bdebf2e5-9545-4c56-a02d-4de56fc97c11"
-          (reference "#PWR01204") (unit 1)
+          (reference "#PWR013") (unit 1)
         )
       )
@@
   (symbol (lib_id "Device:C") (at 146.05 88.9 90) (unit 1)
     (in_bom yes) (on_board yes) (dnp no) (fields_autoplaced)
-    (property "Reference" "C1201" (at 146.05 81.28 90)
+    (property "Reference" "C277" (at 146.05 81.28 90)
       (effects (font (size 1.27 1.27)))
     )
@@
       (project "AMS-board-2024"
         (path "/3a719eb3-09ce-4343-8f6e-20cc0aaf5261/6c88c007-deae-4ed6-a37c-9d5c4c750b8f/bdebf2e5-9545-4c56-a02d-4de56fc97c11"
-          (reference "C1201") (unit 1)
+          (reference "C277") (unit 1)
         )
       )
@@
   (symbol (lib_id "power:GND") (at 114.3 99.06 0) (unit 1)
     (in_bom yes) (on_board yes) (dnp no) (fields_autoplaced)
-    (property "Reference" "#PWR01203" (at 114.3 105.41 0)
+    (property "Reference" "#PWR016" (at 114.3 105.41 0)
       (effects (font (size 1.27 1.27)) hide)
     )
@@
       (project "AMS-board-2024"
         (path "/3a719eb3-09ce-4343-8f6e-20cc0aaf5261/6c88c007-deae-4ed6-a37c-9d5c4c750b8f/bdebf2e5-9545-4c56-a02d-4de56fc97c11"
-          (reference "#PWR01203") (unit 1)
+          (reference "#PWR016") (unit 1)
         )
       )
@@
   (symbol (lib_id "power:GND") (at 139.7 88.9 270) (unit 1)
     (in_bom yes) (on_board yes) (dnp no) (fields_autoplaced)
-    (property "Reference" "#PWR01205" (at 133.35 88.9 0)
+    (property "Reference" "#PWR017" (at 133.35 88.9 0)
       (effects (font (size 1.27 1.27)) hide)
     )
@@
       (project "AMS-board-2024"
         (path "/3a719eb3-09ce-4343-8f6e-20cc0aaf5261/6c88c007-deae-4ed6-a37c-9d5c4c750b8f/bdebf2e5-9545-4c56-a02d-4de56fc97c11"
-          (reference "#PWR01205") (unit 1)
+          (reference "#PWR017") (unit 1)
         )
       )
@@
   (symbol (lib_id "Device:C") (at 104.14 73.66 0) (unit 1)
     (in_bom yes) (on_board yes) (dnp no) (fields_autoplaced)
-    (property "Reference" "C1202" (at 107.95 72.39 0)
+    (property "Reference" "C276" (at 107.95 72.39 0)
       (effects (font (size 1.27 1.27)) (justify left))
     )
@@
       (project "AMS-board-2024"
         (path "/3a719eb3-09ce-4343-8f6e-20cc0aaf5261/6c88c007-deae-4ed6-a37c-9d5c4c750b8f/bdebf2e5-9545-4c56-a02d-4de56fc97c11"
-          (reference "C1202") (unit 1)
+          (reference "C276") (unit 1)
         )
       )
@@
   (symbol (lib_id "ProjectEV:Interface_TCAN1042DQ1") (at 114.3 88.9 0) (unit 1)
     (in_bom yes) (on_board yes) (dnp no)
-    (property "Reference" "U1201" (at 115.57 78.74 0)
+    (property "Reference" "U11" (at 115.57 78.74 0)
       (effects (font (size 1.27 1.27)) (justify left))
     )
@@
       (project "AMS-board-2024"
         (path "/3a719eb3-09ce-4343-8f6e-20cc0aaf5261/6c88c007-deae-4ed6-a37c-9d5c4c750b8f/bdebf2e5-9545-4c56-a02d-4de56fc97c11"
-          (reference "U1201") (unit 1)
+          (reference "U11") (unit 1)
         )
       )
@@
   (symbol (lib_id "power:GND") (at 165.1 121.92 0) (unit 1)
     (in_bom yes) (on_board yes) (dnp no) (fields_autoplaced)
-    (property "Reference" "#PWR01206" (at 165.1 128.27 0)
+    (property "Reference" "#PWR018" (at 165.1 128.27 0)
       (effects (font (size 1.27 1.27)) hide)
     )
@@
       (project "AMS-board-2024"
         (path "/3a719eb3-09ce-4343-8f6e-20cc0aaf5261/6c88c007-deae-4ed6-a37c-9d5c4c750b8f/bdebf2e5-9545-4c56-a02d-4de56fc97c11"
-          (reference "#PWR01206") (unit 1)
+          (reference "#PWR018") (unit 1)
         )
       )
@@
   (symbol (lib_id "Device:R") (at 101.6 97.79 0) (unit 1)
     (in_bom yes) (on_board yes) (dnp no) (fields_autoplaced)
-    (property "Reference" "R1203" (at 104.14 96.52 0)
+    (property "Reference" "R545" (at 104.14 96.52 0)
       (effects (font (size 1.27 1.27)) (justify left))
     )
@@
       (project "AMS-board-2024"
         (path "/3a719eb3-09ce-4343-8f6e-20cc0aaf5261/6c88c007-deae-4ed6-a37c-9d5c4c750b8f/bdebf2e5-9545-4c56-a02d-4de56fc97c11"
-          (reference "R1203") (unit 1)
+          (reference "R545") (unit 1)
         )
       )
@@
   (symbol (lib_id "Device:R") (at 152.4 95.25 0) (unit 1)
     (in_bom yes) (on_board yes) (dnp no) (fields_autoplaced)
-    (property "Reference" "R1202" (at 154.94 93.98 0)
+    (property "Reference" "R547" (at 154.94 93.98 0)
       (effects (font (size 1.27 1.27)) (justify left))
     )
@@
       (project "AMS-board-2024"
         (path "/3a719eb3-09ce-4343-8f6e-20cc0aaf5261/6c88c007-deae-4ed6-a37c-9d5c4c750b8f/bdebf2e5-9545-4c56-a02d-4de56fc97c11"
-          (reference "R1202") (unit 1)
-        )
-      )
+          (reference "R547") (unit 1)
+        )
+      )
