File: AMS-board-2024/SPI-2-wire-interface.kicad_sch (KiCad schematic)
At the start: 13 parts, among them U1101 LTC6820

Commit message: 修正
GNDが抜けていたので追加
Connections:
- net GND: now also C1101.1, C1102.1
Changed lines of the file:
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@@
+    (stroke (width 0) (type default))
+  )
+  (wire (pts (xy 177.8 127) (xy 180.34 127))
     (stroke (width 0) (type default))
   )
@@
   )
   (wire (pts (xy 142.24 88.9) (xy 142.24 86.36))
+    (stroke (width 0) (type default))
+  )
+  (wire (pts (xy 228.6 127) (xy 231.14 127))
     (stroke (width 0) (type default))
   )
@@
     )
   )
+  (symbol (lib_id "power:GND") (at 177.8 127 270) (unit 1)
+    (in_bom yes) (on_board yes) (dnp no) (fields_autoplaced)
+    (property "Reference" "#PWR01111" (at 171.45 127 0)
+      (effects (font (size 1.27 1.27)) hide)
+    )
+    (property "Value" "GND" (at 173.99 127 90)
+      (effects (font (size 1.27 1.27)) (justify right))
+    )
+    (property "Footprint" "" (at 177.8 127 0)
+      (effects (font (size 1.27 1.27)) hide)
+    )
+    (property "Datasheet" "" (at 177.8 127 0)
+      (effects (font (size 1.27 1.27)) hide)
+    )
+    (pin "1")
+    (instances
+      (project "AMS-board-2024"
+        (path "/3a719eb3-09ce-4343-8f6e-20cc0aaf5261/6c88c007-deae-4ed6-a37c-9d5c4c750b8f/e78e9a17-6dfa-4790-b63f-83a7a3017fa5"
+          (reference "#PWR01111") (unit 1)
+        )
+      )
+    )
+  )
   (symbol (lib_id "power:VCC") (at 88.9 80.01 0) (unit 1)
     (in_bom yes) (on_board yes) (dnp no) (fields_autoplaced)
@@
         )
       )
+    )
+  )
+  (symbol (lib_id "power:GND") (at 228.6 127 270) (unit 1)
+    (in_bom yes) (on_board yes) (dnp no) (fields_autoplaced)
+    (property "Reference" "#PWR01112" (at 222.25 127 0)
+      (effects (font (size 1.27 1.27)) hide)
+    )
+    (property "Value" "GND" (at 224.79 127 90)
+      (effects (font (size 1.27 1.27)) (justify right))
+    )
+    (property "Footprint" "" (at 228.6 127 0)
+      (effects (font (size 1.27 1.27)) hide)
+    )
+    (property "Datasheet" "" (at 228.6 127 0)
+      (effects (font (size 1.27 1.27)) hide)
+    )
+    (pin "1")
+    (instances
+      (project "AMS-board-2024"
+        (path "/3a719eb3-09ce-4343-8f6e-20cc0aaf5261/6c88c007-deae-4ed6-a37c-9d5c4c750b8f/e78e9a17-6dfa-4790-b63f-83a7a3017fa5"
+          (reference "#PWR01112") (unit 1)
+        )
+      )

Commit message: 修正
アノテーション方法の変更：最初の空き番号から使用
Parts:
- renumbered C1103 to C273, C1101 to C274, C1102 to C275, FL1101 to FL17, R1101 to R537, R1102 to R538, R1107 to R539, R1108 to R540, R1103 to R541, R1104 to R542, R1105 to R543, R1106 to R544, U1101 to U10
