File: AMS-board-2024/MCU.kicad_sch (KiCad schematic)
At the start: 1 part, among them U1001 R7FA4M1AB3CFM#AA0

Commit message: シート追加
CANトランシーバ回路
Other:
- added sheet CAN Transceiver (CAN-transceiver.kicad_sch)
Changed lines of the file:
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@@
+    )
+  )
+  (sheet (at 50.8 76.2) (size 12.7 12.7) (fields_autoplaced)
+    (stroke (width 0.1524) (type solid))
+    (fill (color 0 0 0 0.0000))
+    (property "Sheetname" "CAN Transceiver" (at 50.8 75.4884 0)
+      (effects (font (size 1.27 1.27)) (justify left bottom))
+    )
+    (property "Sheetfile" "CAN-transceiver.kicad_sch" (at 50.8 89.4846 0)
+      (effects (font (size 1.27 1.27)) (justify left top))
+    )
+    (pin "TXD" input (at 50.8 78.74 180)
+      (effects (font (size 1.27 1.27)) (justify left))
+    )
+    (pin "RXD" output (at 50.8 86.36 180)
+      (effects (font (size 1.27 1.27)) (justify left))
+    )
+    (pin "CANH" bidirectional (at 63.5 78.74 0)
+      (effects (font (size 1.27 1.27)) (justify right))
+    )
+    (pin "CANL" bidirectional (at 63.5 86.36 0)
+      (effects (font (size 1.27 1.27)) (justify right))
+    )
+    (instances
+      (project "AMS-board-2024"
+        (path "/3a719eb3-09ce-4343-8f6e-20cc0aaf5261/6c88c007-deae-4ed6-a37c-9d5c4c750b8f" (page "12"))
+      )
     )
   )

Commit message: 修正
アノテーション方法の変更：最初の空き番号から使用
Parts:
- renumbered U1001 to U9
Changed lines of the file:
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@@
   (symbol (lib_id "ProjectEV:MCU_R7FA4M1AB3CFM#AA0") (at 127 88.9 0) (unit 1)
     (in_bom yes) (on_board yes) (dnp no) (fields_autoplaced)
-    (property "Reference" "U1001" (at 136.8141 132.08 0)
+    (property "Reference" "U9" (at 136.8141 132.08 0)
       (effects (font (size 1.27 1.27)) (justify left))
     )
@@
       (project "AMS-board-2024"
         (path "/3a719eb3-09ce-4343-8f6e-20cc0aaf5261/6c88c007-deae-4ed6-a37c-9d5c4c750b8f"
-          (reference "U1001") (unit 1)
+          (reference "U9") (unit 1)
         )
       )

Commit message: シート削除
削除したシート内の回路はMCU.kicad_schに統合
Parts:
- added C273: C, symbol Device:C
- added C274, C275, C277: 10n, Capacitor_SMD:C_0603_1608Metric, symbol Device:C
- added C276: 0.1u, Capacitor_SMD:C_0603_1608Metric, symbol Device:C
- added D105: NUP2105L, ProjectEV:Package_SOT-23_NUP2105L, symbol ProjectEV:PowerProtection_NUP2105L
- added FL17: DLW43SH101XK2, ProjectEV:CommonModeChoke_DLW43SH101, symbol ProjectEV:CommonModeChoke_DLW43SH101
- added R537, R538, R539, R540: 1k, Resistor_SMD:R_0603_1608Metric, symbol Device:R
- added R541, R542, R546, R547: 60.4, Resistor_SMD:R_0603_1608Metric, symbol Device:R
- added R543, R544: 294, Resistor_SMD:R_0603_1608Metric, symbol Device:R
- added R545: 15k, Resistor_SMD:R_0603_1608Metric, symbol Device:R
- added U10: LTC6820, ProjectEV:Package_MSOP-16_3x4.039mm_P0.5mm_LTC6820, symbol ProjectEV:Interface_LTC6820
- added U11: TCAN1042DQ1, ProjectEV:Package_SOIC-8_3.9x4.9mm_P1.27mm, symbol ProjectEV:Interface_TCAN1042DQ1
Connections:
- net at U9.34 (P109/TDO/SWO): now also R537.2, U10.2 (MOSI)
- net at U9.35 (P110/TDI): now also R538.2, U10.3 (MISO)
- net at U9.36 (P111): now also U10.4 (SCK)
- net at U9.37 (P112): now also U10.5 (~{CS})
- net at U9.45 (P103): now also U11.1 (TXD)
- net at U9.46 (P102): now also U11.4 (RXD)
- new net: C274.2, R541.1, R542.2
- new net: C277.2, R546.2, R547.1
- new net: FL17.1, R542.1, U10.10 (IM)
- new net: FL17.4, R541.2, U10.11 (IP)
- new net: R539.1, R540.2, U10.15 (ICMP)
- new net: R540.1, U10.16 (IBIAS)
- new net: C275.2, R543.1, R544.2
- new net: R545.1, U11.8 (STB)
- new net CANH: D105.2 (K), R546.1, U11.7 (CANH)
- new net CANL: D105.1 (K), R547.2, U11.6 (CANL)
- new net GND: C273.2, C274.1, C275.1, C276.2, C277.1, D105.3 (A), R539.2, R545.2, U10.1 (EN), U10.13 (SLOW), U10.14 (GND), U11.2 (GND)
- new net IM: FL17.2, R544.1
- new net IP: FL17.3, R543.2
- new net VCC: C273.1, C276.1, R537.1, R538.1, U10.12 (MSTR), U10.6 (VDDS), U10.7 (POL), U10.8 (PHA), U10.9 (VDD), U11.3 (VCC)
Other:
- removed sheet CAN Transceiver
- removed sheet SPI 2-wire Interface
- moved on the sheet: U9

Commit message: CANにコモンモードチョーク追加
Parts:
- added FL18: DLW43SH101XK2, ProjectEV:CommonModeChoke_DLW43SH101, symbol ProjectEV:CommonModeChoke_DLW43SH101
Connections:
- net CANH: now also FL17.3; no longer U11.7 (CANH)
- net CANL: now also FL17.2; no longer U11.6 (CANL)
- net IM: now also FL18.2; no longer FL17.2
- net IP: now also FL18.3; no longer FL17.3
- net at R542.1, U10.10 (IM): now also FL18.1; no longer FL17.1
- net at R541.2, U10.11 (IP): now also FL18.4; no longer FL17.4
- new net: FL17.1, U11.6 (CANL)
- new net: FL17.4, U11.7 (CANH)
Other:
- moved on the sheet: C277, D105, FL17, R546, R547

Commit message: リセット、MD等周辺回路の追加
Parts:
- added C278, C279, C280, C281, C284: 0.1u, Capacitor_SMD:C_0603_1608Metric, symbol Device:C
- added C282, C283: 4.7u, Capacitor_SMD:C_0805_2012Metric, symbol Device:C
- added C285, C286: 8p, Capacitor_SMD:C_0402_1005Metric, symbol Device:C
- added R548, R549, R550, R551, R552, R555: 15k, Resistor_SMD:R_0603_1608Metric, symbol Device:R
- added R553: 100k, Resistor_SMD:R_0603_1608Metric, symbol Device:R
- added R554: 13.7k, Resistor_SMD:R_0603_1608Metric, symbol Device:R
- added SW1: DS04-254-01BK-SMT, ProjectEV:SW_DS04-254-01BK-SMT, symbol ProjectEV:SW_DS04-254-2-01BK-SMT
- added SW2: PTS636-SL43-SMTR, ProjectEV:SW_PTS636-43-SMTR, symbol ProjectEV:SW_PTS636-43-SMTR
- added Y1: ABM8W, ProjectEV:Crystal_ABM8W, symbol ProjectEV:Crystal_ABM8W
Connections:
- net GND: now also U9.17 (VSS_USB), U9.40 (VSS_2), U9.57 (AVSS0), U9.8 (VSS_1), C278.1, C279.1, C280.1, C281.1, C282.1, C283.2, C284.1, C285.2, C286.2, R552.2, R554.2, SW1.2, SW2.2, Y1.2, Y1.4
- net VCC: now also R548.1, R549.1, R550.1, R553.1, R555.1
- net at U9.10 (P212/EXTAL): now also C286.1, Y1.1
- net +5V: now reaches U9.11 (VCC_1)
- net +5V: now also U9.21 (VCC_USB_LDO), U9.39 (VCC_2), C278.2, C279.2, C284.2
- net at U9.16 (P407): now also R550.2, R551.1
- net USB_DN: now reaches U9.18 (P915/USB_DM)
- net USB_DP: now reaches U9.19 (P914/USB_DP)
- net +3V3: now reaches U9.20 (VCC_USB)
- net +3V3: now also U9.4 (VBATT), C281.2, C282.2
- net at U9.25 (RES): now also R549.2, SW2.1
- net at U9.26 (P201/MD): now also R548.2, SW1.1
- net at U9.27 (P200): now also R555.2
- net at U9.49 (P500): now also R553.2, R554.1
- net at U9.5 (VCL): now also C283.1
- net +5VA: now reaches U9.56 (AVCC0)
- net +5VA: now also C280.2
- net at U9.9 (P213/XTAL): now also C285.1, Y1.3
- new net: R551.2, R552.1
- no-connect marks 0 -> 8

Commit message: 微修正
Connections:
- net USB_DN: no longer U9.18 (P915/USB_DM)
- net USB_DP: no longer U9.19 (P914/USB_DP)
Other:
- moved on the sheet: C273, C274, C275, C276, C277, D105, FL17, FL18, R537, R538, R539, R540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

Commit message: USBアイソレータ追加
Parts:
- removed R551, R552: 15k, Resistor_SMD:R_0603_1608Metric, symbol Device:R
- added C287, C288, C289, C290: 0.1u, Capacitor_SMD:C_0603_1608Metric, symbol Device:C
- added R556, R557, R558, R559: 24, Resistor_SMD:R_0603_1608Metric, symbol Device:R
- added U12: ADUM3160, ProjectEV:Package_SOIC-16W_7.5x10.3mm_P1.27mm, symbol ProjectEV:Interface_ADUM3160
Connections:
- net GND: now also R550.2, C289.1, C290.2, U12.15 (GND2), U12.9 (GND2)
- net VCC: now also C289.2, U12.16 (VBUS2); no longer R550.1
- net USB_VBUS: now reaches U9.16 (P407)
- net USB_VBUS: now also R550.1, C290.1, U12.12 (PIN), U12.13 (SPD), U12.14 (VDD2); no longer R550.2
- net at U9.18 (P915/USB_DM): now also R558.2
- net at U9.19 (P914/USB_DP): now also R559.2
- new net: R557.2, U12.6 (UD-)
- new net: R558.1, U12.11 (DD-)
- new net: R559.1, U12.10 (DD+)
- new net: C287.2, U12.3 (VDD1), U12.4 (PDEN), U12.5 (SPU)
- new net: R556.2, U12.7 (UD+)
- new net GNDD: C287.1, C288.1, U12.2 (GND1), U12.8 (GND1)
- new net USB_UDN: R557.1
- new net USB_UDP: R556.1
- new net VBUS: C288.2, U12.1 (VBUS1)

Commit message: LEDとそのドライバ追加
Parts:
- added D109, D110, D112: LED, LED_SMD:LED_0603_1608Metric, symbol Device:LED
- added D111: DRTR5V0U2SR, ProjectEV:Package_SOT-143_DRTR5V0U2SR, symbol ProjectEV:TVS_DRTR5V0U2SR
- added Q107, Q108, Q109: 2N7002K-AU, ProjectEV:Package_SOT-23_2N7002K-AU, symbol ProjectEV:Transistor_2N7002K-AU
- added R600, R605, R608: 5.1k, Resistor_SMD:R_0603_1608Metric, symbol Device:R
- added R601, R602, R606: 100, Resistor_SMD:R_0603_1608Metric, symbol Device:R
- added R603, R604, R607: 1M, Resistor_SMD:R_0603_1608Metric, symbol Device:R
Connections:
- net GND: now also D109.1 (K), D110.1 (K), Q107.2 (S), Q108.2 (S), Q109.2 (S), R603.1, R604.1, R607.1
- net GNDD: now also D111.1
- net USB_UDN: now also D111.2
- net USB_UDP: now also D111.3
- net VBUS: now also D111.4
- net VCC: now also R600.1, R605.1, R608.1; no longer C289.2, U12.16 (VBUS2)
- net P109_D11_MOSI: now reaches R537.2, U10.2 (MOSI), U9.34 (P109/TDO/SWO)
- net USB_DDN: now reaches R558.2, U9.18 (P915/USB_DM)
- net P110_D12_MISO: now reaches R538.2, U10.3 (MISO), U9.35 (P110/TDI)
- net P111_D13_SCK: now reaches U10.4 (SCK), U9.36 (P111)
- net P112_D10_~{CS}: now reaches U10.5 (~{CS}), U9.37 (P112)
- net USB_DDP: now reaches R559.2, U9.19 (P914/USB_DP)
- net P304_D8: now reaches U9.28 (P304)
- net P303_D9: now reaches U9.29 (P303)
- net P107_D7: now reaches U9.41 (P107)
- net P106_D6: now reaches U9.42 (P106)
- net P105_D2: now reaches U9.43 (P105)
- net P104_D3: now reaches U9.44 (P104)
- net P103_D4_CAN_TX: now reaches U11.1 (TXD), U9.45 (P103)
- net P102_D5_CAN_RX: now reaches U11.4 (RXD), U9.46 (P102)
- net P013: now reaches U9.54 (P013/VREFL)
- net P013: now also R601.1
- net P012: now reaches U9.55 (P012/VREFH)
- net P012: now also R602.1
- new net: D110.2 (A), Q108.3 (D), R605.2
- new net: Q107.1 (G), R602.2, R603.2
- new net: D109.2 (A), Q107.3 (D), R600.2
- new net: Q108.1 (G), R601.2, R604.2
- new net: D112.1 (K), Q109.3 (D)
- new net: D112.2 (A), R608.2
- new net: Q109.1 (G), R606.2, R607.2
- new net VCCQ: C289.2, U12.16 (VBUS2)
