File: AMS-board-2024/MCU.kicad_sch (KiCad schematic)
At the start: 65 parts, among them Q107 2N7002K-AU, Q108 2N7002K-AU, Q109 2N7002K-AU, SW1 DS04-254-01BK-SMT, SW2 PTS636-SL43-SMTR, U10 LTC6820, U11 TCAN1042DQ1, U12 ADUM3160, U9 R7FA4M1AB3CFM#AA0, Y1 ABM8W

Commit message: デジタルI/O入出力回路追加
Parts:
- added C355, C356, C357, C358, C359, C360: 0.1u, Capacitor_SMD:C_0603_1608Metric, symbol Device:C
- added D117, D118, D119, D120, D121, D122, D123, D124: BAT46W-7-F, ProjectEV:D_SOD-123_BAT46W-7-F, symbol ProjectEV:D_BAT46W-7-F
- added R609 (x8): 100k, Resistor_SMD:R_0603_1608Metric, symbol Device:R
- added R633, R635, R637, R639: 100, Resistor_SMD:R_0603_1608Metric, symbol Device:R
- added R634, R636, R638, R640: 1M, Resistor_SMD:R_0603_1608Metric, symbol Device:R
- added U13, U19: TPS2561-Q1, ProjectEV:Package_VSON-10-1EP_3x3mm_TPS2561-Q1, symbol ProjectEV:Power_TPS2561-Q1
Connections:
- net +5V: now also C273.1, C276.1, R537.1, R538.1, R548.1, R549.1, R553.1, R555.1, U10.12 (MSTR), U10.6 (VDDS), U10.7 (POL), U10.8 (PHA), U10.9 (VDD), U11.3 (VCC), C355.1, C356.1, D117.1 (K), D119.1 (K), D121.1 (K), D123.1 (K), U13.2 (IN), U13.3 (IN), U19.2 (IN), U19.3 (IN)
- net GND: now also C355.2, C356.2, C357.2, C358.2, C359.2, C360.2, D118.2 (A), D120.2 (A), D122.2 (A), D124.2 (A), R609.2, R609.2, R609.2, R609.2, R634.1, R636.1, R638.1, R640.1, U13.1 (GND), U13.11 (PAD), U19.1 (GND), U19.11 (PAD)
- net P104_D3: now also D117.2 (A), D118.1 (K), R633.2, R634.2
- net P105_D2: now also D119.2 (A), D120.1 (K), R635.2, R636.2
- net P106_D6: now also D121.2 (A), D122.1 (K), R637.2, R638.2
- net P107_D7: now also D123.2 (A), D124.1 (K), R639.2, R640.2
- net P301_RXD_D0: now also R609.1
- net P302_TXD_D1: now also R609.1
- net P303_D9: now also R609.1
- net P304_D8: now also R609.1
- net VCC: no longer C273.1, C276.1, R537.1, R538.1, R548.1, R549.1, R553.1, R555.1, U10.12 (MSTR), U10.6 (VDDS), U10.7 (POL), U10.8 (PHA), U10.9 (VDD), U11.3 (VCC)
- net ~{RESET}: now reaches R549.2, SW2.1, U9.25 (RES)
- new net: C359.1, C360.1, R609.2, U19.10 (~{FAULT1}), U19.4 (EN1)
- new net: R609.1, R609.1, U13.7 (ILIM)
- new net: R609.2, U19.5 (EN2), U19.6 (~{FAULT2})
- new net: R609.1, R609.1, U19.7 (ILIM)
- new net: C357.1, R609.2, U13.5 (EN2), U13.6 (~{FAULT2})
- new net: C358.1, R609.2, U13.10 (~{FAULT1}), U13.4 (EN1)
- new net D0: U13.9 (OUT1)
- new net D1: U13.8 (OUT2)
- new net D2: R635.1
- new net D3: R633.1
- new net D6: R637.1
- new net D7: R639.1
- new net D8: U19.8 (OUT2)
- new net D9: U19.9 (OUT1)
Other:
- note added: "I_{LIMIT} = 1 ~ 1.2 A"
- moved on the sheet: C273, C274, C275, C276, C277, C287, C288, C289, C290, D105, D111, FL17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

Commit message: パワーオンリセット回路追加
Parts:
- added C361: 0.1u, Capacitor_SMD:C_0603_1608Metric, symbol Device:C
- added C362: 1000p, Capacitor_SMD:C_0603_1608Metric, symbol Device:C
- added C363: 10u, Capacitor_SMD:C_0603_1608Metric, symbol Device:C
- added U20: BD5230G-2MTR, ProjectEV:Package_SSOP-5_1.6x2.9mm_P0.95mm, symbol ProjectEV:Power_BD5230
- R549: value 15k -> 100k
- U13, U19: value TPS2561-Q1 -> TPS2561QDRCRQ1
- renumbered R609 to R625, R609 to R626, R609 to R627, R609 to R628, R609 to R629, R609 to R630, R609 to R631, R609 to R632
Connections:
- net +5V: now also C363.1, U20.2 (VDD)
- net GND: now also C361.2, C362.2, C363.2, U20.3 (GND)
- net ~{RESET}: now also C362.1, U20.1 (VOUT)
- new net: C361.1, U20.5 (CT)

Commit message: マイコン周辺回路完成
入力保護、温度センサ、EEPROMなど
Parts:
- removed R634: 1M, Resistor_SMD:R_0603_1608Metric, symbol Device:R
- added C319, C323, C324, C343, C344: 0.1u, Capacitor_SMD:C_0603_1608Metric, symbol Device:C
- added D111, D112, D115, D116: BAT46W-7-F, ProjectEV:D_SOD-123_BAT46W-7-F, symbol ProjectEV:D_BAT46W-7-F
- added D122: LED, LED_SMD:LED_0603_1608Metric, symbol Device:LED
- added Q108: 2N7002K-AU, ProjectEV:Package_SOT-23_2N7002K-AU, symbol ProjectEV:Transistor_2N7002K-AU
- added R584, R597, R598, R631: 100, Resistor_SMD:R_0603_1608Metric, symbol Device:R
- added R588, R600, R601, R632: 1M, Resistor_SMD:R_0603_1608Metric, symbol Device:R
- added R614, R620: 5.1k, Resistor_SMD:R_0603_1608Metric, symbol Device:R
- added R622, R623: 15k, Resistor_SMD:R_0603_1608Metric, symbol Device:R
- added U14: TMP101-Q1, ProjectEV:Package_SOT-23-6_TMP101-Q1, symbol ProjectEV:Sensor_TMP101-Q1
- added U15: NV24C16SNVLT3G, ProjectEV:Package_TSOP-5_NV24C16SNVLT3G, symbol ProjectEV:Memory_NV24C16SNVLT3G
- R633: value 100 -> 5.1k
- renumbered C275 to C313, C277 to C314, C287 to C315, C274 to C316, C288 to C317, C289 to C318, C276 to C320, C290 to C321, C273 to C322, C281 to C325, C283 to C326, C284 to C327, C279 to C328, C363 to C329, C361 to C330, C280 to C331, C282 to C332, C278 to C333, C362 to C334, C286 to C335, C285 to C336, C358 to C337, C359 to C338, C357 to C339, C360 to C340, C355 to C341, C356 to C342, D119 to D106, D120 to D107, D121 to D108, D122 to D109, D111 to D110, D123 to D113, D124 to D114, D109 to D119, D110 to D120, D112 to D121, FL18 to FL17, FL17 to FL18, Q107 to Q105, Q108 to Q106, Q109 to Q107, R635 to R577, R637 to R578, R636 to R579, R638 to R580, R543 to R581, R544 to R582, R556 to R583, R557 to R585, R546 to R586, R547 to R587, R639 to R589, R640 to R590, R539 to R591, R541 to R592, R542 to R593, R540 to R594, R558 to R595, R545 to R596, R559 to R599, R537 to R602, R538 to R603, R555 to R604, R548 to R605, R550 to R606, R549 to R607, R602 to R608, R553 to R609, R554 to R610, R603 to R611, R600 to R612, R601 to R613, R604 to R615, R629 to R616, R630 to R617, R631 to R618, R632 to R619, R605 to R621, R606 to R624, R627 to R626, R607 to R627, R626 to R628, R628 to R629, R608 to R630, U11 to U10, U10 to U11, U9 to U12, U20 to U13, U13 to U16, U19 to U17, U12 to U9
Connections:
- net D3 is gone; now on net VCC: R633.1
- net +5V: now also C343.1, C344.1, D111.1 (K), D115.1 (K), R614.1, R620.1, R622.1, R623.1, U14.4 (V+), U15.4 (VCC)
- net GND: now also C319.2, C323.2, C324.2, C343.2, C344.2, D112.2 (A), D116.2 (A), D122.1 (K), Q108.2 (S), R588.1, R600.1, R601.1, R632.1
- net P000_AMP+_A1: now also C319.1, D111.2 (A), D112.1 (K), R584.2, R588.2
- net P001_AMP-_A2: now also C323.1, D115.2 (A), D116.1 (K), R597.2, R600.2
- net P002_AMPO_A3: now also D117.2 (A), D118.1 (K), C324.1, R598.2, R601.2
- net P100_SCL_A5: now also R614.2, U14.1 (SCL), U15.1 (SCL)
- net P101_SDA_A4: now also R620.2, U14.6 (SDA), U15.3 (SDA)
- net P104_D3: now also R623.2, U15.5 (WP); no longer D117.2 (A), D118.1 (K), R633.2
- net IM renamed IN
- new net: D122.2 (A), Q108.3 (D), R633.2
- new net: Q108.1 (G), R631.2, R632.2
- new net: U14.2 (GND), U14.5 (ADD0)
- new net A1: R584.1
- new net A2: R597.1
- new net A3: R598.1
- new net ~{OverTemp}: R622.2, R631.1, U14.3 (ALERT)
Other:
- moved on the sheet: C314, C320, C338, C340, C342, D105, D106, D107, D113, D114, D119, D120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

Commit message: およそ回路図完成
Parts:
- C322: value C -> 0.1u; footprint (none) -> Capacitor_SMD:C_0603_1608Metric
Changed lines of the file:
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@@
       (effects (font (size 1.27 1.27)) (justify left))
     )
-    (property "Value" "C" (at 146.05 259.08 0)
+    (property "Value" "0.1u" (at 146.05 259.08 0)
       (effects (font (size 1.27 1.27)) (justify left))
     )
-    (property "Footprint" "" (at 143.2052 261.62 0)
+    (property "Footprint" "Capacitor_SMD:C_0603_1608Metric" (at 143.2052 261.62 0)
       (effects (font (size 1.27 1.27)) hide)
     )

Commit message: 設定値記載
Parts:
- removed R628, R629: 100k, Resistor_SMD:R_0603_1608Metric, symbol Device:R
Other:
- note added: "I_{LIMIT} = 473 ~ 644 mA"
- note added: "t_{PLH} = 538 ms DCバイアス特性により変動"
- note removed: "I_{LIMIT} = 1 ~ 1.2 A"
Changed lines of the file:
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@@
   (junction (at 368.3 228.6) (diameter 0) (color 0 0 0 0)
   )
-  (junction (at 482.6 233.68) (diameter 0) (color 0 0 0 0)
-  )
   (junction (at 165.1 165.1) (diameter 0) (color 0 0 0 0)
   )
@@
   (junction (at 342.9 157.48) (diameter 0) (color 0 0 0 0)
   )
-  (junction (at 482.6 195.58) (diameter 0) (color 0 0 0 0)
-  )
   (junction (at 107.95 281.94) (diameter 0) (color 0 0 0 0)
   )
@@
   (junction (at 419.1 323.85) (diameter 0) (color 0 0 0 0)
   )
-  (junction (at 482.6 246.38) (diameter 0) (color 0 0 0 0)
-  )
-  (junction (at 482.6 182.88) (diameter 0) (color 0 0 0 0)
-  )
   (junction (at 226.06 210.82) (diameter 0) (color 0 0 0 0)
   )
@@
     (stroke (width 0) (type default))
   )
-  (wire (pts (xy 482.6 233.68) (xy 495.3 233.68))
-    (stroke (width 0) (type default))
-  )
   (wire (pts (xy 317.5 182.88) (xy 320.04 182.88))
     (stroke (width 0) (type default))
@@
     (stroke (width 0) (type default))
   )
-  (wire (pts (xy 495.3 246.38) (xy 495.3 243.84))
-    (stroke (width 0) (type default))
-  )
   (wire (pts (xy 431.8 73.66) (xy 457.2 73.66))
     (stroke (width 0) (type default))
@@
     (stroke (width 0) (type default))
   )
-  (wire (pts (xy 482.6 195.58) (xy 482.6 198.12))
-    (stroke (width 0) (type default))
-  )
   (wire (pts (xy 114.3 213.36) (xy 114.3 215.9))
     (stroke (width 0) (type default))
@@
     (stroke (width 0) (type default))
   )
-  (wire (pts (xy 482.6 195.58) (xy 482.6 193.04))
+  (wire (pts (xy 482.6 193.04) (xy 482.6 198.12))
     (stroke (width 0) (type default))
   )
@@
     (stroke (width 0) (type default))
   )
-  (wire (pts (xy 482.6 182.88) (xy 495.3 182.88))
-    (stroke (width 0) (type default))
-  )
   (wire (pts (xy 368.3 237.49) (xy 368.3 240.03))
     (stroke (width 0) (type default))
@@
     (stroke (width 0) (type default))
   )
-  (wire (pts (xy 482.6 246.38) (xy 495.3 246.38))
-    (stroke (width 0) (type default))
-  )
   (wire (pts (xy 228.6 187.96) (xy 228.6 50.8))
     (stroke (width 0) (type default))
@@
     (stroke (width 0) (type default))
   )
-  (wire (pts (xy 482.6 246.38) (xy 482.6 248.92))
+  (wire (pts (xy 482.6 243.84) (xy 482.6 248.92))
     (stroke (width 0) (type default))
   )
@@
     (stroke (width 0) (type default))
   )
-  (wire (pts (xy 495.3 195.58) (xy 482.6 195.58))
-    (stroke (width 0) (type default))
-  )
   (wire (pts (xy 264.16 185.42) (xy 266.7 185.42))
     (stroke (width 0) (type default))
   )
-  (wire (pts (xy 495.3 193.04) (xy 495.3 195.58))
-    (stroke (width 0) (type default))
-  )
   (wire (pts (xy 101.6 101.6) (xy 101.6 104.14))
     (stroke (width 0) (type default))
@@
     (stroke (width 0) (type default))
   )
-  (wire (pts (xy 495.3 182.88) (xy 495.3 185.42))
-    (stroke (width 0) (type default))
-  )
   (wire (pts (xy 177.8 264.16) (xy 177.8 276.86))
     (stroke (width 0) (type default))
@@
     (stroke (width 0) (type default))
   )
-  (wire (pts (xy 495.3 233.68) (xy 495.3 236.22))
-    (stroke (width 0) (type default))
-  )
   (wire (pts (xy 129.54 31.75) (xy 129.54 30.48))
     (stroke (width 0) (type default))
@@
     (stroke (width 0) (type default))
   )
-  (wire (pts (xy 482.6 243.84) (xy 482.6 246.38))
-    (stroke (width 0) (type default))
-  )
   (wire (pts (xy 431.8 336.55) (xy 431.8 339.09))
     (stroke (width 0) (type default))
@@
     (stroke (width 0) (type default))
   )
-  (text "I_{LIMIT} = 1 ~ 1.2 A" (at 497.84 185.42 0)
+  (text "I_{LIMIT} = 473 ~ 644 mA" (at 485.14 185.42 0)
     (effects (font (size 1.27 1.27)) (justify left bottom))
   )
-  (text "I_{LIMIT} = 1 ~ 1.2 A" (at 497.84 236.22 0)
+  (text "t_{PLH} = 538 ms\nDCバイアス特性により変動" (at 270.51 273.05 0)
+    (effects (font (size 1.27 1.27)) (justify left bottom))
+  )
+  (text "I_{LIMIT} = 473 ~ 644 mA" (at 485.14 236.22 0)
     (effects (font (size 1.27 1.27)) (justify left bottom))
   )
@@
     )
   )
-  (symbol (lib_id "Device:R") (at 495.3 189.23 0) (unit 1)
-    (in_bom yes) (on_board yes) (dnp no) (fields_autoplaced)
-    (property "Reference" "R628" (at 497.84 187.96 0)
-      (effects (font (size 1.27 1.27)) (justify left))
-    )
-    (property "Value" "100k" (at 497.84 190.5 0)
-      (effects (font (size 1.27 1.27)) (justify left))
-    )
-    (property "Footprint" "Resistor_SMD:R_0603_1608Metric" (at 493.522 189.23 90)
-      (effects (font (size 1.27 1.27)) hide)
-    )
-    (property "Datasheet" "~" (at 495.3 189.23 0)
-      (effects (font (size 1.27 1.27)) hide)
-    )
-    (pin "1")
-    (pin "2")
-    (instances
-      (project "AMS-board-2024"
-        (path "/3a719eb3-09ce-4343-8f6e-20cc0aaf5261/6c88c007-deae-4ed6-a37c-9d5c4c750b8f"
-          (reference "R628") (unit 1)
-        )
-      )
-    )
-  )
   (symbol (lib_id "Device:C") (at 262.89 133.35 0) (unit 1)
     (in_bom yes) (on_board yes) (dnp no) (fields_autoplaced)
@@
         )
       )
-    )
-  )
-  (symbol (lib_id "Device:R") (at 495.3 240.03 0) (unit 1)
-    (in_bom yes) (on_board yes) (dnp no) (fields_autoplaced)
-    (property "Reference" "R629" (at 497.84 238.76 0)
-      (effects (font (size 1.27 1.27)) (justify left))
-    )
-    (property "Value" "100k" (at 497.84 241.3 0)
-      (effects (font (size 1.27 1.27)) (justify left))
-    )
-    (property "Footprint" "Resistor_SMD:R_0603_1608Metric" (at 493.522 240.03 90)
-      (effects (font (size 1.27 1.27)) hide)
-    )
-    (property "Datasheet" "~" (at 495.3 240.03 0)
-      (effects (font (size 1.27 1.27)) hide)
-    )
-    (pin "1")
-    (pin "2")
-    (instances
-      (project "AMS-board-2024"
-        (path "/3a719eb3-09ce-4343-8f6e-20cc0aaf5261/6c88c007-deae-4ed6-a37c-9d5c4c750b8f"
-          (reference "R629") (unit 1)
-        )
-      )

Commit message: アノテーションし直し
Parts:
- renumbered C313 to C311, C314 to C312, C315 to C313, C316 to C314, C317 to C315, C318 to C316, C319 to C317, C320 to C318, C321 to C319, C322 to C320, C323 to C321, C324 to C322, C325 to C323, C326 to C324, C327 to C325, C328 to C326, C329 to C327, C330 to C328, C331 to C329, C332 to C330, C333 to C331, C334 to C332, C335 to C333, C336 to C334, C337 to C335, C338 to C336, C339 to C337, C340 to C338, C341 to C339, C342 to C340, C343 to C341, C344 to C342, D105 to D185, D106 to D186, D107 to D187, D108 to D188, D109 to D189, D110 to D190, D111 to D191, D112 to D192, D113 to D193, D114 to D194, D115 to D195, D116 to D196, D117 to D197, D118 to D198, D119 to D199, D120 to D200, D121 to D201, D122 to D202, FL17 to FL16, FL18 to FL17, R577 to R575, R578 to R576, R579 to R577, R580 to R578, R581 to R579, R582 to R580, R583 to R581, R584 to R582, R585 to R583, R586 to R584, R587 to R585, R588 to R586, R589 to R587, R590 to R588, R591 to R589, R592 to R590, R593 to R591, R594 to R592, R595 to R593, R596 to R594, R597 to R595, R598 to R596, R599 to R597, R600 to R598, R601 to R599, R602 to R600, R603 to R601, R604 to R602, R605 to R603, R606 to R604, R607 to R605, R608 to R606, R609 to R607, R610 to R608, R611 to R609, R612 to R610, R613 to R611, R614 to R612, R615 to R613, R616 to R614, R617 to R615, R618 to R616, R619 to R617, R620 to R618, R621 to R619, R622 to R620, R623 to R621, R624 to R622, R625 to R623, R626 to R624, R627 to R625, R630 to R626, R631 to R627, R632 to R628, R633 to R629

Commit message: ERC実行、修正
ラベル修正、未配線部分修正、PWR_FLAG追加
Parts:
- removed D185: NUP2105L, ProjectEV:Package_SOT-23_NUP2105L, symbol ProjectEV:PowerProtection_NUP2105L
- added C367: 1u, Capacitor_SMD:C_0603_1608Metric, symbol Device:C
- added D185: NUP2105L, ProjectEV:Package_SOT-23_NUP2105L, symbol ProjectEV:TVS_NUP2105L
- added L26, L27: BLM18PG471SN1D, ProjectEV:L_BLM18xxxxxxN1x, symbol ProjectEV:L_BLM18PG471SN1D
- added R648: 5.1k, Resistor_SMD:R_0603_1608Metric, symbol Device:R
Connections:
- net VCC is gone; now on net +5V: R610.1, R619.1, R626.1, R629.1
- net +5V: now also L27.1, R648.1
- net +5VA: now also L27.2
- net CANH: now also D185.2 (K)
- net CANL: now also D185.1 (K)
- net GND: now also U14.2 (GND), U14.5 (ADD0), U15.2 (VSS), C367.2, D185.3 (A)
- net at U12.59 (P010/VREFH0): now also C367.1, L26.2
- new net AREF: L26.1, R648.2
Other:
- moved on the sheet: C317, C321, C322, D191, D192, D195, D196, D197, D198, R582, R586, R595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

Commit message: ラベル修正
Connections:
- net AREF renamed S10_AREF
- net P000_AMP+_A1 renamed S10_P000_AMP+_A1
- net P001_AMP-_A2 renamed S10_P001_AMP-_A2
- net P002_AMPO_A3 renamed S10_P002_AMPO_A3
- net P012 renamed S10_P012
- net P013 renamed S10_P013
- net P100_SCL_A5 renamed S10_P100_SCL_A5
- net P101_SDA_A4 renamed S10_P101_SDA_A4
- net P102_D5_CAN_RX renamed S10_P102_D5_CAN_RX
- net P103_D4_CAN_TX renamed S10_P103_D4_CAN_TX
- net P104_D3 renamed S10_P104_D3
- net P105_D2 renamed S10_P105_D2
- net P106_D6 renamed S10_P106_D6
- net P107_D7 renamed S10_P107_D7
- net P109_D11_MOSI renamed S10_P109_D11_MOSI
- net P110_D12_MISO renamed S10_P110_D12_MISO
- net P111_D13_SCK renamed S10_P111_D13_SCK
- net P112_D10_~{CS} renamed S10_P112_D10_~{CS}
- net P301_RXD_D0 renamed S10_P301_RXD_D0
- net P302_TXD_D1 renamed S10_P302_TXD_D1
- net P303_D9 renamed S10_P303_D9
- net P304_D8 renamed S10_P304_D8
- net USB_DDN renamed S10_USB_DDN
- net USB_DDP renamed S10_USB_DDP
- net USB_VBUS renamed S10_USB_VBUS
- net ~{OverTemp} renamed S10_~{OverTemp}
Other:
- moved on the sheet: C367, D199, L26, L27, Q105, R606, R609, R610
