File: AMS-board-2024/MCU.kicad_sch (KiCad schematic)
At the start: 127 parts, among them Q105 2N7002K-AU, Q106 2N7002K-AU, Q107 2N7002K-AU, Q108 2N7002K-AU, SW1 DS04-254-01BK-SMT, SW2 PTS636-SL43-SMTR, U10 TCAN1042DQ1, U11 LTC6820, U12 R7FA4M1AB3CFM#AA0, U13 BD5230G-2MTR, U14 TMP101-Q1, U15 NV24C16SNVLT3G, U16 TPS2561QDRCRQ1, U17 TPS2561QDRCRQ1, U9 ADUM3160, Y1 ABM8W

Commit message: アノテーションし直し
Parts:
- renumbered C311 to C312, C312 to C313, C313 to C314, C317 to C315, C314 to C316, C315 to C317, C316 to C318, C318 to C319, C319 to C320, C320 to C321, C321 to C322, C322 to C323, C367 to C324, C323 to C325, C324 to C326, C325 to C327, C326 to C328, C327 to C329, C328 to C330, C329 to C331, C330 to C332, C331 to C333, C332 to C334, C333 to C335, C334 to C336, C335 to C337, C336 to C338, C337 to C339, C338 to C340, C339 to C341, C340 to C342, C341 to C343, C342 to C344, L27 to L26, L26 to L27, R575 to R577, R576 to R578, R577 to R579, R578 to R580, R582 to R581, R579 to R582, R580 to R583, R586 to R584, R581 to R585, R583 to R586, R584 to R587, R585 to R588, R587 to R589, R588 to R590, R589 to R591, R590 to R592, R591 to R593, R592 to R594, R598 to R597, R599 to R598, R593 to R599, R594 to R600, R597 to R601, R600 to R602, R601 to R603, R648 to R604, R602 to R605, R603 to R606, R604 to R607, R605 to R608, R606 to R609, R609 to R610, R607 to R611, R608 to R612, R610 to R613, R611 to R614, R612 to R615, R613 to R616, R614 to R617, R615 to R618, R616 to R619, R617 to R620, R618 to R621, R619 to R622, R620 to R623, R621 to R624, R622 to R625, R623 to R626, R624 to R627, R625 to R628, R626 to R629, R627 to R630, R628 to R631, R629 to R632

Commit message: 階層シート内の電源シンボル修正
階層シート内で電源シンボルをなるべく使わないようにする
修正途中
Connections:
- net VBUS: no longer C317.2, D190.4, U9.1 (VBUS1)
- net GNDD renamed VBUS-_U
- new net VBUS+_U: C317.2, D190.4, U9.1 (VBUS1)
Other:
- moved on the sheet: C314

Commit message: ラベル修正とテキスト等の追加
階層シート内の電源シンボルをまとめて階層ラベルとして上層に出し、上層のシートで電源シンボルに接続
Connections:
- net +3V3 renamed S10_+3V3
- net +5V renamed VCC
- net +5VA renamed S10_+5VA
- net VBUS renamed VBUS+_D
Other:
- moved on the sheet: C312, C313, C314, C316, C317, C318, C319, C320, C321, C323, C324, C325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

Commit message: チップ抵抗、チップコンデンササイズ修正
Parts:
- C312, C313, C314, C315, C316, C317, C318, C319, C320, C321, C322, C323, C324, C325, C327, C328, C330, C331, C333, C334, C337, C338, C339, C340, C341, C342, C343, C344: footprint Capacitor_SMD:C_0603_1608Metric -> Capacitor_SMD:C_0402_1005Metric
- R577, R578, R581, R589, R591, R594, R595, R596, R602, R603, R604, R608, R609, R611, R612, R613, R614, R615, R617, R618, R619, R620, R621, R622, R625, R626, R627, R629, R630, R632: footprint Resistor_SMD:R_0603_1608Metric -> Resistor_SMD:R_0402_1005Metric

Commit message: アノテーションし直し、
Parts:
- renumbered C314 to C296, C315 to C297, C317 to C298, C318 to C299, C312 to C300, C320 to C301, C313 to C302, C322 to C303, C316 to C304, C319 to C305, C321 to C306, C323 to C307, C324 to C308, C325 to C309, C326 to C310, C327 to C311, C328 to C312, C329 to C313, C330 to C314, C331 to C315, C332 to C316, C333 to C317, C334 to C318, C335 to C319, C336 to C320, C337 to C321, C338 to C322, C339 to C323, C340 to C324, C341 to C325, C342 to C326, C343 to C327, C344 to C328, D190 to D153, D191 to D154, D192 to D155, D186 to D156, D187 to D157, D188 to D158, D189 to D159, D185 to D160, D195 to D161, D196 to D162, D193 to D163, D194 to D164, D197 to D165, D198 to D166, D199 to D167, D200 to D168, D201 to D169, D202 to D170, R581 to R545, R577 to R546, R584 to R547, R579 to R548, R585 to R549, R586 to R550, R578 to R551, R580 to R552, R595 to R553, R582 to R554, R583 to R555, R597 to R556, R589 to R557, R599 to R558, R587 to R559, R588 to R560, R590 to R561, R601 to R562, R591 to R563, R592 to R564, R593 to R565, R594 to R566, R596 to R567, R598 to R568, R600 to R569, R602 to R570, R603 to R571, R604 to R572, R609 to R573, R610 to R574, R613 to R575, R605 to R576, R606 to R577, R607 to R578, R608 to R579, R614 to R580, R616 to R581, R611 to R582, R612 to R583, R622 to R584, R615 to R585, R617 to R586, R618 to R587, R619 to R588, R620 to R589, R625 to R590, R621 to R591, R628 to R592, R629 to R593, R623 to R594, R624 to R595, R630 to R596, R626 to R597, R627 to R598, R631 to R599, R632 to R600

Commit message: 絶縁パルストランス数削減
Parts:
- renumbered L26 to L19, L27 to L20
Changed lines of the file:
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@@
   (symbol (lib_id "ProjectEV:L_BLM18PG471SN1D") (at 311.15 165.1 90) (unit 1)
     (in_bom yes) (on_board yes) (dnp no)
-    (property "Reference" "L27" (at 311.15 160.02 90)
+    (property "Reference" "L20" (at 311.15 160.02 90)
       (effects (font (size 1.27 1.27)))
     )
@@
       (project "AMS-board-2024"
         (path "/3a719eb3-09ce-4343-8f6e-20cc0aaf5261/6c88c007-deae-4ed6-a37c-9d5c4c750b8f"
-          (reference "L27") (unit 1)
+          (reference "L20") (unit 1)
         )
       )
@@
   (symbol (lib_id "ProjectEV:L_BLM18PG471SN1D") (at 295.91 177.8 90) (unit 1)
     (in_bom yes) (on_board yes) (dnp no) (fields_autoplaced)
-    (property "Reference" "L26" (at 295.91 172.72 90)
+    (property "Reference" "L19" (at 295.91 172.72 90)
       (effects (font (size 1.27 1.27)))
     )
@@
       (project "AMS-board-2024"
         (path "/3a719eb3-09ce-4343-8f6e-20cc0aaf5261/6c88c007-deae-4ed6-a37c-9d5c4c750b8f"
-          (reference "L26") (unit 1)
-        )
-      )
+          (reference "L19") (unit 1)
+        )
+      )

Commit message: 5V OUT バッファ回路修正
Connections:
- net at C322.1, R588.2, U17.10 (~{FAULT1})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: no longer C324.1
- net at R589.2, U17.5 (EN2), U17.6 (~{FAULT2}): now also C324.1
Changed lines of the file:
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@@
   (junction (at 500.38 231.14) (diameter 0) (color 0 0 0 0)
   )
-  (junction (at 513.08 231.14) (diameter 0) (color 0 0 0 0)
-  )
   (junction (at 133.35 238.76) (diameter 0) (color 0 0 0 0)
   )
@@
   )
   (junction (at 213.36 182.88) (diameter 0) (color 0 0 0 0)
+  )
+  (junction (at 513.08 236.22) (diameter 0) (color 0 0 0 0)
   )
   (junction (at 58.42 317.5) (diameter 0) (color 0 0 0 0)
@@
     (stroke (width 0) (type default))
   )
-  (wire (pts (xy 500.38 231.14) (xy 513.08 231.14))
+  (wire (pts (xy 500.38 231.14) (xy 520.7 231.14))
     (stroke (width 0) (type default))
   )
@@
     (stroke (width 0) (type default))
   )
+  (wire (pts (xy 513.08 236.22) (xy 495.3 236.22))
+    (stroke (width 0) (type default))
+  )
   (wire (pts (xy 381 304.8) (xy 381 320.04))
     (stroke (width 0) (type default))
@@
     (stroke (width 0) (type default))
   )
+  (wire (pts (xy 513.08 236.22) (xy 513.08 238.76))
+    (stroke (width 0) (type default))
+  )
   (wire (pts (xy 396.24 127) (xy 396.24 129.54))
     (stroke (width 0) (type default))
@@
     (stroke (width 0) (type default))
   )
-  (wire (pts (xy 520.7 236.22) (xy 495.3 236.22))
+  (wire (pts (xy 520.7 236.22) (xy 513.08 236.22))
     (stroke (width 0) (type default))
   )
@@
     (stroke (width 0) (type default))
   )
-  (wire (pts (xy 513.08 231.14) (xy 513.08 238.76))
-    (stroke (width 0) (type default))
-  )
   (wire (pts (xy 133.35 238.76) (xy 114.3 238.76))
     (stroke (width 0) (type default))
@@
     (stroke (width 0) (type default))
   )
-  (wire (pts (xy 513.08 231.14) (xy 520.7 231.14))
-    (stroke (width 0) (type default))
-  )

Commit message: 4.7uFのMLCCのチップサイズ変更
Parts:
- C310, C316: footprint Capacitor_SMD:C_0805_2012Metric -> Capacitor_SMD:C_0603_1608Metric
Changed lines of the file:
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@@
       (effects (font (size 1.27 1.27)) (justify left))
     )
-    (property "Footprint" "Capacitor_SMD:C_0805_2012Metric" (at 341.3252 238.76 0)
+    (property "Footprint" "Capacitor_SMD:C_0603_1608Metric" (at 341.3252 238.76 0)
       (effects (font (size 1.27 1.27)) hide)
     )
@@
       (effects (font (size 1.27 1.27)) (justify left))
     )
-    (property "Footprint" "Capacitor_SMD:C_0805_2012Metric" (at 385.7752 137.16 0)
-      (effects (font (size 1.27 1.27)) hide)
-    )
+    (property "Footprint" "Capacitor_SMD:C_0603_1608Metric" (at 385.7752 137.16 0)
+      (effects (font (size 1.27 1.27)) hide)
+    )
