File: AMS-board-2024/battery-module-monitor-8.kicad_sch (KiCad schematic)
At the start: 144 parts, among them Q901 BSS308PE, Q902 BSS308PE, Q903 BSS308PE, Q904 BSS308PE, Q905 BSS308PE, Q906 BSS308PE, Q907 BSS308PE, Q908 BSS308PE, Q909 BSS308PE, Q910 BSS308PE, Q911 BSS308PE, Q912 BSS308PE, Q913 NSV1C201MZ4, U901 LTC6811-1

Commit message: 修正
アノテーション方法の変更：最初の空き番号から使用
Parts:
- renumbered C901 to C239, C902 to C240, C903 to C241, C904 to C242, C905 to C243, C906 to C244, C907 to C245, C908 to C246, C909 to C247, C910 to C248, C911 to C249, C912 to C250, C913 to C251, C914 to C252, C915 to C253, C916 to C254, C917 to C255, C918 to C256, C919 to C257, C920 to C258, C921 to C259, C922 to C260, C923 to C261, C924 to C262, C925 to C263, C926 to C264, C927 to C265, C928 to C266, C929 to C267, C930 to C268, C931 to C269, C932 to C270, C933 to C271, C934 to C272, D909 to D100, D910 to D101, D911 to D102, D912 to D103, D913 to D104, D901 to D92, D902 to D93, D903 to D94, D904 to D95, D905 to D96, D906 to D97, D907 to D98, D908 to D99, F909 to F100, F910 to F101, F911 to F102, F912 to F103, F913 to F104, F901 to F92, F902 to F93, F903 to F94, F904 to F95, F905 to F96, F906 to F97, F907 to F98, F908 to F99, FL901 to FL15, FL902 to FL16, L901 to L8, Q909 to Q100, Q910 to Q101, Q911 to Q102, Q912 to Q103, Q913 to Q104, Q901 to Q92, Q902 to Q93, Q903 to Q94, Q904 to Q95, Q905 to Q96, Q906 to Q97, Q907 to Q98, Q908 to Q99, R901 to R470, R902 to R471, R903 to R472, R904 to R473, R905 to R474, R906 to R475, R907 to R476, R908 to R477, R909 to R478, R910 to R479, R911 to R480, R912 to R481, R913 to R482, R914 to R483, R915 to R484, R916 to R485, R917 to R486, R918 to R487, R919 to R488, R920 to R489, R921 to R490, R922 to R491, R923 to R492, R924 to R493, R925 to R494, R926 to R495, R927 to R496, R928 to R497, R929 to R498, R930 to R499, R931 to R500, R932 to R501, R933 to R502, R934 to R503, R935 to R504, R936 to R505, R937 to R506, R938 to R507, R939 to R508, R940 to R509, R941 to R510, R942 to R511, R943 to R512, R944 to R513, R945 to R514, R946 to R515, R947 to R516, R948 to R517, R949 to R518, R950 to R519, R951 to R520, R952 to R521, R953 to R522, R954 to R523, R955 to R524, R956 to R525, R957 to R526, R958 to R527, R959 to R528, R960 to R529, R961 to R530, R962 to R531, R963 to R532, R964 to R533, R965 to R534, R966 to R535, R967 to R536, U901 to U8

Commit message: GNDシンボル追加
Connections:
- net GND1: now reaches C269.1
- net GND1: now also C239.2, C240.2, C241.2, C242.2, C243.2, C244.2, C245.2, C246.2, C247.2, C248.2, C249.2, C250.2, C263.2, C264.2, C265.1, C266.1, C267.2, C268.1, C270.2, C271.1, C272.1, L8.2, R524.1, U8.30 (V-), U8.31 (V-)

Commit message: GPIO周辺回路の修正
Parts:
- added C326, C327, C328, C329, C330: 0.1u, Capacitor_SMD:C_0603_1608Metric, symbol Device:C
- added R593, R594, R595, R596, R597: 10k, Resistor_SMD:R_0603_1608Metric, symbol Device:R
- R520, R523, R525, R526, R531: value 10k -> 100
Connections:
- net GND1: now also C326.2, C327.2, C328.2, C329.2, C330.2
- net Thermistor1+: now also R520.2, R593.2; no longer R531.1, U8.27 (GPIO1)
- net Thermistor2+: now also R523.2, R594.2; no longer R526.1, U8.28 (GPIO2)
- net Thermistor3+: now also R525.2, R595.2; no longer R525.1, U8.29 (GPIO3)
- net Thermistor4+: now also R526.2, R596.2; no longer R523.1, U8.32 (GPIO4)
- net Thermistor5+: now also R531.2, R597.2; no longer R520.1, U8.33 (GPIO5)
- net VREG: now reaches C267.1, Q104.3 (E), R522.1, U8.37 (VREG), U8.40 (ISOMD)
- new net: C327.1, R526.1, U8.32 (GPIO4)
- new net: C330.1, R520.1, U8.27 (GPIO1)
- new net: C329.1, R523.1, U8.28 (GPIO2)
- new net: C328.1, R525.1, U8.29 (GPIO3)
- new net: C326.1, R531.1, U8.33 (GPIO5)
- new net VREF_3V: C265.2, R593.1, R594.1, R595.1, R596.1, R597.1, U8.34 (VREF2)

Commit message: テキスト修正
Other:
- note added: "レギュレーション上必要なサーミスタは 96 CELL x 25 % = 24 本. GPIO1~3 をサーミスタに使用し、 GPIO4, 5 は別用途で使用してもOK. GPIO4, 5 のプルアップは必要に応じて実装."
- note removed: "レギュレーション上必要なサーミスタは 3 x 8 = 24 本. GPIO1~3 をサーミスタに使用し、 GPIO4, 5 は別用途で使用してもOK. GPIO4, 5 のプルアップは必要に応じて実装."
Changed lines of the file:
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@@
-    (effects (font (size 1.27 1.27)) (justify left bottom))
-  )
-  (text "レギュレーション上必要なサーミスタは 3 x 8 = 24 本.\nGPIO1~3 をサーミスタに使用し、\nGPIO4, 5 は別用途で使用してもOK.\nGPIO4, 5 のプルアップは必要に応じて実装."
-    (at 469.9 283.21 0)
     (effects (font (size 1.27 1.27)) (justify left bottom))
   )
@@
     (effects (font (size 1.27 1.27)) (justify left bottom))
   )
+  (text "レギュレーション上必要なサーミスタは 96 CELL x 25 % = 24 本.\nGPIO1~3 をサーミスタに使用し、\nGPIO4, 5 は別用途で使用してもOK.\nGPIO4, 5 のプルアップは必要に応じて実装."
+    (at 469.9 283.21 0)
+    (effects (font (size 1.27 1.27)) (justify left bottom))
+  )

Commit message: ヒューズ変更
Parts:
- removed F100, F101, F102, F103, F104, F92, F93, F94, F95, F96, F97, F98, F99: C1F 500, Fuse:Fuse_1206_3216Metric, symbol Device:Fuse
- added F66, F67, F68, F69, F70, F71, F72, F73, F74, F75, F76, F77, F78: 0679L1000-05, ProjectEV:Fuse_0679L, symbol ProjectEV:Fuse_0679L1000-05
Connections:
- net CELL0: now also F78.1
- net CELL1: now also F77.1
- net CELL10: now also F68.1
- net CELL11: now also F67.1
- net CELL12: now also F66.1
- net CELL2: now also F76.1
- net CELL3: now also F75.1
- net CELL4: now also F74.1
- net CELL5: now also F73.1
- net CELL6: now also F72.1
- net CELL7: now also F71.1
- net CELL8: now also F70.1
- net CELL9: now also F69.1
- net at Q99.2 (S), R476.2, R488.2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: now also F73.2
- net at Q95.2 (S), R472.2, R484.2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: now also F69.2
- net at D92.1 (K), Q103.2 (S), R480.2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: now also F77.2
- net at Q94.2 (S), R471.2, R483.2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: now also F68.2
- net at Q97.2 (S), R474.2, R486.2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: now also F71.2
- net at Q93.2 (S), R470.2, R482.2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: now also F67.2
- net at Q98.2 (S), R475.2, R487.2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: now also F72.2
- net at D92.2 (A), L8.1, R481.2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: now also F78.2
- net at Q101.2 (S), R478.2, R490.2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: now also F75.2
- net at Q92.2 (S), R506.1, R519.1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: now also F66.2
- net at Q100.2 (S), R477.2, R489.2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: now also F74.2
- net at Q96.2 (S), R473.2, R485.2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: now also F70.2
- net at Q102.2 (S), R479.2, R491.2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: now also F76.2

Commit message: アノテーションし直し
Parts:
- renumbered C239 to C274, C240 to C275, C241 to C276, C242 to C277, C243 to C278, C244 to C279, C245 to C280, C246 to C281, C247 to C282, C248 to C283, C249 to C284, C250 to C285, C251 to C286, C252 to C287, C253 to C288, C254 to C289, C255 to C290, C256 to C291, C257 to C292, C258 to C293, C259 to C294, C260 to C295, C261 to C296, C262 to C297, C263 to C298, C264 to C299, C326 to C300, C265 to C301, C327 to C302, C266 to C303, C267 to C304, C328 to C305, C268 to C306, C269 to C307, C329 to C308, C330 to C309, C270 to C310, C271 to C311, C272 to C312, F74 to F100, F75 to F101, F76 to F102, F77 to F103, F78 to F104, F66 to F92, F67 to F93, F68 to F94, F69 to F95, F70 to F96, F71 to F97, F72 to F98, F73 to F99, R470 to R505, R471 to R506, R472 to R507, R473 to R508, R474 to R509, R475 to R510, R476 to R511, R477 to R512, R478 to R513, R479 to R514, R480 to R515, R481 to R516, R482 to R517, R483 to R518, R484 to R519, R485 to R520, R486 to R521, R487 to R522, R488 to R523, R489 to R524, R490 to R525, R491 to R526, R492 to R527, R493 to R528, R494 to R529, R495 to R530, R496 to R531, R497 to R532, R498 to R533, R499 to R534, R500 to R535, R501 to R536, R502 to R537, R503 to R538, R504 to R539, R505 to R540, R506 to R541, R507 to R542, R508 to R543, R509 to R544, R510 to R545, R511 to R546, R512 to R547, R513 to R548, R514 to R549, R515 to R550, R516 to R551, R517 to R552, R518 to R553, R519 to R554, R521 to R555, R522 to R556, R524 to R557, R527 to R558, R528 to R559, R529 to R560, R530 to R561, R532 to R562, R520 to R563, R523 to R564, R525 to R565, R526 to R566, R531 to R567, R593 to R568, R533 to R569, R534 to R570, R535 to R571, R536 to R572, R594 to R573, R595 to R574, R596 to R575, R597 to R576

Commit message: GPIO入力保護回路追加
Parts:
- added D200, D201, D202, D203, D204, D205, D206, D207, D208, D209: BAT46W-7-F, ProjectEV:D_SOD-123_BAT46W-7-F, symbol ProjectEV:D_BAT46W-7-F
Connections:
- net GND1: now also D201.2 (A), D203.2 (A), D205.2 (A), D207.2 (A), D209.2 (A)
- net VREG: now also D200.1 (K), D202.1 (K), D204.1 (K), D206.1 (K), D208.1 (K)
- net at C302.1, R566.1, U8.32 (GPIO4): now also D206.2 (A), D207.1 (K)
- net at C309.1, R563.1, U8.27 (GPIO1): now also D200.2 (A), D201.1 (K)
- net at C308.1, R564.1, U8.28 (GPIO2): now also D202.2 (A), D203.1 (K)
- net at C305.1, R565.1, U8.29 (GPIO3): now also D204.2 (A), D205.1 (K)
- net at C300.1, R567.1, U8.33 (GPIO5): now also D208.2 (A), D209.1 (K)
Other:
- moved on the sheet: R563, R564, R565, R566, R567, R568, R573, R574, R575, R576

Commit message: モジュールモニタの最後のisoSPIの使用しない箇所を削除
Parts:
- removed C306, C311: 10n, Capacitor_SMD:C_0603_1608Metric, symbol Device:C
- removed FL15: DLW43SH101XK2, ProjectEV:CommonModeChoke_DLW43SH101, symbol ProjectEV:CommonModeChoke_DLW43SH101
- removed R558, R559: 60.4, Resistor_SMD:R_0603_1608Metric, symbol Device:R
- removed R569, R570: 294, Resistor_SMD:R_0603_1608Metric, symbol Device:R
Connections:
- no-connect marks 2 -> 4
