File: AMS-board-2024/battery-module-monitor-8.kicad_sch (KiCad schematic)
At the start: 157 parts, among them Q100 BSS308PE, Q101 BSS308PE, Q102 BSS308PE, Q103 BSS308PE, Q104 NSV1C201MZ4, Q92 BSS308PE, Q93 BSS308PE, Q94 BSS308PE, Q95 BSS308PE, Q96 BSS308PE, Q97 BSS308PE, Q98 BSS308PE, Q99 BSS308PE, U8 LTC6811-1

Commit message: アノテーションし直し
Parts:
- renumbered C307 to C306, C308 to C307, C309 to C308, C310 to C309, C312 to C310, D92 to D162, D93 to D163, D94 to D164, D95 to D165, D96 to D166, D97 to D167, D98 to D168, D99 to D169, D100 to D170, D101 to D171, D102 to D172, D103 to D173, D104 to D174, D202 to D175, D203 to D176, D206 to D177, D207 to D178, D200 to D179, D201 to D180, D204 to D181, D205 to D182, D208 to D183, D209 to D184, FL16 to FL15, L8 to L24, R505 to R507, R506 to R508, R507 to R509, R508 to R510, R509 to R511, R510 to R512, R511 to R513, R512 to R514, R513 to R515, R514 to R516, R515 to R517, R516 to R518, R517 to R519, R518 to R520, R519 to R521, R520 to R522, R521 to R523, R522 to R524, R523 to R525, R524 to R526, R525 to R527, R526 to R528, R527 to R529, R528 to R530, R529 to R531, R530 to R532, R531 to R533, R532 to R534, R533 to R535, R534 to R536, R535 to R537, R536 to R538, R537 to R539, R538 to R540, R539 to R541, R540 to R542, R541 to R543, R542 to R544, R543 to R545, R544 to R546, R545 to R547, R546 to R548, R547 to R549, R548 to R550, R549 to R551, R550 to R552, R551 to R553, R552 to R554, R553 to R555, R554 to R556, R555 to R557, R556 to R558, R557 to R559, R571 to R563, R572 to R564, R563 to R565, R564 to R566, R565 to R567, R566 to R568, R567 to R569, R568 to R570, R573 to R571, R574 to R572, R575 to R573, R576 to R574

Commit message: ERC実行、修正
ラベル修正、未配線部分修正、PWR_FLAG追加
Connections:
- net GND1 is gone; now on net GND8: C274.2, C275.2, C276.2, C277.2, C278.2, C279.2, C280.2, C281.2, C282.2, C283.2, C284.2, C285.2, C298.2, C299.2, C300.2, C301.1, C302.2, C303.1, C304.2, C305.2, C306.1, C307.2, C308.2, C309.2, C310.1, D176.2 (A), D178.2 (A), D180.2 (A), D182.2 (A), D184.2 (A), L24.2, R559.1, U8.30 (V-), U8.31 (V-)
- net GND8: now reaches U8.36 (SWTEN)
- net VREG renamed VREG8
Changed lines of the file:
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@@
   (junction (at 127 259.08) (diameter 0) (color 0 0 0 0)
   )
+  (junction (at 292.1 165.1) (diameter 0) (color 0 0 0 0)
+  )
+  (junction (at 101.6 381) (diameter 0) (color 0 0 0 0)
+  )
   (junction (at 127 245.11) (diameter 0) (color 0 0 0 0)
   )
@@
     (stroke (width 0) (type default))
   )
-  (wire (pts (xy 101.6 378.46) (xy 101.6 379.73))
+  (wire (pts (xy 101.6 378.46) (xy 101.6 381))
     (stroke (width 0) (type default))
   )
@@
     (stroke (width 0) (type default))
   )
+  (wire (pts (xy 96.52 381) (xy 101.6 381))
+    (stroke (width 0) (type default))
+  )
   (wire (pts (xy 236.22 287.02) (xy 236.22 228.6))
     (stroke (width 0) (type default))
@@
     (stroke (width 0) (type default))
   )
+  (wire (pts (xy 101.6 381) (xy 101.6 383.54))
+    (stroke (width 0) (type default))
+  )
   (wire (pts (xy 127 210.82) (xy 127 212.09))
     (stroke (width 0) (type default))
@@
     (stroke (width 0) (type default))
   )
+  (wire (pts (xy 304.8 223.52) (xy 307.34 223.52))
+    (stroke (width 0) (type default))
+  )
   (wire (pts (xy 165.1 365.76) (xy 165.1 350.52))
     (stroke (width 0) (type default))
@@
     (effects (font (size 1.27 1.27)) (justify left))
   )
-  (hierarchical_label "GND" (shape output) (at 419.1 228.6 0) (fields_autoplaced)
+  (hierarchical_label "GND8" (shape output) (at 419.1 228.6 0) (fields_autoplaced)
     (effects (font (size 1.27 1.27)) (justify left))
   )
@@
     (effects (font (size 1.27 1.27)) (justify right))
   )
-  (hierarchical_label "VREG" (shape output) (at 419.1 223.52 0) (fields_autoplaced)
+  (hierarchical_label "VREG8" (shape output) (at 419.1 223.52 0) (fields_autoplaced)
     (effects (font (size 1.27 1.27)) (justify left))
   )
@@
     )
   )
-  (symbol (lib_id "ProjectEV:GND8") (at 101.6 379.73 0) (unit 1)
+  (symbol (lib_id "ProjectEV:GND8") (at 101.6 383.54 0) (unit 1)
     (in_bom yes) (on_board yes) (dnp no) (fields_autoplaced)
-    (property "Reference" "#PWR0309" (at 101.6 386.08 0)
+    (property "Reference" "#PWR0309" (at 101.6 389.89 0)
       (effects (font (size 1.27 1.27)) hide)
     )
-    (property "Value" "GND8" (at 101.6 384.81 0)
+    (property "Value" "GND8" (at 101.6 388.62 0)
       (effects (font (size 1.27 1.27)))
     )
-    (property "Footprint" "" (at 101.6 379.73 0)
+    (property "Footprint" "" (at 101.6 383.54 0)
       (effects (font (size 1.27 1.27)) hide)
     )
-    (property "Datasheet" "" (at 101.6 379.73 0)
+    (property "Datasheet" "" (at 101.6 383.54 0)
       (effects (font (size 1.27 1.27)) hide)
     )
@@
     )
   )
+  (symbol (lib_id "ProjectEV:GND8") (at 307.34 223.52 90) (unit 1)
+    (in_bom yes) (on_board yes) (dnp no) (fields_autoplaced)
+    (property "Reference" "#PWR0433" (at 313.69 223.52 0)
+      (effects (font (size 1.27 1.27)) hide)
+    )
+    (property "Value" "GND8" (at 311.15 223.52 90)
+      (effects (font (size 1.27 1.27)) (justify right))
+    )
+    (property "Footprint" "" (at 307.34 223.52 0)
+      (effects (font (size 1.27 1.27)) hide)
+    )
+    (property "Datasheet" "" (at 307.34 223.52 0)
+      (effects (font (size 1.27 1.27)) hide)
+    )
+    (pin "1")
+    (instances
+      (project "AMS-board-2024"
+        (path "/3a719eb3-09ce-4343-8f6e-20cc0aaf5261/89a445cf-4dca-4c05-9556-2d66db3a69e6"
+          (reference "#PWR0433") (unit 1)
+        )
+      )
+    )
+  )
+  (symbol (lib_id "power:PWR_FLAG") (at 96.52 381 0) (unit 1)
+    (in_bom yes) (on_board yes) (dnp no) (fields_autoplaced)
+    (property "Reference" "#FLG017" (at 96.52 379.095 0)
+      (effects (font (size 1.27 1.27)) hide)
+    )
+    (property "Value" "PWR_FLAG" (at 96.52 375.92 0)
+      (effects (font (size 1.27 1.27)))
+    )
+    (property "Footprint" "" (at 96.52 381 0)
+      (effects (font (size 1.27 1.27)) hide)
+    )
+    (property "Datasheet" "~" (at 96.52 381 0)
+      (effects (font (size 1.27 1.27)) hide)
+    )
+    (pin "1")
+    (instances
+      (project "AMS-board-2024"
+        (path "/3a719eb3-09ce-4343-8f6e-20cc0aaf5261/89a445cf-4dca-4c05-9556-2d66db3a69e6"
+          (reference "#FLG017") (unit 1)
+        )
+      )
+    )
+  )
   (symbol (lib_id "ProjectEV:GND8") (at 152.4 134.62 0) (unit 1)
     (in_bom yes) (on_board yes) (dnp no) (fields_autoplaced)
@@
         )
       )
+    )
+  )
+  (symbol (lib_id "power:PWR_FLAG") (at 292.1 165.1 0) (unit 1)
+    (in_bom yes) (on_board yes) (dnp no) (fields_autoplaced)
+    (property "Reference" "#FLG09" (at 292.1 163.195 0)
+      (effects (font (size 1.27 1.27)) hide)
+    )
+    (property "Value" "PWR_FLAG" (at 292.1 160.02 0)
+      (effects (font (size 1.27 1.27)))
+    )
+    (property "Footprint" "" (at 292.1 165.1 0)
+      (effects (font (size 1.27 1.27)) hide)
+    )
+    (property "Datasheet" "~" (at 292.1 165.1 0)
+      (effects (font (size 1.27 1.27)) hide)
+    )
+    (pin "1")
+    (instances
+      (project "AMS-board-2024"
+        (path "/3a719eb3-09ce-4343-8f6e-20cc0aaf5261/89a445cf-4dca-4c05-9556-2d66db3a69e6"
+          (reference "#FLG09") (unit 1)
+        )
+      )

Commit message: 終端抵抗追加
Parts:
- added C373: 10n, Capacitor_SMD:C_0603_1608Metric, symbol Device:C
- added R662, R663: 60.4, Resistor_SMD:R_0603_1608Metric, symbol Device:R
Connections:
- net GND8: now also C373.1
- net at U8.47 (IMB): now also R663.1
- net at U8.48 (IPB): now also R662.2
- new net: C373.2, R662.1, R663.2
- no-connect marks 4 -> 2
Changed lines of the file:
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@@
   (junction (at 393.7 139.7) (diameter 0) (color 0 0 0 0)
   )
+  (junction (at 342.9 88.9) (diameter 0) (color 0 0 0 0)
+  )
   (junction (at 127 269.24) (diameter 0) (color 0 0 0 0)
   )
@@
   (no_connect (at 304.8 210.82))
   (no_connect (at 304.8 208.28))
-  (no_connect (at 304.8 185.42))
-  (no_connect (at 304.8 187.96))
   (wire (pts (xy 114.3 293.37) (xy 127 293.37))
     (stroke (width 0) (type default))
@@
     (stroke (width 0) (type default))
   )
+  (wire (pts (xy 342.9 101.6) (xy 309.88 101.6))
+    (stroke (width 0) (type default))
+  )
   (wire (pts (xy 149.86 148.59) (xy 152.4 148.59))
     (stroke (width 0) (type default))
@@
     (stroke (width 0) (type default))
   )
+  (wire (pts (xy 304.8 185.42) (xy 307.34 185.42))
+    (stroke (width 0) (type default))
+  )
   (wire (pts (xy 76.2 220.98) (xy 85.09 220.98))
     (stroke (width 0) (type default))
@@
     (stroke (width 0) (type default))
   )
+  (wire (pts (xy 307.34 76.2) (xy 342.9 76.2))
+    (stroke (width 0) (type default))
+  )
   (wire (pts (xy 223.52 213.36) (xy 279.4 213.36))
     (stroke (width 0) (type default))
@@
     (stroke (width 0) (type default))
   )
+  (wire (pts (xy 309.88 187.96) (xy 304.8 187.96))
+    (stroke (width 0) (type default))
+  )
   (wire (pts (xy 152.4 196.85) (xy 165.1 196.85))
     (stroke (width 0) (type default))
@@
     (stroke (width 0) (type default))
   )
+  (wire (pts (xy 331.47 88.9) (xy 332.74 88.9))
+    (stroke (width 0) (type default))
+  )
   (wire (pts (xy 127 269.24) (xy 127 267.97))
     (stroke (width 0) (type default))
@@
     (stroke (width 0) (type default))
   )
+  (wire (pts (xy 307.34 185.42) (xy 307.34 76.2))
+    (stroke (width 0) (type default))
+  )
   (wire (pts (xy 368.3 340.36) (xy 368.3 342.9))
     (stroke (width 0) (type default))
@@
     (stroke (width 0) (type default))
   )
+  (wire (pts (xy 342.9 99.06) (xy 342.9 101.6))
+    (stroke (width 0) (type default))
+  )
   (wire (pts (xy 152.4 245.11) (xy 165.1 245.11))
     (stroke (width 0) (type default))
@@
     (stroke (width 0) (type default))
   )
+  (wire (pts (xy 342.9 88.9) (xy 342.9 91.44))
+    (stroke (width 0) (type default))
+  )
   (wire (pts (xy 127 172.72) (xy 142.24 172.72))
     (stroke (width 0) (type default))
@@
     (stroke (width 0) (type default))
   )
+  (wire (pts (xy 342.9 76.2) (xy 342.9 78.74))
+    (stroke (width 0) (type default))
+  )
   (wire (pts (xy 355.6 223.52) (xy 355.6 215.9))
     (stroke (width 0) (type default))
@@
     (stroke (width 0) (type default))
   )
+  (wire (pts (xy 342.9 86.36) (xy 342.9 88.9))
+    (stroke (width 0) (type default))
+  )
   (wire (pts (xy 124.46 331.47) (xy 127 331.47))
     (stroke (width 0) (type default))
@@
     (stroke (width 0) (type default))
   )
+  (wire (pts (xy 340.36 88.9) (xy 342.9 88.9))
+    (stroke (width 0) (type default))
+  )
   (wire (pts (xy 114.3 340.36) (xy 114.3 341.63))
     (stroke (width 0) (type default))
@@
     (stroke (width 0) (type default))
   )
+  (wire (pts (xy 309.88 101.6) (xy 309.88 187.96))
+    (stroke (width 0) (type default))
+  )
   (wire (pts (xy 114.3 243.84) (xy 114.3 245.11))
     (stroke (width 0) (type default))
@@
     )
   )
+  (symbol (lib_id "Device:R") (at 342.9 95.25 180) (unit 1)
+    (in_bom yes) (on_board yes) (dnp no) (fields_autoplaced)
+    (property "Reference" "R663" (at 345.44 93.98 0)
+      (effects (font (size 1.27 1.27)) (justify right))
+    )
+    (property "Value" "60.4" (at 345.44 96.52 0)
+      (effects (font (size 1.27 1.27)) (justify right))
+    )
+    (property "Footprint" "Resistor_SMD:R_0603_1608Metric" (at 344.678 95.25 90)
+      (effects (font (size 1.27 1.27)) hide)
+    )
+    (property "Datasheet" "~" (at 342.9 95.25 0)
+      (effects (font (size 1.27 1.27)) hide)
+    )
+    (pin "1")
+    (pin "2")
+    (instances
+      (project "AMS-board-2024"
+        (path "/3a719eb3-09ce-4343-8f6e-20cc0aaf5261/89a445cf-4dca-4c05-9556-2d66db3a69e6"
+          (reference "R663") (unit 1)
+        )
+      )
+    )
+  )
   (symbol (lib_id "Device:R") (at 139.7 347.98 90) (unit 1)
     (in_bom yes) (on_board yes) (dnp no)
@@
     )
   )
+  (symbol (lib_id "ProjectEV:GND8") (at 331.47 88.9 270) (unit 1)
+    (in_bom yes) (on_board yes) (dnp no) (fields_autoplaced)
+    (property "Reference" "#PWR0447" (at 325.12 88.9 0)
+      (effects (font (size 1.27 1.27)) hide)
+    )
+    (property "Value" "GND8" (at 327.66 88.9 90)
+      (effects (font (size 1.27 1.27)) (justify right))
+    )
+    (property "Footprint" "" (at 331.47 88.9 0)
+      (effects (font (size 1.27 1.27)) hide)
+    )
+    (property "Datasheet" "" (at 331.47 88.9 0)
+      (effects (font (size 1.27 1.27)) hide)
+    )
+    (pin "1")
+    (instances
+      (project "AMS-board-2024"
+        (path "/3a719eb3-09ce-4343-8f6e-20cc0aaf5261/89a445cf-4dca-4c05-9556-2d66db3a69e6"
+          (reference "#PWR0447") (unit 1)
+        )
+      )
+    )
+  )
   (symbol (lib_id "ProjectEV:GND8") (at 381 368.3 0) (unit 1)
     (in_bom yes) (on_board yes) (dnp no) (fields_autoplaced)
@@
     )
   )
+  (symbol (lib_id "Device:R") (at 342.9 82.55 180) (unit 1)
+    (in_bom yes) (on_board yes) (dnp no) (fields_autoplaced)
+    (property "Reference" "R662" (at 345.44 81.28 0)
+      (effects (font (size 1.27 1.27)) (justify right))
+    )
+    (property "Value" "60.4" (at 345.44 83.82 0)
+      (effects (font (size 1.27 1.27)) (justify right))
+    )
+    (property "Footprint" "Resistor_SMD:R_0603_1608Metric" (at 344.678 82.55 90)
+      (effects (font (size 1.27 1.27)) hide)
+    )
+    (property "Datasheet" "~" (at 342.9 82.55 0)
+      (effects (font (size 1.27 1.27)) hide)
+    )
+    (pin "1")
+    (pin "2")
+    (instances
+      (project "AMS-board-2024"
+        (path "/3a719eb3-09ce-4343-8f6e-20cc0aaf5261/89a445cf-4dca-4c05-9556-2d66db3a69e6"
+          (reference "R662") (unit 1)
+        )
+      )
+    )
+  )
   (symbol (lib_id "Device:LED") (at 120.65 138.43 0) (unit 1)
     (in_bom yes) (on_board yes) (dnp no)
@@
         )
       )
+    )
+  )
+  (symbol (lib_id "Device:C") (at 336.55 88.9 90) (unit 1)
+    (in_bom yes) (on_board yes) (dnp no) (fields_autoplaced)
+    (property "Reference" "C373" (at 336.55 81.28 90)
+      (effects (font (size 1.27 1.27)))
+    )
+    (property "Value" "10n" (at 336.55 83.82 90)
+      (effects (font (size 1.27 1.27)))
+    )
+    (property "Footprint" "Capacitor_SMD:C_0603_1608Metric" (at 340.36 87.9348 0)
+      (effects (font (size 1.27 1.27)) hide)
+    )
+    (property "Datasheet" "~" (at 336.55 88.9 0)
+      (effects (font (size 1.27 1.27)) hide)
+    )
+    (pin "1")
+    (pin "2")
+    (instances
+      (project "AMS-board-2024"
+        (path "/3a719eb3-09ce-4343-8f6e-20cc0aaf5261/89a445cf-4dca-4c05-9556-2d66db3a69e6"
+          (reference "C373") (unit 1)
+        )
+      )

Commit message: ラベル修正
Connections:
- net VREG8 renamed VREG
Changed lines of the file:
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@@
     (effects (font (size 1.27 1.27)) (justify left bottom))
   )
-  (label "VREG8" (at 365.76 317.5 0) (fields_autoplaced)
+  (label "S9_VREG" (at 365.76 317.5 0) (fields_autoplaced)
     (effects (font (size 1.27 1.27)) (justify left bottom))
   )
-  (label "VREG8" (at 365.76 266.7 0) (fields_autoplaced)
+  (label "S9_VREG" (at 378.46 292.1 0) (fields_autoplaced)
     (effects (font (size 1.27 1.27)) (justify left bottom))
   )
-  (label "VREG8" (at 378.46 241.3 0) (fields_autoplaced)
+  (label "S9_VREG" (at 378.46 342.9 0) (fields_autoplaced)
     (effects (font (size 1.27 1.27)) (justify left bottom))
   )
-  (label "VREG8" (at 378.46 292.1 0) (fields_autoplaced)
+  (label "S9_VREG" (at 342.9 215.9 0) (fields_autoplaced)
     (effects (font (size 1.27 1.27)) (justify left bottom))
   )
-  (label "VREG8" (at 342.9 215.9 0) (fields_autoplaced)
+  (label "S9_VREG" (at 365.76 266.7 0) (fields_autoplaced)
     (effects (font (size 1.27 1.27)) (justify left bottom))
   )
-  (label "VREG8" (at 378.46 342.9 0) (fields_autoplaced)
+  (label "S9_VREG" (at 378.46 241.3 0) (fields_autoplaced)
     (effects (font (size 1.27 1.27)) (justify left bottom))
   )
@@
     (effects (font (size 1.27 1.27)) (justify right))
   )
-  (hierarchical_label "VREG8" (shape output) (at 419.1 223.52 0) (fields_autoplaced)
+  (hierarchical_label "VREG" (shape output) (at 419.1 223.52 0) (fields_autoplaced)
     (effects (font (size 1.27 1.27)) (justify left))
   )

Commit message: アノテーションし直し
Parts:
- renumbered C373 to C306, C306 to C307, C307 to C308, C308 to C309, C309 to C310, C310 to C311, L24 to L25, R662 to R560, R663 to R561, R560 to R562, R561 to R563, R562 to R564, R563 to R565, R564 to R566, R565 to R567, R566 to R568, R567 to R569, R568 to R570, R569 to R571, R570 to R572, R571 to R573, R572 to R574, R573 to R575, R574 to R576

Commit message: ラベル修正とテキスト等の追加
階層シート内の電源シンボルをまとめて階層ラベルとして上層に出し、上層のシートで電源シンボルに接続
Connections:
- net GND8 renamed GND
- net GND: no longer C301.1, C303.1, C304.2, C310.2, R559.1, U8.36 (SWTEN)
- new net: C301.1, C303.1, C304.2, C310.2, R559.1, U8.36 (SWTEN)

Commit message: LTC6811のシンボルを更新
Parts:
- U8: footprint ProjectEV:SSOP-48_5.3x12.8mm_P0.5mm_LTC6811 -> ProjectEV:Package_SSOP-48_5.3x12.8mm_P0.5mm_LTC6811
Changed lines of the file:
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@@
       (effects (font (size 1.27 1.27)) (justify left))
     )
-    (property "Footprint" "ProjectEV:SSOP-48_5.3x12.8mm_P0.5mm_LTC6811" (at 290.83 213.36 0)
+    (property "Footprint" "ProjectEV:Package_SSOP-48_5.3x12.8mm_P0.5mm_LTC6811" (at 290.83 213.36 0)
       (effects (font (size 1.27 1.27)) hide)
     )

Commit message: チップ抵抗、チップコンデンササイズ修正
Parts:
- C286, C287, C288, C289, C290, C291, C292, C293, C294, C295, C296, C297, C298, C300, C301, C302, C303, C304, C305, C306, C307, C308, C309, C311: footprint Capacitor_SMD:C_0603_1608Metric -> Capacitor_SMD:C_0402_1005Metric
- R531, R532, R533, R534, R535, R536, R537, R538, R539, R540, R541, R542, R543, R544, R545, R546, R547, R548, R549, R550, R551, R552, R553, R554, R555, R556, R557, R559, R564, R567, R568, R569, R570, R571, R572, R573, R574, R575, R576: footprint Resistor_SMD:R_0603_1608Metric -> Resistor_SMD:R_0402_1005Metric
