File: AMS-board-2024/battery-module-monitor-8.kicad_sch (KiCad schematic)
At the start: 160 parts, among them Q100 BSS308PE, Q101 BSS308PE, Q102 BSS308PE, Q103 BSS308PE, Q104 NSV1C201MZ4, Q92 BSS308PE, Q93 BSS308PE, Q94 BSS308PE, Q95 BSS308PE, Q96 BSS308PE, Q97 BSS308PE, Q98 BSS308PE, Q99 BSS308PE, U8 LTC6811-1

Commit message: 温度センサ用コネクタ変更、大まかな位置決定
Parts:
- removed C300, C302: 0.1u, Capacitor_SMD:C_0402_1005Metric, symbol Device:C
- removed D177, D178, D183, D184: BAT46W-7-F, ProjectEV:D_SOD-123_BAT46W-7-F, symbol ProjectEV:D_BAT46W-7-F
- removed R570, R571: 100, Resistor_SMD:R_0402_1005Metric, symbol Device:R
- removed R575, R576: 10k, Resistor_SMD:R_0402_1005Metric, symbol Device:R
Connections:
- net VREF_3V: no longer names the net of C301.2, R572.1, R573.1, R574.1, U8.34 (VREF2)
- net VREG: no longer names the net of C304.1, D175.1 (K), D179.1 (K), D181.1 (K), Q104.3 (E), R558.1, U8.37 (VREG), U8.40 (ISOMD)
- no-connect marks 2 -> 4

Commit message: アノテーションし直し、
Parts:
- R528: renamed from R556; footprint Resistor_SMD:R_0402_1005Metric -> Resistor_SMD:R_0603_1608Metric
- R536: renamed from R564; footprint Resistor_SMD:R_0402_1005Metric -> Resistor_SMD:R_0603_1608Metric
- renumbered C274 to C260, C275 to C261, C276 to C262, C277 to C263, C278 to C264, C279 to C265, C280 to C266, C281 to C267, C282 to C268, C283 to C269, C284 to C270, C285 to C271, C286 to C272, C287 to C273, C288 to C274, C289 to C275, C290 to C276, C291 to C277, C292 to C278, C293 to C279, C294 to C280, C295 to C281, C296 to C282, C297 to C283, C298 to C284, C299 to C285, C301 to C286, C303 to C287, C304 to C288, C305 to C289, C306 to C290, C307 to C291, C308 to C292, C309 to C293, C310 to C294, C311 to C295, D162 to D134, D163 to D135, D164 to D136, D165 to D137, D166 to D138, D167 to D139, D168 to D140, D169 to D141, D170 to D142, D171 to D143, D172 to D144, D173 to D145, D174 to D146, D175 to D147, D176 to D148, D179 to D149, D180 to D150, D181 to D151, D182 to D152, R507 to R479, R508 to R480, R509 to R481, R510 to R482, R511 to R483, R512 to R484, R513 to R485, R514 to R486, R515 to R487, R516 to R488, R517 to R489, R518 to R490, R519 to R491, R520 to R492, R521 to R493, R522 to R494, R523 to R495, R524 to R496, R525 to R497, R526 to R498, R527 to R499, R528 to R500, R529 to R501, R530 to R502, R531 to R503, R532 to R504, R533 to R505, R534 to R506, R535 to R507, R536 to R508, R537 to R509, R538 to R510, R539 to R511, R540 to R512, R541 to R513, R542 to R514, R543 to R515, R544 to R516, R545 to R517, R546 to R518, R547 to R519, R548 to R520, R549 to R521, R550 to R522, R551 to R523, R552 to R524, R553 to R525, R554 to R526, R555 to R527, R557 to R529, R558 to R530, R559 to R531, R560 to R532, R561 to R533, R562 to R534, R563 to R535, R565 to R537, R566 to R538, R567 to R539, R568 to R540, R569 to R541, R572 to R542, R573 to R543, R574 to R544

Commit message: 絶縁パルストランス数削減
Parts:
- renumbered L25 to L18
Changed lines of the file:
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@@
   (symbol (lib_id "ProjectEV:L_MH3261") (at 101.6 374.65 0) (unit 1)
     (in_bom yes) (on_board yes) (dnp no) (fields_autoplaced)
-    (property "Reference" "L25" (at 102.87 373.38 0)
+    (property "Reference" "L18" (at 102.87 373.38 0)
       (effects (font (size 1.27 1.27)) (justify left))
     )
@@
       (project "AMS-board-2024"
         (path "/3a719eb3-09ce-4343-8f6e-20cc0aaf5261/89a445cf-4dca-4c05-9556-2d66db3a69e6"
-          (reference "L25") (unit 1)
+          (reference "L18") (unit 1)
         )
       )

Commit message: 一部GNDへつながっていなかったので修正
Connections:
- net GND: now also C286.1, C287.1, C288.2, C294.2, R531.1, U8.36 (SWTEN)
Changed lines of the file:
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@@
   (junction (at 345.44 238.76) (diameter 0) (color 0 0 0 0)
   )
+  (junction (at 320.04 231.14) (diameter 0) (color 0 0 0 0)
+  )
   (junction (at 393.7 114.3) (diameter 0) (color 0 0 0 0)
   )
@@
   )
   (junction (at 114.3 148.59) (diameter 0) (color 0 0 0 0)
+  )
+  (junction (at 320.04 259.08) (diameter 0) (color 0 0 0 0)
   )
   (junction (at 165.1 245.11) (diameter 0) (color 0 0 0 0)
@@
     (stroke (width 0) (type default))
   )
+  (wire (pts (xy 320.04 231.14) (xy 320.04 259.08))
+    (stroke (width 0) (type default))
+  )
   (wire (pts (xy 127 257.81) (xy 127 259.08))
     (stroke (width 0) (type default))
@@
     (stroke (width 0) (type default))
   )
+  (wire (pts (xy 320.04 231.14) (xy 337.82 231.14))
+    (stroke (width 0) (type default))
+  )
   (wire (pts (xy 309.88 187.96) (xy 304.8 187.96))
     (stroke (width 0) (type default))
@@
     (stroke (width 0) (type default))
   )
-  (wire (pts (xy 317.5 231.14) (xy 337.82 231.14))
-    (stroke (width 0) (type default))
-  )
+  (wire (pts (xy 317.5 231.14) (xy 320.04 231.14))
+    (stroke (width 0) (type default))
+  )

Commit message: 抵抗修正
3.3k -> 3k (1608)
15k -> 100k (1005, プルアップ/ダウン), 5.1k (1005, LED用)
Parts:
- R503, R504, R505, R506, R507, R508, R509, R510, R511, R512, R513, R514: value 3.3k -> 3k; footprint Resistor_SMD:R_0402_1005Metric -> Resistor_SMD:R_0603_1608Metric
Changed lines of the file:
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@@
       (effects (font (size 1.27 1.27)))
     )
-    (property "Value" "3.3k" (at 139.7 345.44 90)
-      (effects (font (size 1.27 1.27)))
-    )
-    (property "Footprint" "Resistor_SMD:R_0402_1005Metric" (at 139.7 349.758 90)
+    (property "Value" "3k" (at 139.7 345.44 90)
+      (effects (font (size 1.27 1.27)))
+    )
+    (property "Footprint" "Resistor_SMD:R_0603_1608Metric" (at 139.7 349.758 90)
       (effects (font (size 1.27 1.27)) hide)
     )
@@
       (effects (font (size 1.27 1.27)))
     )
-    (property "Value" "3.3k" (at 139.7 176.53 90)
-      (effects (font (size 1.27 1.27)))
-    )
-    (property "Footprint" "Resistor_SMD:R_0402_1005Metric" (at 139.7 180.848 90)
+    (property "Value" "3k" (at 139.7 176.53 90)
+      (effects (font (size 1.27 1.27)))
+    )
+    (property "Footprint" "Resistor_SMD:R_0603_1608Metric" (at 139.7 180.848 90)
       (effects (font (size 1.27 1.27)) hide)
     )
@@
       (effects (font (size 1.27 1.27)))
     )
-    (property "Value" "3.3k" (at 139.7 128.27 90)
-      (effects (font (size 1.27 1.27)))
-    )
-    (property "Footprint" "Resistor_SMD:R_0402_1005Metric" (at 139.7 132.588 90)
+    (property "Value" "3k" (at 139.7 128.27 90)
+      (effects (font (size 1.27 1.27)))
+    )
+    (property "Footprint" "Resistor_SMD:R_0603_1608Metric" (at 139.7 132.588 90)
       (effects (font (size 1.27 1.27)) hide)
     )
@@
       (effects (font (size 1.27 1.27)))
     )
-    (property "Value" "3.3k" (at 139.7 104.14 90)
-      (effects (font (size 1.27 1.27)))
-    )
-    (property "Footprint" "Resistor_SMD:R_0402_1005Metric" (at 139.7 108.458 90)
+    (property "Value" "3k" (at 139.7 104.14 90)
+      (effects (font (size 1.27 1.27)))
+    )
+    (property "Footprint" "Resistor_SMD:R_0603_1608Metric" (at 139.7 108.458 90)
       (effects (font (size 1.27 1.27)) hide)
     )
@@
       (effects (font (size 1.27 1.27)))
     )
-    (property "Value" "3.3k" (at 139.7 248.92 90)
-      (effects (font (size 1.27 1.27)))
-    )
-    (property "Footprint" "Resistor_SMD:R_0402_1005Metric" (at 139.7 253.238 90)
+    (property "Value" "3k" (at 139.7 248.92 90)
+      (effects (font (size 1.27 1.27)))
+    )
+    (property "Footprint" "Resistor_SMD:R_0603_1608Metric" (at 139.7 253.238 90)
       (effects (font (size 1.27 1.27)) hide)
     )
@@
       (effects (font (size 1.27 1.27)))
     )
-    (property "Value" "3.3k" (at 139.7 224.79 90)
-      (effects (font (size 1.27 1.27)))
-    )
-    (property "Footprint" "Resistor_SMD:R_0402_1005Metric" (at 139.7 229.108 90)
+    (property "Value" "3k" (at 139.7 224.79 90)
+      (effects (font (size 1.27 1.27)))
+    )
+    (property "Footprint" "Resistor_SMD:R_0603_1608Metric" (at 139.7 229.108 90)
       (effects (font (size 1.27 1.27)) hide)
     )
@@
       (effects (font (size 1.27 1.27)))
     )
-    (property "Value" "3.3k" (at 139.7 297.18 90)
-      (effects (font (size 1.27 1.27)))
-    )
-    (property "Footprint" "Resistor_SMD:R_0402_1005Metric" (at 139.7 301.498 90)
+    (property "Value" "3k" (at 139.7 297.18 90)
+      (effects (font (size 1.27 1.27)))
+    )
+    (property "Footprint" "Resistor_SMD:R_0603_1608Metric" (at 139.7 301.498 90)
       (effects (font (size 1.27 1.27)) hide)
     )
@@
       (effects (font (size 1.27 1.27)))
     )
-    (property "Value" "3.3k" (at 139.7 200.66 90)
-      (effects (font (size 1.27 1.27)))
-    )
-    (property "Footprint" "Resistor_SMD:R_0402_1005Metric" (at 139.7 204.978 90)
+    (property "Value" "3k" (at 139.7 200.66 90)
+      (effects (font (size 1.27 1.27)))
+    )
+    (property "Footprint" "Resistor_SMD:R_0603_1608Metric" (at 139.7 204.978 90)
       (effects (font (size 1.27 1.27)) hide)
     )
@@
       (effects (font (size 1.27 1.27)))
     )
-    (property "Value" "3.3k" (at 139.7 152.4 90)
-      (effects (font (size 1.27 1.27)))
-    )
-    (property "Footprint" "Resistor_SMD:R_0402_1005Metric" (at 139.7 156.718 90)
+    (property "Value" "3k" (at 139.7 152.4 90)
+      (effects (font (size 1.27 1.27)))
+    )
+    (property "Footprint" "Resistor_SMD:R_0603_1608Metric" (at 139.7 156.718 90)
       (effects (font (size 1.27 1.27)) hide)
     )
@@
       (effects (font (size 1.27 1.27)))
     )
-    (property "Value" "3.3k" (at 139.7 273.05 90)
-      (effects (font (size 1.27 1.27)))
-    )
-    (property "Footprint" "Resistor_SMD:R_0402_1005Metric" (at 139.7 277.368 90)
+    (property "Value" "3k" (at 139.7 273.05 90)
+      (effects (font (size 1.27 1.27)))
+    )
+    (property "Footprint" "Resistor_SMD:R_0603_1608Metric" (at 139.7 277.368 90)
       (effects (font (size 1.27 1.27)) hide)
     )
@@
       (effects (font (size 1.27 1.27)))
     )
-    (property "Value" "3.3k" (at 139.7 321.31 90)
-      (effects (font (size 1.27 1.27)))
-    )
-    (property "Footprint" "Resistor_SMD:R_0402_1005Metric" (at 139.7 325.628 90)
+    (property "Value" "3k" (at 139.7 321.31 90)
+      (effects (font (size 1.27 1.27)))
+    )
+    (property "Footprint" "Resistor_SMD:R_0603_1608Metric" (at 139.7 325.628 90)
       (effects (font (size 1.27 1.27)) hide)
     )
@@
       (effects (font (size 1.27 1.27)))
     )
-    (property "Value" "3.3k" (at 139.7 80.01 90)
-      (effects (font (size 1.27 1.27)))
-    )
-    (property "Footprint" "Resistor_SMD:R_0402_1005Metric" (at 139.7 84.328 90)
-      (effects (font (size 1.27 1.27)) hide)
-    )
+    (property "Value" "3k" (at 139.7 80.01 90)
+      (effects (font (size 1.27 1.27)))
+    )
+    (property "Footprint" "Resistor_SMD:R_0603_1608Metric" (at 139.7 84.328 90)
+      (effects (font (size 1.27 1.27)) hide)
+    )

Commit message: アノテーションし直し
Parts:
- renumbered C260 to C269, C261 to C270, C262 to C271, C263 to C272, C264 to C273, C265 to C274, C266 to C275, C267 to C276, C268 to C277, C269 to C278, C270 to C279, C271 to C280, C272 to C281, C273 to C282, C274 to C283, C275 to C284, C276 to C285, C277 to C286, C278 to C287, C279 to C288, C280 to C289, C281 to C290, C282 to C291, C283 to C292, C284 to C293, C285 to C294, C286 to C295, C287 to C296, C288 to C297, C289 to C298, C290 to C299, C291 to C300, C292 to C301, C293 to C302, C294 to C303, C295 to C304, L18 to L14
