File: AMS-board-2024/AMS-board-2024.kicad_sch (KiCad schematic)
At the start: 45 parts, among them J1 19427-0049, J10 19427-0049, J11 19427-0049, J12 19427-0049, J13 19427-0049, J14 19427-0049, J15 19427-0040, J16 19427-0040, J17 19427-0049, J18 19427-0049, J19 19427-0017, J2 19427-0049, J20 19427-0018, J21 19427-0040, J22 PinHeader_02x05_P1.00mm, J23 19427-0040, J24 5077CR-16-SMC2-BK-TR, J3 19427-0049, J4 19427-0049, J5 19427-0049, J6 19427-0049, J7 19427-0049, J8 19427-0049, J9 19427-0049

Commit message: 高電圧コネクタのMPの接続をNCに修正
Connections:
- net Battery Stack Monitor/V_{BAT}-: no longer J15.MP (MountPin), J16.MP (MountPin)
- no-connect marks 67 -> 69
Changed lines of the file:
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@@
   (junction (at 388.62 74.93) (diameter 0) (color 0 0 0 0)
   )
-  (junction (at 226.06 215.9) (diameter 0) (color 0 0 0 0)
-  )
   (junction (at 355.6 187.96) (diameter 0) (color 0 0 0 0)
   )
@@
   )
   (junction (at 289.56 208.28) (diameter 0) (color 0 0 0 0)
-  )
-  (junction (at 226.06 208.28) (diameter 0) (color 0 0 0 0)
   )
   (junction (at 381 74.93) (diameter 0) (color 0 0 0 0)
@@
   (no_connect (at 365.76 66.04))
   (no_connect (at 86.36 271.78))
+  (no_connect (at 218.44 231.14))
   (no_connect (at 170.18 175.26))
   (no_connect (at 175.26 271.78))
   (no_connect (at 45.72 149.86))
+  (no_connect (at 218.44 213.36))
   (no_connect (at 170.18 88.9))
   (no_connect (at 223.52 63.5))
@@
     (stroke (width 0) (type default))
   )
-  (wire (pts (xy 223.52 208.28) (xy 226.06 208.28))
+  (wire (pts (xy 223.52 208.28) (xy 228.6 208.28))
     (stroke (width 0) (type default))
   )
@@
     (stroke (width 0) (type default))
   )
-  (wire (pts (xy 226.06 215.9) (xy 226.06 208.28))
-    (stroke (width 0) (type default))
-  )
   (wire (pts (xy 134.62 116.84) (xy 139.7 116.84))
     (stroke (width 0) (type default))
@@
     (stroke (width 0) (type default))
   )
-  (wire (pts (xy 226.06 215.9) (xy 226.06 233.68))
-    (stroke (width 0) (type default))
-  )
   (wire (pts (xy 170.18 76.2) (xy 165.1 76.2))
     (stroke (width 0) (type default))
@@
     (stroke (width 0) (type default))
   )
-  (wire (pts (xy 218.44 231.14) (xy 218.44 233.68))
-    (stroke (width 0) (type default))
-  )
   (wire (pts (xy 76.2 119.38) (xy 81.28 119.38))
     (stroke (width 0) (type default))
@@
     (stroke (width 0) (type default))
   )
-  (wire (pts (xy 218.44 215.9) (xy 226.06 215.9))
-    (stroke (width 0) (type default))
-  )
   (wire (pts (xy 134.62 132.08) (xy 139.7 132.08))
     (stroke (width 0) (type default))
@@
     (stroke (width 0) (type default))
   )
-  (wire (pts (xy 218.44 213.36) (xy 218.44 215.9))
-    (stroke (width 0) (type default))
-  )
   (wire (pts (xy 254 213.36) (xy 259.08 213.36))
     (stroke (width 0) (type default))
@@
     (stroke (width 0) (type default))
   )
-  (wire (pts (xy 226.06 233.68) (xy 218.44 233.68))
-    (stroke (width 0) (type default))
-  )
   (wire (pts (xy 78.74 116.84) (xy 78.74 114.3))
     (stroke (width 0) (type default))
@@
     (stroke (width 0) (type default))
   )
-  (wire (pts (xy 226.06 208.28) (xy 228.6 208.28))
-    (stroke (width 0) (type default))
-  )

Commit message: 階層シート内の電源シンボル修正
階層シート内で電源シンボルをなるべく使わないようにする
修正途中
Connections:
- net Battery Module Monitor 1/Thermistor1- is gone; now on net Battery Module Monitor 1/GND: J9.5 (Pin_5)
- net Battery Module Monitor 1/Thermistor2- is gone; now on net Battery Module Monitor 1/GND: J9.7 (Pin_7)
- net Battery Module Monitor 1/Thermistor3- is gone; now on net Battery Module Monitor 1/GND: J9.9 (Pin_9)
- net Battery Module Monitor 1/Thermistor4- is gone; now on net Battery Module Monitor 1/GND: J9.11 (Pin_11)
- net Battery Module Monitor 1/Thermistor5- is gone; now on net Battery Module Monitor 1/GND: J9.13 (Pin_13)
- net Battery Module Monitor 2/Thermistor1- is gone; now on net Battery Module Monitor 2/GND: J10.5 (Pin_5)
- net Battery Module Monitor 2/Thermistor2- is gone; now on net Battery Module Monitor 2/GND: J10.7 (Pin_7)
- net Battery Module Monitor 2/Thermistor3- is gone; now on net Battery Module Monitor 2/GND: J10.9 (Pin_9)
- net Battery Module Monitor 2/Thermistor4- is gone; now on net Battery Module Monitor 2/GND: J10.11 (Pin_11)
- net Battery Module Monitor 2/Thermistor5- is gone; now on net Battery Module Monitor 2/GND: J10.13 (Pin_13)
- net Battery Module Monitor 3/Thermistor1- is gone; now on net Battery Module Monitor 3/GND: J11.5 (Pin_5)
- net Battery Module Monitor 3/Thermistor2- is gone; now on net Battery Module Monitor 3/GND: J11.7 (Pin_7)
- net Battery Module Monitor 3/Thermistor3- is gone; now on net Battery Module Monitor 3/GND: J11.9 (Pin_9)
- net Battery Module Monitor 3/Thermistor4- is gone; now on net Battery Module Monitor 3/GND: J11.11 (Pin_11)
- net Battery Module Monitor 3/Thermistor5- is gone; now on net Battery Module Monitor 3/GND: J11.13 (Pin_13)
- net Battery Module Monitor 1/GND1 renamed Battery Module Monitor 1/GND
- net Battery Module Monitor 2/GND2 renamed Battery Module Monitor 2/GND
- net Battery Module Monitor 3/GND3 renamed Battery Module Monitor 3/GND
Other:
- sheet Battery Module Monitor 1 ports: added GND; removed GND1, Thermistor1-, Thermistor2-, Thermistor3-, Thermistor4-, Thermistor5-
- sheet Battery Module Monitor 2 ports: added GND; removed GND2, Thermistor1-, Thermistor2-, Thermistor3-, Thermistor4-, Thermistor5-
- sheet Battery Module Monitor 3 ports: added GND; removed GND3, Thermistor1-, Thermistor2-, Thermistor3-, Thermistor4-, Thermistor5-
- sheet MCU ports: added VBUS+_U, VBUS-_U; removed none
- moved on the sheet: J21
