File: AMS-board-2024/AMS-board-2024.kicad_sch (KiCad schematic)
At the start: 46 parts, among them J1 XH_6pin_Side, J10 XH_6pin_Side, J11 XH_7pin_Side, J12 XH_6pin_Side, J13 XH_7pin_Side, J14 XH_6pin_Side, J15 XH_7pin_Side, J16 XH_6pin_Side, J17 XH_6pin_Side, J18 XH_6pin_Side, J19 19427-0040, J2 XH_7pin_Side, J20 19427-0040, J21 XH_6pin_Side, J22 XH_7pin_Side, J23 XH_6pin_Side, J24 XH_7pin_Side, J25 XH_6pin_Side, J26 XH_6pin_Side, J27 XH_2pin_Side, J28 XH_6pin_Side, J29 XH_8pin_Side, J3 XH_6pin_Side, J30 PinHeader_02x05_P1.00mm, J31 XH_2pin_Side, J32 5077CR-16-SMC2-BK-TR, J4 XH_7pin_Side, J5 XH_6pin_Side, J6 XH_7pin_Side, J7 XH_6pin_Side, J8 XH_6pin_Side, J9 XH_6pin_Side

Commit message: VBUSのPWR_FLAG追加
Changed lines of the file:
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@@
   (junction (at 256.54 68.58) (diameter 0) (color 0 0 0 0)
+  )
+  (junction (at 363.22 73.66) (diameter 0) (color 0 0 0 0)
   )
   (junction (at 78.74 78.74) (diameter 0) (color 0 0 0 0)
@@
   )
   (wire (pts (xy 167.64 231.14) (xy 170.18 231.14))
+    (stroke (width 0) (type default))
+  )
+  (wire (pts (xy 355.6 73.66) (xy 363.22 73.66))
     (stroke (width 0) (type default))
   )
@@
         )
       )
+    )
+  )
+  (symbol (lib_id "power:PWR_FLAG") (at 355.6 73.66 0) (unit 1)
+    (in_bom yes) (on_board yes) (dnp no) (fields_autoplaced)
+    (property "Reference" "#FLG028" (at 355.6 71.755 0)
+      (effects (font (size 1.27 1.27)) hide)
+    )
+    (property "Value" "PWR_FLAG" (at 355.6 68.58 0)
+      (effects (font (size 1.27 1.27)))
+    )
+    (property "Footprint" "" (at 355.6 73.66 0)
+      (effects (font (size 1.27 1.27)) hide)
+    )
+    (property "Datasheet" "~" (at 355.6 73.66 0)
+      (effects (font (size 1.27 1.27)) hide)
+    )
+    (pin "1")
+    (instances
+      (project "AMS-board-2024"
+        (path "/3a719eb3-09ce-4343-8f6e-20cc0aaf5261"
+          (reference "#FLG028") (unit 1)
+        )
+      )

Commit message: 固定用穴追加
Parts:
- removed J29: XH_8pin_Side, Connector_JST:JST_XH_S8B-XH-A_1x08_P2.50mm_Horizontal, symbol Connector_Generic:Conn_01x08
- added C382: 1000p, Capacitor_SMD:C_1206_3216Metric, symbol Device:C
- added H3, H4, H5, H6, H7, H8: MountingHole_Pad, MountingHole:MountingHole_6.4mm_M6_Pad_Via, symbol Mechanical:MountingHole_Pad
- added J29, J33: XH_5pin_Side, Connector_JST:JST_XH_S5B-XH-A_1x05_P2.50mm_Horizontal, symbol Connector_Generic:Conn_01x05
Connections:
- net +5V: now also J29.1 (Pin_1), J33.1 (Pin_1)
- net GND: now also C382.2, J29.2 (Pin_2), J33.2 (Pin_2)
- net MCU/A1: now also J33.3 (Pin_3)
- net MCU/A2: now also J33.4 (Pin_4)
- net MCU/A3: now also J33.5 (Pin_5)
- net MCU/D2: now also J29.3 (Pin_3)
- net MCU/D6: now also J29.4 (Pin_4)
- net MCU/D7: now also J29.5 (Pin_5)
- new net: C382.1, H3.1
- no-connect marks 5 -> 10
Other:
- note added: "1kV, 3216"

Commit message: 5V OUT のピンアサイン修正
Connections:
- net MCU/D0: now also J28.5 (Pin_5); no longer J28.3 (Pin_3)
- net MCU/D1: now also J28.6 (Pin_6); no longer J28.4 (Pin_4)
- net MCU/D8: now also J28.3 (Pin_3); no longer J28.5 (Pin_5)
- net MCU/D9: now also J28.4 (Pin_4); no longer J28.6 (Pin_6)
Changed lines of the file:
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@@
       (effects (font (size 1.27 1.27)) (justify left))
     )
-    (pin "D9" output (at 317.5 154.94 180)
+    (pin "D9" output (at 317.5 149.86 180)
       (effects (font (size 1.27 1.27)) (justify left))
     )
-    (pin "D8" output (at 317.5 152.4 180)
+    (pin "D8" output (at 317.5 147.32 180)
       (effects (font (size 1.27 1.27)) (justify left))
     )
-    (pin "D1" output (at 317.5 149.86 180)
+    (pin "D1" output (at 317.5 154.94 180)
       (effects (font (size 1.27 1.27)) (justify left))
     )
-    (pin "D0" output (at 317.5 147.32 180)
+    (pin "D0" output (at 317.5 152.4 180)
       (effects (font (size 1.27 1.27)) (justify left))
     )

Commit message: 5V OUT ピンアサイン修正
Connections:
- net MCU/D0: now also J28.3 (Pin_3); no longer J28.5 (Pin_5)
- net MCU/D1: now also J28.4 (Pin_4); no longer J28.6 (Pin_6)
- net MCU/D8: now also J28.5 (Pin_5); no longer J28.3 (Pin_3)
- net MCU/D9: now also J28.6 (Pin_6); no longer J28.4 (Pin_4)
Changed lines of the file:
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@@
       (effects (font (size 1.27 1.27)) (justify left))
     )
-    (pin "D9" output (at 317.5 149.86 180)
+    (pin "D9" output (at 317.5 154.94 180)
       (effects (font (size 1.27 1.27)) (justify left))
     )
-    (pin "D8" output (at 317.5 147.32 180)
+    (pin "D8" output (at 317.5 152.4 180)
       (effects (font (size 1.27 1.27)) (justify left))
     )
-    (pin "D1" output (at 317.5 154.94 180)
+    (pin "D1" output (at 317.5 149.86 180)
       (effects (font (size 1.27 1.27)) (justify left))
     )
-    (pin "D0" output (at 317.5 152.4 180)
+    (pin "D0" output (at 317.5 147.32 180)
       (effects (font (size 1.27 1.27)) (justify left))
     )

Commit message: セル監視用コネクタを表面実装XHに変更
Parts:
- removed J1, J10, J12, J14, J16, J17, J18, J21, J23, J25, J26, J3, J5, J7, J8, J9: XH_6pin_Side, Connector_JST:JST_XH_S6B-XH-A_1x06_P2.50mm_Horizontal, symbol Connector_Generic:Conn_01x06
- removed J11, J13, J15, J2, J22, J24, J4, J6: XH_7pin_Side, Connector_JST:JST_XH_S7B-XH-A_1x07_P2.50mm_Horizontal, symbol Connector_Generic:Conn_01x07
- added J1, J10, J13, J16, J21, J24, J34, J35, J36, J37, J38, J39, J4, J40, J41, J7: XH_6pin_SMT, ProjectEV:Connector_S6B-XH-SM4-TB, symbol ProjectEV:Connector_XH_6pin_SMT
- added J11, J14, J17, J2, J22, J25, J5, J8: XH_3pin_SMT, ProjectEV:Connector_S3B-XH-SM4-TB, symbol ProjectEV:Connector_XH_3pin_SMT
- added J12, J15, J18, J23, J26, J3, J6, J9: XH_4pin_SMT, ProjectEV:Connector_S4B-XH-SM4-TB, symbol ProjectEV:Connector_XH_4pin_SMT
Connections:
- net Battery Module Monitor 1/CELL0: now also J3.4 (Pin_4)
- net Battery Module Monitor 1/CELL1: now also J3.3 (Pin_3)
- net Battery Module Monitor 1/CELL10: now also J1.3 (Pin_3)
- net Battery Module Monitor 1/CELL11: now also J1.2 (Pin_2)
- net Battery Module Monitor 1/CELL12: now also J1.1 (Pin_1)
- net Battery Module Monitor 1/CELL2: now also J3.2 (Pin_2)
- net Battery Module Monitor 1/CELL3: now also J3.1 (Pin_1)
- net Battery Module Monitor 1/CELL4: now also J2.3 (Pin_3)
- net Battery Module Monitor 1/CELL5: now also J2.2 (Pin_2)
- net Battery Module Monitor 1/CELL6: now also J2.1 (Pin_1)
- net Battery Module Monitor 1/CELL7: now also J1.6 (Pin_6)
- net Battery Module Monitor 1/CELL8: now also J1.5 (Pin_5)
- net Battery Module Monitor 1/CELL9: now also J1.4 (Pin_4)
- net Battery Module Monitor 1/Thermistor1+: now also J34.1 (Pin_1)
- net Battery Module Monitor 1/Thermistor2+: now also J34.3 (Pin_3)
- net Battery Module Monitor 1/Thermistor3+: now also J34.5 (Pin_5)
- net Battery Module Monitor 2/CELL0: now also J6.4 (Pin_4)
- net Battery Module Monitor 2/CELL1: now also J6.3 (Pin_3)
- net Battery Module Monitor 2/CELL10: now also J4.3 (Pin_3)
- net Battery Module Monitor 2/CELL11: now also J4.2 (Pin_2)
- net Battery Module Monitor 2/CELL12: now also J4.1 (Pin_1)
- net Battery Module Monitor 2/CELL2: now also J6.2 (Pin_2)
- net Battery Module Monitor 2/CELL3: now also J6.1 (Pin_1)
- net Battery Module Monitor 2/CELL4: now also J5.3 (Pin_3)
- net Battery Module Monitor 2/CELL5: now also J5.2 (Pin_2)
- net Battery Module Monitor 2/CELL6: now also J5.1 (Pin_1)
- net Battery Module Monitor 2/CELL7: now also J4.6 (Pin_6)
- net Battery Module Monitor 2/CELL8: now also J4.5 (Pin_5)
- net Battery Module Monitor 2/CELL9: now also J4.4 (Pin_4)
- net Battery Module Monitor 2/Thermistor1+: now also J35.1 (Pin_1)
- net Battery Module Monitor 2/Thermistor2+: now also J35.3 (Pin_3)
- net Battery Module Monitor 2/Thermistor3+: now also J35.5 (Pin_5)
- net Battery Module Monitor 3/CELL0: now also J9.4 (Pin_4)
- net Battery Module Monitor 3/CELL1: now also J9.3 (Pin_3)
- net Battery Module Monitor 3/CELL10: now also J7.3 (Pin_3)
- net Battery Module Monitor 3/CELL11: now also J7.2 (Pin_2)
- net Battery Module Monitor 3/CELL12: now also J7.1 (Pin_1)
- net Battery Module Monitor 3/CELL2: now also J9.2 (Pin_2)
- net Battery Module Monitor 3/CELL3: now also J9.1 (Pin_1)
- net Battery Module Monitor 3/CELL4: now also J8.3 (Pin_3)
- net Battery Module Monitor 3/CELL5: now also J8.2 (Pin_2)
- net Battery Module Monitor 3/CELL6: now also J8.1 (Pin_1)
- net Battery Module Monitor 3/CELL7: now also J7.6 (Pin_6)
- net Battery Module Monitor 3/CELL8: now also J7.5 (Pin_5)
- net Battery Module Monitor 3/CELL9: now also J7.4 (Pin_4)
- net Battery Module Monitor 3/Thermistor1+: now also J36.1 (Pin_1)
- net Battery Module Monitor 3/Thermistor2+: now also J36.3 (Pin_3)
- net Battery Module Monitor 3/Thermistor3+: now also J36.5 (Pin_5)
- net Battery Module Monitor 4/CELL0: now also J12.4 (Pin_4)
- net Battery Module Monitor 4/CELL1: now also J12.3 (Pin_3)
- net Battery Module Monitor 4/CELL10: now also J10.3 (Pin_3)
- net Battery Module Monitor 4/CELL11: now also J10.2 (Pin_2)
- net Battery Module Monitor 4/CELL12: now also J10.1 (Pin_1)
- net Battery Module Monitor 4/CELL2: now also J12.2 (Pin_2)
- net Battery Module Monitor 4/CELL3: now also J12.1 (Pin_1)
- net Battery Module Monitor 4/CELL4: now also J11.3 (Pin_3)
- net Battery Module Monitor 4/CELL5: now also J11.2 (Pin_2)
- net Battery Module Monitor 4/CELL6: now also J11.1 (Pin_1)
- net Battery Module Monitor 4/CELL7: now also J10.6 (Pin_6)
- net Battery Module Monitor 4/CELL8: now also J10.5 (Pin_5)
- net Battery Module Monitor 4/CELL9: now also J10.4 (Pin_4)
- net Battery Module Monitor 4/Thermistor1+: now also J37.1 (Pin_1)
- net Battery Module Monitor 4/Thermistor2+: now also J37.3 (Pin_3)
- net Battery Module Monitor 4/Thermistor3+: now also J37.5 (Pin_5)
- net Battery Module Monitor 5/CELL0: now also J15.4 (Pin_4)
- net Battery Module Monitor 5/CELL1: now also J15.3 (Pin_3)
- net Battery Module Monitor 5/CELL10: now also J13.3 (Pin_3)
- net Battery Module Monitor 5/CELL11: now also J13.2 (Pin_2)
- net Battery Module Monitor 5/CELL12: now also J13.1 (Pin_1)
- net Battery Module Monitor 5/CELL2: now also J15.2 (Pin_2)
- net Battery Module Monitor 5/CELL3: now also J15.1 (Pin_1)
- net Battery Module Monitor 5/CELL4: now also J14.3 (Pin_3)
- net Battery Module Monitor 5/CELL5: now also J14.2 (Pin_2)
- net Battery Module Monitor 5/CELL6: now also J14.1 (Pin_1)
- net Battery Module Monitor 5/CELL7: now also J13.6 (Pin_6)
- net Battery Module Monitor 5/CELL8: now also J13.5 (Pin_5)
- net Battery Module Monitor 5/CELL9: now also J13.4 (Pin_4)
- net Battery Module Monitor 5/Thermistor1+: now also J38.1 (Pin_1)
- net Battery Module Monitor 5/Thermistor2+: now also J38.3 (Pin_3)
- net Battery Module Monitor 5/Thermistor3+: now also J38.5 (Pin_5)
- net Battery Module Monitor 6/CELL0: now also J18.4 (Pin_4)
- net Battery Module Monitor 6/CELL1: now also J18.3 (Pin_3)
- net Battery Module Monitor 6/CELL10: now also J16.3 (Pin_3)
- net Battery Module Monitor 6/CELL11: now also J16.2 (Pin_2)
- net Battery Module Monitor 6/CELL12: now also J16.1 (Pin_1)
- net Battery Module Monitor 6/CELL2: now also J18.2 (Pin_2)
- net Battery Module Monitor 6/CELL3: now also J18.1 (Pin_1)
- net Battery Module Monitor 6/CELL4: now also J17.3 (Pin_3)
- net Battery Module Monitor 6/CELL5: now also J17.2 (Pin_2)
- net Battery Module Monitor 6/CELL6: now also J17.1 (Pin_1)
- net Battery Module Monitor 6/CELL7: now also J16.6 (Pin_6)
- net Battery Module Monitor 6/CELL8: now also J16.5 (Pin_5)
- net Battery Module Monitor 6/CELL9: now also J16.4 (Pin_4)
- net Battery Module Monitor 6/Thermistor1+: now also J39.1 (Pin_1)
- net Battery Module Monitor 6/Thermistor2+: now also J39.3 (Pin_3)
- net Battery Module Monitor 6/Thermistor3+: now also J39.5 (Pin_5)
- net Battery Module Monitor 7/CELL0: now also J23.4 (Pin_4)
- net Battery Module Monitor 7/CELL1: now also J23.3 (Pin_3)
- net Battery Module Monitor 7/CELL10: now also J21.3 (Pin_3)
- net Battery Module Monitor 7/CELL11: now also J21.2 (Pin_2)
- net Battery Module Monitor 7/CELL12: now also J21.1 (Pin_1)
- net Battery Module Monitor 7/CELL2: now also J23.2 (Pin_2)
- net Battery Module Monitor 7/CELL3: now also J23.1 (Pin_1)
- net Battery Module Monitor 7/CELL4: now also J22.3 (Pin_3)
- net Battery Module Monitor 7/CELL5: now also J22.2 (Pin_2)
- net Battery Module Monitor 7/CELL6: now also J22.1 (Pin_1)
- net Battery Module Monitor 7/CELL7: now also J21.6 (Pin_6)
- net Battery Module Monitor 7/CELL8: now also J21.5 (Pin_5)
- net Battery Module Monitor 7/CELL9: now also J21.4 (Pin_4)
- net Battery Module Monitor 7/Thermistor1+: now also J40.1 (Pin_1)
- net Battery Module Monitor 7/Thermistor2+: now also J40.3 (Pin_3)
- net Battery Module Monitor 7/Thermistor3+: now also J40.5 (Pin_5)
- net Battery Module Monitor 8/CELL0: now also J26.4 (Pin_4)
- net Battery Module Monitor 8/CELL1: now also J26.3 (Pin_3)
- net Battery Module Monitor 8/CELL10: now also J24.3 (Pin_3)
- net Battery Module Monitor 8/CELL11: now also J24.2 (Pin_2)
- net Battery Module Monitor 8/CELL12: now also J24.1 (Pin_1)
- net Battery Module Monitor 8/CELL2: now also J26.2 (Pin_2)
- net Battery Module Monitor 8/CELL3: now also J26.1 (Pin_1)
- net Battery Module Monitor 8/CELL4: now also J25.3 (Pin_3)
- net Battery Module Monitor 8/CELL5: now also J25.2 (Pin_2)
- net Battery Module Monitor 8/CELL6: now also J25.1 (Pin_1)
- net Battery Module Monitor 8/CELL7: now also J24.6 (Pin_6)
- net Battery Module Monitor 8/CELL8: now also J24.5 (Pin_5)
- net Battery Module Monitor 8/CELL9: now also J24.4 (Pin_4)
- net Battery Module Monitor 8/Thermistor1+: now also J41.1 (Pin_1)
- net Battery Module Monitor 8/Thermistor2+: now also J41.3 (Pin_3)
- net Battery Module Monitor 8/Thermistor3+: now also J41.5 (Pin_5)
- net GND1: now also J34.2 (Pin_2), J34.4 (Pin_4), J34.6 (Pin_6)
- net GND2: now also J35.2 (Pin_2), J35.4 (Pin_4), J35.6 (Pin_6)
- net GND3: now also J36.2 (Pin_2), J36.4 (Pin_4), J36.6 (Pin_6)
- net GND4: now also J37.2 (Pin_2), J37.4 (Pin_4), J37.6 (Pin_6)
- net GND5: now also J38.2 (Pin_2), J38.4 (Pin_4), J38.6 (Pin_6)
- net GND6: now also J39.2 (Pin_2), J39.4 (Pin_4), J39.6 (Pin_6)
- net GND7: now also J40.2 (Pin_2), J40.4 (Pin_4), J40.6 (Pin_6)
- net GND8: now also J41.2 (Pin_2), J41.4 (Pin_4), J41.6 (Pin_6)
- no-connect marks 10 -> 42

Commit message: モジュール内のisoSPIをコンデンサ接続に変更
Parts:
- removed L1, L4, L6, L8: CEEH96B, ProjectEV:Transformer_CEEH96B, symbol ProjectEV:Transfomer_CEEH96B
- added C383, C384, C385, C386, C387, C388, C389, C390: 10n, Capacitor_SMD:C_1206_3216Metric, symbol Device:C
Connections:
- net Battery Module Monitor 1/IH_N: now also C384.1
- net Battery Module Monitor 1/IH_P: now also C383.1
- net Battery Module Monitor 2/IL_N: now also C384.2
- net Battery Module Monitor 2/IL_P: now also C383.2
- net Battery Module Monitor 3/IH_N: now also C386.1
- net Battery Module Monitor 3/IH_P: now also C385.1
- net Battery Module Monitor 4/IL_N: now also C386.2
- net Battery Module Monitor 4/IL_P: now also C385.2
- net Battery Module Monitor 5/IH_N: now also C388.1
- net Battery Module Monitor 5/IH_P: now also C387.1
- net Battery Module Monitor 6/IL_N: now also C388.2
- net Battery Module Monitor 6/IL_P: now also C387.2
- net Battery Module Monitor 7/IH_N: now also C390.1
- net Battery Module Monitor 7/IH_P: now also C389.1
- net Battery Module Monitor 8/IL_N: now also C390.2
- net Battery Module Monitor 8/IL_P: now also C389.2
Other:
- moved on the sheet: L2

Commit message: セル監視コネクタを34691-0200に変更
Parts:
- removed J1, J10, J13, J16, J21, J24, J34, J35, J36, J37, J38, J39, J4, J40, J41, J7: XH_6pin_SMT, ProjectEV:Connector_S6B-XH-SM4-TB, symbol ProjectEV:Connector_XH_6pin_SMT
- removed J11, J14, J17, J2, J22, J25, J5, J8: XH_3pin_SMT, ProjectEV:Connector_S3B-XH-SM4-TB, symbol ProjectEV:Connector_XH_3pin_SMT
- removed J12, J15, J18, J23, J26, J3, J6, J9: XH_4pin_SMT, ProjectEV:Connector_S4B-XH-SM4-TB, symbol ProjectEV:Connector_XH_4pin_SMT
- added J1, J2, J3, J4, J5, J6, J7, J8: 34691-0200, ProjectEV:Connector_34691-0200, symbol ProjectEV:Connector_34691-0200
Connections:
- net Battery Module Monitor 1/CELL0: now also J1.7 (Pin_7)
- net Battery Module Monitor 1/CELL1: now also J1.16 (Pin_16)
- net Battery Module Monitor 1/CELL10: now also J1.2 (Pin_2)
- net Battery Module Monitor 1/CELL11: now also J1.11 (Pin_11)
- net Battery Module Monitor 1/CELL12: now also J1.1 (Pin_1)
- net Battery Module Monitor 1/CELL2: now also J1.6 (Pin_6)
- net Battery Module Monitor 1/CELL3: now also J1.15 (Pin_15)
- net Battery Module Monitor 1/CELL4: now also J1.5 (Pin_5)
- net Battery Module Monitor 1/CELL5: now also J1.14 (Pin_14)
- net Battery Module Monitor 1/CELL6: now also J1.4 (Pin_4)
- net Battery Module Monitor 1/CELL7: now also J1.13 (Pin_13)
- net Battery Module Monitor 1/CELL8: now also J1.3 (Pin_3)
- net Battery Module Monitor 1/CELL9: now also J1.12 (Pin_12)
- net Battery Module Monitor 1/Thermistor1+: now also J1.8 (Pin_8)
- net Battery Module Monitor 1/Thermistor2+: now also J1.9 (Pin_9)
- net Battery Module Monitor 1/Thermistor3+: now also J1.10 (Pin_10)
- net Battery Module Monitor 2/CELL0: now also J2.7 (Pin_7)
- net Battery Module Monitor 2/CELL1: now also J2.16 (Pin_16)
- net Battery Module Monitor 2/CELL10: now also J2.2 (Pin_2)
- net Battery Module Monitor 2/CELL11: now also J2.11 (Pin_11)
- net Battery Module Monitor 2/CELL12: now also J2.1 (Pin_1)
- net Battery Module Monitor 2/CELL2: now also J2.6 (Pin_6)
- net Battery Module Monitor 2/CELL3: now also J2.15 (Pin_15)
- net Battery Module Monitor 2/CELL4: now also J2.5 (Pin_5)
- net Battery Module Monitor 2/CELL5: now also J2.14 (Pin_14)
- net Battery Module Monitor 2/CELL6: now also J2.4 (Pin_4)
- net Battery Module Monitor 2/CELL7: now also J2.13 (Pin_13)
- net Battery Module Monitor 2/CELL8: now also J2.3 (Pin_3)
- net Battery Module Monitor 2/CELL9: now also J2.12 (Pin_12)
- net Battery Module Monitor 2/Thermistor1+: now also J2.8 (Pin_8)
- net Battery Module Monitor 2/Thermistor2+: now also J2.9 (Pin_9)
- net Battery Module Monitor 2/Thermistor3+: now also J2.10 (Pin_10)
- net Battery Module Monitor 3/CELL0: now also J3.7 (Pin_7)
- net Battery Module Monitor 3/CELL1: now also J3.16 (Pin_16)
- net Battery Module Monitor 3/CELL10: now also J3.2 (Pin_2)
- net Battery Module Monitor 3/CELL11: now also J3.11 (Pin_11)
- net Battery Module Monitor 3/CELL12: now also J3.1 (Pin_1)
- net Battery Module Monitor 3/CELL2: now also J3.6 (Pin_6)
- net Battery Module Monitor 3/CELL3: now also J3.15 (Pin_15)
- net Battery Module Monitor 3/CELL4: now also J3.5 (Pin_5)
- net Battery Module Monitor 3/CELL5: now also J3.14 (Pin_14)
- net Battery Module Monitor 3/CELL6: now also J3.4 (Pin_4)
- net Battery Module Monitor 3/CELL7: now also J3.13 (Pin_13)
- net Battery Module Monitor 3/CELL8: now also J3.3 (Pin_3)
- net Battery Module Monitor 3/CELL9: now also J3.12 (Pin_12)
- net Battery Module Monitor 3/Thermistor1+: now also J3.8 (Pin_8)
- net Battery Module Monitor 3/Thermistor2+: now also J3.9 (Pin_9)
- net Battery Module Monitor 3/Thermistor3+: now also J3.10 (Pin_10)
- net Battery Module Monitor 4/CELL0: now also J4.7 (Pin_7)
- net Battery Module Monitor 4/CELL1: now also J4.16 (Pin_16)
- net Battery Module Monitor 4/CELL10: now also J4.2 (Pin_2)
- net Battery Module Monitor 4/CELL11: now also J4.11 (Pin_11)
- net Battery Module Monitor 4/CELL12: now also J4.1 (Pin_1)
- net Battery Module Monitor 4/CELL2: now also J4.6 (Pin_6)
- net Battery Module Monitor 4/CELL3: now also J4.15 (Pin_15)
- net Battery Module Monitor 4/CELL4: now also J4.5 (Pin_5)
- net Battery Module Monitor 4/CELL5: now also J4.14 (Pin_14)
- net Battery Module Monitor 4/CELL6: now also J4.4 (Pin_4)
- net Battery Module Monitor 4/CELL7: now also J4.13 (Pin_13)
- net Battery Module Monitor 4/CELL8: now also J4.3 (Pin_3)
- net Battery Module Monitor 4/CELL9: now also J4.12 (Pin_12)
- net Battery Module Monitor 4/Thermistor1+: now also J4.8 (Pin_8)
- net Battery Module Monitor 4/Thermistor2+: now also J4.9 (Pin_9)
- net Battery Module Monitor 4/Thermistor3+: now also J4.10 (Pin_10)
- net Battery Module Monitor 5/CELL0: now also J5.7 (Pin_7)
- net Battery Module Monitor 5/CELL1: now also J5.16 (Pin_16)
- net Battery Module Monitor 5/CELL10: now also J5.2 (Pin_2)
- net Battery Module Monitor 5/CELL11: now also J5.11 (Pin_11)
- net Battery Module Monitor 5/CELL12: now also J5.1 (Pin_1)
- net Battery Module Monitor 5/CELL2: now also J5.6 (Pin_6)
- net Battery Module Monitor 5/CELL3: now also J5.15 (Pin_15)
- net Battery Module Monitor 5/CELL4: now also J5.5 (Pin_5)
- net Battery Module Monitor 5/CELL5: now also J5.14 (Pin_14)
- net Battery Module Monitor 5/CELL6: now also J5.4 (Pin_4)
- net Battery Module Monitor 5/CELL7: now also J5.13 (Pin_13)
- net Battery Module Monitor 5/CELL8: now also J5.3 (Pin_3)
- net Battery Module Monitor 5/CELL9: now also J5.12 (Pin_12)
- net Battery Module Monitor 5/Thermistor1+: now also J5.8 (Pin_8)
- net Battery Module Monitor 5/Thermistor2+: now also J5.9 (Pin_9)
- net Battery Module Monitor 5/Thermistor3+: now also J5.10 (Pin_10)
- net Battery Module Monitor 6/CELL0: now also J6.7 (Pin_7)
- net Battery Module Monitor 6/CELL1: now also J6.16 (Pin_16)
- net Battery Module Monitor 6/CELL10: now also J6.2 (Pin_2)
- net Battery Module Monitor 6/CELL11: now also J6.11 (Pin_11)
- net Battery Module Monitor 6/CELL12: now also J6.1 (Pin_1)
- net Battery Module Monitor 6/CELL2: now also J6.6 (Pin_6)
- net Battery Module Monitor 6/CELL3: now also J6.15 (Pin_15)
- net Battery Module Monitor 6/CELL4: now also J6.5 (Pin_5)
- net Battery Module Monitor 6/CELL5: now also J6.14 (Pin_14)
- net Battery Module Monitor 6/CELL6: now also J6.4 (Pin_4)
- net Battery Module Monitor 6/CELL7: now also J6.13 (Pin_13)
- net Battery Module Monitor 6/CELL8: now also J6.3 (Pin_3)
- net Battery Module Monitor 6/CELL9: now also J6.12 (Pin_12)
- net Battery Module Monitor 6/Thermistor1+: now also J6.8 (Pin_8)
- net Battery Module Monitor 6/Thermistor2+: now also J6.9 (Pin_9)
- net Battery Module Monitor 6/Thermistor3+: now also J6.10 (Pin_10)
- net Battery Module Monitor 7/CELL0: now also J7.7 (Pin_7)
- net Battery Module Monitor 7/CELL1: now also J7.16 (Pin_16)
- net Battery Module Monitor 7/CELL10: now also J7.2 (Pin_2)
- net Battery Module Monitor 7/CELL11: now also J7.11 (Pin_11)
- net Battery Module Monitor 7/CELL12: now also J7.1 (Pin_1)
- net Battery Module Monitor 7/CELL2: now also J7.6 (Pin_6)
- net Battery Module Monitor 7/CELL3: now also J7.15 (Pin_15)
- net Battery Module Monitor 7/CELL4: now also J7.5 (Pin_5)
- net Battery Module Monitor 7/CELL5: now also J7.14 (Pin_14)
- net Battery Module Monitor 7/CELL6: now also J7.4 (Pin_4)
- net Battery Module Monitor 7/CELL7: now also J7.13 (Pin_13)
- net Battery Module Monitor 7/CELL8: now also J7.3 (Pin_3)
- net Battery Module Monitor 7/CELL9: now also J7.12 (Pin_12)
- net Battery Module Monitor 7/Thermistor1+: now also J7.8 (Pin_8)
- net Battery Module Monitor 7/Thermistor2+: now also J7.9 (Pin_9)
- net Battery Module Monitor 7/Thermistor3+: now also J7.10 (Pin_10)
- net Battery Module Monitor 8/CELL0: now also J8.7 (Pin_7)
- net Battery Module Monitor 8/CELL1: now also J8.16 (Pin_16)
- net Battery Module Monitor 8/CELL10: now also J8.2 (Pin_2)
- net Battery Module Monitor 8/CELL11: now also J8.11 (Pin_11)
- net Battery Module Monitor 8/CELL12: now also J8.1 (Pin_1)
- net Battery Module Monitor 8/CELL2: now also J8.6 (Pin_6)
- net Battery Module Monitor 8/CELL3: now also J8.15 (Pin_15)
- net Battery Module Monitor 8/CELL4: now also J8.5 (Pin_5)
- net Battery Module Monitor 8/CELL5: now also J8.14 (Pin_14)
- net Battery Module Monitor 8/CELL6: now also J8.4 (Pin_4)
- net Battery Module Monitor 8/CELL7: now also J8.13 (Pin_13)
- net Battery Module Monitor 8/CELL8: now also J8.3 (Pin_3)
- net Battery Module Monitor 8/CELL9: now also J8.12 (Pin_12)
- net Battery Module Monitor 8/Thermistor1+: now also J8.8 (Pin_8)
- net Battery Module Monitor 8/Thermistor2+: now also J8.9 (Pin_9)
- net Battery Module Monitor 8/Thermistor3+: now also J8.10 (Pin_10)
- net GND1: now also J1.18 (Pin_18), J1.19 (Pin_19), J1.20 (Pin_20)
- net GND2: now also J2.18 (Pin_18), J2.19 (Pin_19), J2.20 (Pin_20)
- net GND3: now also J3.18 (Pin_18), J3.19 (Pin_19), J3.20 (Pin_20)
- net GND4: now also J4.18 (Pin_18), J4.19 (Pin_19), J4.20 (Pin_20)
- net GND5: now also J5.18 (Pin_18), J5.19 (Pin_19), J5.20 (Pin_20)
- net GND6: now also J6.18 (Pin_18), J6.19 (Pin_19), J6.20 (Pin_20)
- net GND7: now also J7.18 (Pin_18), J7.19 (Pin_19), J7.20 (Pin_20)
- net GND8: now also J8.18 (Pin_18), J8.19 (Pin_19), J8.20 (Pin_20)
- no-connect marks 42 -> 18

Commit message: アノテーションし直し
Parts:
- renumbered C383 to C1, C384 to C2, C385 to C3, C386 to C4, C387 to C5, C388 to C6, C389 to C7, C390 to C8, C382 to C9, H6 to H5, H5 to H6, J8 to J10, J27 to J11, J28 to J12, J29 to J13, J33 to J14, J30 to J15, J31 to J16, J32 to J17, J19 to J7, J20 to J8, J7 to J9, L2 to L1, L3 to L2, L5 to L3, L7 to L4, L9 to L5, L10 to L6
