File: AMS-board-2024/battery-module-monitor-2.kicad_sch (KiCad schematic)
At the start: 144 parts, among them Q301 BSS308PE, Q302 BSS308PE, Q303 BSS308PE, Q304 BSS308PE, Q305 BSS308PE, Q306 BSS308PE, Q307 BSS308PE, Q308 BSS308PE, Q309 BSS308PE, Q310 BSS308PE, Q311 BSS308PE, Q312 BSS308PE, Q313 NSV1C201MZ4, U301 LTC6811-1

Commit message: 修正
アノテーション方法の変更：最初の空き番号から使用
Parts:
- renumbered C301 to C35, C302 to C36, C303 to C37, C304 to C38, C305 to C39, C306 to C40, C307 to C41, C308 to C42, C309 to C43, C310 to C44, C311 to C45, C312 to C46, C313 to C47, C314 to C48, C315 to C49, C316 to C50, C317 to C51, C318 to C52, C319 to C53, C320 to C54, C321 to C55, C322 to C56, C323 to C57, C324 to C58, C325 to C59, C326 to C60, C327 to C61, C328 to C62, C329 to C63, C330 to C64, C331 to C65, C332 to C66, C333 to C67, C334 to C68, D301 to D14, D302 to D15, D303 to D16, D304 to D17, D305 to D18, D306 to D19, D307 to D20, D308 to D21, D309 to D22, D310 to D23, D311 to D24, D312 to D25, D313 to D26, F301 to F14, F302 to F15, F303 to F16, F304 to F17, F305 to F18, F306 to F19, F307 to F20, F308 to F21, F309 to F22, F310 to F23, F311 to F24, F312 to F25, F313 to F26, FL301 to FL3, FL302 to FL4, L301 to L2, Q301 to Q14, Q302 to Q15, Q303 to Q16, Q304 to Q17, Q305 to Q18, Q306 to Q19, Q307 to Q20, Q308 to Q21, Q309 to Q22, Q310 to Q23, Q311 to Q24, Q312 to Q25, Q313 to Q26, R333 to R100, R334 to R101, R335 to R102, R336 to R103, R337 to R104, R338 to R105, R339 to R106, R340 to R107, R341 to R108, R342 to R109, R343 to R110, R344 to R111, R345 to R112, R346 to R113, R347 to R114, R348 to R115, R349 to R116, R350 to R117, R351 to R118, R352 to R119, R353 to R120, R354 to R121, R355 to R122, R356 to R123, R357 to R124, R358 to R125, R359 to R126, R360 to R127, R361 to R128, R362 to R129, R363 to R130, R364 to R131, R365 to R132, R366 to R133, R367 to R134, R301 to R68, R302 to R69, R303 to R70, R304 to R71, R305 to R72, R306 to R73, R307 to R74, R308 to R75, R309 to R76, R310 to R77, R311 to R78, R312 to R79, R313 to R80, R314 to R81, R315 to R82, R316 to R83, R317 to R84, R318 to R85, R319 to R86, R320 to R87, R321 to R88, R322 to R89, R323 to R90, R324 to R91, R325 to R92, R326 to R93, R327 to R94, R328 to R95, R329 to R96, R330 to R97, R331 to R98, R332 to R99, U301 to U2

Commit message: GNDシンボル追加
Connections:
- net GND2: now reaches L2.2
- net GND2: now also C35.2, C36.2, C37.2, C38.2, C39.2, C40.2, C41.2, C42.2, C43.2, C44.2, C45.2, C46.2, C59.2, C60.2, C61.1, C62.1, C63.2, C64.1, C65.1, C66.2, C67.1, C68.1, R122.1, U2.30 (V-), U2.31 (V-)

Commit message: GPIO周辺回路の修正
Parts:
- added C296, C297, C298, C299, C300: 0.1u, Capacitor_SMD:C_0603_1608Metric, symbol Device:C
- added R563, R564, R565, R566, R567: 100, Resistor_SMD:R_0603_1608Metric, symbol Device:R
Connections:
- net GND2: now also C296.2, C297.2, C298.2, C299.2, C300.2
- net Thermistor1+: now also R118.2, R563.2; no longer R129.1, U2.27 (GPIO1)
- net Thermistor2+: now also R121.2, R564.2; no longer R124.1, U2.28 (GPIO2)
- net Thermistor3+: now also R123.2, R565.2; no longer R123.1, U2.29 (GPIO3)
- net Thermistor4+: now also R124.2, R566.2; no longer R121.1, U2.32 (GPIO4)
- net Thermistor5+: now also R129.2, R567.2; no longer R118.1, U2.33 (GPIO5)
- net VREG: now reaches C63.1, Q26.3 (E), R120.1, U2.37 (VREG), U2.40 (ISOMD)
- new net: C299.1, R564.1, U2.28 (GPIO2)
- new net: C297.1, R566.1, U2.32 (GPIO4)
- new net: C298.1, R565.1, U2.29 (GPIO3)
- new net: C300.1, R563.1, U2.27 (GPIO1)
- new net: C296.1, R567.1, U2.33 (GPIO5)
- new net VREF_3V: C61.2, R118.1, R121.1, R123.1, R124.1, R129.1, U2.34 (VREF2)
Other:
- moved on the sheet: R118, R121, R123, R124, R129

Commit message: テキスト修正
Other:
- note added: "レギュレーション上必要なサーミスタは 96 CELL x 25 % = 24 本. GPIO1~3 をサーミスタに使用し、 GPIO4, 5 は別用途で使用してもOK. GPIO4, 5 のプルアップは必要に応じて実装."
- note removed: "レギュレーション上必要なサーミスタは 3 x 8 = 24 本. GPIO1~3 をサーミスタに使用し、 GPIO4, 5 は別用途で使用してもOK. GPIO4, 5 のプルアップは必要に応じて実装."
Changed lines of the file:
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@@
-    (effects (font (size 1.27 1.27)) (justify left bottom))
-  )
-  (text "レギュレーション上必要なサーミスタは 3 x 8 = 24 本.\nGPIO1~3 をサーミスタに使用し、\nGPIO4, 5 は別用途で使用してもOK.\nGPIO4, 5 のプルアップは必要に応じて実装."
-    (at 469.9 283.21 0)
     (effects (font (size 1.27 1.27)) (justify left bottom))
   )
@@
     (effects (font (size 1.27 1.27)) (justify left bottom))
   )
+  (text "レギュレーション上必要なサーミスタは 96 CELL x 25 % = 24 本.\nGPIO1~3 をサーミスタに使用し、\nGPIO4, 5 は別用途で使用してもOK.\nGPIO4, 5 のプルアップは必要に応じて実装."
+    (at 469.9 283.21 0)
+    (effects (font (size 1.27 1.27)) (justify left bottom))
+  )

Commit message: ヒューズ変更
Parts:
- removed F14, F15, F16, F17, F18, F19, F20, F21, F22, F23, F24, F25, F26: C1F 500, Fuse:Fuse_1206_3216Metric, symbol Device:Fuse
- added F301, F302, F303, F304, F305, F306, F307, F308, F309, F310, F311, F312, F313: 0679L1000-05, ProjectEV:Fuse_0679L, symbol ProjectEV:Fuse_0679L1000-05
Connections:
- net CELL0: now also F313.1
- net CELL1: now also F312.1
- net CELL10: now also F303.1
- net CELL11: now also F302.1
- net CELL12: now also F301.1
- net CELL2: now also F311.1
- net CELL3: now also F310.1
- net CELL4: now also F309.1
- net CELL5: now also F308.1
- net CELL6: now also F307.1
- net CELL7: now also F306.1
- net CELL8: now also F305.1
- net CELL9: now also F304.1
- net at Q14.2 (S), R104.1, R117.1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: now also F301.2
- net at Q22.2 (S), R112.1, R75.2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: now also F309.2
- net at Q17.2 (S), R107.1, R70.2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: now also F304.2
- net at D14.2 (A), L2.1, R116.1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: now also F313.2
- net at Q23.2 (S), R113.1, R76.2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: now also F310.2
- net at D14.1 (K), Q25.2 (S), R115.1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: now also F312.2
- net at Q16.2 (S), R106.1, R69.2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: now also F303.2
- net at Q24.2 (S), R114.1, R77.2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: now also F311.2
- net at Q20.2 (S), R110.1, R73.2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: now also F307.2
- net at Q21.2 (S), R111.1, R74.2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: now also F308.2
- net at Q18.2 (S), R108.1, R71.2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: now also F305.2
- net at Q15.2 (S), R105.1, R68.2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: now also F302.2
- net at Q19.2 (S), R109.1, R72.2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: now also F306.2

Commit message: アノテーションし直し
Parts:
- renumbered C35 to C40, C36 to C41, C37 to C42, C38 to C43, C39 to C44, C40 to C45, C41 to C46, C42 to C47, C43 to C48, C44 to C49, C45 to C50, C46 to C51, C47 to C52, C48 to C53, C49 to C54, C50 to C55, C51 to C56, C52 to C57, C53 to C58, C54 to C59, C55 to C60, C56 to C61, C57 to C62, C58 to C63, C59 to C64, C60 to C65, C296 to C66, C61 to C67, C297 to C68, C62 to C69, C63 to C70, C298 to C71, C64 to C72, C65 to C73, C299 to C74, C300 to C75, C66 to C76, C67 to C77, C68 to C78, F301 to F14, F302 to F15, F303 to F16, F304 to F17, F305 to F18, F306 to F19, F307 to F20, F308 to F21, F309 to F22, F310 to F23, F311 to F24, F312 to F25, F313 to F26, R95 to R100, R96 to R101, R97 to R102, R98 to R103, R99 to R104, R100 to R105, R101 to R106, R102 to R107, R103 to R108, R104 to R109, R105 to R110, R106 to R111, R107 to R112, R108 to R113, R109 to R114, R110 to R115, R111 to R116, R112 to R117, R113 to R118, R114 to R119, R115 to R120, R116 to R121, R117 to R122, R119 to R123, R120 to R124, R122 to R125, R125 to R126, R126 to R127, R127 to R128, R128 to R129, R563 to R131, R564 to R132, R565 to R133, R566 to R134, R567 to R135, R118 to R136, R131 to R137, R132 to R138, R133 to R139, R134 to R140, R121 to R141, R123 to R142, R124 to R143, R129 to R144, R68 to R73, R69 to R74, R70 to R75, R71 to R76, R72 to R77, R73 to R78, R74 to R79, R75 to R80, R76 to R81, R77 to R82, R78 to R83, R79 to R84, R80 to R85, R81 to R86, R82 to R87, R83 to R88, R84 to R89, R85 to R90, R86 to R91, R87 to R92, R88 to R93, R89 to R94, R90 to R95, R91 to R96, R92 to R97, R93 to R98, R94 to R99

Commit message: GPIO入力保護回路追加
Parts:
- added D130, D131, D132, D133, D134, D135, D136, D137, D138, D139: BAT46W-7-F, ProjectEV:D_SOD-123_BAT46W-7-F, symbol ProjectEV:D_BAT46W-7-F
Connections:
- net GND2: now also D130.2 (A), D133.2 (A), D135.2 (A), D137.2 (A), D139.2 (A)
- net VREG: now also D131.1 (K), D132.1 (K), D134.1 (K), D136.1 (K), D138.1 (K)
- net at C74.1, R132.1, U2.28 (GPIO2): now also D132.2 (A), D133.1 (K)
- net at C68.1, R134.1, U2.32 (GPIO4): now also D136.2 (A), D137.1 (K)
- net at C71.1, R133.1, U2.29 (GPIO3): now also D134.2 (A), D135.1 (K)
- net at C75.1, R131.1, U2.27 (GPIO1): now also D130.1 (K), D131.2 (A)
- net at C66.1, R135.1, U2.33 (GPIO5): now also D138.2 (A), D139.1 (K)
Other:
- moved on the sheet: R131, R132, R133, R134, R135, R136, R141, R142, R143, R144

Commit message: アノテーションし直し
Parts:
- renumbered D14 to D24, D15 to D25, D16 to D26, D17 to D27, D18 to D28, D19 to D29, D20 to D30, D21 to D31, D22 to D32, D23 to D33, D24 to D34, D25 to D35, D26 to D36, D132 to D37, D133 to D38, D136 to D39, D137 to D40, D131 to D41, D130 to D42, D134 to D43, D135 to D44, D138 to D45, D139 to D46, L2 to L18, R98 to R100, R99 to R101, R100 to R102, R101 to R103, R102 to R104, R103 to R105, R104 to R106, R105 to R107, R106 to R108, R107 to R109, R108 to R110, R109 to R111, R110 to R112, R111 to R113, R112 to R114, R113 to R115, R114 to R116, R115 to R117, R116 to R118, R117 to R119, R118 to R120, R119 to R121, R120 to R122, R121 to R123, R122 to R124, R123 to R125, R124 to R126, R125 to R127, R126 to R128, R127 to R129, R128 to R130, R129 to R131, R130 to R132, R137 to R133, R138 to R134, R139 to R135, R140 to R136, R131 to R137, R132 to R138, R133 to R139, R134 to R140, R135 to R141, R136 to R142, R141 to R143, R142 to R144, R143 to R145, R144 to R146, R73 to R75, R74 to R76, R75 to R77, R76 to R78, R77 to R79, R78 to R80, R79 to R81, R80 to R82, R81 to R83, R82 to R84, R83 to R85, R84 to R86, R85 to R87, R86 to R88, R87 to R89, R88 to R90, R89 to R91, R90 to R92, R91 to R93, R92 to R94, R93 to R95, R94 to R96, R95 to R97, R96 to R98, R97 to R99
