File: AMS-board-2024/battery-module-monitor-2.kicad_sch (KiCad schematic)
At the start: 164 parts, among them Q14 BSS308PE, Q15 BSS308PE, Q16 BSS308PE, Q17 BSS308PE, Q18 BSS308PE, Q19 BSS308PE, Q20 BSS308PE, Q21 BSS308PE, Q22 BSS308PE, Q23 BSS308PE, Q24 BSS308PE, Q25 BSS308PE, Q26 NSV1C201MZ4, U2 LTC6811-1

Commit message: ERC実行、修正
ラベル修正、未配線部分修正、PWR_FLAG追加
Connections:
- net GND2: now also U2.36 (SWTEN)
- net VREG renamed VREG2
Changed lines of the file:
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@@
   (junction (at 307.34 246.38) (diameter 0) (color 0 0 0 0)
   )
+  (junction (at 292.1 165.1) (diameter 0) (color 0 0 0 0)
+  )
   (junction (at 332.74 241.3) (diameter 0) (color 0 0 0 0)
   )
+  (junction (at 101.6 381) (diameter 0) (color 0 0 0 0)
+  )
   (junction (at 101.6 341.63) (diameter 0) (color 0 0 0 0)
   )
@@
     (stroke (width 0) (type default))
   )
+  (wire (pts (xy 304.8 223.52) (xy 307.34 223.52))
+    (stroke (width 0) (type default))
+  )
   (wire (pts (xy 134.62 251.46) (xy 135.89 251.46))
     (stroke (width 0) (type default))
@@
     (stroke (width 0) (type default))
   )
+  (wire (pts (xy 96.52 381) (xy 101.6 381))
+    (stroke (width 0) (type default))
+  )
   (wire (pts (xy 335.28 220.98) (xy 337.82 220.98))
     (stroke (width 0) (type default))
@@
     (stroke (width 0) (type default))
   )
+  (wire (pts (xy 101.6 381) (xy 101.6 383.54))
+    (stroke (width 0) (type default))
+  )
   (wire (pts (xy 424.18 241.3) (xy 406.4 241.3))
     (stroke (width 0) (type default))
@@
     (stroke (width 0) (type default))
   )
-  (wire (pts (xy 101.6 378.46) (xy 101.6 379.73))
+  (wire (pts (xy 101.6 378.46) (xy 101.6 381))
     (stroke (width 0) (type default))
   )
@@
     (effects (font (size 1.27 1.27)) (justify right))
   )
-  (hierarchical_label "VREG" (shape output) (at 419.1 223.52 0) (fields_autoplaced)
+  (hierarchical_label "VREG2" (shape output) (at 419.1 223.52 0) (fields_autoplaced)
     (effects (font (size 1.27 1.27)) (justify left))
   )
@@
     (effects (font (size 1.27 1.27)) (justify left))
   )
-  (hierarchical_label "GND" (shape output) (at 419.1 228.6 0) (fields_autoplaced)
+  (hierarchical_label "GND2" (shape output) (at 419.1 228.6 0) (fields_autoplaced)
     (effects (font (size 1.27 1.27)) (justify left))
   )
@@
     )
   )
+  (symbol (lib_id "power:PWR_FLAG") (at 96.52 381 0) (unit 1)
+    (in_bom yes) (on_board yes) (dnp no) (fields_autoplaced)
+    (property "Reference" "#FLG010" (at 96.52 379.095 0)
+      (effects (font (size 1.27 1.27)) hide)
+    )
+    (property "Value" "PWR_FLAG" (at 96.52 375.92 0)
+      (effects (font (size 1.27 1.27)))
+    )
+    (property "Footprint" "" (at 96.52 381 0)
+      (effects (font (size 1.27 1.27)) hide)
+    )
+    (property "Datasheet" "~" (at 96.52 381 0)
+      (effects (font (size 1.27 1.27)) hide)
+    )
+    (pin "1")
+    (instances
+      (project "AMS-board-2024"
+        (path "/3a719eb3-09ce-4343-8f6e-20cc0aaf5261/283ab3c5-5baf-4497-bb23-492a3bdd3023"
+          (reference "#FLG010") (unit 1)
+        )
+      )
+    )
+  )
   (symbol (lib_id "Device:LED") (at 120.65 114.3 0) (unit 1)
     (in_bom yes) (on_board yes) (dnp no)
@@
     )
   )
+  (symbol (lib_id "power:GND2") (at 307.34 223.52 90) (unit 1)
+    (in_bom yes) (on_board yes) (dnp no) (fields_autoplaced)
+    (property "Reference" "#PWR0438" (at 313.69 223.52 0)
+      (effects (font (size 1.27 1.27)) hide)
+    )
+    (property "Value" "GND2" (at 311.15 223.52 90)
+      (effects (font (size 1.27 1.27)) (justify right))
+    )
+    (property "Footprint" "" (at 307.34 223.52 0)
+      (effects (font (size 1.27 1.27)) hide)
+    )
+    (property "Datasheet" "" (at 307.34 223.52 0)
+      (effects (font (size 1.27 1.27)) hide)
+    )
+    (pin "1")
+    (instances
+      (project "AMS-board-2024"
+        (path "/3a719eb3-09ce-4343-8f6e-20cc0aaf5261/283ab3c5-5baf-4497-bb23-492a3bdd3023"
+          (reference "#PWR0438") (unit 1)
+        )
+      )
+    )
+  )
   (symbol (lib_id "ProjectEV:Fuse_0679L1000-05") (at 88.9 76.2 90) (unit 1)
     (in_bom yes) (on_board yes) (dnp no) (fields_autoplaced)
@@
     )
   )
-  (symbol (lib_id "power:GND2") (at 101.6 379.73 0) (unit 1)
+  (symbol (lib_id "power:GND2") (at 101.6 383.54 0) (unit 1)
     (in_bom yes) (on_board yes) (dnp no) (fields_autoplaced)
-    (property "Reference" "#PWR063" (at 101.6 386.08 0)
+    (property "Reference" "#PWR063" (at 101.6 389.89 0)
       (effects (font (size 1.27 1.27)) hide)
     )
-    (property "Value" "GND2" (at 101.6 384.81 0)
+    (property "Value" "GND2" (at 101.6 388.62 0)
       (effects (font (size 1.27 1.27)))
     )
-    (property "Footprint" "" (at 101.6 379.73 0)
+    (property "Footprint" "" (at 101.6 383.54 0)
       (effects (font (size 1.27 1.27)) hide)
     )
-    (property "Datasheet" "" (at 101.6 379.73 0)
+    (property "Datasheet" "" (at 101.6 383.54 0)
       (effects (font (size 1.27 1.27)) hide)
     )
@@
         )
       )
+    )
+  )
+  (symbol (lib_id "power:PWR_FLAG") (at 292.1 165.1 0) (unit 1)
+    (in_bom yes) (on_board yes) (dnp no) (fields_autoplaced)
+    (property "Reference" "#FLG03" (at 292.1 163.195 0)
+      (effects (font (size 1.27 1.27)) hide)
+    )
+    (property "Value" "PWR_FLAG" (at 292.1 160.02 0)
+      (effects (font (size 1.27 1.27)))
+    )
+    (property "Footprint" "" (at 292.1 165.1 0)
+      (effects (font (size 1.27 1.27)) hide)
+    )
+    (property "Datasheet" "~" (at 292.1 165.1 0)
+      (effects (font (size 1.27 1.27)) hide)
+    )
+    (pin "1")
+    (instances
+      (project "AMS-board-2024"
+        (path "/3a719eb3-09ce-4343-8f6e-20cc0aaf5261/283ab3c5-5baf-4497-bb23-492a3bdd3023"
+          (reference "#FLG03") (unit 1)
+        )
+      )

Commit message: ラベル修正
Connections:
- net VREG2 renamed VREG
Changed lines of the file:
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@@
     (effects (font (size 1.27 1.27)) (justify left bottom))
   )
-  (label "VREG2" (at 378.46 241.3 0) (fields_autoplaced)
+  (label "S3_VREG" (at 378.46 292.1 0) (fields_autoplaced)
     (effects (font (size 1.27 1.27)) (justify left bottom))
   )
-  (label "VREG2" (at 378.46 292.1 0) (fields_autoplaced)
+  (label "S3_VREG" (at 342.9 215.9 0) (fields_autoplaced)
     (effects (font (size 1.27 1.27)) (justify left bottom))
   )
-  (label "VREG2" (at 365.76 266.7 0) (fields_autoplaced)
+  (label "S3_VREG" (at 378.46 342.9 0) (fields_autoplaced)
     (effects (font (size 1.27 1.27)) (justify left bottom))
   )
-  (label "VREG2" (at 342.9 215.9 0) (fields_autoplaced)
+  (label "S3_VREG" (at 378.46 241.3 0) (fields_autoplaced)
     (effects (font (size 1.27 1.27)) (justify left bottom))
   )
-  (label "VREG2" (at 365.76 317.5 0) (fields_autoplaced)
+  (label "S3_VREG" (at 365.76 317.5 0) (fields_autoplaced)
     (effects (font (size 1.27 1.27)) (justify left bottom))
   )
-  (label "VREG2" (at 378.46 342.9 0) (fields_autoplaced)
+  (label "S3_VREG" (at 365.76 266.7 0) (fields_autoplaced)
     (effects (font (size 1.27 1.27)) (justify left bottom))
   )
@@
     (effects (font (size 1.27 1.27)) (justify right))
   )
-  (hierarchical_label "VREG2" (shape output) (at 419.1 223.52 0) (fields_autoplaced)
+  (hierarchical_label "VREG" (shape output) (at 419.1 223.52 0) (fields_autoplaced)
     (effects (font (size 1.27 1.27)) (justify left))
   )

Commit message: アノテーションし直し
Parts:
- renumbered L18 to L19

Commit message: 階層シート内の電源シンボル修正
階層シート内で電源シンボルをなるべく使わないようにする
修正途中
Connections:
- net GND2 renamed GND

Commit message: LTC6811のシンボルを更新
Parts:
- U2: footprint ProjectEV:SSOP-48_5.3x12.8mm_P0.5mm_LTC6811 -> ProjectEV:Package_SSOP-48_5.3x12.8mm_P0.5mm_LTC6811
Changed lines of the file:
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@@
       (effects (font (size 1.27 1.27)) (justify left))
     )
-    (property "Footprint" "ProjectEV:SSOP-48_5.3x12.8mm_P0.5mm_LTC6811" (at 290.83 213.36 0)
+    (property "Footprint" "ProjectEV:Package_SSOP-48_5.3x12.8mm_P0.5mm_LTC6811" (at 290.83 213.36 0)
       (effects (font (size 1.27 1.27)) hide)
     )

Commit message: チップ抵抗、チップコンデンササイズ修正
Parts:
- C52, C53, C54, C55, C56, C57, C58, C59, C60, C61, C62, C63, C64, C66, C67, C68, C69, C70, C71, C72, C73, C74, C75, C77, C78: footprint Capacitor_SMD:C_0603_1608Metric -> Capacitor_SMD:C_0402_1005Metric
- R100, R101, R102, R103, R104, R105, R106, R107, R108, R109, R110, R111, R112, R113, R114, R115, R116, R117, R118, R119, R120, R121, R122, R123, R124, R125, R127, R132, R137, R138, R139, R140, R141, R142, R143, R144, R145, R146, R99: footprint Resistor_SMD:R_0603_1608Metric -> Resistor_SMD:R_0402_1005Metric

Commit message: 温度センサ用コネクタ変更、大まかな位置決定
Parts:
- removed C66, C68: 0.1u, Capacitor_SMD:C_0402_1005Metric, symbol Device:C
- removed D39, D40, D45, D46: BAT46W-7-F, ProjectEV:D_SOD-123_BAT46W-7-F, symbol ProjectEV:D_BAT46W-7-F
- removed R140, R141: 100, Resistor_SMD:R_0402_1005Metric, symbol Device:R
- removed R145, R146: 10k, Resistor_SMD:R_0402_1005Metric, symbol Device:R
Connections:
- net VREF_3V: no longer names the net of C67.2, R142.1, R143.1, R144.1, U2.34 (VREF2)
- net VREG: no longer names the net of C70.1, D37.1 (K), D41.1 (K), D43.1 (K), Q26.3 (E), R126.1, U2.37 (VREG), U2.40 (ISOMD)
- no-connect marks 2 -> 4

Commit message: アノテーションし直し、
Parts:
- R120: renamed from R124; footprint Resistor_SMD:R_0402_1005Metric -> Resistor_SMD:R_0603_1608Metric
- R128: renamed from R132; footprint Resistor_SMD:R_0402_1005Metric -> Resistor_SMD:R_0603_1608Metric
- renumbered C40 to C38, C41 to C39, C42 to C40, C43 to C41, C44 to C42, C45 to C43, C46 to C44, C47 to C45, C48 to C46, C49 to C47, C50 to C48, C51 to C49, C52 to C50, C53 to C51, C54 to C52, C55 to C53, C56 to C54, C57 to C55, C58 to C56, C59 to C57, C60 to C58, C61 to C59, C62 to C60, C63 to C61, C64 to C62, C65 to C63, C67 to C64, C69 to C65, C70 to C66, C71 to C67, C72 to C68, C73 to C69, C74 to C70, C75 to C71, C76 to C72, C77 to C73, C78 to C74, D24 to D20, D25 to D21, D26 to D22, D27 to D23, D28 to D24, D29 to D25, D30 to D26, D31 to D27, D32 to D28, D33 to D29, D34 to D30, D35 to D31, D36 to D32, D37 to D33, D38 to D34, D41 to D35, D42 to D36, D43 to D37, D44 to D38, R104 to R100, R105 to R101, R106 to R102, R107 to R103, R108 to R104, R109 to R105, R110 to R106, R111 to R107, R112 to R108, R113 to R109, R114 to R110, R115 to R111, R116 to R112, R117 to R113, R118 to R114, R119 to R115, R120 to R116, R121 to R117, R122 to R118, R123 to R119, R125 to R121, R126 to R122, R127 to R123, R128 to R124, R129 to R125, R130 to R126, R131 to R127, R133 to R129, R134 to R130, R135 to R131, R136 to R132, R137 to R133, R138 to R134, R139 to R135, R142 to R136, R143 to R137, R144 to R138, R75 to R71, R76 to R72, R77 to R73, R78 to R74, R79 to R75, R80 to R76, R81 to R77, R82 to R78, R83 to R79, R84 to R80, R85 to R81, R86 to R82, R87 to R83, R88 to R84, R89 to R85, R90 to R86, R91 to R87, R92 to R88, R93 to R89, R94 to R90, R95 to R91, R96 to R92, R97 to R93, R98 to R94, R99 to R95, R100 to R96, R101 to R97, R102 to R98, R103 to R99
