File: AMS-board-2024/battery-module-monitor-2.kicad_sch (KiCad schematic)
At the start: 154 parts, among them Q14 BSS308PE, Q15 BSS308PE, Q16 BSS308PE, Q17 BSS308PE, Q18 BSS308PE, Q19 BSS308PE, Q20 BSS308PE, Q21 BSS308PE, Q22 BSS308PE, Q23 BSS308PE, Q24 BSS308PE, Q25 BSS308PE, Q26 NSV1C201MZ4, U2 LTC6811-1

Commit message: 絶縁パルストランス数削減
Parts:
- renumbered L19 to L12
Changed lines of the file:
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@@
   (symbol (lib_id "ProjectEV:L_MH3261") (at 101.6 374.65 0) (unit 1)
     (in_bom yes) (on_board yes) (dnp no) (fields_autoplaced)
-    (property "Reference" "L19" (at 102.87 373.38 0)
+    (property "Reference" "L12" (at 102.87 373.38 0)
       (effects (font (size 1.27 1.27)) (justify left))
     )
@@
       (project "AMS-board-2024"
         (path "/3a719eb3-09ce-4343-8f6e-20cc0aaf5261/283ab3c5-5baf-4497-bb23-492a3bdd3023"
-          (reference "L19") (unit 1)
+          (reference "L12") (unit 1)
         )
       )

Commit message: 抵抗修正
3.3k -> 3k (1608)
15k -> 100k (1005, プルアップ/ダウン), 5.1k (1005, LED用)
Parts:
- R100, R101, R102, R103, R104, R105, R106, R95, R96, R97, R98, R99: value 3.3k -> 3k; footprint Resistor_SMD:R_0402_1005Metric -> Resistor_SMD:R_0603_1608Metric
Changed lines of the file:
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@@
       (effects (font (size 1.27 1.27)))
     )
-    (property "Value" "3.3k" (at 139.7 297.18 90)
+    (property "Value" "3k" (at 139.7 297.18 90)
       (effects (font (size 1.27 1.27)))
     )
-    (property "Footprint" "Resistor_SMD:R_0402_1005Metric" (at 139.7 301.498 90)
+    (property "Footprint" "Resistor_SMD:R_0603_1608Metric" (at 139.7 301.498 90)
       (effects (font (size 1.27 1.27)) hide)
     )
@@
       (effects (font (size 1.27 1.27)))
     )
-    (property "Value" "3.3k" (at 139.7 152.4 90)
+    (property "Value" "3k" (at 139.7 152.4 90)
       (effects (font (size 1.27 1.27)))
     )
-    (property "Footprint" "Resistor_SMD:R_0402_1005Metric" (at 139.7 156.718 90)
+    (property "Footprint" "Resistor_SMD:R_0603_1608Metric" (at 139.7 156.718 90)
       (effects (font (size 1.27 1.27)) hide)
     )
@@
       (effects (font (size 1.27 1.27)))
     )
-    (property "Value" "3.3k" (at 139.7 176.53 90)
+    (property "Value" "3k" (at 139.7 176.53 90)
       (effects (font (size 1.27 1.27)))
     )
-    (property "Footprint" "Resistor_SMD:R_0402_1005Metric" (at 139.7 180.848 90)
+    (property "Footprint" "Resistor_SMD:R_0603_1608Metric" (at 139.7 180.848 90)
       (effects (font (size 1.27 1.27)) hide)
     )
@@
       (effects (font (size 1.27 1.27)))
     )
-    (property "Value" "3.3k" (at 139.7 224.79 90)
+    (property "Value" "3k" (at 139.7 224.79 90)
       (effects (font (size 1.27 1.27)))
     )
-    (property "Footprint" "Resistor_SMD:R_0402_1005Metric" (at 139.7 229.108 90)
+    (property "Footprint" "Resistor_SMD:R_0603_1608Metric" (at 139.7 229.108 90)
       (effects (font (size 1.27 1.27)) hide)
     )
@@
       (effects (font (size 1.27 1.27)))
     )
-    (property "Value" "3.3k" (at 139.7 345.44 90)
+    (property "Value" "3k" (at 139.7 345.44 90)
       (effects (font (size 1.27 1.27)))
     )
-    (property "Footprint" "Resistor_SMD:R_0402_1005Metric" (at 139.7 349.758 90)
+    (property "Footprint" "Resistor_SMD:R_0603_1608Metric" (at 139.7 349.758 90)
       (effects (font (size 1.27 1.27)) hide)
     )
@@
       (effects (font (size 1.27 1.27)))
     )
-    (property "Value" "3.3k" (at 139.7 321.31 90)
+    (property "Value" "3k" (at 139.7 321.31 90)
       (effects (font (size 1.27 1.27)))
     )
-    (property "Footprint" "Resistor_SMD:R_0402_1005Metric" (at 139.7 325.628 90)
+    (property "Footprint" "Resistor_SMD:R_0603_1608Metric" (at 139.7 325.628 90)
       (effects (font (size 1.27 1.27)) hide)
     )
@@
       (effects (font (size 1.27 1.27)))
     )
-    (property "Value" "3.3k" (at 139.7 248.92 90)
+    (property "Value" "3k" (at 139.7 248.92 90)
       (effects (font (size 1.27 1.27)))
     )
-    (property "Footprint" "Resistor_SMD:R_0402_1005Metric" (at 139.7 253.238 90)
+    (property "Footprint" "Resistor_SMD:R_0603_1608Metric" (at 139.7 253.238 90)
       (effects (font (size 1.27 1.27)) hide)
     )
@@
       (effects (font (size 1.27 1.27)))
     )
-    (property "Value" "3.3k" (at 139.7 273.05 90)
+    (property "Value" "3k" (at 139.7 273.05 90)
       (effects (font (size 1.27 1.27)))
     )
-    (property "Footprint" "Resistor_SMD:R_0402_1005Metric" (at 139.7 277.368 90)
+    (property "Footprint" "Resistor_SMD:R_0603_1608Metric" (at 139.7 277.368 90)
       (effects (font (size 1.27 1.27)) hide)
     )
@@
       (effects (font (size 1.27 1.27)))
     )
-    (property "Value" "3.3k" (at 139.7 200.66 90)
+    (property "Value" "3k" (at 139.7 200.66 90)
       (effects (font (size 1.27 1.27)))
     )
-    (property "Footprint" "Resistor_SMD:R_0402_1005Metric" (at 139.7 204.978 90)
+    (property "Footprint" "Resistor_SMD:R_0603_1608Metric" (at 139.7 204.978 90)
       (effects (font (size 1.27 1.27)) hide)
     )
@@
       (effects (font (size 1.27 1.27)))
     )
-    (property "Value" "3.3k" (at 139.7 80.01 90)
+    (property "Value" "3k" (at 139.7 80.01 90)
       (effects (font (size 1.27 1.27)))
     )
-    (property "Footprint" "Resistor_SMD:R_0402_1005Metric" (at 139.7 84.328 90)
+    (property "Footprint" "Resistor_SMD:R_0603_1608Metric" (at 139.7 84.328 90)
       (effects (font (size 1.27 1.27)) hide)
     )
@@
       (effects (font (size 1.27 1.27)))
     )
-    (property "Value" "3.3k" (at 139.7 128.27 90)
+    (property "Value" "3k" (at 139.7 128.27 90)
       (effects (font (size 1.27 1.27)))
     )
-    (property "Footprint" "Resistor_SMD:R_0402_1005Metric" (at 139.7 132.588 90)
+    (property "Footprint" "Resistor_SMD:R_0603_1608Metric" (at 139.7 132.588 90)
       (effects (font (size 1.27 1.27)) hide)
     )
@@
       (effects (font (size 1.27 1.27)))
     )
-    (property "Value" "3.3k" (at 139.7 104.14 90)
+    (property "Value" "3k" (at 139.7 104.14 90)
       (effects (font (size 1.27 1.27)))
     )
-    (property "Footprint" "Resistor_SMD:R_0402_1005Metric" (at 139.7 108.458 90)
+    (property "Footprint" "Resistor_SMD:R_0603_1608Metric" (at 139.7 108.458 90)
       (effects (font (size 1.27 1.27)) hide)
     )

Commit message: アノテーションし直し
Parts:
- renumbered C38 to C47, C39 to C48, C40 to C49, C41 to C50, C42 to C51, C43 to C52, C44 to C53, C45 to C54, C46 to C55, C47 to C56, C48 to C57, C49 to C58, C50 to C59, C51 to C60, C52 to C61, C53 to C62, C54 to C63, C55 to C64, C56 to C65, C57 to C66, C58 to C67, C59 to C68, C60 to C69, C61 to C70, C62 to C71, C63 to C72, C64 to C73, C65 to C74, C66 to C75, C67 to C76, C68 to C77, C69 to C78, C70 to C79, C71 to C80, C72 to C81, C73 to C82, C74 to C83, L12 to L8
