File: AMS-board-2024/battery-module-monitor-3.kicad_sch (KiCad schematic)
At the start: 144 parts, among them Q401 BSS308PE, Q402 BSS308PE, Q403 BSS308PE, Q404 BSS308PE, Q405 BSS308PE, Q406 BSS308PE, Q407 BSS308PE, Q408 BSS308PE, Q409 BSS308PE, Q410 BSS308PE, Q411 BSS308PE, Q412 BSS308PE, Q413 NSV1C201MZ4, U401 LTC6811-1

Commit message: 修正
アノテーション方法の変更：最初の空き番号から使用
Parts:
- renumbered C432 to C100, C433 to C101, C434 to C102, C401 to C69, C402 to C70, C403 to C71, C404 to C72, C405 to C73, C406 to C74, C407 to C75, C408 to C76, C409 to C77, C410 to C78, C411 to C79, C412 to C80, C413 to C81, C414 to C82, C415 to C83, C416 to C84, C417 to C85, C418 to C86, C419 to C87, C420 to C88, C421 to C89, C422 to C90, C423 to C91, C424 to C92, C425 to C93, C426 to C94, C427 to C95, C428 to C96, C429 to C97, C430 to C98, C431 to C99, D401 to D27, D402 to D28, D403 to D29, D404 to D30, D405 to D31, D406 to D32, D407 to D33, D408 to D34, D409 to D35, D410 to D36, D411 to D37, D412 to D38, D413 to D39, F401 to F27, F402 to F28, F403 to F29, F404 to F30, F405 to F31, F406 to F32, F407 to F33, F408 to F34, F409 to F35, F410 to F36, F411 to F37, F412 to F38, F413 to F39, FL401 to FL5, FL402 to FL6, L401 to L3, Q401 to Q27, Q402 to Q28, Q403 to Q29, Q404 to Q30, Q405 to Q31, Q406 to Q32, Q407 to Q33, Q408 to Q34, Q409 to Q35, Q410 to Q36, Q411 to Q37, Q412 to Q38, Q413 to Q39, R401 to R135, R402 to R136, R403 to R137, R404 to R138, R405 to R139, R406 to R140, R407 to R141, R408 to R142, R409 to R143, R410 to R144, R411 to R145, R412 to R146, R413 to R147, R414 to R148, R415 to R149, R416 to R150, R417 to R151, R418 to R152, R419 to R153, R420 to R154, R421 to R155, R422 to R156, R423 to R157, R424 to R158, R425 to R159, R426 to R160, R427 to R161, R428 to R162, R429 to R163, R430 to R164, R431 to R165, R432 to R166, R433 to R167, R434 to R168, R435 to R169, R436 to R170, R437 to R171, R438 to R172, R439 to R173, R440 to R174, R441 to R175, R442 to R176, R443 to R177, R444 to R178, R445 to R179, R446 to R180, R447 to R181, R448 to R182, R449 to R183, R450 to R184, R451 to R185, R452 to R186, R453 to R187, R454 to R188, R455 to R189, R456 to R190, R457 to R191, R458 to R192, R459 to R193, R460 to R194, R461 to R195, R462 to R196, R463 to R197, R464 to R198, R465 to R199, R466 to R200, R467 to R201, U401 to U3

Commit message: GNDシンボル追加
Connections:
- net GND3: now reaches C74.2
- net GND3: now also C100.2, C101.1, C102.1, C69.2, C70.2, C71.2, C72.2, C73.2, C75.2, C76.2, C77.2, C78.2, C79.2, C80.2, C93.2, C94.2, C95.1, C96.1, C97.2, C98.1, C99.1, L3.2, R189.1, U3.30 (V-), U3.31 (V-)

Commit message: GPIO周辺回路の修正
Parts:
- added C301, C302, C303, C304, C305: 0.1u, Capacitor_SMD:C_0603_1608Metric, symbol Device:C
- added R568, R569, R570, R571, R572: 10k, Resistor_SMD:R_0603_1608Metric, symbol Device:R
- R185, R188, R190, R191, R196: value 10k -> 100
Connections:
- net GND3: now also C301.2, C302.2, C303.2, C304.2, C305.2
- net Thermistor1+: now also R185.2, R568.2; no longer R196.1, U3.27 (GPIO1)
- net Thermistor2+: now also R188.2, R569.2; no longer R191.1, U3.28 (GPIO2)
- net Thermistor3+: now also R190.2, R570.2; no longer R190.1, U3.29 (GPIO3)
- net Thermistor4+: now also R191.2, R571.2; no longer R188.1, U3.32 (GPIO4)
- net Thermistor5+: now also R196.2, R572.2; no longer R185.1, U3.33 (GPIO5)
- net VREG: now reaches C97.1, Q39.3 (E), R187.1, U3.37 (VREG), U3.40 (ISOMD)
- new net: C301.1, R196.1, U3.33 (GPIO5)
- new net: C303.1, R190.1, U3.29 (GPIO3)
- new net: C302.1, R191.1, U3.32 (GPIO4)
- new net: C304.1, R188.1, U3.28 (GPIO2)
- new net: C305.1, R185.1, U3.27 (GPIO1)
- new net VREF_3V: C95.2, R568.1, R569.1, R570.1, R571.1, R572.1, U3.34 (VREF2)

Commit message: テキスト修正
Other:
- note added: "レギュレーション上必要なサーミスタは 96 CELL x 25 % = 24 本. GPIO1~3 をサーミスタに使用し、 GPIO4, 5 は別用途で使用してもOK. GPIO4, 5 のプルアップは必要に応じて実装."
- note removed: "レギュレーション上必要なサーミスタは 3 x 8 = 24 本. GPIO1~3 をサーミスタに使用し、 GPIO4, 5 は別用途で使用してもOK. GPIO4, 5 のプルアップは必要に応じて実装."
Changed lines of the file:
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@@
+    (effects (font (size 1.27 1.27)) (justify left bottom))
+  )
+  (text "レギュレーション上必要なサーミスタは 96 CELL x 25 % = 24 本.\nGPIO1~3 をサーミスタに使用し、\nGPIO4, 5 は別用途で使用してもOK.\nGPIO4, 5 のプルアップは必要に応じて実装."
+    (at 469.9 283.21 0)
     (effects (font (size 1.27 1.27)) (justify left bottom))
   )
@@
     (effects (font (size 1.27 1.27)) (justify left bottom))
   )
-  (text "レギュレーション上必要なサーミスタは 3 x 8 = 24 本.\nGPIO1~3 をサーミスタに使用し、\nGPIO4, 5 は別用途で使用してもOK.\nGPIO4, 5 のプルアップは必要に応じて実装."
-    (at 469.9 283.21 0)
-    (effects (font (size 1.27 1.27)) (justify left bottom))
-  )

Commit message: ヒューズ変更
Parts:
- removed F27, F28, F29, F30, F31, F32, F33, F34, F35, F36, F37, F38, F39: C1F 500, Fuse:Fuse_1206_3216Metric, symbol Device:Fuse
- added F1, F10, F11, F12, F13, F2, F3, F4, F5, F6, F7, F8, F9: 0679L1000-05, ProjectEV:Fuse_0679L, symbol ProjectEV:Fuse_0679L1000-05
Connections:
- net CELL0: now also F13.1
- net CELL1: now also F12.1
- net CELL10: now also F3.1
- net CELL11: now also F2.1
- net CELL12: now also F1.1
- net CELL2: now also F11.1
- net CELL3: now also F10.1
- net CELL4: now also F9.1
- net CELL5: now also F8.1
- net CELL6: now also F7.1
- net CELL7: now also F6.1
- net CELL8: now also F5.1
- net CELL9: now also F4.1
- net at Q32.2 (S), R139.2, R151.2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: now also F6.2
- net at Q31.2 (S), R138.2, R150.2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: now also F5.2
- net at Q33.2 (S), R140.2, R152.2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: now also F7.2
- net at Q35.2 (S), R142.2, R154.2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: now also F9.2
- net at Q36.2 (S), R143.2, R155.2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: now also F10.2
- net at Q37.2 (S), R144.2, R156.2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: now also F11.2
- net at D27.1 (K), Q38.2 (S), R145.2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: now also F12.2
- net at D27.2 (A), L3.1, R146.2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: now also F13.2
- net at Q34.2 (S), R141.2, R153.2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: now also F8.2
- net at Q28.2 (S), R135.2, R147.2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: now also F2.2
- net at Q27.2 (S), R171.1, R184.1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: now also F1.2
- net at Q29.2 (S), R136.2, R148.2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: now also F3.2
- net at Q30.2 (S), R137.2, R149.2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: now also F4.2

Commit message: アノテーションし直し
Parts:
- renumbered C90 to C100, C91 to C101, C92 to C102, C93 to C103, C94 to C104, C301 to C105, C95 to C106, C302 to C107, C96 to C108, C97 to C109, C303 to C110, C98 to C111, C99 to C112, C304 to C113, C305 to C114, C100 to C115, C101 to C116, C102 to C117, C69 to C79, C70 to C80, C71 to C81, C72 to C82, C73 to C83, C74 to C84, C75 to C85, C76 to C86, C77 to C87, C78 to C88, C79 to C89, C80 to C90, C81 to C91, C82 to C92, C83 to C93, C84 to C94, C85 to C95, C86 to C96, C87 to C97, C88 to C98, C89 to C99, F1 to F27, F2 to F28, F3 to F29, F4 to F30, F5 to F31, F6 to F32, F7 to F33, F8 to F34, F9 to F35, F10 to F36, F11 to F37, F12 to F38, F13 to F39, R135 to R145, R136 to R146, R137 to R147, R138 to R148, R139 to R149, R140 to R150, R141 to R151, R142 to R152, R143 to R153, R144 to R154, R145 to R155, R146 to R156, R147 to R157, R148 to R158, R149 to R159, R150 to R160, R151 to R161, R152 to R162, R153 to R163, R154 to R164, R155 to R165, R156 to R166, R157 to R167, R158 to R168, R159 to R169, R160 to R170, R161 to R171, R162 to R172, R163 to R173, R164 to R174, R165 to R175, R166 to R176, R167 to R177, R168 to R178, R169 to R179, R170 to R180, R171 to R181, R172 to R182, R173 to R183, R174 to R184, R175 to R185, R176 to R186, R177 to R187, R178 to R188, R179 to R189, R180 to R190, R181 to R191, R182 to R192, R183 to R193, R184 to R194, R186 to R195, R187 to R196, R189 to R197, R192 to R198, R193 to R199, R194 to R200, R195 to R201, R197 to R202, R185 to R203, R188 to R204, R190 to R205, R191 to R206, R196 to R207, R568 to R208, R198 to R209, R199 to R210, R200 to R211, R201 to R212, R569 to R213, R570 to R214, R571 to R215, R572 to R216

Commit message: GPIO入力保護回路追加
Parts:
- added D150, D151, D152, D153, D154, D155, D156, D157, D158, D159: BAT46W-7-F, ProjectEV:D_SOD-123_BAT46W-7-F, symbol ProjectEV:D_BAT46W-7-F
Connections:
- net GND3: now also D151.2 (A), D153.2 (A), D155.2 (A), D157.2 (A), D159.2 (A)
- net VREG: now also D150.1 (K), D152.1 (K), D154.1 (K), D156.1 (K), D158.1 (K)
- net at C105.1, R207.1, U3.33 (GPIO5): now also D158.2 (A), D159.1 (K)
- net at C110.1, R205.1, U3.29 (GPIO3): now also D154.2 (A), D155.1 (K)
- net at C107.1, R206.1, U3.32 (GPIO4): now also D156.2 (A), D157.1 (K)
- net at C113.1, R204.1, U3.28 (GPIO2): now also D152.2 (A), D153.1 (K)
- net at C114.1, R203.1, U3.27 (GPIO1): now also D150.2 (A), D151.1 (K)
Other:
- moved on the sheet: R203, R204, R205, R206, R207, R208, R213, R214, R215, R216

Commit message: アノテーションし直し
Parts:
- renumbered D27 to D47, D28 to D48, D29 to D49, D30 to D50, D31 to D51, D32 to D52, D33 to D53, D34 to D54, D35 to D55, D36 to D56, D37 to D57, D38 to D58, D39 to D59, D152 to D60, D153 to D61, D156 to D62, D157 to D63, D150 to D64, D151 to D65, D154 to D66, D155 to D67, D158 to D68, D159 to D69, L3 to L19, R145 to R147, R146 to R148, R147 to R149, R148 to R150, R149 to R151, R150 to R152, R151 to R153, R152 to R154, R153 to R155, R154 to R156, R155 to R157, R156 to R158, R157 to R159, R158 to R160, R159 to R161, R160 to R162, R161 to R163, R162 to R164, R163 to R165, R164 to R166, R165 to R167, R166 to R168, R167 to R169, R168 to R170, R169 to R171, R170 to R172, R171 to R173, R172 to R174, R173 to R175, R174 to R176, R175 to R177, R176 to R178, R177 to R179, R178 to R180, R179 to R181, R180 to R182, R181 to R183, R182 to R184, R183 to R185, R184 to R186, R185 to R187, R186 to R188, R187 to R189, R188 to R190, R189 to R191, R190 to R192, R191 to R193, R192 to R194, R193 to R195, R194 to R196, R195 to R197, R196 to R198, R197 to R199, R198 to R200, R199 to R201, R200 to R202, R201 to R203, R202 to R204, R209 to R205, R210 to R206, R211 to R207, R212 to R208, R203 to R209, R204 to R210, R205 to R211, R206 to R212, R207 to R213, R208 to R214, R213 to R215, R214 to R216, R215 to R217, R216 to R218
