File: AMS-board-2024/battery-module-monitor-3.kicad_sch (KiCad schematic)
At the start: 164 parts, among them Q27 BSS308PE, Q28 BSS308PE, Q29 BSS308PE, Q30 BSS308PE, Q31 BSS308PE, Q32 BSS308PE, Q33 BSS308PE, Q34 BSS308PE, Q35 BSS308PE, Q36 BSS308PE, Q37 BSS308PE, Q38 BSS308PE, Q39 NSV1C201MZ4, U3 LTC6811-1

Commit message: ERC実行、修正
ラベル修正、未配線部分修正、PWR_FLAG追加
Connections:
- net GND3: now also U3.36 (SWTEN)
- net VREG renamed VREG3
Changed lines of the file:
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@@
 (kicad_sch (version 20230121) (generator eeschema)
   (paper "A2")
+  (junction (at 101.6 381) (diameter 0) (color 0 0 0 0)
+  )
   (junction (at 342.9 114.3) (diameter 0) (color 0 0 0 0)
   )
@@
   (junction (at 127 331.47) (diameter 0) (color 0 0 0 0)
   )
+  (junction (at 292.1 165.1) (diameter 0) (color 0 0 0 0)
+  )
   (junction (at 441.96 241.3) (diameter 0) (color 0 0 0 0)
   )
@@
     (stroke (width 0) (type default))
   )
-  (wire (pts (xy 101.6 378.46) (xy 101.6 379.73))
+  (wire (pts (xy 101.6 378.46) (xy 101.6 381))
     (stroke (width 0) (type default))
   )
@@
     (stroke (width 0) (type default))
   )
+  (wire (pts (xy 101.6 381) (xy 101.6 383.54))
+    (stroke (width 0) (type default))
+  )
   (wire (pts (xy 246.38 238.76) (xy 279.4 238.76))
     (stroke (width 0) (type default))
@@
     (stroke (width 0) (type default))
   )
+  (wire (pts (xy 304.8 223.52) (xy 307.34 223.52))
+    (stroke (width 0) (type default))
+  )
   (wire (pts (xy 152.4 148.59) (xy 152.4 149.86))
     (stroke (width 0) (type default))
@@
     (stroke (width 0) (type default))
   )
+  (wire (pts (xy 96.52 381) (xy 101.6 381))
+    (stroke (width 0) (type default))
+  )
   (wire (pts (xy 279.4 190.5) (xy 246.38 190.5))
     (stroke (width 0) (type default))
@@
     (effects (font (size 1.27 1.27)) (justify right))
   )
-  (hierarchical_label "VREG" (shape output) (at 419.1 223.52 0) (fields_autoplaced)
+  (hierarchical_label "VREG3" (shape output) (at 419.1 223.52 0) (fields_autoplaced)
     (effects (font (size 1.27 1.27)) (justify left))
   )
@@
     (effects (font (size 1.27 1.27)) (justify left))
   )
-  (hierarchical_label "GND" (shape output) (at 419.1 228.6 0) (fields_autoplaced)
+  (hierarchical_label "GND3" (shape output) (at 419.1 228.6 0) (fields_autoplaced)
     (effects (font (size 1.27 1.27)) (justify left))
   )
@@
     )
   )
+  (symbol (lib_id "power:GND3") (at 307.34 223.52 90) (unit 1)
+    (in_bom yes) (on_board yes) (dnp no) (fields_autoplaced)
+    (property "Reference" "#PWR0439" (at 313.69 223.52 0)
+      (effects (font (size 1.27 1.27)) hide)
+    )
+    (property "Value" "GND3" (at 311.15 223.52 90)
+      (effects (font (size 1.27 1.27)) (justify right))
+    )
+    (property "Footprint" "" (at 307.34 223.52 0)
+      (effects (font (size 1.27 1.27)) hide)
+    )
+    (property "Datasheet" "" (at 307.34 223.52 0)
+      (effects (font (size 1.27 1.27)) hide)
+    )
+    (pin "1")
+    (instances
+      (project "AMS-board-2024"
+        (path "/3a719eb3-09ce-4343-8f6e-20cc0aaf5261/1e87e362-5c61-4f39-a903-ecfc3a14ee8d"
+          (reference "#PWR0439") (unit 1)
+        )
+      )
+    )
+  )
   (symbol (lib_id "ProjectEV:Fuse_0679L1000-05") (at 88.9 269.24 90) (unit 1)
     (in_bom yes) (on_board yes) (dnp no) (fields_autoplaced)
@@
     )
   )
-  (symbol (lib_id "power:GND3") (at 101.6 379.73 0) (unit 1)
+  (symbol (lib_id "power:GND3") (at 101.6 383.54 0) (unit 1)
     (in_bom yes) (on_board yes) (dnp no) (fields_autoplaced)
-    (property "Reference" "#PWR0104" (at 101.6 386.08 0)
+    (property "Reference" "#PWR0104" (at 101.6 389.89 0)
       (effects (font (size 1.27 1.27)) hide)
     )
-    (property "Value" "GND3" (at 101.6 384.81 0)
+    (property "Value" "GND3" (at 101.6 388.62 0)
       (effects (font (size 1.27 1.27)))
     )
-    (property "Footprint" "" (at 101.6 379.73 0)
+    (property "Footprint" "" (at 101.6 383.54 0)
       (effects (font (size 1.27 1.27)) hide)
     )
-    (property "Datasheet" "" (at 101.6 379.73 0)
+    (property "Datasheet" "" (at 101.6 383.54 0)
       (effects (font (size 1.27 1.27)) hide)
     )
@@
     )
   )
+  (symbol (lib_id "power:PWR_FLAG") (at 292.1 165.1 0) (unit 1)
+    (in_bom yes) (on_board yes) (dnp no) (fields_autoplaced)
+    (property "Reference" "#FLG04" (at 292.1 163.195 0)
+      (effects (font (size 1.27 1.27)) hide)
+    )
+    (property "Value" "PWR_FLAG" (at 292.1 160.02 0)
+      (effects (font (size 1.27 1.27)))
+    )
+    (property "Footprint" "" (at 292.1 165.1 0)
+      (effects (font (size 1.27 1.27)) hide)
+    )
+    (property "Datasheet" "~" (at 292.1 165.1 0)
+      (effects (font (size 1.27 1.27)) hide)
+    )
+    (pin "1")
+    (instances
+      (project "AMS-board-2024"
+        (path "/3a719eb3-09ce-4343-8f6e-20cc0aaf5261/1e87e362-5c61-4f39-a903-ecfc3a14ee8d"
+          (reference "#FLG04") (unit 1)
+        )
+      )
+    )
+  )
   (symbol (lib_id "Device:R") (at 146.05 124.46 90) (unit 1)
     (in_bom yes) (on_board yes) (dnp no)
@@
         )
       )
+    )
+  )
+  (symbol (lib_id "power:PWR_FLAG") (at 96.52 381 0) (unit 1)
+    (in_bom yes) (on_board yes) (dnp no) (fields_autoplaced)
+    (property "Reference" "#FLG012" (at 96.52 379.095 0)
+      (effects (font (size 1.27 1.27)) hide)
+    )
+    (property "Value" "PWR_FLAG" (at 96.52 375.92 0)
+      (effects (font (size 1.27 1.27)))
+    )
+    (property "Footprint" "" (at 96.52 381 0)
+      (effects (font (size 1.27 1.27)) hide)
+    )
+    (property "Datasheet" "~" (at 96.52 381 0)
+      (effects (font (size 1.27 1.27)) hide)
+    )
+    (pin "1")
+    (instances
+      (project "AMS-board-2024"
+        (path "/3a719eb3-09ce-4343-8f6e-20cc0aaf5261/1e87e362-5c61-4f39-a903-ecfc3a14ee8d"
+          (reference "#FLG012") (unit 1)
+        )
+      )

Commit message: ラベル修正
Connections:
- net VREG3 renamed VREG
Changed lines of the file:
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@@
     (effects (font (size 1.27 1.27)) (justify left bottom))
   )
-  (label "VREG3" (at 365.76 317.5 0) (fields_autoplaced)
+  (label "S4_VREG" (at 378.46 342.9 0) (fields_autoplaced)
     (effects (font (size 1.27 1.27)) (justify left bottom))
   )
-  (label "VREG3" (at 378.46 241.3 0) (fields_autoplaced)
+  (label "S4_VREG" (at 378.46 241.3 0) (fields_autoplaced)
     (effects (font (size 1.27 1.27)) (justify left bottom))
   )
-  (label "VREG3" (at 378.46 292.1 0) (fields_autoplaced)
+  (label "S4_VREG" (at 378.46 292.1 0) (fields_autoplaced)
     (effects (font (size 1.27 1.27)) (justify left bottom))
   )
-  (label "VREG3" (at 378.46 342.9 0) (fields_autoplaced)
+  (label "S4_VREG" (at 365.76 317.5 0) (fields_autoplaced)
     (effects (font (size 1.27 1.27)) (justify left bottom))
   )
-  (label "VREG3" (at 342.9 215.9 0) (fields_autoplaced)
+  (label "S4_VREG" (at 342.9 215.9 0) (fields_autoplaced)
     (effects (font (size 1.27 1.27)) (justify left bottom))
   )
-  (label "VREG3" (at 365.76 266.7 0) (fields_autoplaced)
+  (label "S4_VREG" (at 365.76 266.7 0) (fields_autoplaced)
     (effects (font (size 1.27 1.27)) (justify left bottom))
   )
@@
     (effects (font (size 1.27 1.27)) (justify right))
   )
-  (hierarchical_label "VREG3" (shape output) (at 419.1 223.52 0) (fields_autoplaced)
+  (hierarchical_label "VREG" (shape output) (at 419.1 223.52 0) (fields_autoplaced)
     (effects (font (size 1.27 1.27)) (justify left))
   )

Commit message: アノテーションし直し
Parts:
- renumbered L19 to L20

Commit message: 階層シート内の電源シンボル修正
階層シート内で電源シンボルをなるべく使わないようにする
修正途中
Connections:
- net VREF_3V: now also D60.1 (K), D62.1 (K), D64.1 (K), D66.1 (K), D68.1 (K)
- net VREG: no longer D60.1 (K), D62.1 (K), D64.1 (K), D66.1 (K), D68.1 (K)
- net GND3 renamed GND

Commit message: ラベル修正とテキスト等の追加
階層シート内の電源シンボルをまとめて階層ラベルとして上層に出し、上層のシートで電源シンボルに接続
Connections:
- net VREF_3V: no longer D60.1 (K), D62.1 (K), D64.1 (K), D66.1 (K), D68.1 (K)
- net VREG: now also D60.1 (K), D62.1 (K), D64.1 (K), D66.1 (K), D68.1 (K)
Changed lines of the file:
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@@
 (kicad_sch (version 20230121) (generator eeschema)
   (paper "A2")
+  (junction (at 381 241.3) (diameter 0) (color 0 0 0 0)
+  )
   (junction (at 101.6 381) (diameter 0) (color 0 0 0 0)
   )
@@
   (junction (at 355.6 215.9) (diameter 0) (color 0 0 0 0)
   )
+  (junction (at 381 223.52) (diameter 0) (color 0 0 0 0)
+  )
   (junction (at 381 127) (diameter 0) (color 0 0 0 0)
   )
@@
   (junction (at 330.2 127) (diameter 0) (color 0 0 0 0)
   )
-  (junction (at 373.38 241.3) (diameter 0) (color 0 0 0 0)
-  )
   (junction (at 127 220.98) (diameter 0) (color 0 0 0 0)
   )
@@
   )
   (junction (at 165.1 381) (diameter 0) (color 0 0 0 0)
-  )
-  (junction (at 373.38 233.68) (diameter 0) (color 0 0 0 0)
   )
   (junction (at 165.1 317.5) (diameter 0) (color 0 0 0 0)
@@
     (stroke (width 0) (type default))
   )
-  (wire (pts (xy 373.38 233.68) (xy 406.4 233.68))
+  (wire (pts (xy 355.6 233.68) (xy 406.4 233.68))
     (stroke (width 0) (type default))
   )
@@
     (stroke (width 0) (type default))
   )
+  (wire (pts (xy 381 223.52) (xy 381 241.3))
+    (stroke (width 0) (type default))
+  )
   (wire (pts (xy 335.28 231.14) (xy 335.28 259.08))
     (stroke (width 0) (type default))
@@
     (stroke (width 0) (type default))
   )
+  (wire (pts (xy 381 223.52) (xy 355.6 223.52))
+    (stroke (width 0) (type default))
+  )
   (wire (pts (xy 393.7 124.46) (xy 393.7 127))
     (stroke (width 0) (type default))
@@
     (stroke (width 0) (type default))
   )
-  (wire (pts (xy 419.1 223.52) (xy 355.6 223.52))
+  (wire (pts (xy 419.1 223.52) (xy 381 223.52))
     (stroke (width 0) (type default))
   )
@@
     (stroke (width 0) (type default))
   )
-  (wire (pts (xy 373.38 233.68) (xy 373.38 241.3))
-    (stroke (width 0) (type default))
-  )
   (wire (pts (xy 127 196.85) (xy 127 195.58))
     (stroke (width 0) (type default))
@@
   )
   (wire (pts (xy 152.4 256.54) (xy 154.94 256.54))
-    (stroke (width 0) (type default))
-  )
-  (wire (pts (xy 355.6 233.68) (xy 373.38 233.68))
     (stroke (width 0) (type default))
   )
@@
     (effects (font (size 1.27 1.27)) (justify left bottom))
   )
-  (label "S4_VREG" (at 342.9 215.9 0) (fields_autoplaced)
-    (effects (font (size 1.27 1.27)) (justify left bottom))
-  )

Commit message: LTC6811のシンボルを更新
Parts:
- U3: footprint ProjectEV:SSOP-48_5.3x12.8mm_P0.5mm_LTC6811 -> ProjectEV:Package_SSOP-48_5.3x12.8mm_P0.5mm_LTC6811
Changed lines of the file:
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@@
       (effects (font (size 1.27 1.27)) (justify left))
     )
-    (property "Footprint" "ProjectEV:SSOP-48_5.3x12.8mm_P0.5mm_LTC6811" (at 290.83 213.36 0)
+    (property "Footprint" "ProjectEV:Package_SSOP-48_5.3x12.8mm_P0.5mm_LTC6811" (at 290.83 213.36 0)
       (effects (font (size 1.27 1.27)) hide)
     )

Commit message: チップ抵抗、チップコンデンササイズ修正
Parts:
- C100, C101, C102, C103, C105, C106, C107, C108, C109, C110, C111, C112, C113, C114, C116, C117, C91, C92, C93, C94, C95, C96, C97, C98, C99: footprint Capacitor_SMD:C_0603_1608Metric -> Capacitor_SMD:C_0402_1005Metric
- R171, R172, R173, R174, R175, R176, R177, R178, R179, R180, R181, R182, R183, R184, R185, R186, R187, R188, R189, R190, R191, R192, R193, R194, R195, R196, R197, R199, R204, R209, R210, R211, R212, R213, R214, R215, R216, R217, R218: footprint Resistor_SMD:R_0603_1608Metric -> Resistor_SMD:R_0402_1005Metric

Commit message: 温度センサ用コネクタ変更、大まかな位置決定
Parts:
- removed C105, C107: 0.1u, Capacitor_SMD:C_0402_1005Metric, symbol Device:C
- removed D62, D63, D68, D69: BAT46W-7-F, ProjectEV:D_SOD-123_BAT46W-7-F, symbol ProjectEV:D_BAT46W-7-F
- removed R212, R213: 100, Resistor_SMD:R_0402_1005Metric, symbol Device:R
- removed R217, R218: 10k, Resistor_SMD:R_0402_1005Metric, symbol Device:R
Connections:
- net VREF_3V: no longer names the net of C106.2, R214.1, R215.1, R216.1, U3.34 (VREF2)
- net VREG: no longer names the net of C109.1, D60.1 (K), D64.1 (K), D66.1 (K), Q39.3 (E), R198.1, U3.37 (VREG), U3.40 (ISOMD)
- no-connect marks 2 -> 4
