File: AMS-board-2024/battery-module-monitor-3.kicad_sch (KiCad schematic)
At the start: 154 parts, among them Q27 BSS308PE, Q28 BSS308PE, Q29 BSS308PE, Q30 BSS308PE, Q31 BSS308PE, Q32 BSS308PE, Q33 BSS308PE, Q34 BSS308PE, Q35 BSS308PE, Q36 BSS308PE, Q37 BSS308PE, Q38 BSS308PE, Q39 NSV1C201MZ4, U3 LTC6811-1

Commit message: アノテーションし直し、
Parts:
- R188: renamed from R196; footprint Resistor_SMD:R_0402_1005Metric -> Resistor_SMD:R_0603_1608Metric
- R196: renamed from R204; footprint Resistor_SMD:R_0402_1005Metric -> Resistor_SMD:R_0603_1608Metric
- renumbered C104 to C100, C106 to C101, C108 to C102, C109 to C103, C110 to C104, C111 to C105, C112 to C106, C113 to C107, C114 to C108, C115 to C109, C116 to C110, C117 to C111, C79 to C75, C80 to C76, C81 to C77, C82 to C78, C83 to C79, C84 to C80, C85 to C81, C86 to C82, C87 to C83, C88 to C84, C89 to C85, C90 to C86, C91 to C87, C92 to C88, C93 to C89, C94 to C90, C95 to C91, C96 to C92, C97 to C93, C98 to C94, C99 to C95, C100 to C96, C101 to C97, C102 to C98, C103 to C99, D47 to D39, D48 to D40, D49 to D41, D50 to D42, D51 to D43, D52 to D44, D53 to D45, D54 to D46, D55 to D47, D56 to D48, D57 to D49, D58 to D50, D59 to D51, D60 to D52, D61 to D53, D64 to D54, D65 to D55, D66 to D56, D67 to D57, R147 to R139, R148 to R140, R149 to R141, R150 to R142, R151 to R143, R152 to R144, R153 to R145, R154 to R146, R155 to R147, R156 to R148, R157 to R149, R158 to R150, R159 to R151, R160 to R152, R161 to R153, R162 to R154, R163 to R155, R164 to R156, R165 to R157, R166 to R158, R167 to R159, R168 to R160, R169 to R161, R170 to R162, R171 to R163, R172 to R164, R173 to R165, R174 to R166, R175 to R167, R176 to R168, R177 to R169, R178 to R170, R179 to R171, R180 to R172, R181 to R173, R182 to R174, R183 to R175, R184 to R176, R185 to R177, R186 to R178, R187 to R179, R188 to R180, R189 to R181, R190 to R182, R191 to R183, R192 to R184, R193 to R185, R194 to R186, R195 to R187, R197 to R189, R198 to R190, R199 to R191, R200 to R192, R201 to R193, R202 to R194, R203 to R195, R205 to R197, R206 to R198, R207 to R199, R208 to R200, R209 to R201, R210 to R202, R211 to R203, R214 to R204, R215 to R205, R216 to R206

Commit message: 絶縁パルストランス数削減
Parts:
- renumbered L20 to L13
Changed lines of the file:
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@@
   (symbol (lib_id "ProjectEV:L_MH3261") (at 101.6 374.65 0) (unit 1)
     (in_bom yes) (on_board yes) (dnp no) (fields_autoplaced)
-    (property "Reference" "L20" (at 102.87 373.38 0)
+    (property "Reference" "L13" (at 102.87 373.38 0)
       (effects (font (size 1.27 1.27)) (justify left))
     )
@@
       (project "AMS-board-2024"
         (path "/3a719eb3-09ce-4343-8f6e-20cc0aaf5261/1e87e362-5c61-4f39-a903-ecfc3a14ee8d"
-          (reference "L20") (unit 1)
+          (reference "L13") (unit 1)
         )
       )

Commit message: 抵抗修正
3.3k -> 3k (1608)
15k -> 100k (1005, プルアップ/ダウン), 5.1k (1005, LED用)
Parts:
- R163, R164, R165, R166, R167, R168, R169, R170, R171, R172, R173, R174: value 3.3k -> 3k; footprint Resistor_SMD:R_0402_1005Metric -> Resistor_SMD:R_0603_1608Metric
Changed lines of the file:
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@@
       (effects (font (size 1.27 1.27)))
     )
-    (property "Value" "3.3k" (at 139.7 152.4 90)
+    (property "Value" "3k" (at 139.7 152.4 90)
       (effects (font (size 1.27 1.27)))
     )
-    (property "Footprint" "Resistor_SMD:R_0402_1005Metric" (at 139.7 156.718 90)
+    (property "Footprint" "Resistor_SMD:R_0603_1608Metric" (at 139.7 156.718 90)
       (effects (font (size 1.27 1.27)) hide)
     )
@@
       (effects (font (size 1.27 1.27)))
     )
-    (property "Value" "3.3k" (at 139.7 297.18 90)
+    (property "Value" "3k" (at 139.7 297.18 90)
       (effects (font (size 1.27 1.27)))
     )
-    (property "Footprint" "Resistor_SMD:R_0402_1005Metric" (at 139.7 301.498 90)
+    (property "Footprint" "Resistor_SMD:R_0603_1608Metric" (at 139.7 301.498 90)
       (effects (font (size 1.27 1.27)) hide)
     )
@@
       (effects (font (size 1.27 1.27)))
     )
-    (property "Value" "3.3k" (at 139.7 273.05 90)
+    (property "Value" "3k" (at 139.7 273.05 90)
       (effects (font (size 1.27 1.27)))
     )
-    (property "Footprint" "Resistor_SMD:R_0402_1005Metric" (at 139.7 277.368 90)
+    (property "Footprint" "Resistor_SMD:R_0603_1608Metric" (at 139.7 277.368 90)
       (effects (font (size 1.27 1.27)) hide)
     )
@@
       (effects (font (size 1.27 1.27)))
     )
-    (property "Value" "3.3k" (at 139.7 104.14 90)
+    (property "Value" "3k" (at 139.7 104.14 90)
       (effects (font (size 1.27 1.27)))
     )
-    (property "Footprint" "Resistor_SMD:R_0402_1005Metric" (at 139.7 108.458 90)
+    (property "Footprint" "Resistor_SMD:R_0603_1608Metric" (at 139.7 108.458 90)
       (effects (font (size 1.27 1.27)) hide)
     )
@@
       (effects (font (size 1.27 1.27)))
     )
-    (property "Value" "3.3k" (at 139.7 200.66 90)
+    (property "Value" "3k" (at 139.7 200.66 90)
       (effects (font (size 1.27 1.27)))
     )
-    (property "Footprint" "Resistor_SMD:R_0402_1005Metric" (at 139.7 204.978 90)
+    (property "Footprint" "Resistor_SMD:R_0603_1608Metric" (at 139.7 204.978 90)
       (effects (font (size 1.27 1.27)) hide)
     )
@@
       (effects (font (size 1.27 1.27)))
     )
-    (property "Value" "3.3k" (at 139.7 80.01 90)
+    (property "Value" "3k" (at 139.7 80.01 90)
       (effects (font (size 1.27 1.27)))
     )
-    (property "Footprint" "Resistor_SMD:R_0402_1005Metric" (at 139.7 84.328 90)
+    (property "Footprint" "Resistor_SMD:R_0603_1608Metric" (at 139.7 84.328 90)
       (effects (font (size 1.27 1.27)) hide)
     )
@@
       (effects (font (size 1.27 1.27)))
     )
-    (property "Value" "3.3k" (at 139.7 224.79 90)
+    (property "Value" "3k" (at 139.7 224.79 90)
       (effects (font (size 1.27 1.27)))
     )
-    (property "Footprint" "Resistor_SMD:R_0402_1005Metric" (at 139.7 229.108 90)
+    (property "Footprint" "Resistor_SMD:R_0603_1608Metric" (at 139.7 229.108 90)
       (effects (font (size 1.27 1.27)) hide)
     )
@@
       (effects (font (size 1.27 1.27)))
     )
-    (property "Value" "3.3k" (at 139.7 176.53 90)
+    (property "Value" "3k" (at 139.7 176.53 90)
       (effects (font (size 1.27 1.27)))
     )
-    (property "Footprint" "Resistor_SMD:R_0402_1005Metric" (at 139.7 180.848 90)
+    (property "Footprint" "Resistor_SMD:R_0603_1608Metric" (at 139.7 180.848 90)
       (effects (font (size 1.27 1.27)) hide)
     )
@@
       (effects (font (size 1.27 1.27)))
     )
-    (property "Value" "3.3k" (at 139.7 321.31 90)
+    (property "Value" "3k" (at 139.7 321.31 90)
       (effects (font (size 1.27 1.27)))
     )
-    (property "Footprint" "Resistor_SMD:R_0402_1005Metric" (at 139.7 325.628 90)
+    (property "Footprint" "Resistor_SMD:R_0603_1608Metric" (at 139.7 325.628 90)
       (effects (font (size 1.27 1.27)) hide)
     )
@@
       (effects (font (size 1.27 1.27)))
     )
-    (property "Value" "3.3k" (at 139.7 345.44 90)
+    (property "Value" "3k" (at 139.7 345.44 90)
       (effects (font (size 1.27 1.27)))
     )
-    (property "Footprint" "Resistor_SMD:R_0402_1005Metric" (at 139.7 349.758 90)
+    (property "Footprint" "Resistor_SMD:R_0603_1608Metric" (at 139.7 349.758 90)
       (effects (font (size 1.27 1.27)) hide)
     )
@@
       (effects (font (size 1.27 1.27)))
     )
-    (property "Value" "3.3k" (at 139.7 128.27 90)
+    (property "Value" "3k" (at 139.7 128.27 90)
       (effects (font (size 1.27 1.27)))
     )
-    (property "Footprint" "Resistor_SMD:R_0402_1005Metric" (at 139.7 132.588 90)
+    (property "Footprint" "Resistor_SMD:R_0603_1608Metric" (at 139.7 132.588 90)
       (effects (font (size 1.27 1.27)) hide)
     )
@@
       (effects (font (size 1.27 1.27)))
     )
-    (property "Value" "3.3k" (at 139.7 248.92 90)
+    (property "Value" "3k" (at 139.7 248.92 90)
       (effects (font (size 1.27 1.27)))
     )
-    (property "Footprint" "Resistor_SMD:R_0402_1005Metric" (at 139.7 253.238 90)
+    (property "Footprint" "Resistor_SMD:R_0603_1608Metric" (at 139.7 253.238 90)
       (effects (font (size 1.27 1.27)) hide)
     )

Commit message: アノテーションし直し
Parts:
- renumbered C91 to C100, C92 to C101, C93 to C102, C94 to C103, C95 to C104, C96 to C105, C97 to C106, C98 to C107, C99 to C108, C100 to C109, C101 to C110, C102 to C111, C103 to C112, C104 to C113, C105 to C114, C106 to C115, C107 to C116, C108 to C117, C109 to C118, C110 to C119, C111 to C120, C75 to C84, C76 to C85, C77 to C86, C78 to C87, C79 to C88, C80 to C89, C81 to C90, C82 to C91, C83 to C92, C84 to C93, C85 to C94, C86 to C95, C87 to C96, C88 to C97, C89 to C98, C90 to C99, L13 to L9
