File: AMS-board-2024/battery-module-monitor-4.kicad_sch (KiCad schematic)
At the start: 144 parts, among them Q501 BSS308PE, Q502 BSS308PE, Q503 BSS308PE, Q504 BSS308PE, Q505 BSS308PE, Q506 BSS308PE, Q507 BSS308PE, Q508 BSS308PE, Q509 BSS308PE, Q510 BSS308PE, Q511 BSS308PE, Q512 BSS308PE, Q513 NSV1C201MZ4, U501 LTC6811-1

Commit message: 修正
アノテーション方法の変更：最初の空き番号から使用
Parts:
- renumbered C501 to C103, C502 to C104, C503 to C105, C504 to C106, C505 to C107, C506 to C108, C507 to C109, C508 to C110, C509 to C111, C510 to C112, C511 to C113, C512 to C114, C513 to C115, C514 to C116, C515 to C117, C516 to C118, C517 to C119, C518 to C120, C519 to C121, C520 to C122, C521 to C123, C522 to C124, C523 to C125, C524 to C126, C525 to C127, C526 to C128, C527 to C129, C528 to C130, C529 to C131, C530 to C132, C531 to C133, C532 to C134, C533 to C135, C534 to C136, D501 to D40, D502 to D41, D503 to D42, D504 to D43, D505 to D44, D506 to D45, D507 to D46, D508 to D47, D509 to D48, D510 to D49, D511 to D50, D512 to D51, D513 to D52, F501 to F40, F502 to F41, F503 to F42, F504 to F43, F505 to F44, F506 to F45, F507 to F46, F508 to F47, F509 to F48, F510 to F49, F511 to F50, F512 to F51, F513 to F52, FL501 to FL7, FL502 to FL8, L501 to L4, Q501 to Q40, Q502 to Q41, Q503 to Q42, Q504 to Q43, Q505 to Q44, Q506 to Q45, Q507 to Q46, Q508 to Q47, Q509 to Q48, Q510 to Q49, Q511 to Q50, Q512 to Q51, Q513 to Q52, R501 to R202, R502 to R203, R503 to R204, R504 to R205, R505 to R206, R506 to R207, R507 to R208, R508 to R209, R509 to R210, R510 to R211, R511 to R212, R512 to R213, R513 to R214, R514 to R215, R515 to R216, R516 to R217, R517 to R218, R518 to R219, R519 to R220, R520 to R221, R521 to R222, R522 to R223, R523 to R224, R524 to R225, R525 to R226, R526 to R227, R527 to R228, R528 to R229, R529 to R230, R530 to R231, R531 to R232, R532 to R233, R533 to R234, R534 to R235, R535 to R236, R536 to R237, R537 to R238, R538 to R239, R539 to R240, R540 to R241, R541 to R242, R542 to R243, R543 to R244, R544 to R245, R545 to R246, R546 to R247, R547 to R248, R548 to R249, R549 to R250, R550 to R251, R551 to R252, R552 to R253, R553 to R254, R554 to R255, R555 to R256, R556 to R257, R557 to R258, R558 to R259, R559 to R260, R560 to R261, R561 to R262, R562 to R263, R563 to R264, R564 to R265, R565 to R266, R566 to R267, R567 to R268, U501 to U4

Commit message: GNDシンボル追加
Connections:
- net GND1: now reaches C133.1
- net GND1: now also C103.2, C104.2, C105.2, C106.2, C107.2, C108.2, C109.2, C110.2, C111.2, C112.2, C113.2, C114.2, C127.2, C128.2, C129.1, C130.1, C131.2, C132.1, C134.2, C135.1, C136.1, L4.2, R256.1, U4.30 (V-), U4.31 (V-)

Commit message: GPIO周辺回路の修正
Parts:
- added C306, C307, C308, C309, C310: 0.1u, Capacitor_SMD:C_0603_1608Metric, symbol Device:C
- added R573, R574, R575, R576, R577: 10k, Resistor_SMD:R_0603_1608Metric, symbol Device:R
- R252, R255, R257, R258, R263: value 10k -> 100
Connections:
- net GND1: now also C306.2, C307.2, C308.2, C309.2, C310.2
- net Thermistor1+: now also R252.2, R573.2; no longer R263.1, U4.27 (GPIO1)
- net Thermistor2+: now also R255.2, R574.2; no longer R258.1, U4.28 (GPIO2)
- net Thermistor3+: now also R257.2, R575.2; no longer R257.1, U4.29 (GPIO3)
- net Thermistor4+: now also R258.2, R576.2; no longer R255.1, U4.32 (GPIO4)
- net Thermistor5+: now also R263.2, R577.2; no longer R252.1, U4.33 (GPIO5)
- net VREG: now reaches C131.1, Q52.3 (E), R254.1, U4.37 (VREG), U4.40 (ISOMD)
- new net: C310.1, R252.1, U4.27 (GPIO1)
- new net: C309.1, R255.1, U4.28 (GPIO2)
- new net: C308.1, R257.1, U4.29 (GPIO3)
- new net: C307.1, R258.1, U4.32 (GPIO4)
- new net: C306.1, R263.1, U4.33 (GPIO5)
- new net VREF_3V: C129.2, R573.1, R574.1, R575.1, R576.1, R577.1, U4.34 (VREF2)

Commit message: テキスト修正
Other:
- note added: "レギュレーション上必要なサーミスタは 96 CELL x 25 % = 24 本. GPIO1~3 をサーミスタに使用し、 GPIO4, 5 は別用途で使用してもOK. GPIO4, 5 のプルアップは必要に応じて実装."
- note removed: "レギュレーション上必要なサーミスタは 3 x 8 = 24 本. GPIO1~3 をサーミスタに使用し、 GPIO4, 5 は別用途で使用してもOK. GPIO4, 5 のプルアップは必要に応じて実装."
Changed lines of the file:
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@@
+    (effects (font (size 1.27 1.27)) (justify left bottom))
+  )
+  (text "レギュレーション上必要なサーミスタは 96 CELL x 25 % = 24 本.\nGPIO1~3 をサーミスタに使用し、\nGPIO4, 5 は別用途で使用してもOK.\nGPIO4, 5 のプルアップは必要に応じて実装."
+    (at 469.9 283.21 0)
     (effects (font (size 1.27 1.27)) (justify left bottom))
   )
@@
     (effects (font (size 1.27 1.27)) (justify left bottom))
   )
-  (text "レギュレーション上必要なサーミスタは 3 x 8 = 24 本.\nGPIO1~3 をサーミスタに使用し、\nGPIO4, 5 は別用途で使用してもOK.\nGPIO4, 5 のプルアップは必要に応じて実装."
-    (at 469.9 283.21 0)
-    (effects (font (size 1.27 1.27)) (justify left bottom))
-  )

Commit message: ヒューズ変更
Parts:
- removed F40, F41, F42, F43, F44, F45, F46, F47, F48, F49, F50, F51, F52: C1F 500, Fuse:Fuse_1206_3216Metric, symbol Device:Fuse
- added F14, F15, F16, F17, F18, F19, F20, F21, F22, F23, F24, F25, F26: 0679L1000-05, ProjectEV:Fuse_0679L, symbol ProjectEV:Fuse_0679L1000-05
Connections:
- net CELL0: now also F26.1
- net CELL1: now also F25.1
- net CELL10: now also F16.1
- net CELL11: now also F15.1
- net CELL12: now also F14.1
- net CELL2: now also F24.1
- net CELL3: now also F23.1
- net CELL4: now also F22.1
- net CELL5: now also F21.1
- net CELL6: now also F20.1
- net CELL7: now also F19.1
- net CELL8: now also F18.1
- net CELL9: now also F17.1
- net at Q46.2 (S), R207.2, R219.2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: now also F20.2
- net at Q43.2 (S), R204.2, R216.2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: now also F17.2
- net at Q48.2 (S), R209.2, R221.2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: now also F22.2
- net at D40.1 (K), Q51.2 (S), R212.2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: now also F25.2
- net at Q42.2 (S), R203.2, R215.2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: now also F16.2
- net at Q45.2 (S), R206.2, R218.2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: now also F19.2
- net at Q47.2 (S), R208.2, R220.2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: now also F21.2
- net at Q49.2 (S), R210.2, R222.2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: now also F23.2
- net at Q50.2 (S), R211.2, R223.2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: now also F24.2
- net at Q40.2 (S), R238.1, R251.1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: now also F14.2
- net at Q41.2 (S), R202.2, R214.2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: now also F15.2
- net at Q44.2 (S), R205.2, R217.2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: now also F18.2
- net at D40.2 (A), L4.1, R213.2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: now also F26.2

Commit message: アノテーションし直し
Parts:
- renumbered C103 to C118, C104 to C119, C105 to C120, C106 to C121, C107 to C122, C108 to C123, C109 to C124, C110 to C125, C111 to C126, C112 to C127, C113 to C128, C114 to C129, C115 to C130, C116 to C131, C117 to C132, C118 to C133, C119 to C134, C120 to C135, C121 to C136, C122 to C137, C123 to C138, C124 to C139, C125 to C140, C126 to C141, C127 to C142, C128 to C143, C306 to C144, C129 to C145, C307 to C146, C130 to C147, C131 to C148, C308 to C149, C132 to C150, C133 to C151, C309 to C152, C310 to C153, C134 to C154, C135 to C155, C136 to C156, F14 to F40, F15 to F41, F16 to F42, F17 to F43, F18 to F44, F19 to F45, F20 to F46, F21 to F47, F22 to F48, F23 to F49, F24 to F50, F25 to F51, F26 to F52, R202 to R217, R203 to R218, R204 to R219, R205 to R220, R206 to R221, R207 to R222, R208 to R223, R209 to R224, R210 to R225, R211 to R226, R212 to R227, R213 to R228, R214 to R229, R215 to R230, R216 to R231, R217 to R232, R218 to R233, R219 to R234, R220 to R235, R221 to R236, R222 to R237, R223 to R238, R224 to R239, R225 to R240, R226 to R241, R227 to R242, R228 to R243, R229 to R244, R230 to R245, R231 to R246, R232 to R247, R233 to R248, R234 to R249, R235 to R250, R236 to R251, R237 to R252, R238 to R253, R239 to R254, R240 to R255, R241 to R256, R242 to R257, R243 to R258, R244 to R259, R245 to R260, R246 to R261, R247 to R262, R248 to R263, R249 to R264, R250 to R265, R251 to R266, R253 to R267, R254 to R268, R256 to R269, R259 to R270, R260 to R271, R261 to R272, R262 to R273, R264 to R274, R252 to R275, R255 to R276, R257 to R277, R258 to R278, R263 to R279, R573 to R280, R265 to R281, R266 to R282, R267 to R283, R268 to R284, R574 to R285, R575 to R286, R576 to R287, R577 to R288

Commit message: GPIO入力保護回路追加
Parts:
- added D160, D161, D162, D163, D164, D165, D166, D167, D168, D169: BAT46W-7-F, ProjectEV:D_SOD-123_BAT46W-7-F, symbol ProjectEV:D_BAT46W-7-F
Connections:
- net GND1: now also D161.2 (A), D163.2 (A), D165.2 (A), D167.2 (A), D169.2 (A)
- net VREG: now also D160.1 (K), D162.1 (K), D164.1 (K), D166.1 (K), D168.1 (K)
- net at C153.1, R275.1, U4.27 (GPIO1): now also D160.2 (A), D161.1 (K)
- net at C152.1, R276.1, U4.28 (GPIO2): now also D162.2 (A), D163.1 (K)
- net at C149.1, R277.1, U4.29 (GPIO3): now also D164.2 (A), D165.1 (K)
- net at C146.1, R278.1, U4.32 (GPIO4): now also D166.2 (A), D167.1 (K)
- net at C144.1, R279.1, U4.33 (GPIO5): now also D168.2 (A), D169.1 (K)
Other:
- moved on the sheet: R275, R276, R277, R278, R279, R280, R285, R286, R287, R288

Commit message: アノテーションし直し
Parts:
- renumbered D40 to D70, D41 to D71, D42 to D72, D43 to D73, D44 to D74, D45 to D75, D46 to D76, D47 to D77, D48 to D78, D49 to D79, D50 to D80, D51 to D81, D52 to D82, D162 to D83, D163 to D84, D166 to D85, D167 to D86, D160 to D87, D161 to D88, D164 to D89, D165 to D90, D168 to D91, D169 to D92, L4 to L20, R217 to R219, R218 to R220, R219 to R221, R220 to R222, R221 to R223, R222 to R224, R223 to R225, R224 to R226, R225 to R227, R226 to R228, R227 to R229, R228 to R230, R229 to R231, R230 to R232, R231 to R233, R232 to R234, R233 to R235, R234 to R236, R235 to R237, R236 to R238, R237 to R239, R238 to R240, R239 to R241, R240 to R242, R241 to R243, R242 to R244, R243 to R245, R244 to R246, R245 to R247, R246 to R248, R247 to R249, R248 to R250, R249 to R251, R250 to R252, R251 to R253, R252 to R254, R253 to R255, R254 to R256, R255 to R257, R256 to R258, R257 to R259, R258 to R260, R259 to R261, R260 to R262, R261 to R263, R262 to R264, R263 to R265, R264 to R266, R265 to R267, R266 to R268, R267 to R269, R268 to R270, R269 to R271, R270 to R272, R271 to R273, R272 to R274, R273 to R275, R274 to R276, R281 to R277, R282 to R278, R283 to R279, R284 to R280, R275 to R281, R276 to R282, R277 to R283, R278 to R284, R279 to R285, R280 to R286, R285 to R287, R286 to R288, R287 to R289, R288 to R290
