File: AMS-board-2024/battery-module-monitor-4.kicad_sch (KiCad schematic)
At the start: 154 parts, among them Q40 BSS308PE, Q41 BSS308PE, Q42 BSS308PE, Q43 BSS308PE, Q44 BSS308PE, Q45 BSS308PE, Q46 BSS308PE, Q47 BSS308PE, Q48 BSS308PE, Q49 BSS308PE, Q50 BSS308PE, Q51 BSS308PE, Q52 NSV1C201MZ4, U4 LTC6811-1

Commit message: アノテーションし直し、
Parts:
- R256: renamed from R268; footprint Resistor_SMD:R_0402_1005Metric -> Resistor_SMD:R_0603_1608Metric
- R264: renamed from R276; footprint Resistor_SMD:R_0402_1005Metric -> Resistor_SMD:R_0603_1608Metric
- renumbered C118 to C112, C119 to C113, C120 to C114, C121 to C115, C122 to C116, C123 to C117, C124 to C118, C125 to C119, C126 to C120, C127 to C121, C128 to C122, C129 to C123, C130 to C124, C131 to C125, C132 to C126, C133 to C127, C134 to C128, C135 to C129, C136 to C130, C137 to C131, C138 to C132, C139 to C133, C140 to C134, C141 to C135, C142 to C136, C143 to C137, C145 to C138, C147 to C139, C148 to C140, C149 to C141, C150 to C142, C151 to C143, C152 to C144, C153 to C145, C154 to C146, C155 to C147, C156 to C148, D70 to D58, D71 to D59, D72 to D60, D73 to D61, D74 to D62, D75 to D63, D76 to D64, D77 to D65, D78 to D66, D79 to D67, D80 to D68, D81 to D69, D82 to D70, D83 to D71, D84 to D72, D87 to D73, D88 to D74, D89 to D75, D90 to D76, R219 to R207, R220 to R208, R221 to R209, R222 to R210, R223 to R211, R224 to R212, R225 to R213, R226 to R214, R227 to R215, R228 to R216, R229 to R217, R230 to R218, R231 to R219, R232 to R220, R233 to R221, R234 to R222, R235 to R223, R236 to R224, R237 to R225, R238 to R226, R239 to R227, R240 to R228, R241 to R229, R242 to R230, R243 to R231, R244 to R232, R245 to R233, R246 to R234, R247 to R235, R248 to R236, R249 to R237, R250 to R238, R251 to R239, R252 to R240, R253 to R241, R254 to R242, R255 to R243, R256 to R244, R257 to R245, R258 to R246, R259 to R247, R260 to R248, R261 to R249, R262 to R250, R263 to R251, R264 to R252, R265 to R253, R266 to R254, R267 to R255, R269 to R257, R270 to R258, R271 to R259, R272 to R260, R273 to R261, R274 to R262, R275 to R263, R277 to R265, R278 to R266, R279 to R267, R280 to R268, R281 to R269, R282 to R270, R283 to R271, R286 to R272, R287 to R273, R288 to R274
