File: AMS-board-2024/battery-module-monitor-5.kicad_sch (KiCad schematic)
At the start: 144 parts, among them Q601 BSS308PE, Q602 BSS308PE, Q603 BSS308PE, Q604 BSS308PE, Q605 BSS308PE, Q606 BSS308PE, Q607 BSS308PE, Q608 BSS308PE, Q609 BSS308PE, Q610 BSS308PE, Q611 BSS308PE, Q612 BSS308PE, Q613 NSV1C201MZ4, U601 LTC6811-1

Commit message: 修正
アノテーション方法の変更：最初の空き番号から使用
Parts:
- renumbered C601 to C137, C602 to C138, C603 to C139, C604 to C140, C605 to C141, C606 to C142, C607 to C143, C608 to C144, C609 to C145, C610 to C146, C611 to C147, C612 to C148, C613 to C149, C614 to C150, C615 to C151, C616 to C152, C617 to C153, C618 to C154, C619 to C155, C620 to C156, C621 to C157, C622 to C158, C623 to C159, C624 to C160, C625 to C161, C626 to C162, C627 to C163, C628 to C164, C629 to C165, C630 to C166, C631 to C167, C632 to C168, C633 to C169, C634 to C170, D601 to D53, D602 to D54, D603 to D55, D604 to D56, D605 to D57, D606 to D58, D607 to D59, D608 to D60, D609 to D61, D610 to D62, D611 to D63, D612 to D64, D613 to D65, F601 to F53, F602 to F54, F603 to F55, F604 to F56, F605 to F57, F606 to F58, F607 to F59, F608 to F60, F609 to F61, F610 to F62, F611 to F63, F612 to F64, F613 to F65, FL602 to FL10, FL601 to FL9, L601 to L5, Q601 to Q53, Q602 to Q54, Q603 to Q55, Q604 to Q56, Q605 to Q57, Q606 to Q58, Q607 to Q59, Q608 to Q60, Q609 to Q61, Q610 to Q62, Q611 to Q63, Q612 to Q64, Q613 to Q65, R601 to R269, R602 to R270, R603 to R271, R604 to R272, R605 to R273, R606 to R274, R607 to R275, R608 to R276, R609 to R277, R610 to R278, R611 to R279, R612 to R280, R613 to R281, R614 to R282, R615 to R283, R616 to R284, R617 to R285, R618 to R286, R619 to R287, R620 to R288, R621 to R289, R622 to R290, R623 to R291, R624 to R292, R625 to R293, R626 to R294, R627 to R295, R628 to R296, R629 to R297, R630 to R298, R631 to R299, R632 to R300, R633 to R301, R634 to R302, R635 to R303, R636 to R304, R637 to R305, R638 to R306, R639 to R307, R640 to R308, R641 to R309, R642 to R310, R643 to R311, R644 to R312, R645 to R313, R646 to R314, R647 to R315, R648 to R316, R649 to R317, R650 to R318, R651 to R319, R652 to R320, R653 to R321, R654 to R322, R655 to R323, R656 to R324, R657 to R325, R658 to R326, R659 to R327, R660 to R328, R661 to R329, R662 to R330, R663 to R331, R664 to R332, R665 to R333, R666 to R334, R667 to R335, U601 to U5

Commit message: GNDシンボル追加
Connections:
- net GND1: now reaches C161.2
- net GND1: now also C137.2, C138.2, C139.2, C140.2, C141.2, C142.2, C143.2, C144.2, C145.2, C146.2, C147.2, C148.2, C162.2, C163.1, C164.1, C165.2, C166.1, C167.1, C168.2, C169.1, C170.1, L5.2, R323.1, U5.30 (V-), U5.31 (V-)

Commit message: GPIO周辺回路の修正
Parts:
- added C311, C312, C313, C314, C315: 0.1u, Capacitor_SMD:C_0603_1608Metric, symbol Device:C
- added R578, R579, R580, R581, R582: 10k, Resistor_SMD:R_0603_1608Metric, symbol Device:R
- R319, R322, R324, R325, R330: value 10k -> 100
Connections:
- net GND1: now also C311.2, C312.2, C313.2, C314.2, C315.2
- net Thermistor1+: now also R319.2, R578.2; no longer R330.1, U5.27 (GPIO1)
- net Thermistor2+: now also R322.2, R579.2; no longer R325.1, U5.28 (GPIO2)
- net Thermistor3+: now also R324.2, R580.2; no longer R324.1, U5.29 (GPIO3)
- net Thermistor4+: now also R325.2, R581.2; no longer R322.1, U5.32 (GPIO4)
- net Thermistor5+: now also R330.2, R582.2; no longer R319.1, U5.33 (GPIO5)
- net VREG: now reaches C165.1, Q65.3 (E), R321.1, U5.37 (VREG), U5.40 (ISOMD)
- new net: C314.1, R322.1, U5.28 (GPIO2)
- new net: C312.1, R325.1, U5.32 (GPIO4)
- new net: C311.1, R330.1, U5.33 (GPIO5)
- new net: C313.1, R324.1, U5.29 (GPIO3)
- new net: C315.1, R319.1, U5.27 (GPIO1)
- new net VREF_3V: C163.2, R578.1, R579.1, R580.1, R581.1, R582.1, U5.34 (VREF2)

Commit message: テキスト修正
Other:
- note added: "レギュレーション上必要なサーミスタは 96 CELL x 25 % = 24 本. GPIO1~3 をサーミスタに使用し、 GPIO4, 5 は別用途で使用してもOK. GPIO4, 5 のプルアップは必要に応じて実装."
- note removed: "レギュレーション上必要なサーミスタは 3 x 8 = 24 本. GPIO1~3 をサーミスタに使用し、 GPIO4, 5 は別用途で使用してもOK. GPIO4, 5 のプルアップは必要に応じて実装."
Changed lines of the file:
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@@
-    (effects (font (size 1.27 1.27)) (justify left bottom))
-  )
-  (text "レギュレーション上必要なサーミスタは 3 x 8 = 24 本.\nGPIO1~3 をサーミスタに使用し、\nGPIO4, 5 は別用途で使用してもOK.\nGPIO4, 5 のプルアップは必要に応じて実装."
-    (at 469.9 283.21 0)
     (effects (font (size 1.27 1.27)) (justify left bottom))
   )
@@
     (effects (font (size 1.27 1.27)) (justify left bottom))
   )
+  (text "レギュレーション上必要なサーミスタは 96 CELL x 25 % = 24 本.\nGPIO1~3 をサーミスタに使用し、\nGPIO4, 5 は別用途で使用してもOK.\nGPIO4, 5 のプルアップは必要に応じて実装."
+    (at 469.9 283.21 0)
+    (effects (font (size 1.27 1.27)) (justify left bottom))
+  )

Commit message: ヒューズ変更
Parts:
- removed F53, F54, F55, F56, F57, F58, F59, F60, F61, F62, F63, F64, F65: C1F 500, Fuse:Fuse_1206_3216Metric, symbol Device:Fuse
- added F27, F28, F29, F30, F31, F32, F33, F34, F35, F36, F37, F38, F39: 0679L1000-05, ProjectEV:Fuse_0679L, symbol ProjectEV:Fuse_0679L1000-05
Connections:
- net CELL0: now also F39.1
- net CELL1: now also F38.1
- net CELL10: now also F29.1
- net CELL11: now also F28.1
- net CELL12: now also F27.1
- net CELL2: now also F37.1
- net CELL3: now also F36.1
- net CELL4: now also F35.1
- net CELL5: now also F34.1
- net CELL6: now also F33.1
- net CELL7: now also F32.1
- net CELL8: now also F31.1
- net CELL9: now also F30.1
- net at Q53.2 (S), R305.1, R318.1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: now also F27.2
- net at Q54.2 (S), R269.2, R281.2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: now also F28.2
- net at Q56.2 (S), R271.2, R283.2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: now also F30.2
- net at Q58.2 (S), R273.2, R285.2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: now also F32.2
- net at Q57.2 (S), R272.2, R284.2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: now also F31.2
- net at Q60.2 (S), R275.2, R287.2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: now also F34.2
- net at D53.1 (K), Q64.2 (S), R279.2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: now also F38.2
- net at Q55.2 (S), R270.2, R282.2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: now also F29.2
- net at Q59.2 (S), R274.2, R286.2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: now also F33.2
- net at D53.2 (A), L5.1, R280.2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: now also F39.2
- net at Q61.2 (S), R276.2, R288.2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: now also F35.2
- net at Q62.2 (S), R277.2, R289.2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: now also F36.2
- net at Q63.2 (S), R278.2, R290.2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: now also F37.2

Commit message: アノテーションし直し
Parts:
- renumbered C137 to C157, C138 to C158, C139 to C159, C140 to C160, C141 to C161, C142 to C162, C143 to C163, C144 to C164, C145 to C165, C146 to C166, C147 to C167, C148 to C168, C149 to C169, C150 to C170, C151 to C171, C152 to C172, C153 to C173, C154 to C174, C155 to C175, C156 to C176, C157 to C177, C158 to C178, C159 to C179, C160 to C180, C161 to C181, C162 to C182, C311 to C183, C163 to C184, C312 to C185, C164 to C186, C165 to C187, C313 to C188, C166 to C189, C167 to C190, C314 to C191, C315 to C192, C168 to C193, C169 to C194, C170 to C195, F27 to F53, F28 to F54, F29 to F55, F30 to F56, F31 to F57, F32 to F58, F33 to F59, F34 to F60, F35 to F61, F36 to F62, F37 to F63, F38 to F64, F39 to F65, R269 to R289, R270 to R290, R271 to R291, R272 to R292, R273 to R293, R274 to R294, R275 to R295, R276 to R296, R277 to R297, R278 to R298, R279 to R299, R280 to R300, R281 to R301, R282 to R302, R283 to R303, R284 to R304, R285 to R305, R286 to R306, R287 to R307, R288 to R308, R289 to R309, R290 to R310, R291 to R311, R292 to R312, R293 to R313, R294 to R314, R295 to R315, R296 to R316, R297 to R317, R298 to R318, R299 to R319, R300 to R320, R301 to R321, R302 to R322, R303 to R323, R304 to R324, R305 to R325, R306 to R326, R307 to R327, R308 to R328, R309 to R329, R310 to R330, R311 to R331, R312 to R332, R313 to R333, R314 to R334, R315 to R335, R316 to R336, R317 to R337, R318 to R338, R320 to R339, R321 to R340, R323 to R341, R326 to R342, R327 to R343, R328 to R344, R329 to R345, R331 to R346, R319 to R347, R322 to R348, R324 to R349, R325 to R350, R330 to R351, R578 to R352, R332 to R353, R333 to R354, R334 to R355, R335 to R356, R579 to R357, R580 to R358, R581 to R359, R582 to R360

Commit message: GPIO入力保護回路追加
Parts:
- added D170, D171, D172, D173, D174, D175, D176, D177, D178, D179: BAT46W-7-F, ProjectEV:D_SOD-123_BAT46W-7-F, symbol ProjectEV:D_BAT46W-7-F
Connections:
- net GND1: now also D171.2 (A), D173.2 (A), D175.2 (A), D177.2 (A), D179.2 (A)
- net VREG: now also D170.1 (K), D172.1 (K), D174.1 (K), D176.1 (K), D178.1 (K)
- net at C191.1, R348.1, U5.28 (GPIO2): now also D172.2 (A), D173.1 (K)
- net at C185.1, R350.1, U5.32 (GPIO4): now also D176.2 (A), D177.1 (K)
- net at C183.1, R351.1, U5.33 (GPIO5): now also D178.2 (A), D179.1 (K)
- net at C188.1, R349.1, U5.29 (GPIO3): now also D174.2 (A), D175.1 (K)
- net at C192.1, R347.1, U5.27 (GPIO1): now also D170.2 (A), D171.1 (K)
Other:
- moved on the sheet: R347, R348, R349, R350, R351, R352, R357, R358, R359, R360

Commit message: アノテーションし直し
Parts:
- renumbered D60 to D100, D61 to D101, D62 to D102, D63 to D103, D64 to D104, D65 to D105, D172 to D106, D173 to D107, D176 to D108, D177 to D109, D170 to D110, D171 to D111, D174 to D112, D175 to D113, D178 to D114, D179 to D115, D53 to D93, D54 to D94, D55 to D95, D56 to D96, D57 to D97, D58 to D98, D59 to D99, L5 to L21, R289 to R291, R290 to R292, R291 to R293, R292 to R294, R293 to R295, R294 to R296, R295 to R297, R296 to R298, R297 to R299, R298 to R300, R299 to R301, R300 to R302, R301 to R303, R302 to R304, R303 to R305, R304 to R306, R305 to R307, R306 to R308, R307 to R309, R308 to R310, R309 to R311, R310 to R312, R311 to R313, R312 to R314, R313 to R315, R314 to R316, R315 to R317, R316 to R318, R317 to R319, R318 to R320, R319 to R321, R320 to R322, R321 to R323, R322 to R324, R323 to R325, R324 to R326, R325 to R327, R326 to R328, R327 to R329, R328 to R330, R329 to R331, R330 to R332, R331 to R333, R332 to R334, R333 to R335, R334 to R336, R335 to R337, R336 to R338, R337 to R339, R338 to R340, R339 to R341, R340 to R342, R341 to R343, R342 to R344, R343 to R345, R344 to R346, R345 to R347, R346 to R348, R353 to R349, R354 to R350, R355 to R351, R356 to R352, R347 to R353, R348 to R354, R349 to R355, R350 to R356, R351 to R357, R352 to R358, R357 to R359, R358 to R360, R359 to R361, R360 to R362
