File: AMS-board-2024/battery-module-monitor-5.kicad_sch (KiCad schematic)
At the start: 164 parts, among them Q53 BSS308PE, Q54 BSS308PE, Q55 BSS308PE, Q56 BSS308PE, Q57 BSS308PE, Q58 BSS308PE, Q59 BSS308PE, Q60 BSS308PE, Q61 BSS308PE, Q62 BSS308PE, Q63 BSS308PE, Q64 BSS308PE, Q65 NSV1C201MZ4, U5 LTC6811-1

Commit message: ERC実行、修正
ラベル修正、未配線部分修正、PWR_FLAG追加
Connections:
- net GND1 is gone; now on net GND5: C157.2, C158.2, C159.2, C160.2, C161.2, C162.2, C163.2, C164.2, C165.2, C166.2, C167.2, C168.2, C181.2, C182.2, C183.2, C184.1, C185.2, C186.1, C187.2, C188.2, C189.1, C190.1, C191.2, C192.2, C193.2, C194.1, C195.1, D107.2 (A), D109.2 (A), D111.2 (A), D113.2 (A), D115.2 (A), L21.2, R343.1, U5.30 (V-), U5.31 (V-)
- net GND5: now reaches U5.36 (SWTEN)
- net VREG renamed VREG5
Changed lines of the file:
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@@
   (junction (at 292.1 252.73) (diameter 0) (color 0 0 0 0)
   )
+  (junction (at 292.1 165.1) (diameter 0) (color 0 0 0 0)
+  )
   (junction (at 368.3 279.4) (diameter 0) (color 0 0 0 0)
   )
@@
   (junction (at 114.3 196.85) (diameter 0) (color 0 0 0 0)
   )
+  (junction (at 101.6 381) (diameter 0) (color 0 0 0 0)
+  )
   (junction (at 165.1 317.5) (diameter 0) (color 0 0 0 0)
   )
@@
     (stroke (width 0) (type default))
   )
+  (wire (pts (xy 96.52 381) (xy 101.6 381))
+    (stroke (width 0) (type default))
+  )
   (wire (pts (xy 149.86 317.5) (xy 152.4 317.5))
     (stroke (width 0) (type default))
@@
     (stroke (width 0) (type default))
   )
+  (wire (pts (xy 101.6 381) (xy 101.6 383.54))
+    (stroke (width 0) (type default))
+  )
   (wire (pts (xy 304.8 246.38) (xy 307.34 246.38))
     (stroke (width 0) (type default))
@@
     (stroke (width 0) (type default))
   )
+  (wire (pts (xy 304.8 223.52) (xy 307.34 223.52))
+    (stroke (width 0) (type default))
+  )
   (wire (pts (xy 304.8 236.22) (xy 358.14 236.22))
     (stroke (width 0) (type default))
@@
     (stroke (width 0) (type default))
   )
-  (wire (pts (xy 101.6 378.46) (xy 101.6 379.73))
+  (wire (pts (xy 101.6 378.46) (xy 101.6 381))
     (stroke (width 0) (type default))
   )
@@
     (effects (font (size 1.27 1.27)) (justify right))
   )
-  (hierarchical_label "VREG" (shape output) (at 419.1 223.52 0) (fields_autoplaced)
+  (hierarchical_label "VREG5" (shape output) (at 419.1 223.52 0) (fields_autoplaced)
     (effects (font (size 1.27 1.27)) (justify left))
   )
@@
     (effects (font (size 1.27 1.27)) (justify left))
   )
-  (hierarchical_label "GND" (shape output) (at 419.1 228.6 0) (fields_autoplaced)
+  (hierarchical_label "GND5" (shape output) (at 419.1 228.6 0) (fields_autoplaced)
     (effects (font (size 1.27 1.27)) (justify left))
   )
@@
     )
   )
+  (symbol (lib_id "power:PWR_FLAG") (at 96.52 381 0) (unit 1)
+    (in_bom yes) (on_board yes) (dnp no) (fields_autoplaced)
+    (property "Reference" "#FLG014" (at 96.52 379.095 0)
+      (effects (font (size 1.27 1.27)) hide)
+    )
+    (property "Value" "PWR_FLAG" (at 96.52 375.92 0)
+      (effects (font (size 1.27 1.27)))
+    )
+    (property "Footprint" "" (at 96.52 381 0)
+      (effects (font (size 1.27 1.27)) hide)
+    )
+    (property "Datasheet" "~" (at 96.52 381 0)
+      (effects (font (size 1.27 1.27)) hide)
+    )
+    (pin "1")
+    (instances
+      (project "AMS-board-2024"
+        (path "/3a719eb3-09ce-4343-8f6e-20cc0aaf5261/05d6ad3e-cff9-48e6-bf87-71a8eb2b1b95"
+          (reference "#FLG014") (unit 1)
+        )
+      )
+    )
+  )
   (symbol (lib_id "ProjectEV:GND5") (at 152.4 207.01 0) (unit 1)
     (in_bom yes) (on_board yes) (dnp no) (fields_autoplaced)
@@
     )
   )
+  (symbol (lib_id "ProjectEV:GND5") (at 307.34 223.52 90) (unit 1)
+    (in_bom yes) (on_board yes) (dnp no) (fields_autoplaced)
+    (property "Reference" "#PWR0435" (at 313.69 223.52 0)
+      (effects (font (size 1.27 1.27)) hide)
+    )
+    (property "Value" "GND5" (at 311.15 223.52 90)
+      (effects (font (size 1.27 1.27)) (justify right))
+    )
+    (property "Footprint" "" (at 307.34 223.52 0)
+      (effects (font (size 1.27 1.27)) hide)
+    )
+    (property "Datasheet" "" (at 307.34 223.52 0)
+      (effects (font (size 1.27 1.27)) hide)
+    )
+    (pin "1")
+    (instances
+      (project "AMS-board-2024"
+        (path "/3a719eb3-09ce-4343-8f6e-20cc0aaf5261/05d6ad3e-cff9-48e6-bf87-71a8eb2b1b95"
+          (reference "#PWR0435") (unit 1)
+        )
+      )
+    )
+  )
   (symbol (lib_id "ProjectEV:GND5") (at 320.04 231.14 90) (unit 1)
     (in_bom yes) (on_board yes) (dnp no) (fields_autoplaced)
@@
     )
   )
-  (symbol (lib_id "ProjectEV:GND5") (at 101.6 379.73 0) (unit 1)
+  (symbol (lib_id "ProjectEV:GND5") (at 101.6 383.54 0) (unit 1)
     (in_bom yes) (on_board yes) (dnp no) (fields_autoplaced)
-    (property "Reference" "#PWR0186" (at 101.6 386.08 0)
+    (property "Reference" "#PWR0186" (at 101.6 389.89 0)
       (effects (font (size 1.27 1.27)) hide)
     )
-    (property "Value" "GND5" (at 101.6 384.81 0)
+    (property "Value" "GND5" (at 101.6 388.62 0)
       (effects (font (size 1.27 1.27)))
     )
-    (property "Footprint" "" (at 101.6 379.73 0)
+    (property "Footprint" "" (at 101.6 383.54 0)
       (effects (font (size 1.27 1.27)) hide)
     )
-    (property "Datasheet" "" (at 101.6 379.73 0)
+    (property "Datasheet" "" (at 101.6 383.54 0)
       (effects (font (size 1.27 1.27)) hide)
     )
@@
         )
       )
+    )
+  )
+  (symbol (lib_id "power:PWR_FLAG") (at 292.1 165.1 0) (unit 1)
+    (in_bom yes) (on_board yes) (dnp no) (fields_autoplaced)
+    (property "Reference" "#FLG06" (at 292.1 163.195 0)
+      (effects (font (size 1.27 1.27)) hide)
+    )
+    (property "Value" "PWR_FLAG" (at 292.1 160.02 0)
+      (effects (font (size 1.27 1.27)))
+    )
+    (property "Footprint" "" (at 292.1 165.1 0)
+      (effects (font (size 1.27 1.27)) hide)
+    )
+    (property "Datasheet" "~" (at 292.1 165.1 0)
+      (effects (font (size 1.27 1.27)) hide)
+    )
+    (pin "1")
+    (instances
+      (project "AMS-board-2024"
+        (path "/3a719eb3-09ce-4343-8f6e-20cc0aaf5261/05d6ad3e-cff9-48e6-bf87-71a8eb2b1b95"
+          (reference "#FLG06") (unit 1)
+        )
+      )

Commit message: ラベル修正
Connections:
- net VREG5 renamed VREG
Changed lines of the file:
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@@
     (effects (font (size 1.27 1.27)) (justify left bottom))
   )
-  (label "VREG5" (at 342.9 215.9 0) (fields_autoplaced)
+  (label "S6_VREG" (at 378.46 292.1 0) (fields_autoplaced)
     (effects (font (size 1.27 1.27)) (justify left bottom))
   )
-  (label "VREG5" (at 365.76 317.5 0) (fields_autoplaced)
+  (label "S6_VREG" (at 342.9 215.9 0) (fields_autoplaced)
     (effects (font (size 1.27 1.27)) (justify left bottom))
   )
-  (label "VREG5" (at 378.46 342.9 0) (fields_autoplaced)
+  (label "S6_VREG" (at 378.46 342.9 0) (fields_autoplaced)
     (effects (font (size 1.27 1.27)) (justify left bottom))
   )
-  (label "VREG5" (at 378.46 241.3 0) (fields_autoplaced)
+  (label "S6_VREG" (at 365.76 266.7 0) (fields_autoplaced)
     (effects (font (size 1.27 1.27)) (justify left bottom))
   )
-  (label "VREG5" (at 378.46 292.1 0) (fields_autoplaced)
+  (label "S6_VREG" (at 365.76 317.5 0) (fields_autoplaced)
     (effects (font (size 1.27 1.27)) (justify left bottom))
   )
-  (label "VREG5" (at 365.76 266.7 0) (fields_autoplaced)
+  (label "S6_VREG" (at 378.46 241.3 0) (fields_autoplaced)
     (effects (font (size 1.27 1.27)) (justify left bottom))
   )
@@
     (effects (font (size 1.27 1.27)) (justify right))
   )
-  (hierarchical_label "VREG5" (shape output) (at 419.1 223.52 0) (fields_autoplaced)
+  (hierarchical_label "VREG" (shape output) (at 419.1 223.52 0) (fields_autoplaced)
     (effects (font (size 1.27 1.27)) (justify left))
   )

Commit message: アノテーションし直し
Parts:
- renumbered L21 to L22

Commit message: ラベル修正とテキスト等の追加
階層シート内の電源シンボルをまとめて階層ラベルとして上層に出し、上層のシートで電源シンボルに接続
Connections:
- net GND5: no longer names the net of C157.2, C158.2, C159.2, C160.2, C161.2, C162.2, C163.2, C164.2, C165.2, C166.2, C167.2, C168.2, C181.2, C182.2, C189.1, C190.1, C194.1, C195.1, L22.2, U5.30 (V-), U5.31 (V-)
- net GND5: no longer C183.2, C184.1, C185.2, C186.1, C187.2, C188.2, C191.2, C192.2, C193.2, D107.2 (A), D109.2 (A), D111.2 (A), D113.2 (A), D115.2 (A), R343.1, U5.36 (SWTEN)
- new net: C183.2, C184.1, C185.2, C186.1, C187.2, C188.2, C191.2, C192.2, C193.2, R343.1, U5.36 (SWTEN)
- new net GND: D107.2 (A), D109.2 (A), D111.2 (A), D113.2 (A), D115.2 (A)

Commit message: LTC6811のシンボルを更新
Parts:
- U5: footprint ProjectEV:SSOP-48_5.3x12.8mm_P0.5mm_LTC6811 -> ProjectEV:Package_SSOP-48_5.3x12.8mm_P0.5mm_LTC6811
Changed lines of the file:
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@@
       (effects (font (size 1.27 1.27)) (justify left))
     )
-    (property "Footprint" "ProjectEV:SSOP-48_5.3x12.8mm_P0.5mm_LTC6811" (at 290.83 213.36 0)
+    (property "Footprint" "ProjectEV:Package_SSOP-48_5.3x12.8mm_P0.5mm_LTC6811" (at 290.83 213.36 0)
       (effects (font (size 1.27 1.27)) hide)
     )

Commit message: チップ抵抗、チップコンデンササイズ修正
Parts:
- C169, C170, C171, C172, C173, C174, C175, C176, C177, C178, C179, C180, C181, C183, C184, C185, C186, C187, C188, C189, C190, C191, C192, C194, C195: footprint Capacitor_SMD:C_0603_1608Metric -> Capacitor_SMD:C_0402_1005Metric
- R315, R316, R317, R318, R319, R320, R321, R322, R323, R324, R325, R326, R327, R328, R329, R330, R331, R332, R333, R334, R335, R336, R337, R338, R339, R340, R341, R343, R348, R353, R354, R355, R356, R357, R358, R359, R360, R361, R362: footprint Resistor_SMD:R_0603_1608Metric -> Resistor_SMD:R_0402_1005Metric

Commit message: 温度センサ用コネクタ変更、大まかな位置決定
Parts:
- removed C183, C185: 0.1u, Capacitor_SMD:C_0402_1005Metric, symbol Device:C
- removed D108, D109, D114, D115: BAT46W-7-F, ProjectEV:D_SOD-123_BAT46W-7-F, symbol ProjectEV:D_BAT46W-7-F
- removed R356, R357: 100, Resistor_SMD:R_0402_1005Metric, symbol Device:R
- removed R361, R362: 10k, Resistor_SMD:R_0402_1005Metric, symbol Device:R
Connections:
- net GND: now also C157.2, C158.2, C159.2, C160.2, C161.2, C162.2, C163.2, C164.2, C165.2, C166.2, C167.2, C168.2, C181.2, C182.2, C184.1, C186.1, C187.2, C188.2, C189.1, C190.1, C191.2, C192.2, C193.2, C194.1, C195.1, L22.2, R343.1, U5.30 (V-), U5.31 (V-), U5.36 (SWTEN)
- net VREF_3V: no longer names the net of C184.2, R358.1, R359.1, R360.1, U5.34 (VREF2)
- net VREG: no longer names the net of C187.1, D106.1 (K), D110.1 (K), D112.1 (K), Q65.3 (E), R342.1, U5.37 (VREG), U5.40 (ISOMD)
- no-connect marks 2 -> 4

Commit message: アノテーションし直し、
Parts:
- R324: renamed from R340; footprint Resistor_SMD:R_0402_1005Metric -> Resistor_SMD:R_0603_1608Metric
- R332: renamed from R348; footprint Resistor_SMD:R_0402_1005Metric -> Resistor_SMD:R_0603_1608Metric
- renumbered C157 to C149, C158 to C150, C159 to C151, C160 to C152, C161 to C153, C162 to C154, C163 to C155, C164 to C156, C165 to C157, C166 to C158, C167 to C159, C168 to C160, C169 to C161, C170 to C162, C171 to C163, C172 to C164, C173 to C165, C174 to C166, C175 to C167, C176 to C168, C177 to C169, C178 to C170, C179 to C171, C180 to C172, C181 to C173, C182 to C174, C184 to C175, C186 to C176, C187 to C177, C188 to C178, C189 to C179, C190 to C180, C191 to C181, C192 to C182, C193 to C183, C194 to C184, C195 to C185, D93 to D77, D94 to D78, D95 to D79, D96 to D80, D97 to D81, D98 to D82, D99 to D83, D100 to D84, D101 to D85, D102 to D86, D103 to D87, D104 to D88, D105 to D89, D106 to D90, D107 to D91, D110 to D92, D111 to D93, D112 to D94, D113 to D95, R291 to R275, R292 to R276, R293 to R277, R294 to R278, R295 to R279, R296 to R280, R297 to R281, R298 to R282, R299 to R283, R300 to R284, R301 to R285, R302 to R286, R303 to R287, R304 to R288, R305 to R289, R306 to R290, R307 to R291, R308 to R292, R309 to R293, R310 to R294, R311 to R295, R312 to R296, R313 to R297, R314 to R298, R315 to R299, R316 to R300, R317 to R301, R318 to R302, R319 to R303, R320 to R304, R321 to R305, R322 to R306, R323 to R307, R324 to R308, R325 to R309, R326 to R310, R327 to R311, R328 to R312, R329 to R313, R330 to R314, R331 to R315, R332 to R316, R333 to R317, R334 to R318, R335 to R319, R336 to R320, R337 to R321, R338 to R322, R339 to R323, R341 to R325, R342 to R326, R343 to R327, R344 to R328, R345 to R329, R346 to R330, R347 to R331, R349 to R333, R350 to R334, R351 to R335, R352 to R336, R353 to R337, R354 to R338, R355 to R339, R358 to R340, R359 to R341, R360 to R342
