File: AMS-board-2024/battery-module-monitor-6.kicad_sch (KiCad schematic)
At the start: 144 parts, among them Q701 BSS308PE, Q702 BSS308PE, Q703 BSS308PE, Q704 BSS308PE, Q705 BSS308PE, Q706 BSS308PE, Q707 BSS308PE, Q708 BSS308PE, Q709 BSS308PE, Q710 BSS308PE, Q711 BSS308PE, Q712 BSS308PE, Q713 NSV1C201MZ4, U701 LTC6811-1

Commit message: 修正
アノテーション方法の変更：最初の空き番号から使用
Parts:
- renumbered C701 to C171, C702 to C172, C703 to C173, C704 to C174, C705 to C175, C706 to C176, C707 to C177, C708 to C178, C709 to C179, C710 to C180, C711 to C181, C712 to C182, C713 to C183, C714 to C184, C715 to C185, C716 to C186, C717 to C187, C718 to C188, C719 to C189, C720 to C190, C721 to C191, C722 to C192, C723 to C193, C724 to C194, C725 to C195, C726 to C196, C727 to C197, C728 to C198, C729 to C199, C730 to C200, C731 to C201, C732 to C202, C733 to C203, C734 to C204, D701 to D66, D702 to D67, D703 to D68, D704 to D69, D705 to D70, D706 to D71, D707 to D72, D708 to D73, D709 to D74, D710 to D75, D711 to D76, D712 to D77, D713 to D78, F701 to F66, F702 to F67, F703 to F68, F704 to F69, F705 to F70, F706 to F71, F707 to F72, F708 to F73, F709 to F74, F710 to F75, F711 to F76, F712 to F77, F713 to F78, FL701 to FL11, FL702 to FL12, L701 to L6, Q701 to Q66, Q702 to Q67, Q703 to Q68, Q704 to Q69, Q705 to Q70, Q706 to Q71, Q707 to Q72, Q708 to Q73, Q709 to Q74, Q710 to Q75, Q711 to Q76, Q712 to Q77, Q713 to Q78, R701 to R336, R702 to R337, R703 to R338, R704 to R339, R705 to R340, R706 to R341, R707 to R342, R708 to R343, R709 to R344, R710 to R345, R711 to R346, R712 to R347, R713 to R348, R714 to R349, R715 to R350, R716 to R351, R717 to R352, R718 to R353, R719 to R354, R720 to R355, R721 to R356, R722 to R357, R723 to R358, R724 to R359, R725 to R360, R726 to R361, R727 to R362, R728 to R363, R729 to R364, R730 to R365, R731 to R366, R732 to R367, R733 to R368, R734 to R369, R735 to R370, R736 to R371, R737 to R372, R738 to R373, R739 to R374, R740 to R375, R741 to R376, R742 to R377, R743 to R378, R744 to R379, R745 to R380, R746 to R381, R747 to R382, R748 to R383, R749 to R384, R750 to R385, R751 to R386, R752 to R387, R753 to R388, R754 to R389, R755 to R390, R756 to R391, R757 to R392, R758 to R393, R759 to R394, R760 to R395, R761 to R396, R762 to R397, R763 to R398, R764 to R399, R765 to R400, R766 to R401, R767 to R402, U701 to U6

Commit message: GNDシンボル追加
Connections:
- net GND1: now reaches C171.2
- net GND1: now also C172.2, C173.2, C174.2, C175.2, C176.2, C177.2, C178.2, C179.2, C180.2, C181.2, C182.2, C195.2, C196.2, C197.1, C198.1, C199.2, C200.1, C201.1, C202.2, C203.1, C204.1, L6.2, R390.1, U6.30 (V-), U6.31 (V-)

Commit message: GPIO周辺回路の修正
Parts:
- added C316, C317, C318, C319, C320: 0.1u, Capacitor_SMD:C_0603_1608Metric, symbol Device:C
- added R583, R584, R585, R586, R587: 10k, Resistor_SMD:R_0603_1608Metric, symbol Device:R
- R386, R389, R391, R392, R397: value 10k -> 100
Connections:
- net GND1: now also C316.2, C317.2, C318.2, C319.2, C320.2
- net Thermistor1+: now also R386.2, R583.2; no longer R397.1, U6.27 (GPIO1)
- net Thermistor2+: now also R389.2, R584.2; no longer R392.1, U6.28 (GPIO2)
- net Thermistor3+: now also R391.2, R585.2; no longer R391.1, U6.29 (GPIO3)
- net Thermistor4+: now also R392.2, R586.2; no longer R389.1, U6.32 (GPIO4)
- net Thermistor5+: now also R397.2, R587.2; no longer R386.1, U6.33 (GPIO5)
- net VREG: now reaches C199.1, Q78.3 (E), R388.1, U6.37 (VREG), U6.40 (ISOMD)
- new net: C316.1, R397.1, U6.33 (GPIO5)
- new net: C317.1, R392.1, U6.32 (GPIO4)
- new net: C318.1, R391.1, U6.29 (GPIO3)
- new net: C319.1, R389.1, U6.28 (GPIO2)
- new net: C320.1, R386.1, U6.27 (GPIO1)
- new net VREF_3V: C197.2, R583.1, R584.1, R585.1, R586.1, R587.1, U6.34 (VREF2)

Commit message: テキスト修正
Other:
- note added: "レギュレーション上必要なサーミスタは 96 CELL x 25 % = 24 本. GPIO1~3 をサーミスタに使用し、 GPIO4, 5 は別用途で使用してもOK. GPIO4, 5 のプルアップは必要に応じて実装."
- note removed: "レギュレーション上必要なサーミスタは 3 x 8 = 24 本. GPIO1~3 をサーミスタに使用し、 GPIO4, 5 は別用途で使用してもOK. GPIO4, 5 のプルアップは必要に応じて実装."
Changed lines of the file:
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@@
-    (effects (font (size 1.27 1.27)) (justify left bottom))
-  )
-  (text "レギュレーション上必要なサーミスタは 3 x 8 = 24 本.\nGPIO1~3 をサーミスタに使用し、\nGPIO4, 5 は別用途で使用してもOK.\nGPIO4, 5 のプルアップは必要に応じて実装."
-    (at 469.9 283.21 0)
     (effects (font (size 1.27 1.27)) (justify left bottom))
   )
@@
     (effects (font (size 1.27 1.27)) (justify left bottom))
   )
+  (text "レギュレーション上必要なサーミスタは 96 CELL x 25 % = 24 本.\nGPIO1~3 をサーミスタに使用し、\nGPIO4, 5 は別用途で使用してもOK.\nGPIO4, 5 のプルアップは必要に応じて実装."
+    (at 469.9 283.21 0)
+    (effects (font (size 1.27 1.27)) (justify left bottom))
+  )

Commit message: ヒューズ変更
Parts:
- removed F66, F67, F68, F69, F70, F71, F72, F73, F74, F75, F76, F77, F78: C1F 500, Fuse:Fuse_1206_3216Metric, symbol Device:Fuse
- added F40, F41, F42, F43, F44, F45, F46, F47, F48, F49, F50, F51, F52: 0679L1000-05, ProjectEV:Fuse_0679L, symbol ProjectEV:Fuse_0679L1000-05
Connections:
- net CELL0: now also F52.1
- net CELL1: now also F51.1
- net CELL10: now also F42.1
- net CELL11: now also F41.1
- net CELL12: now also F40.1
- net CELL2: now also F50.1
- net CELL3: now also F49.1
- net CELL4: now also F48.1
- net CELL5: now also F47.1
- net CELL6: now also F46.1
- net CELL7: now also F45.1
- net CELL8: now also F44.1
- net CELL9: now also F43.1
- net at D66.2 (A), L6.1, R347.2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: now also F52.2
- net at Q71.2 (S), R340.2, R352.2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: now also F45.2
- net at D66.1 (K), Q77.2 (S), R346.2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: now also F51.2
- net at Q69.2 (S), R338.2, R350.2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: now also F43.2
- net at Q75.2 (S), R344.2, R356.2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: now also F49.2
- net at Q72.2 (S), R341.2, R353.2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: now also F46.2
- net at Q67.2 (S), R336.2, R348.2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: now also F41.2
- net at Q66.2 (S), R372.1, R385.1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: now also F40.2
- net at Q73.2 (S), R342.2, R354.2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: now also F47.2
- net at Q70.2 (S), R339.2, R351.2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: now also F44.2
- net at Q74.2 (S), R343.2, R355.2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: now also F48.2
- net at Q76.2 (S), R345.2, R357.2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: now also F50.2
- net at Q68.2 (S), R337.2, R349.2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: now also F42.2

Commit message: アノテーションし直し
Parts:
- renumbered C171 to C196, C172 to C197, C173 to C198, C174 to C199, C175 to C200, C176 to C201, C177 to C202, C178 to C203, C179 to C204, C180 to C205, C181 to C206, C182 to C207, C183 to C208, C184 to C209, C185 to C210, C186 to C211, C187 to C212, C188 to C213, C189 to C214, C190 to C215, C191 to C216, C192 to C217, C193 to C218, C194 to C219, C195 to C220, C196 to C221, C316 to C222, C197 to C223, C317 to C224, C198 to C225, C199 to C226, C318 to C227, C200 to C228, C201 to C229, C319 to C230, C320 to C231, C202 to C232, C203 to C233, C204 to C234, F40 to F66, F41 to F67, F42 to F68, F43 to F69, F44 to F70, F45 to F71, F46 to F72, F47 to F73, F48 to F74, F49 to F75, F50 to F76, F51 to F77, F52 to F78, R336 to R361, R337 to R362, R338 to R363, R339 to R364, R340 to R365, R341 to R366, R342 to R367, R343 to R368, R344 to R369, R345 to R370, R346 to R371, R347 to R372, R348 to R373, R349 to R374, R350 to R375, R351 to R376, R352 to R377, R353 to R378, R354 to R379, R355 to R380, R356 to R381, R357 to R382, R358 to R383, R359 to R384, R360 to R385, R361 to R386, R362 to R387, R363 to R388, R364 to R389, R365 to R390, R366 to R391, R367 to R392, R368 to R393, R369 to R394, R370 to R395, R371 to R396, R372 to R397, R373 to R398, R374 to R399, R375 to R400, R376 to R401, R377 to R402, R378 to R403, R379 to R404, R380 to R405, R381 to R406, R382 to R407, R383 to R408, R384 to R409, R385 to R410, R387 to R411, R388 to R412, R390 to R413, R393 to R414, R394 to R415, R395 to R416, R396 to R417, R398 to R418, R386 to R419, R389 to R420, R391 to R421, R392 to R422, R397 to R423, R583 to R424, R399 to R425, R400 to R426, R401 to R427, R402 to R428, R584 to R429, R585 to R430, R586 to R431, R587 to R432

Commit message: GPIO入力保護回路追加
Parts:
- added D180, D181, D182, D183, D184, D185, D186, D187, D188, D189: BAT46W-7-F, ProjectEV:D_SOD-123_BAT46W-7-F, symbol ProjectEV:D_BAT46W-7-F
Connections:
- net GND1: now also D181.2 (A), D183.2 (A), D185.2 (A), D187.2 (A), D189.2 (A)
- net VREG: now also D180.1 (K), D182.1 (K), D184.1 (K), D186.1 (K), D188.1 (K)
- net at C222.1, R423.1, U6.33 (GPIO5): now also D188.2 (A), D189.1 (K)
- net at C224.1, R422.1, U6.32 (GPIO4): now also D186.2 (A), D187.1 (K)
- net at C227.1, R421.1, U6.29 (GPIO3): now also D184.2 (A), D185.1 (K)
- net at C230.1, R420.1, U6.28 (GPIO2): now also D182.2 (A), D183.1 (K)
- net at C231.1, R419.1, U6.27 (GPIO1): now also D180.2 (A), D181.1 (K)
Other:
- moved on the sheet: R419, R420, R421, R422, R423, R424, R429, R430, R431, R432

Commit message: アノテーションし直し
Parts:
- renumbered D66 to D116, D67 to D117, D68 to D118, D69 to D119, D70 to D120, D71 to D121, D72 to D122, D73 to D123, D74 to D124, D75 to D125, D76 to D126, D77 to D127, D78 to D128, D182 to D129, D183 to D130, D186 to D131, D187 to D132, D180 to D133, D181 to D134, D184 to D135, D185 to D136, D188 to D137, D189 to D138, L6 to L22, R361 to R363, R362 to R364, R363 to R365, R364 to R366, R365 to R367, R366 to R368, R367 to R369, R368 to R370, R369 to R371, R370 to R372, R371 to R373, R372 to R374, R373 to R375, R374 to R376, R375 to R377, R376 to R378, R377 to R379, R378 to R380, R379 to R381, R380 to R382, R381 to R383, R382 to R384, R383 to R385, R384 to R386, R385 to R387, R386 to R388, R387 to R389, R388 to R390, R389 to R391, R390 to R392, R391 to R393, R392 to R394, R393 to R395, R394 to R396, R395 to R397, R396 to R398, R397 to R399, R398 to R400, R399 to R401, R400 to R402, R401 to R403, R402 to R404, R403 to R405, R404 to R406, R405 to R407, R406 to R408, R407 to R409, R408 to R410, R409 to R411, R410 to R412, R411 to R413, R412 to R414, R413 to R415, R414 to R416, R415 to R417, R416 to R418, R417 to R419, R418 to R420, R425 to R421, R426 to R422, R427 to R423, R428 to R424, R419 to R425, R420 to R426, R421 to R427, R422 to R428, R423 to R429, R424 to R430, R429 to R431, R430 to R432, R431 to R433, R432 to R434
