File: AMS-board-2024/battery-module-monitor-6.kicad_sch (KiCad schematic)
At the start: 154 parts, among them Q66 BSS308PE, Q67 BSS308PE, Q68 BSS308PE, Q69 BSS308PE, Q70 BSS308PE, Q71 BSS308PE, Q72 BSS308PE, Q73 BSS308PE, Q74 BSS308PE, Q75 BSS308PE, Q76 BSS308PE, Q77 BSS308PE, Q78 NSV1C201MZ4, U6 LTC6811-1

Commit message: アノテーションし直し、
Parts:
- R392: renamed from R412; footprint Resistor_SMD:R_0402_1005Metric -> Resistor_SMD:R_0603_1608Metric
- R400: renamed from R420; footprint Resistor_SMD:R_0402_1005Metric -> Resistor_SMD:R_0603_1608Metric
- renumbered C196 to C186, C197 to C187, C198 to C188, C199 to C189, C200 to C190, C201 to C191, C202 to C192, C203 to C193, C204 to C194, C205 to C195, C206 to C196, C207 to C197, C208 to C198, C209 to C199, C210 to C200, C211 to C201, C212 to C202, C213 to C203, C214 to C204, C215 to C205, C216 to C206, C217 to C207, C218 to C208, C219 to C209, C220 to C210, C221 to C211, C223 to C212, C225 to C213, C226 to C214, C227 to C215, C228 to C216, C229 to C217, C230 to C218, C231 to C219, C232 to C220, C233 to C221, C234 to C222, D120 to D100, D121 to D101, D122 to D102, D123 to D103, D124 to D104, D125 to D105, D126 to D106, D127 to D107, D128 to D108, D129 to D109, D130 to D110, D133 to D111, D134 to D112, D135 to D113, D136 to D114, D116 to D96, D117 to D97, D118 to D98, D119 to D99, R363 to R343, R364 to R344, R365 to R345, R366 to R346, R367 to R347, R368 to R348, R369 to R349, R370 to R350, R371 to R351, R372 to R352, R373 to R353, R374 to R354, R375 to R355, R376 to R356, R377 to R357, R378 to R358, R379 to R359, R380 to R360, R381 to R361, R382 to R362, R383 to R363, R384 to R364, R385 to R365, R386 to R366, R387 to R367, R388 to R368, R389 to R369, R390 to R370, R391 to R371, R392 to R372, R393 to R373, R394 to R374, R395 to R375, R396 to R376, R397 to R377, R398 to R378, R399 to R379, R400 to R380, R401 to R381, R402 to R382, R403 to R383, R404 to R384, R405 to R385, R406 to R386, R407 to R387, R408 to R388, R409 to R389, R410 to R390, R411 to R391, R413 to R393, R414 to R394, R415 to R395, R416 to R396, R417 to R397, R418 to R398, R419 to R399, R421 to R401, R422 to R402, R423 to R403, R424 to R404, R425 to R405, R426 to R406, R427 to R407, R430 to R408, R431 to R409, R432 to R410
