File: AMS-board-2024/battery-module-monitor-6.kicad_sch (KiCad schematic)
At the start: 154 parts, among them Q66 BSS308PE, Q67 BSS308PE, Q68 BSS308PE, Q69 BSS308PE, Q70 BSS308PE, Q71 BSS308PE, Q72 BSS308PE, Q73 BSS308PE, Q74 BSS308PE, Q75 BSS308PE, Q76 BSS308PE, Q77 BSS308PE, Q78 NSV1C201MZ4, U6 LTC6811-1

Commit message: 絶縁パルストランス数削減
Parts:
- renumbered L23 to L16
Changed lines of the file:
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@@
   (symbol (lib_id "ProjectEV:L_MH3261") (at 101.6 374.65 0) (unit 1)
     (in_bom yes) (on_board yes) (dnp no) (fields_autoplaced)
-    (property "Reference" "L23" (at 102.87 373.38 0)
+    (property "Reference" "L16" (at 102.87 373.38 0)
       (effects (font (size 1.27 1.27)) (justify left))
     )
@@
       (project "AMS-board-2024"
         (path "/3a719eb3-09ce-4343-8f6e-20cc0aaf5261/1ec1bfe3-7fe8-447f-81d8-7e7cb948fc43"
-          (reference "L23") (unit 1)
+          (reference "L16") (unit 1)
         )
       )

Commit message: 抵抗修正
3.3k -> 3k (1608)
15k -> 100k (1005, プルアップ/ダウン), 5.1k (1005, LED用)
Parts:
- R367, R368, R369, R370, R371, R372, R373, R374, R375, R376, R377, R378: value 3.3k -> 3k; footprint Resistor_SMD:R_0402_1005Metric -> Resistor_SMD:R_0603_1608Metric
Changed lines of the file:
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@@
       (effects (font (size 1.27 1.27)))
     )
-    (property "Value" "3.3k" (at 139.7 80.01 90)
-      (effects (font (size 1.27 1.27)))
-    )
-    (property "Footprint" "Resistor_SMD:R_0402_1005Metric" (at 139.7 84.328 90)
+    (property "Value" "3k" (at 139.7 80.01 90)
+      (effects (font (size 1.27 1.27)))
+    )
+    (property "Footprint" "Resistor_SMD:R_0603_1608Metric" (at 139.7 84.328 90)
       (effects (font (size 1.27 1.27)) hide)
     )
@@
       (effects (font (size 1.27 1.27)))
     )
-    (property "Value" "3.3k" (at 139.7 345.44 90)
-      (effects (font (size 1.27 1.27)))
-    )
-    (property "Footprint" "Resistor_SMD:R_0402_1005Metric" (at 139.7 349.758 90)
+    (property "Value" "3k" (at 139.7 345.44 90)
+      (effects (font (size 1.27 1.27)))
+    )
+    (property "Footprint" "Resistor_SMD:R_0603_1608Metric" (at 139.7 349.758 90)
       (effects (font (size 1.27 1.27)) hide)
     )
@@
       (effects (font (size 1.27 1.27)))
     )
-    (property "Value" "3.3k" (at 139.7 176.53 90)
-      (effects (font (size 1.27 1.27)))
-    )
-    (property "Footprint" "Resistor_SMD:R_0402_1005Metric" (at 139.7 180.848 90)
+    (property "Value" "3k" (at 139.7 176.53 90)
+      (effects (font (size 1.27 1.27)))
+    )
+    (property "Footprint" "Resistor_SMD:R_0603_1608Metric" (at 139.7 180.848 90)
       (effects (font (size 1.27 1.27)) hide)
     )
@@
       (effects (font (size 1.27 1.27)))
     )
-    (property "Value" "3.3k" (at 139.7 297.18 90)
-      (effects (font (size 1.27 1.27)))
-    )
-    (property "Footprint" "Resistor_SMD:R_0402_1005Metric" (at 139.7 301.498 90)
+    (property "Value" "3k" (at 139.7 297.18 90)
+      (effects (font (size 1.27 1.27)))
+    )
+    (property "Footprint" "Resistor_SMD:R_0603_1608Metric" (at 139.7 301.498 90)
       (effects (font (size 1.27 1.27)) hide)
     )
@@
       (effects (font (size 1.27 1.27)))
     )
-    (property "Value" "3.3k" (at 139.7 224.79 90)
-      (effects (font (size 1.27 1.27)))
-    )
-    (property "Footprint" "Resistor_SMD:R_0402_1005Metric" (at 139.7 229.108 90)
+    (property "Value" "3k" (at 139.7 224.79 90)
+      (effects (font (size 1.27 1.27)))
+    )
+    (property "Footprint" "Resistor_SMD:R_0603_1608Metric" (at 139.7 229.108 90)
       (effects (font (size 1.27 1.27)) hide)
     )
@@
       (effects (font (size 1.27 1.27)))
     )
-    (property "Value" "3.3k" (at 139.7 200.66 90)
-      (effects (font (size 1.27 1.27)))
-    )
-    (property "Footprint" "Resistor_SMD:R_0402_1005Metric" (at 139.7 204.978 90)
+    (property "Value" "3k" (at 139.7 200.66 90)
+      (effects (font (size 1.27 1.27)))
+    )
+    (property "Footprint" "Resistor_SMD:R_0603_1608Metric" (at 139.7 204.978 90)
       (effects (font (size 1.27 1.27)) hide)
     )
@@
       (effects (font (size 1.27 1.27)))
     )
-    (property "Value" "3.3k" (at 139.7 321.31 90)
-      (effects (font (size 1.27 1.27)))
-    )
-    (property "Footprint" "Resistor_SMD:R_0402_1005Metric" (at 139.7 325.628 90)
+    (property "Value" "3k" (at 139.7 321.31 90)
+      (effects (font (size 1.27 1.27)))
+    )
+    (property "Footprint" "Resistor_SMD:R_0603_1608Metric" (at 139.7 325.628 90)
       (effects (font (size 1.27 1.27)) hide)
     )
@@
       (effects (font (size 1.27 1.27)))
     )
-    (property "Value" "3.3k" (at 139.7 104.14 90)
-      (effects (font (size 1.27 1.27)))
-    )
-    (property "Footprint" "Resistor_SMD:R_0402_1005Metric" (at 139.7 108.458 90)
+    (property "Value" "3k" (at 139.7 104.14 90)
+      (effects (font (size 1.27 1.27)))
+    )
+    (property "Footprint" "Resistor_SMD:R_0603_1608Metric" (at 139.7 108.458 90)
       (effects (font (size 1.27 1.27)) hide)
     )
@@
       (effects (font (size 1.27 1.27)))
     )
-    (property "Value" "3.3k" (at 139.7 152.4 90)
-      (effects (font (size 1.27 1.27)))
-    )
-    (property "Footprint" "Resistor_SMD:R_0402_1005Metric" (at 139.7 156.718 90)
+    (property "Value" "3k" (at 139.7 152.4 90)
+      (effects (font (size 1.27 1.27)))
+    )
+    (property "Footprint" "Resistor_SMD:R_0603_1608Metric" (at 139.7 156.718 90)
       (effects (font (size 1.27 1.27)) hide)
     )
@@
       (effects (font (size 1.27 1.27)))
     )
-    (property "Value" "3.3k" (at 139.7 128.27 90)
-      (effects (font (size 1.27 1.27)))
-    )
-    (property "Footprint" "Resistor_SMD:R_0402_1005Metric" (at 139.7 132.588 90)
+    (property "Value" "3k" (at 139.7 128.27 90)
+      (effects (font (size 1.27 1.27)))
+    )
+    (property "Footprint" "Resistor_SMD:R_0603_1608Metric" (at 139.7 132.588 90)
       (effects (font (size 1.27 1.27)) hide)
     )
@@
       (effects (font (size 1.27 1.27)))
     )
-    (property "Value" "3.3k" (at 139.7 248.92 90)
-      (effects (font (size 1.27 1.27)))
-    )
-    (property "Footprint" "Resistor_SMD:R_0402_1005Metric" (at 139.7 253.238 90)
+    (property "Value" "3k" (at 139.7 248.92 90)
+      (effects (font (size 1.27 1.27)))
+    )
+    (property "Footprint" "Resistor_SMD:R_0603_1608Metric" (at 139.7 253.238 90)
       (effects (font (size 1.27 1.27)) hide)
     )
@@
       (effects (font (size 1.27 1.27)))
     )
-    (property "Value" "3.3k" (at 139.7 273.05 90)
-      (effects (font (size 1.27 1.27)))
-    )
-    (property "Footprint" "Resistor_SMD:R_0402_1005Metric" (at 139.7 277.368 90)
-      (effects (font (size 1.27 1.27)) hide)
-    )
+    (property "Value" "3k" (at 139.7 273.05 90)
+      (effects (font (size 1.27 1.27)))
+    )
+    (property "Footprint" "Resistor_SMD:R_0603_1608Metric" (at 139.7 277.368 90)
+      (effects (font (size 1.27 1.27)) hide)
+    )

Commit message: アノテーションし直し
Parts:
- renumbered C186 to C195, C187 to C196, C188 to C197, C189 to C198, C190 to C199, C191 to C200, C192 to C201, C193 to C202, C194 to C203, C195 to C204, C196 to C205, C197 to C206, C198 to C207, C199 to C208, C200 to C209, C201 to C210, C202 to C211, C203 to C212, C204 to C213, C205 to C214, C206 to C215, C207 to C216, C208 to C217, C209 to C218, C210 to C219, C211 to C220, C212 to C221, C213 to C222, C214 to C223, C215 to C224, C216 to C225, C217 to C226, C218 to C227, C219 to C228, C220 to C229, C221 to C230, C222 to C231, L16 to L12
