File: AMS-board-2024/battery-module-monitor-7.kicad_sch (KiCad schematic)
At the start: 144 parts, among them Q801 BSS308PE, Q802 BSS308PE, Q803 BSS308PE, Q804 BSS308PE, Q805 BSS308PE, Q806 BSS308PE, Q807 BSS308PE, Q808 BSS308PE, Q809 BSS308PE, Q810 BSS308PE, Q811 BSS308PE, Q812 BSS308PE, Q813 NSV1C201MZ4, U801 LTC6811-1

Commit message: 修正
アノテーション方法の変更：最初の空き番号から使用
Parts:
- renumbered C801 to C205, C802 to C206, C803 to C207, C804 to C208, C805 to C209, C806 to C210, C807 to C211, C808 to C212, C809 to C213, C810 to C214, C811 to C215, C812 to C216, C813 to C217, C814 to C218, C815 to C219, C816 to C220, C817 to C221, C818 to C222, C819 to C223, C820 to C224, C821 to C225, C822 to C226, C823 to C227, C824 to C228, C825 to C229, C826 to C230, C827 to C231, C828 to C232, C829 to C233, C830 to C234, C831 to C235, C832 to C236, C833 to C237, C834 to C238, D801 to D79, D802 to D80, D803 to D81, D804 to D82, D805 to D83, D806 to D84, D807 to D85, D808 to D86, D809 to D87, D810 to D88, D811 to D89, D812 to D90, D813 to D91, F801 to F79, F802 to F80, F803 to F81, F804 to F82, F805 to F83, F806 to F84, F807 to F85, F808 to F86, F809 to F87, F810 to F88, F811 to F89, F812 to F90, F813 to F91, FL801 to FL13, FL802 to FL14, L801 to L7, Q801 to Q79, Q802 to Q80, Q803 to Q81, Q804 to Q82, Q805 to Q83, Q806 to Q84, Q807 to Q85, Q808 to Q86, Q809 to Q87, Q810 to Q88, Q811 to Q89, Q812 to Q90, Q813 to Q91, R801 to R403, R802 to R404, R803 to R405, R804 to R406, R805 to R407, R806 to R408, R807 to R409, R808 to R410, R809 to R411, R810 to R412, R811 to R413, R812 to R414, R813 to R415, R814 to R416, R815 to R417, R816 to R418, R817 to R419, R818 to R420, R819 to R421, R820 to R422, R821 to R423, R822 to R424, R823 to R425, R824 to R426, R825 to R427, R826 to R428, R827 to R429, R828 to R430, R829 to R431, R830 to R432, R831 to R433, R832 to R434, R833 to R435, R834 to R436, R835 to R437, R836 to R438, R837 to R439, R838 to R440, R839 to R441, R840 to R442, R841 to R443, R842 to R444, R843 to R445, R844 to R446, R845 to R447, R846 to R448, R847 to R449, R848 to R450, R849 to R451, R850 to R452, R851 to R453, R852 to R454, R853 to R455, R854 to R456, R855 to R457, R856 to R458, R857 to R459, R858 to R460, R859 to R461, R860 to R462, R861 to R463, R862 to R464, R863 to R465, R864 to R466, R865 to R467, R866 to R468, R867 to R469, U801 to U7

Commit message: GNDシンボル追加
Connections:
- net GND1: now reaches L7.2
- net GND1: now also C205.2, C206.2, C207.2, C208.2, C209.2, C210.2, C211.2, C212.2, C213.2, C214.2, C215.2, C216.2, C229.2, C230.2, C231.1, C232.1, C233.2, C234.1, C235.1, C236.2, C237.1, C238.1, R457.1, U7.30 (V-), U7.31 (V-)

Commit message: GPIO周辺回路の修正
Parts:
- added C321, C322, C323, C324, C325: 0.1u, Capacitor_SMD:C_0603_1608Metric, symbol Device:C
- added R588, R589, R590, R591, R592: 10k, Resistor_SMD:R_0603_1608Metric, symbol Device:R
- R453, R456, R458, R459, R464: value 10k -> 100
Connections:
- net GND1: now also C321.2, C322.2, C323.2, C324.2, C325.2
- net Thermistor1+: now also R453.2, R588.2; no longer R464.1, U7.27 (GPIO1)
- net Thermistor2+: now also R456.2, R589.2; no longer R459.1, U7.28 (GPIO2)
- net Thermistor3+: now also R458.2, R590.2; no longer R458.1, U7.29 (GPIO3)
- net Thermistor4+: now also R459.2, R591.2; no longer R456.1, U7.32 (GPIO4)
- net Thermistor5+: now also R464.2, R592.2; no longer R453.1, U7.33 (GPIO5)
- net VREG: now reaches C233.1, Q91.3 (E), R455.1, U7.37 (VREG), U7.40 (ISOMD)
- new net: C325.1, R453.1, U7.27 (GPIO1)
- new net: C324.1, R456.1, U7.28 (GPIO2)
- new net: C322.1, R459.1, U7.32 (GPIO4)
- new net: C321.1, R464.1, U7.33 (GPIO5)
- new net: C323.1, R458.1, U7.29 (GPIO3)
- new net VREF_3V: C231.2, R588.1, R589.1, R590.1, R591.1, R592.1, U7.34 (VREF2)

Commit message: テキスト修正
Other:
- note added: "レギュレーション上必要なサーミスタは 96 CELL x 25 % = 24 本. GPIO1~3 をサーミスタに使用し、 GPIO4, 5 は別用途で使用してもOK. GPIO4, 5 のプルアップは必要に応じて実装."
- note removed: "レギュレーション上必要なサーミスタは 3 x 8 = 24 本. GPIO1~3 をサーミスタに使用し、 GPIO4, 5 は別用途で使用してもOK. GPIO4, 5 のプルアップは必要に応じて実装."
Changed lines of the file:
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@@
     (effects (font (size 1.27 1.27)) (justify left bottom))
   )
-  (text "レギュレーション上必要なサーミスタは 3 x 8 = 24 本.\nGPIO1~3 をサーミスタに使用し、\nGPIO4, 5 は別用途で使用してもOK.\nGPIO4, 5 のプルアップは必要に応じて実装."
+  (text "レギュレーション上必要なサーミスタは 96 CELL x 25 % = 24 本.\nGPIO1~3 をサーミスタに使用し、\nGPIO4, 5 は別用途で使用してもOK.\nGPIO4, 5 のプルアップは必要に応じて実装."
     (at 469.9 283.21 0)
     (effects (font (size 1.27 1.27)) (justify left bottom))

Commit message: ヒューズ変更
Parts:
- removed F79, F80, F81, F82, F83, F84, F85, F86, F87, F88, F89, F90, F91: C1F 500, Fuse:Fuse_1206_3216Metric, symbol Device:Fuse
- added F53, F54, F55, F56, F57, F58, F59, F60, F61, F62, F63, F64, F65: 0679L1000-05, ProjectEV:Fuse_0679L, symbol ProjectEV:Fuse_0679L1000-05
Connections:
- net CELL0: now also F65.1
- net CELL1: now also F64.1
- net CELL10: now also F55.1
- net CELL11: now also F54.1
- net CELL12: now also F53.1
- net CELL2: now also F63.1
- net CELL3: now also F62.1
- net CELL4: now also F61.1
- net CELL5: now also F60.1
- net CELL6: now also F59.1
- net CELL7: now also F58.1
- net CELL8: now also F57.1
- net CELL9: now also F56.1
- net at D79.1 (K), Q90.2 (S), R413.2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: now also F64.2
- net at D79.2 (A), L7.1, R414.2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: now also F65.2
- net at Q83.2 (S), R406.2, R418.2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: now also F57.2
- net at Q80.2 (S), R403.2, R415.2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: now also F54.2
- net at Q79.2 (S), R439.1, R452.1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: now also F53.2
- net at Q81.2 (S), R404.2, R416.2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: now also F55.2
- net at Q84.2 (S), R407.2, R419.2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: now also F58.2
- net at Q87.2 (S), R410.2, R422.2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: now also F61.2
- net at Q89.2 (S), R412.2, R424.2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: now also F63.2
- net at Q85.2 (S), R408.2, R420.2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: now also F59.2
- net at Q88.2 (S), R411.2, R423.2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: now also F62.2
- net at Q82.2 (S), R405.2, R417.2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: now also F56.2
- net at Q86.2 (S), R409.2, R421.2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: now also F60.2

Commit message: アノテーションし直し
Parts:
- renumbered C205 to C235, C206 to C236, C207 to C237, C208 to C238, C209 to C239, C210 to C240, C211 to C241, C212 to C242, C213 to C243, C214 to C244, C215 to C245, C216 to C246, C217 to C247, C218 to C248, C219 to C249, C220 to C250, C221 to C251, C222 to C252, C223 to C253, C224 to C254, C225 to C255, C226 to C256, C227 to C257, C228 to C258, C229 to C259, C230 to C260, C321 to C261, C231 to C262, C322 to C263, C232 to C264, C233 to C265, C323 to C266, C234 to C267, C235 to C268, C324 to C269, C325 to C270, C236 to C271, C237 to C272, C238 to C273, F53 to F79, F54 to F80, F55 to F81, F56 to F82, F57 to F83, F58 to F84, F59 to F85, F60 to F86, F61 to F87, F62 to F88, F63 to F89, F64 to F90, F65 to F91, R403 to R433, R404 to R434, R405 to R435, R406 to R436, R407 to R437, R408 to R438, R409 to R439, R410 to R440, R411 to R441, R412 to R442, R413 to R443, R414 to R444, R415 to R445, R416 to R446, R417 to R447, R418 to R448, R419 to R449, R420 to R450, R421 to R451, R422 to R452, R423 to R453, R424 to R454, R425 to R455, R426 to R456, R427 to R457, R428 to R458, R429 to R459, R430 to R460, R431 to R461, R432 to R462, R433 to R463, R434 to R464, R435 to R465, R436 to R466, R437 to R467, R438 to R468, R439 to R469, R440 to R470, R441 to R471, R442 to R472, R443 to R473, R444 to R474, R445 to R475, R446 to R476, R447 to R477, R448 to R478, R449 to R479, R450 to R480, R451 to R481, R452 to R482, R454 to R483, R455 to R484, R457 to R485, R460 to R486, R461 to R487, R462 to R488, R463 to R489, R465 to R490, R453 to R491, R456 to R492, R458 to R493, R459 to R494, R464 to R495, R588 to R496, R466 to R497, R467 to R498, R468 to R499, R469 to R500, R589 to R501, R590 to R502, R591 to R503, R592 to R504

Commit message: GPIO入力保護回路追加
Parts:
- added D190, D191, D192, D193, D194, D195, D196, D197, D198, D199: BAT46W-7-F, ProjectEV:D_SOD-123_BAT46W-7-F, symbol ProjectEV:D_BAT46W-7-F
Connections:
- net GND1: now also D191.2 (A), D193.2 (A), D195.2 (A), D197.2 (A), D199.2 (A)
- net VREG: now also D190.1 (K), D192.1 (K), D194.1 (K), D196.1 (K), D198.1 (K)
- net at C270.1, R491.1, U7.27 (GPIO1): now also D190.2 (A), D191.1 (K)
- net at C269.1, R492.1, U7.28 (GPIO2): now also D192.2 (A), D193.1 (K)
- net at C263.1, R494.1, U7.32 (GPIO4): now also D196.2 (A), D197.1 (K)
- net at C261.1, R495.1, U7.33 (GPIO5): now also D198.2 (A), D199.1 (K)
- net at C266.1, R493.1, U7.29 (GPIO3): now also D194.2 (A), D195.1 (K)
Other:
- moved on the sheet: R491, R492, R493, R494, R495, R496, R501, R502, R503, R504

Commit message: アノテーションし直し
Parts:
- renumbered D79 to D139, D80 to D140, D81 to D141, D82 to D142, D83 to D143, D84 to D144, D85 to D145, D86 to D146, D87 to D147, D88 to D148, D89 to D149, D90 to D150, D91 to D151, D192 to D152, D193 to D153, D196 to D154, D197 to D155, D190 to D156, D191 to D157, D194 to D158, D195 to D159, D198 to D160, D199 to D161, L7 to L23, R433 to R435, R434 to R436, R435 to R437, R436 to R438, R437 to R439, R438 to R440, R439 to R441, R440 to R442, R441 to R443, R442 to R444, R443 to R445, R444 to R446, R445 to R447, R446 to R448, R447 to R449, R448 to R450, R449 to R451, R450 to R452, R451 to R453, R452 to R454, R453 to R455, R454 to R456, R455 to R457, R456 to R458, R457 to R459, R458 to R460, R459 to R461, R460 to R462, R461 to R463, R462 to R464, R463 to R465, R464 to R466, R465 to R467, R466 to R468, R467 to R469, R468 to R470, R469 to R471, R470 to R472, R471 to R473, R472 to R474, R473 to R475, R474 to R476, R475 to R477, R476 to R478, R477 to R479, R478 to R480, R479 to R481, R480 to R482, R481 to R483, R482 to R484, R483 to R485, R484 to R486, R485 to R487, R486 to R488, R487 to R489, R488 to R490, R489 to R491, R490 to R492, R497 to R493, R498 to R494, R499 to R495, R500 to R496, R491 to R497, R492 to R498, R493 to R499, R494 to R500, R495 to R501, R496 to R502, R501 to R503, R502 to R504, R503 to R505, R504 to R506
