File: AMS-board-2024/battery-module-monitor-7.kicad_sch (KiCad schematic)
At the start: 154 parts, among them Q79 BSS308PE, Q80 BSS308PE, Q81 BSS308PE, Q82 BSS308PE, Q83 BSS308PE, Q84 BSS308PE, Q85 BSS308PE, Q86 BSS308PE, Q87 BSS308PE, Q88 BSS308PE, Q89 BSS308PE, Q90 BSS308PE, Q91 NSV1C201MZ4, U7 LTC6811-1

Commit message: アノテーションし直し、
Parts:
- R460: renamed from R484; footprint Resistor_SMD:R_0402_1005Metric -> Resistor_SMD:R_0603_1608Metric
- R468: renamed from R492; footprint Resistor_SMD:R_0402_1005Metric -> Resistor_SMD:R_0603_1608Metric
- renumbered C235 to C223, C236 to C224, C237 to C225, C238 to C226, C239 to C227, C240 to C228, C241 to C229, C242 to C230, C243 to C231, C244 to C232, C245 to C233, C246 to C234, C247 to C235, C248 to C236, C249 to C237, C250 to C238, C251 to C239, C252 to C240, C253 to C241, C254 to C242, C255 to C243, C256 to C244, C257 to C245, C258 to C246, C259 to C247, C260 to C248, C262 to C249, C264 to C250, C265 to C251, C266 to C252, C267 to C253, C268 to C254, C269 to C255, C270 to C256, C271 to C257, C272 to C258, C273 to C259, D139 to D115, D140 to D116, D141 to D117, D142 to D118, D143 to D119, D144 to D120, D145 to D121, D146 to D122, D147 to D123, D148 to D124, D149 to D125, D150 to D126, D151 to D127, D152 to D128, D153 to D129, D156 to D130, D157 to D131, D158 to D132, D159 to D133, R435 to R411, R436 to R412, R437 to R413, R438 to R414, R439 to R415, R440 to R416, R441 to R417, R442 to R418, R443 to R419, R444 to R420, R445 to R421, R446 to R422, R447 to R423, R448 to R424, R449 to R425, R450 to R426, R451 to R427, R452 to R428, R453 to R429, R454 to R430, R455 to R431, R456 to R432, R457 to R433, R458 to R434, R459 to R435, R460 to R436, R461 to R437, R462 to R438, R463 to R439, R464 to R440, R465 to R441, R466 to R442, R467 to R443, R468 to R444, R469 to R445, R470 to R446, R471 to R447, R472 to R448, R473 to R449, R474 to R450, R475 to R451, R476 to R452, R477 to R453, R478 to R454, R479 to R455, R480 to R456, R481 to R457, R482 to R458, R483 to R459, R485 to R461, R486 to R462, R487 to R463, R488 to R464, R489 to R465, R490 to R466, R491 to R467, R493 to R469, R494 to R470, R495 to R471, R496 to R472, R497 to R473, R498 to R474, R499 to R475, R502 to R476, R503 to R477, R504 to R478
