File: AMS-board-2024/battery-module-monitor-7.kicad_sch (KiCad schematic)
At the start: 154 parts, among them Q79 BSS308PE, Q80 BSS308PE, Q81 BSS308PE, Q82 BSS308PE, Q83 BSS308PE, Q84 BSS308PE, Q85 BSS308PE, Q86 BSS308PE, Q87 BSS308PE, Q88 BSS308PE, Q89 BSS308PE, Q90 BSS308PE, Q91 NSV1C201MZ4, U7 LTC6811-1

Commit message: 絶縁パルストランス数削減
Parts:
- renumbered L24 to L17
Changed lines of the file:
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@@
   (symbol (lib_id "ProjectEV:L_MH3261") (at 101.6 374.65 0) (unit 1)
     (in_bom yes) (on_board yes) (dnp no) (fields_autoplaced)
-    (property "Reference" "L24" (at 102.87 373.38 0)
+    (property "Reference" "L17" (at 102.87 373.38 0)
       (effects (font (size 1.27 1.27)) (justify left))
     )
@@
       (project "AMS-board-2024"
         (path "/3a719eb3-09ce-4343-8f6e-20cc0aaf5261/70ce9b75-a01e-4dd0-929c-e9ba1d32d92a"
-          (reference "L24") (unit 1)
+          (reference "L17") (unit 1)
         )
       )

Commit message: 抵抗修正
3.3k -> 3k (1608)
15k -> 100k (1005, プルアップ/ダウン), 5.1k (1005, LED用)
Parts:
- R435, R436, R437, R438, R439, R440, R441, R442, R443, R444, R445, R446: value 3.3k -> 3k; footprint Resistor_SMD:R_0402_1005Metric -> Resistor_SMD:R_0603_1608Metric
Changed lines of the file:
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@@
       (effects (font (size 1.27 1.27)))
     )
-    (property "Value" "3.3k" (at 139.7 321.31 90)
-      (effects (font (size 1.27 1.27)))
-    )
-    (property "Footprint" "Resistor_SMD:R_0402_1005Metric" (at 139.7 325.628 90)
+    (property "Value" "3k" (at 139.7 321.31 90)
+      (effects (font (size 1.27 1.27)))
+    )
+    (property "Footprint" "Resistor_SMD:R_0603_1608Metric" (at 139.7 325.628 90)
       (effects (font (size 1.27 1.27)) hide)
     )
@@
       (effects (font (size 1.27 1.27)))
     )
-    (property "Value" "3.3k" (at 139.7 345.44 90)
-      (effects (font (size 1.27 1.27)))
-    )
-    (property "Footprint" "Resistor_SMD:R_0402_1005Metric" (at 139.7 349.758 90)
+    (property "Value" "3k" (at 139.7 345.44 90)
+      (effects (font (size 1.27 1.27)))
+    )
+    (property "Footprint" "Resistor_SMD:R_0603_1608Metric" (at 139.7 349.758 90)
       (effects (font (size 1.27 1.27)) hide)
     )
@@
       (effects (font (size 1.27 1.27)))
     )
-    (property "Value" "3.3k" (at 139.7 104.14 90)
-      (effects (font (size 1.27 1.27)))
-    )
-    (property "Footprint" "Resistor_SMD:R_0402_1005Metric" (at 139.7 108.458 90)
+    (property "Value" "3k" (at 139.7 104.14 90)
+      (effects (font (size 1.27 1.27)))
+    )
+    (property "Footprint" "Resistor_SMD:R_0603_1608Metric" (at 139.7 108.458 90)
       (effects (font (size 1.27 1.27)) hide)
     )
@@
       (effects (font (size 1.27 1.27)))
     )
-    (property "Value" "3.3k" (at 139.7 128.27 90)
-      (effects (font (size 1.27 1.27)))
-    )
-    (property "Footprint" "Resistor_SMD:R_0402_1005Metric" (at 139.7 132.588 90)
+    (property "Value" "3k" (at 139.7 128.27 90)
+      (effects (font (size 1.27 1.27)))
+    )
+    (property "Footprint" "Resistor_SMD:R_0603_1608Metric" (at 139.7 132.588 90)
       (effects (font (size 1.27 1.27)) hide)
     )
@@
       (effects (font (size 1.27 1.27)))
     )
-    (property "Value" "3.3k" (at 139.7 200.66 90)
-      (effects (font (size 1.27 1.27)))
-    )
-    (property "Footprint" "Resistor_SMD:R_0402_1005Metric" (at 139.7 204.978 90)
+    (property "Value" "3k" (at 139.7 200.66 90)
+      (effects (font (size 1.27 1.27)))
+    )
+    (property "Footprint" "Resistor_SMD:R_0603_1608Metric" (at 139.7 204.978 90)
       (effects (font (size 1.27 1.27)) hide)
     )
@@
       (effects (font (size 1.27 1.27)))
     )
-    (property "Value" "3.3k" (at 139.7 224.79 90)
-      (effects (font (size 1.27 1.27)))
-    )
-    (property "Footprint" "Resistor_SMD:R_0402_1005Metric" (at 139.7 229.108 90)
+    (property "Value" "3k" (at 139.7 224.79 90)
+      (effects (font (size 1.27 1.27)))
+    )
+    (property "Footprint" "Resistor_SMD:R_0603_1608Metric" (at 139.7 229.108 90)
       (effects (font (size 1.27 1.27)) hide)
     )
@@
       (effects (font (size 1.27 1.27)))
     )
-    (property "Value" "3.3k" (at 139.7 248.92 90)
-      (effects (font (size 1.27 1.27)))
-    )
-    (property "Footprint" "Resistor_SMD:R_0402_1005Metric" (at 139.7 253.238 90)
+    (property "Value" "3k" (at 139.7 248.92 90)
+      (effects (font (size 1.27 1.27)))
+    )
+    (property "Footprint" "Resistor_SMD:R_0603_1608Metric" (at 139.7 253.238 90)
       (effects (font (size 1.27 1.27)) hide)
     )
@@
       (effects (font (size 1.27 1.27)))
     )
-    (property "Value" "3.3k" (at 139.7 152.4 90)
-      (effects (font (size 1.27 1.27)))
-    )
-    (property "Footprint" "Resistor_SMD:R_0402_1005Metric" (at 139.7 156.718 90)
+    (property "Value" "3k" (at 139.7 152.4 90)
+      (effects (font (size 1.27 1.27)))
+    )
+    (property "Footprint" "Resistor_SMD:R_0603_1608Metric" (at 139.7 156.718 90)
       (effects (font (size 1.27 1.27)) hide)
     )
@@
       (effects (font (size 1.27 1.27)))
     )
-    (property "Value" "3.3k" (at 139.7 176.53 90)
-      (effects (font (size 1.27 1.27)))
-    )
-    (property "Footprint" "Resistor_SMD:R_0402_1005Metric" (at 139.7 180.848 90)
+    (property "Value" "3k" (at 139.7 176.53 90)
+      (effects (font (size 1.27 1.27)))
+    )
+    (property "Footprint" "Resistor_SMD:R_0603_1608Metric" (at 139.7 180.848 90)
       (effects (font (size 1.27 1.27)) hide)
     )
@@
       (effects (font (size 1.27 1.27)))
     )
-    (property "Value" "3.3k" (at 139.7 80.01 90)
-      (effects (font (size 1.27 1.27)))
-    )
-    (property "Footprint" "Resistor_SMD:R_0402_1005Metric" (at 139.7 84.328 90)
+    (property "Value" "3k" (at 139.7 80.01 90)
+      (effects (font (size 1.27 1.27)))
+    )
+    (property "Footprint" "Resistor_SMD:R_0603_1608Metric" (at 139.7 84.328 90)
       (effects (font (size 1.27 1.27)) hide)
     )
@@
       (effects (font (size 1.27 1.27)))
     )
-    (property "Value" "3.3k" (at 139.7 273.05 90)
-      (effects (font (size 1.27 1.27)))
-    )
-    (property "Footprint" "Resistor_SMD:R_0402_1005Metric" (at 139.7 277.368 90)
+    (property "Value" "3k" (at 139.7 273.05 90)
+      (effects (font (size 1.27 1.27)))
+    )
+    (property "Footprint" "Resistor_SMD:R_0603_1608Metric" (at 139.7 277.368 90)
       (effects (font (size 1.27 1.27)) hide)
     )
@@
       (effects (font (size 1.27 1.27)))
     )
-    (property "Value" "3.3k" (at 139.7 297.18 90)
-      (effects (font (size 1.27 1.27)))
-    )
-    (property "Footprint" "Resistor_SMD:R_0402_1005Metric" (at 139.7 301.498 90)
-      (effects (font (size 1.27 1.27)) hide)
-    )
+    (property "Value" "3k" (at 139.7 297.18 90)
+      (effects (font (size 1.27 1.27)))
+    )
+    (property "Footprint" "Resistor_SMD:R_0603_1608Metric" (at 139.7 301.498 90)
+      (effects (font (size 1.27 1.27)) hide)
+    )

Commit message: アノテーションし直し
Parts:
- renumbered C223 to C232, C224 to C233, C225 to C234, C226 to C235, C227 to C236, C228 to C237, C229 to C238, C230 to C239, C231 to C240, C232 to C241, C233 to C242, C234 to C243, C235 to C244, C236 to C245, C237 to C246, C238 to C247, C239 to C248, C240 to C249, C241 to C250, C242 to C251, C243 to C252, C244 to C253, C245 to C254, C246 to C255, C247 to C256, C248 to C257, C249 to C258, C250 to C259, C251 to C260, C252 to C261, C253 to C262, C254 to C263, C255 to C264, C256 to C265, C257 to C266, C258 to C267, C259 to C268, L17 to L13
