File: AMS-board-2024/battery-module-monitor-1.kicad_sch (KiCad schematic)
At the start: 144 parts, among them Q201 BSS308PE, Q202 BSS308PE, Q203 BSS308PE, Q204 BSS308PE, Q205 BSS308PE, Q206 BSS308PE, Q207 BSS308PE, Q208 BSS308PE, Q209 BSS308PE, Q210 BSS308PE, Q211 BSS308PE, Q212 BSS308PE, Q213 NSV1C201MZ4, U201 LTC6811-1

Commit message: 修正
アノテーション方法の変更：最初の空き番号から使用
Parts:
- renumbered C201 to C1, C210 to C10, C211 to C11, C212 to C12, C213 to C13, C214 to C14, C215 to C15, C216 to C16, C217 to C17, C218 to C18, C219 to C19, C202 to C2, C220 to C20, C221 to C21, C222 to C22, C223 to C23, C224 to C24, C225 to C25, C226 to C26, C227 to C27, C228 to C28, C229 to C29, C203 to C3, C230 to C30, C231 to C31, C232 to C32, C233 to C33, C234 to C34, C204 to C4, C205 to C5, C206 to C6, C207 to C7, C208 to C8, C209 to C9, D201 to D1, D210 to D10, D211 to D11, D212 to D12, D213 to D13, D202 to D2, D203 to D3, D204 to D4, D205 to D5, D206 to D6, D207 to D7, D208 to D8, D209 to D9, F201 to F1, F210 to F10, F211 to F11, F212 to F12, F213 to F13, F202 to F2, F203 to F3, F204 to F4, F205 to F5, F206 to F6, F207 to F7, F208 to F8, F209 to F9, FL201 to FL1, FL202 to FL2, L201 to L1, Q201 to Q1, Q210 to Q10, Q211 to Q11, Q212 to Q12, Q213 to Q13, Q202 to Q2, Q203 to Q3, Q204 to Q4, Q205 to Q5, Q206 to Q6, Q207 to Q7, Q208 to Q8, Q209 to Q9, R201 to R1, R210 to R10, R211 to R11, R212 to R12, R213 to R13, R214 to R14, R215 to R15, R216 to R16, R217 to R17, R218 to R18, R219 to R19, R202 to R2, R220 to R20, R221 to R21, R222 to R22, R223 to R23, R224 to R24, R225 to R25, R226 to R26, R227 to R27, R228 to R28, R229 to R29, R203 to R3, R230 to R30, R231 to R31, R232 to R32, R233 to R33, R234 to R34, R235 to R35, R236 to R36, R237 to R37, R238 to R38, R239 to R39, R204 to R4, R240 to R40, R241 to R41, R242 to R42, R243 to R43, R244 to R44, R245 to R45, R246 to R46, R247 to R47, R248 to R48, R249 to R49, R205 to R5, R250 to R50, R251 to R51, R252 to R52, R253 to R53, R254 to R54, R255 to R55, R256 to R56, R257 to R57, R258 to R58, R259 to R59, R206 to R6, R260 to R60, R261 to R61, R262 to R62, R263 to R63, R264 to R64, R265 to R65, R266 to R66, R267 to R67, R207 to R7, R208 to R8, R209 to R9, U201 to U1

Commit message: GNDシンボル追加
Connections:
- net GND1: now reaches C5.2
- net GND1: now also C1.2, C10.2, C11.2, C12.2, C2.2, C25.2, C26.2, C27.1, C28.1, C29.2, C3.2, C30.1, C31.1, C32.2, C33.1, C34.1, C4.2, C6.2, C7.2, C8.2, C9.2, L1.2, R55.1, U1.30 (V-), U1.31 (V-)

Commit message: GPIO周辺回路の修正
Parts:
- added C291, C292, C293, C294, C295: 0.1u, Capacitor_SMD:C_0603_1608Metric, symbol Device:C
- added R551, R552, R560, R561, R562: 100, Resistor_SMD:R_0603_1608Metric, symbol Device:R
Connections:
- net GND1: now also C291.2, C292.2, C293.2, C294.2, C295.2
- net Thermistor1+: now also R51.2, R551.2; no longer R62.1, U1.27 (GPIO1)
- net Thermistor2+: now also R54.2, R552.2; no longer R57.1, U1.28 (GPIO2)
- net Thermistor3+: now also R56.2, R560.2; no longer R56.1, U1.29 (GPIO3)
- net Thermistor4+: now also R57.2, R561.2; no longer R54.1, U1.32 (GPIO4)
- net Thermistor5+: now also R62.2, R562.2; no longer R51.1, U1.33 (GPIO5)
- net VREG: now reaches C29.1, Q13.3 (E), R53.1, U1.37 (VREG), U1.40 (ISOMD)
- new net: C295.1, R562.1, U1.33 (GPIO5)
- new net: C292.1, R552.1, U1.28 (GPIO2)
- new net: C291.1, R551.1, U1.27 (GPIO1)
- new net: C293.1, R560.1, U1.29 (GPIO3)
- new net: C294.1, R561.1, U1.32 (GPIO4)
- new net VREF_3V: C27.2, R51.1, R54.1, R56.1, R57.1, R62.1, U1.34 (VREF2)
Other:
- moved on the sheet: R51, R54, R56, R57, R62

Commit message: ヒューズ変更
Parts:
- removed F1, F10, F11, F12, F13, F2, F3, F4, F5, F6, F7, F8, F9: C1F 500, Fuse:Fuse_1206_3216Metric, symbol Device:Fuse
- added F201, F202, F203, F204, F205, F206, F207, F208, F209, F210, F211, F212, F213: 0679L1000-05, ProjectEV:Fuse_0679L, symbol ProjectEV:Fuse_0679L1000-05
Connections:
- net CELL0: now also F213.1
- net CELL1: now also F212.1
- net CELL10: now also F203.1
- net CELL11: now also F202.1
- net CELL12: now also F201.1
- net CELL2: now also F211.1
- net CELL3: now also F210.1
- net CELL4: now also F209.1
- net CELL5: now also F208.1
- net CELL6: now also F207.1
- net CELL7: now also F206.1
- net CELL8: now also F205.1
- net CELL9: now also F204.1
- net at Q11.2 (S), R10.2, R22.2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: now also F211.2
- net at Q7.2 (S), R18.2, R43.1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: now also F207.2
- net at Q9.2 (S), R20.2, R45.1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: now also F209.2
- net at Q6.2 (S), R17.2, R42.1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: now also F206.2
- net at Q4.2 (S), R15.2, R3.2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: now also F204.2
- net at Q3.2 (S), R14.2, R2.2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: now also F203.2
- net at D1.1 (K), Q12.2 (S), R11.2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: now also F212.2
- net at Q10.2 (S), R21.2, R46.1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: now also F210.2
- net at D1.2 (A), L1.1, R12.2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: now also F213.2
- net at Q5.2 (S), R16.2, R4.2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: now also F205.2
- net at Q8.2 (S), R19.2, R44.1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: now also F208.2
- net at Q1.2 (S), R37.1, R50.1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: now also F201.2
- net at Q2.2 (S), R1.2, R13.2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: now also F202.2

Commit message: アノテーションし直し
Parts:
- renumbered C295 to C27, C27 to C28, C294 to C29, C28 to C30, C29 to C31, C293 to C32, C30 to C33, C31 to C34, C292 to C35, C291 to C36, C32 to C37, C33 to C38, C34 to C39, F201 to F1, F210 to F10, F211 to F11, F212 to F12, F213 to F13, F202 to F2, F203 to F3, F204 to F4, F205 to F5, F206 to F6, F207 to F7, F208 to F8, F209 to F9, R52 to R51, R53 to R52, R55 to R53, R58 to R54, R59 to R55, R60 to R56, R61 to R57, R63 to R58, R551 to R59, R552 to R60, R560 to R61, R561 to R62, R562 to R63, R51 to R64, R64 to R65, R65 to R66, R66 to R67, R67 to R68, R54 to R69, R56 to R70, R57 to R71, R62 to R72

Commit message: GPIO入力保護回路追加
Parts:
- added D140, D141, D142, D143, D144, D145, D146, D147, D148, D149: BAT46W-7-F, ProjectEV:D_SOD-123_BAT46W-7-F, symbol ProjectEV:D_BAT46W-7-F
Connections:
- net GND1: now also D141.2 (A), D143.2 (A), D145.2 (A), D147.2 (A), D149.2 (A)
- net VREG: now also D140.1 (K), D142.1 (K), D144.1 (K), D146.1 (K), D148.1 (K)
- net at C27.1, R63.1, U1.33 (GPIO5): now also D148.2 (A), D149.1 (K)
- net at C35.1, R60.1, U1.28 (GPIO2): now also D142.2 (A), D143.1 (K)
- net at C36.1, R59.1, U1.27 (GPIO1): now also D140.2 (A), D141.1 (K)
- net at C32.1, R61.1, U1.29 (GPIO3): now also D144.2 (A), D145.1 (K)
- net at C29.1, R62.1, U1.32 (GPIO4): now also D146.2 (A), D147.1 (K)
Other:
- moved on the sheet: R59, R60, R61, R62, R63, R64, R69, R70, R71, R72

Commit message: アノテーションし直し
Parts:
- renumbered D142 to D14, D143 to D15, D146 to D16, D147 to D17, D140 to D18, D141 to D19, D144 to D20, D145 to D21, D148 to D22, D149 to D23, L1 to L17, R8 to R10, R9 to R11, R10 to R12, R11 to R13, R12 to R14, R13 to R15, R14 to R16, R15 to R17, R16 to R18, R17 to R19, R18 to R20, R19 to R21, R20 to R22, R21 to R23, R22 to R24, R23 to R25, R24 to R26, R25 to R27, R26 to R28, R27 to R29, R1 to R3, R28 to R30, R29 to R31, R30 to R32, R31 to R33, R32 to R34, R33 to R35, R34 to R36, R35 to R37, R36 to R38, R37 to R39, R2 to R4, R38 to R40, R39 to R41, R40 to R42, R41 to R43, R42 to R44, R43 to R45, R44 to R46, R45 to R47, R46 to R48, R47 to R49, R3 to R5, R48 to R50, R49 to R51, R50 to R52, R51 to R53, R52 to R54, R53 to R55, R54 to R56, R55 to R57, R56 to R58, R57 to R59, R4 to R6, R58 to R60, R65 to R61, R66 to R62, R67 to R63, R68 to R64, R59 to R65, R60 to R66, R61 to R67, R62 to R68, R63 to R69, R5 to R7, R64 to R70, R69 to R71, R70 to R72, R71 to R73, R72 to R74, R6 to R8, R7 to R9

Commit message: ERC実行、修正
ラベル修正、未配線部分修正、PWR_FLAG追加
Connections:
- net GND1: now also U1.36 (SWTEN)
- net VREG renamed VREG1
