File: AMS-board-2024/battery-module-monitor-1.kicad_sch (KiCad schematic)
At the start: 164 parts, among them Q1 BSS308PE, Q10 BSS308PE, Q11 BSS308PE, Q12 BSS308PE, Q13 NSV1C201MZ4, Q2 BSS308PE, Q3 BSS308PE, Q4 BSS308PE, Q5 BSS308PE, Q6 BSS308PE, Q7 BSS308PE, Q8 BSS308PE, Q9 BSS308PE, U1 LTC6811-1

Commit message: ラベル修正
Connections:
- net VREG1 renamed VREG
Changed lines of the file:
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@@
     (effects (font (size 1.27 1.27)) (justify left bottom))
   )
-  (label "VREG1" (at 365.76 266.7 0) (fields_autoplaced)
+  (label "S2_VREG" (at 378.46 241.3 0) (fields_autoplaced)
     (effects (font (size 1.27 1.27)) (justify left bottom))
   )
-  (label "VREG1" (at 378.46 241.3 0) (fields_autoplaced)
+  (label "S2_VREG" (at 365.76 317.5 0) (fields_autoplaced)
     (effects (font (size 1.27 1.27)) (justify left bottom))
   )
-  (label "VREG1" (at 378.46 342.9 0) (fields_autoplaced)
+  (label "S2_VREG" (at 365.76 266.7 0) (fields_autoplaced)
     (effects (font (size 1.27 1.27)) (justify left bottom))
   )
-  (label "VREG1" (at 378.46 292.1 0) (fields_autoplaced)
+  (label "S2_VREG" (at 378.46 342.9 0) (fields_autoplaced)
     (effects (font (size 1.27 1.27)) (justify left bottom))
   )
-  (label "VREG1" (at 365.76 317.5 0) (fields_autoplaced)
+  (label "S2_VREG" (at 378.46 292.1 0) (fields_autoplaced)
     (effects (font (size 1.27 1.27)) (justify left bottom))
   )
-  (label "VREG1" (at 342.9 215.9 0) (fields_autoplaced)
+  (label "S2_VREG" (at 342.9 215.9 0) (fields_autoplaced)
     (effects (font (size 1.27 1.27)) (justify left bottom))
   )
@@
     (effects (font (size 1.27 1.27)) (justify right))
   )
-  (hierarchical_label "VREG1" (shape output) (at 419.1 223.52 0) (fields_autoplaced)
+  (hierarchical_label "VREG" (shape output) (at 419.1 223.52 0) (fields_autoplaced)
     (effects (font (size 1.27 1.27)) (justify left))
   )

Commit message: アノテーションし直し
Parts:
- renumbered L17 to L18

Commit message: 階層シート内の電源シンボル修正
階層シート内で電源シンボルをなるべく使わないようにする
修正途中
Connections:
- net GND1 renamed GND

Commit message: LTC6811のシンボルを更新
Parts:
- U1: footprint ProjectEV:SSOP-48_5.3x12.8mm_P0.5mm_LTC6811 -> ProjectEV:Package_SSOP-48_5.3x12.8mm_P0.5mm_LTC6811
Changed lines of the file:
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@@
       (effects (font (size 1.27 1.27)) (justify left))
     )
-    (property "Footprint" "ProjectEV:SSOP-48_5.3x12.8mm_P0.5mm_LTC6811" (at 290.83 213.36 0)
+    (property "Footprint" "ProjectEV:Package_SSOP-48_5.3x12.8mm_P0.5mm_LTC6811" (at 290.83 213.36 0)
       (effects (font (size 1.27 1.27)) hide)
     )

Commit message: チップ抵抗、チップコンデンササイズ修正
Parts:
- C13, C14, C15, C16, C17, C18, C19, C20, C21, C22, C23, C24, C25, C27, C28, C29, C30, C31, C32, C33, C34, C35, C36, C38, C39: footprint Capacitor_SMD:C_0603_1608Metric -> Capacitor_SMD:C_0402_1005Metric
- R27, R28, R29, R30, R31, R32, R33, R34, R35, R36, R37, R38, R39, R40, R41, R42, R43, R44, R45, R46, R47, R48, R49, R50, R51, R52, R53, R55, R60, R65, R66, R67, R68, R69, R70, R71, R72, R73, R74: footprint Resistor_SMD:R_0603_1608Metric -> Resistor_SMD:R_0402_1005Metric

Commit message: 温度センサ用コネクタ変更、大まかな位置決定
Parts:
- removed C27, C29: 0.1u, Capacitor_SMD:C_0402_1005Metric, symbol Device:C
- removed D16, D17, D22, D23: BAT46W-7-F, ProjectEV:D_SOD-123_BAT46W-7-F, symbol ProjectEV:D_BAT46W-7-F
- removed R68, R69: 100, Resistor_SMD:R_0402_1005Metric, symbol Device:R
- removed R73, R74: 10k, Resistor_SMD:R_0402_1005Metric, symbol Device:R
Connections:
- net VREF_3V: no longer names the net of C28.2, R70.1, R71.1, R72.1, U1.34 (VREF2)
- net VREG: no longer names the net of C31.1, D14.1 (K), D18.1 (K), D20.1 (K), Q13.3 (E), R54.1, U1.37 (VREG), U1.40 (ISOMD)
- no-connect marks 2 -> 4

Commit message: アノテーションし直し、
Parts:
- R52, R60: footprint Resistor_SMD:R_0402_1005Metric -> Resistor_SMD:R_0603_1608Metric
- renumbered C28 to C27, C30 to C28, C31 to C29, C32 to C30, C33 to C31, C34 to C32, C35 to C33, C36 to C34, C37 to C35, C38 to C36, C39 to C37, D18 to D16, D19 to D17, D20 to D18, D21 to D19, R70 to R68, R71 to R69, R72 to R70

Commit message: 絶縁パルストランス数削減
Parts:
- renumbered L18 to L11
Changed lines of the file:
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@@
   (symbol (lib_id "ProjectEV:L_MH3261") (at 101.6 374.65 0) (unit 1)
     (in_bom yes) (on_board yes) (dnp no) (fields_autoplaced)
-    (property "Reference" "L18" (at 102.87 373.38 0)
+    (property "Reference" "L11" (at 102.87 373.38 0)
       (effects (font (size 1.27 1.27)) (justify left))
     )
@@
       (project "AMS-board-2024"
         (path "/3a719eb3-09ce-4343-8f6e-20cc0aaf5261/9d82a782-0bb3-4a0b-9494-e2cd06769caf"
-          (reference "L18") (unit 1)
+          (reference "L11") (unit 1)
         )
       )
