File: AMS-board-2024/battery-module-monitor-1.kicad_sch (KiCad schematic)
At the start: 154 parts, among them Q1 BSS308PE, Q10 BSS308PE, Q11 BSS308PE, Q12 BSS308PE, Q13 NSV1C201MZ4, Q2 BSS308PE, Q3 BSS308PE, Q4 BSS308PE, Q5 BSS308PE, Q6 BSS308PE, Q7 BSS308PE, Q8 BSS308PE, Q9 BSS308PE, U1 LTC6811-1

Commit message: 抵抗修正
3.3k -> 3k (1608)
15k -> 100k (1005, プルアップ/ダウン), 5.1k (1005, LED用)
Parts:
- R27, R28, R29, R30, R31, R32, R33, R34, R35, R36, R37, R38: value 3.3k -> 3k; footprint Resistor_SMD:R_0402_1005Metric -> Resistor_SMD:R_0603_1608Metric
Changed lines of the file:
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@@
       (effects (font (size 1.27 1.27)))
     )
-    (property "Value" "3.3k" (at 139.7 345.44 90)
-      (effects (font (size 1.27 1.27)))
-    )
-    (property "Footprint" "Resistor_SMD:R_0402_1005Metric" (at 139.7 349.758 90)
+    (property "Value" "3k" (at 139.7 345.44 90)
+      (effects (font (size 1.27 1.27)))
+    )
+    (property "Footprint" "Resistor_SMD:R_0603_1608Metric" (at 139.7 349.758 90)
       (effects (font (size 1.27 1.27)) hide)
     )
@@
       (effects (font (size 1.27 1.27)))
     )
-    (property "Value" "3.3k" (at 139.7 152.4 90)
-      (effects (font (size 1.27 1.27)))
-    )
-    (property "Footprint" "Resistor_SMD:R_0402_1005Metric" (at 139.7 156.718 90)
+    (property "Value" "3k" (at 139.7 152.4 90)
+      (effects (font (size 1.27 1.27)))
+    )
+    (property "Footprint" "Resistor_SMD:R_0603_1608Metric" (at 139.7 156.718 90)
       (effects (font (size 1.27 1.27)) hide)
     )
@@
       (effects (font (size 1.27 1.27)))
     )
-    (property "Value" "3.3k" (at 139.7 128.27 90)
-      (effects (font (size 1.27 1.27)))
-    )
-    (property "Footprint" "Resistor_SMD:R_0402_1005Metric" (at 139.7 132.588 90)
+    (property "Value" "3k" (at 139.7 128.27 90)
+      (effects (font (size 1.27 1.27)))
+    )
+    (property "Footprint" "Resistor_SMD:R_0603_1608Metric" (at 139.7 132.588 90)
       (effects (font (size 1.27 1.27)) hide)
     )
@@
       (effects (font (size 1.27 1.27)))
     )
-    (property "Value" "3.3k" (at 139.7 224.79 90)
-      (effects (font (size 1.27 1.27)))
-    )
-    (property "Footprint" "Resistor_SMD:R_0402_1005Metric" (at 139.7 229.108 90)
+    (property "Value" "3k" (at 139.7 224.79 90)
+      (effects (font (size 1.27 1.27)))
+    )
+    (property "Footprint" "Resistor_SMD:R_0603_1608Metric" (at 139.7 229.108 90)
       (effects (font (size 1.27 1.27)) hide)
     )
@@
       (effects (font (size 1.27 1.27)))
     )
-    (property "Value" "3.3k" (at 139.7 248.92 90)
-      (effects (font (size 1.27 1.27)))
-    )
-    (property "Footprint" "Resistor_SMD:R_0402_1005Metric" (at 139.7 253.238 90)
+    (property "Value" "3k" (at 139.7 248.92 90)
+      (effects (font (size 1.27 1.27)))
+    )
+    (property "Footprint" "Resistor_SMD:R_0603_1608Metric" (at 139.7 253.238 90)
       (effects (font (size 1.27 1.27)) hide)
     )
@@
       (effects (font (size 1.27 1.27)))
     )
-    (property "Value" "3.3k" (at 139.7 80.01 90)
-      (effects (font (size 1.27 1.27)))
-    )
-    (property "Footprint" "Resistor_SMD:R_0402_1005Metric" (at 139.7 84.328 90)
+    (property "Value" "3k" (at 139.7 80.01 90)
+      (effects (font (size 1.27 1.27)))
+    )
+    (property "Footprint" "Resistor_SMD:R_0603_1608Metric" (at 139.7 84.328 90)
       (effects (font (size 1.27 1.27)) hide)
     )
@@
       (effects (font (size 1.27 1.27)))
     )
-    (property "Value" "3.3k" (at 139.7 297.18 90)
-      (effects (font (size 1.27 1.27)))
-    )
-    (property "Footprint" "Resistor_SMD:R_0402_1005Metric" (at 139.7 301.498 90)
+    (property "Value" "3k" (at 139.7 297.18 90)
+      (effects (font (size 1.27 1.27)))
+    )
+    (property "Footprint" "Resistor_SMD:R_0603_1608Metric" (at 139.7 301.498 90)
       (effects (font (size 1.27 1.27)) hide)
     )
@@
       (effects (font (size 1.27 1.27)))
     )
-    (property "Value" "3.3k" (at 139.7 273.05 90)
-      (effects (font (size 1.27 1.27)))
-    )
-    (property "Footprint" "Resistor_SMD:R_0402_1005Metric" (at 139.7 277.368 90)
+    (property "Value" "3k" (at 139.7 273.05 90)
+      (effects (font (size 1.27 1.27)))
+    )
+    (property "Footprint" "Resistor_SMD:R_0603_1608Metric" (at 139.7 277.368 90)
       (effects (font (size 1.27 1.27)) hide)
     )
@@
       (effects (font (size 1.27 1.27)))
     )
-    (property "Value" "3.3k" (at 139.7 200.66 90)
-      (effects (font (size 1.27 1.27)))
-    )
-    (property "Footprint" "Resistor_SMD:R_0402_1005Metric" (at 139.7 204.978 90)
+    (property "Value" "3k" (at 139.7 200.66 90)
+      (effects (font (size 1.27 1.27)))
+    )
+    (property "Footprint" "Resistor_SMD:R_0603_1608Metric" (at 139.7 204.978 90)
       (effects (font (size 1.27 1.27)) hide)
     )
@@
       (effects (font (size 1.27 1.27)))
     )
-    (property "Value" "3.3k" (at 139.7 104.14 90)
-      (effects (font (size 1.27 1.27)))
-    )
-    (property "Footprint" "Resistor_SMD:R_0402_1005Metric" (at 139.7 108.458 90)
+    (property "Value" "3k" (at 139.7 104.14 90)
+      (effects (font (size 1.27 1.27)))
+    )
+    (property "Footprint" "Resistor_SMD:R_0603_1608Metric" (at 139.7 108.458 90)
       (effects (font (size 1.27 1.27)) hide)
     )
@@
       (effects (font (size 1.27 1.27)))
     )
-    (property "Value" "3.3k" (at 139.7 321.31 90)
-      (effects (font (size 1.27 1.27)))
-    )
-    (property "Footprint" "Resistor_SMD:R_0402_1005Metric" (at 139.7 325.628 90)
+    (property "Value" "3k" (at 139.7 321.31 90)
+      (effects (font (size 1.27 1.27)))
+    )
+    (property "Footprint" "Resistor_SMD:R_0603_1608Metric" (at 139.7 325.628 90)
       (effects (font (size 1.27 1.27)) hide)
     )
@@
       (effects (font (size 1.27 1.27)))
     )
-    (property "Value" "3.3k" (at 139.7 176.53 90)
-      (effects (font (size 1.27 1.27)))
-    )
-    (property "Footprint" "Resistor_SMD:R_0402_1005Metric" (at 139.7 180.848 90)
-      (effects (font (size 1.27 1.27)) hide)
-    )
+    (property "Value" "3k" (at 139.7 176.53 90)
+      (effects (font (size 1.27 1.27)))
+    )
+    (property "Footprint" "Resistor_SMD:R_0603_1608Metric" (at 139.7 180.848 90)
+      (effects (font (size 1.27 1.27)) hide)
+    )

Commit message: アノテーションし直し
Parts:
- renumbered C1 to C10, C2 to C11, C3 to C12, C4 to C13, C5 to C14, C6 to C15, C7 to C16, C8 to C17, C9 to C18, C10 to C19, C11 to C20, C12 to C21, C13 to C22, C14 to C23, C15 to C24, C16 to C25, C17 to C26, C18 to C27, C19 to C28, C20 to C29, C21 to C30, C22 to C31, C23 to C32, C24 to C33, C25 to C34, C26 to C35, C27 to C36, C28 to C37, C29 to C38, C30 to C39, C31 to C40, C32 to C41, C33 to C42, C34 to C43, C35 to C44, C36 to C45, C37 to C46, L11 to L7
