File: AMS-board-2024/power.kicad_sch (KiCad schematic)
At the start: 9 parts, among them Q105 AO3401A, Q106 AO3401A, U13 MCP6001T-E/OT

Commit message: 電源回路作成
VBUS絶縁回路以外およそ完成
Parts:
- removed D108: BZX584C5V1-AU, ProjectEV:D_SOD-523_BZX584CxVx-AU, symbol ProjectEV:D_BZX584C5V1-AU
- removed F105: Fuse, symbol Device:Fuse
- removed Q105, Q106: AO3401A, ProjectEV:Package_SOT-23, symbol ProjectEV:Transistor_AO3401A
- added C331, C337, C338, C340, C341, C342, C343, C344, C345: 10u, Capacitor_SMD:C_1206_3216Metric, symbol Device:C
- added C332, C334, C335, C339, C346, C347: 0.1u, Capacitor_SMD:C_0603_1608Metric, symbol Device:C
- added C333: 1u, Capacitor_SMD:C_0603_1608Metric, symbol Device:C
- added C336, C350: 22u, Capacitor_SMD:C_0805_2012Metric, symbol Device:C
- added C348, C349: 22u, symbol Device:C_Polarized
- added D108: SMBJ33CAQ, ProjectEV:D_SMB_SMBJxxxCAQ, symbol ProjectEV:TVS_SMBJ33CAQ
- added D113: LED, LED_SMD:LED_0603_1608Metric, symbol Device:LED
- added D114: SMSZ4690, ProjectEV:D_SOD-123_SMSZ4xxx, symbol ProjectEV:D_SMSZ4690
- added L9: EXLA1V0605-1R5-R, ProjectEV:L_EXLA1V06, symbol ProjectEV:L_EXLA1V06
- added Q105, Q106: DMT6007LFGQ, ProjectEV:Package_PowerDI3333-8_DMT6007LFGQ, symbol ProjectEV:Transistor_DMT6007LFGQ
- added Q110, Q111: 2N7002K-AU, ProjectEV:Package_SOT-23_2N7002K-AU, symbol ProjectEV:Transistor_2N7002K-AU
- added R609, R611, R612, R615: 100k, Resistor_SMD:R_0603_1608Metric, symbol Device:R
- added R610: 24.9k, Resistor_SMD:R_0603_1608Metric, symbol Device:R
- added R613: 13k, Resistor_SMD:R_0603_1608Metric, symbol Device:R
- added R614: 8.2k, Resistor_SMD:R_0603_1608Metric, symbol Device:R
- added R616: 5.1k, Resistor_SMD:R_0603_1608Metric, symbol Device:R
- added R617: 2.2k, Resistor_SMD:R_0603_1608Metric, symbol Device:R
- added R618: 15k, Resistor_SMD:R_0603_1608Metric, symbol Device:R
- added U14: LMR33620APCQRNXRQ1, ProjectEV:Package_VQFN-HR-12_RNX0012C_2x3mm_LMR33620AP-Q1, symbol ProjectEV:Regulator_LMR33620AP-Q1
- added U15: AP74700QW6-7, ProjectEV:Package_SOT-26_AP74700Q, symbol ProjectEV:PowerProtection_AP74700Q
- added U16: LM5060, ProjectEV:Package_VSSOP-10_3x3mm_P0.5mm_LM5060, symbol ProjectEV:PowerProtection_LM5060
- added U17: VOMA617A, ProjectEV:Package_SOP-4_4.57x4.92mm_P2.54mm_VOMA617A, symbol ProjectEV:Isolator_VOMA617A
- R599: value 15k -> 1.2k
Connections:
- net PWRIN+: now reaches D106.2 (A), D107.1 (K)
- net PWRIN+: now also C338.1, C339.1, D108.2 (A2), Q105.1 (S), Q105.2 (S), Q105.3 (S), U15.3 (EN), U15.6 (ANODE)
- net PWRIN-: now reaches R598.2
- net PWRIN-: now also C331.2, C332.2, C333.2, C335.2, C336.2, C340.2, C341.2, C343.2, C344.2, C345.2, C346.2, C347.1, C348.2, C349.2, C350.2, D108.1 (A1), D114.2 (A), Q110.2 (S), Q111.2 (S), R610.2, R614.2, R618.2, U14.1 (PGND), U14.11 (PGND), U14.6 (AGND), U15.2 (GND), U16.6 (GND), U17.2
- net at R599.1: now also C337.1, C342.1, C347.2, C348.1, Q105.5 (D), Q106.1 (S), Q106.2 (S), Q106.3 (S), R612.1, R615.1, U15.4 (CATHODE), U16.2 (VIN), U16.5 (EN)
- net at R599.2: now also U16.1 (SENSE)
- new net: R609.2, R610.1, U14.7 (FB)
- new net: Q111.3 (D), R617.2, U17.1
- new net: C337.2, C341.1
- new net: C346.1, U16.7 (TIMER)
- new net: D113.1 (K), Q110.3 (D)
- new net: C338.2, C340.1
- new net: R612.2, R613.1, U16.4 (UVLO)
- new net: R613.2, R614.1, U16.3 (OVP)
- new net: Q106.4 (G), U16.10 (GATE)
- new net: Q105.4 (G), U15.5 (GATE)
- new net: C339.2, U15.1 (VCP)
- new net: C342.2, C343.1
- new net: C334.2, L9.1, U14.12 (SW)
- new net: C334.1, U14.4 (BOOT)
- new net: C333.1, R611.2, U14.5 (VCC)
- new net: D113.2 (A), R616.2
- new net DCDC_EN: R618.1, U14.9 (EN), U17.3
- new net PG: Q110.1 (G), R611.1, U14.8 (PG)
- new net PWROUT+: C331.1, C332.1, C344.1, C345.1, C349.1, Q106.5 (D), R617.1, U14.10 (VIN), U14.2 (VIN), U16.9 (OUT), U17.4
- new net VOUT+: C335.1, C336.1, C350.1, L9.2, R609.1, R616.1
- new net ~{DCDC_EN}: D114.1 (K), Q111.1 (G), R615.2, U16.8 (nPGD)
Other:
- moved on the sheet: D106, D107, R598, U13

Commit message: VBUS絶縁回路追加
Parts:
- removed U13: MCP6001T-E/OT, ProjectEV:Package_SOT-23-5_MCP6001, symbol ProjectEV:Opamp_MCP6001T-x/OT
- added C351, C352: 0.1u, Capacitor_SMD:C_0603_1608Metric, symbol Device:C
- added C353, C354: 10u, Capacitor_SMD:C_1206_3216Metric, symbol Device:C
- added R619: 0, Resistor_SMD:R_0603_1608Metric, symbol Device:R
- added R620: 100k, Resistor_SMD:R_0603_1608Metric, symbol Device:R
- added U18: UCC12040, ProjectEV:Package_SOIC-16W_7.5x10.3mm_P1.27mm_UCC12040, symbol ProjectEV:Regulator_UCC12040
Connections:
- net VBUS1: now also C352.2, C353.1, R620.1, U18.1 (EN), U18.3 (VINP)
- net VBUS2: now also C351.2, C354.1, R619.1, U18.14 (VISO)
- new net: R619.2, U18.13 (SEL)
- new net: R620.2, U18.5 (SYNC_OK)
- new net VBUS1_GND: C352.1, C353.2, U18.2 (GNDP), U18.4 (SYNC), U18.6 (NC), U18.7 (NC), U18.8 (NC)
- new net VBUS2_GND: C351.1, C354.2, U18.10 (NC), U18.11 (NC), U18.12 (NC), U18.15 (GNDS), U18.16 (GNDS), U18.9 (GNDS)

Commit message: 電源回路完成
入力保護、降圧レギュレータ、VBUS絶縁など
Parts:
- added D115, D116: LED, LED_SMD:LED_0603_1608Metric, symbol Device:LED
- added Q112: BSS308PE, ProjectEV:Package_SOT-23_BSS308PE, symbol ProjectEV:Transistor_BSS308PE
- added Q113: 2N7002K-AU, ProjectEV:Package_SOT-23_2N7002K-AU, symbol ProjectEV:Transistor_2N7002K-AU
- added R621, R622: 5.1k, Resistor_SMD:R_0603_1608Metric, symbol Device:R
- added R623: 1M, Resistor_SMD:R_0603_1608Metric, symbol Device:R
- added R624: 100, Resistor_SMD:R_0603_1608Metric, symbol Device:R
- R618: value 15k -> 100k
Connections:
- net VBUS2_GND is gone; now on net PWRIN-: C351.1, C354.2, U18.10 (NC), U18.11 (NC), U18.12 (NC), U18.15 (GNDS), U18.16 (GNDS), U18.9 (GNDS)
- net PG: now also Q112.1 (G)
- net PWRIN-: now also D115.1 (K), Q113.2 (S), R623.2
- net PWROUT+: now also Q106.1 (S), Q106.2 (S), Q106.3 (S); no longer Q106.5 (D)
- net VOUT+: now also Q112.2 (S), R622.1
- net at C337.1, C342.1, C347.2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: now also Q106.5 (D); no longer Q106.1 (S), Q106.2 (S), Q106.3 (S)
- net at L9.1, U14.12 (SW): now also C334.1; no longer C334.2
- net at U14.4 (BOOT): now also C334.2; no longer C334.1
- net VBUS1 renamed VBUS1+
- net VBUS1_GND renamed VBUS1-
- net VBUS2 renamed VBUS2+
- net VBUS2+: now also Q112.3 (D), R621.1, R624.1
- new net: D115.2 (A), R621.2
- new net: Q113.1 (G), R623.1, R624.2
- new net: D116.2 (A), R622.2
- new net: D116.1 (K), Q113.3 (D)
Other:
- moved on the sheet: C331, C332, C333, C335, C336, C344, C345, C346, C347, C348, C349, C350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

Commit message: アノテーションし直し
Parts:
- renumbered C353 to C345, C352 to C346, C338 to C347, C340 to C348, C339 to C349, C351 to C350, C337 to C351, C341 to C352, C354 to C353, C342 to C354, C343 to C355, C348 to C356, C349 to C357, C331 to C358, C347 to C359, C332 to C360, C333 to C361, C346 to C362, C344 to C363, C345 to C364, C334 to C365, C335 to C366, C336 to C367, C350 to C368, D107 to D123, D106 to D124, D108 to D125, D115 to D126, D114 to D127, D116 to D128, D113 to D129, Q105 to Q109, Q112 to Q110, Q113 to Q112, Q106 to Q113, Q110 to Q114, R598 to R634, R620 to R635, R619 to R636, R621 to R637, R624 to R638, R615 to R639, R617 to R640, R623 to R641, R622 to R642, R612 to R643, R613 to R644, R614 to R645, R618 to R646, R599 to R647, R611 to R648, R609 to R649, R610 to R650, R616 to R651, U15 to U19, U17 to U20, U16 to U21, U14 to U22

Commit message: およそ回路図完成
Parts:
- D123, D124: footprint (none) -> LED_SMD:LED_0603_1608Metric
Changed lines of the file:
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@@
       (effects (font (size 1.27 1.27)) (justify right))
     )
-    (property "Footprint" "" (at 63.5 44.45 0)
+    (property "Footprint" "LED_SMD:LED_0603_1608Metric" (at 63.5 44.45 0)
       (effects (font (size 1.27 1.27)) hide)
     )
@@
       (effects (font (size 1.27 1.27)) (justify left))
     )
-    (property "Footprint" "" (at 50.8 44.45 0)
-      (effects (font (size 1.27 1.27)) hide)
-    )
+    (property "Footprint" "LED_SMD:LED_0603_1608Metric" (at 50.8 44.45 0)
+      (effects (font (size 1.27 1.27)) hide)
+    )

Commit message: 設定値記載
Parts:
- U22: value LMR33620APCQRNXRQ1 -> LMR33630APCQRNXRQ1
Other:
- note added: "5V, 3A"
- note added: "I_{DSTH} = 3.2 A"
- note added: "V_{INMAX} = 30.1 V V_{INMIN} = 9.7 V"
Changed lines of the file:
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@@
     (stroke (width 0) (type default))
+  )
+  (text "V_{INMAX} = 30.1 V\nV_{INMIN} = 9.7 V" (at 196.85 35.56 0)
+    (effects (font (size 1.27 1.27)) (justify left bottom))
+  )
+  (text "I_{DSTH} = 3.2 A" (at 220.98 35.56 0)
+    (effects (font (size 1.27 1.27)) (justify left bottom))
+  )
+  (text "5V, 3A " (at 314.96 124.46 0)
+    (effects (font (size 1.27 1.27)) (justify left bottom))
   )
   (global_label "~{DCDC_EN}" (shape output) (at 175.26 76.2 180) (fields_autoplaced)
@@
       (effects (font (size 1.27 1.27)))
     )
-    (property "Value" "LMR33620APCQRNXRQ1" (at 266.7 121.92 0)
-      (effects (font (size 1.27 1.27)))
-    )
+    (property "Value" "LMR33630APCQRNXRQ1" (at 266.7 121.92 0)
+      (effects (font (size 1.27 1.27)))
+    )

Commit message: アノテーションし直し
Parts:
- renumbered C345 to C343, C346 to C344, C347 to C345, C348 to C346, C349 to C347, C350 to C348, C351 to C349, C352 to C350, C353 to C351, C354 to C352, C355 to C353, C356 to C354, C357 to C355, C358 to C356, C359 to C357, C360 to C358, C361 to C359, C362 to C360, C363 to C361, C364 to C362, C365 to C363, C366 to C364, C367 to C365, C368 to C366, D123 to D203, D124 to D204, D125 to D205, D126 to D206, D127 to D207, D128 to D208, D129 to D209, L9 to L25, R634 to R630, R635 to R631, R636 to R632, R637 to R633, R638 to R634, R639 to R635, R640 to R636, R641 to R637, R642 to R638, R643 to R639, R644 to R640, R645 to R641, R646 to R642, R647 to R643, R648 to R644, R649 to R645, R650 to R646, R651 to R647

Commit message: ERC実行、修正
ラベル修正、未配線部分修正、PWR_FLAG追加
Changed lines of the file:
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@@
     )
   )
-  (symbol (lib_id "ProjectEV:Transistor_2N7002K-AU") (at 175.26 158.75 0) (unit 1)
+  (symbol (lib_name "Transistor_2N7002K-AU_1") (lib_id "ProjectEV:Transistor_2N7002K-AU") (at 175.26 158.75 0) (unit 1)
     (in_bom yes) (on_board yes) (dnp no)
     (property "Reference" "Q111" (at 170.18 152.4 0)
@@
     )
   )
+  (symbol (lib_id "power:PWR_FLAG") (at 279.4 38.1 0) (unit 1)
+    (in_bom yes) (on_board yes) (dnp no) (fields_autoplaced)
+    (property "Reference" "#FLG022" (at 279.4 36.195 0)
+      (effects (font (size 1.27 1.27)) hide)
+    )
+    (property "Value" "PWR_FLAG" (at 279.4 33.02 0)
+      (effects (font (size 1.27 1.27)))
+    )
+    (property "Footprint" "" (at 279.4 38.1 0)
+      (effects (font (size 1.27 1.27)) hide)
+    )
+    (property "Datasheet" "~" (at 279.4 38.1 0)
+      (effects (font (size 1.27 1.27)) hide)
+    )
+    (pin "1")
+    (instances
+      (project "AMS-board-2024"
+        (path "/3a719eb3-09ce-4343-8f6e-20cc0aaf5261/e5bb215a-09a7-47e9-9b6f-2807241074ff"
+          (reference "#FLG022") (unit 1)
+        )
+      )
+    )
+  )
   (symbol (lib_id "ProjectEV:Transistor_BSS308PE") (at 171.45 218.44 90) (unit 1)
     (in_bom yes) (on_board yes) (dnp no) (fields_autoplaced)
@@
     )
   )
-  (symbol (lib_id "ProjectEV:Transistor_2N7002K-AU") (at 340.36 158.75 0) (unit 1)
+  (symbol (lib_name "Transistor_2N7002K-AU_2") (lib_id "ProjectEV:Transistor_2N7002K-AU") (at 340.36 158.75 0) (unit 1)
     (in_bom yes) (on_board yes) (dnp no) (fields_autoplaced)
     (property "Reference" "Q114" (at 346.71 157.48 0)
@@
       (effects (font (size 1.27 1.27) italic) (justify left) hide)
     )
-    (property "Datasheet" "chrome-extension://efaidnbmnnnibpcajpcglclefindmkaj/https://www.panjit.com.tw/upload/datasheet/2N7002K-AU.pdf" (at 345.44 162.56 0)
+    (property "Datasheet" "https://www.panjit.com.tw/upload/datasheet/2N7002K-AU.pdf" (at 345.44 162.56 0)
       (effects (font (size 1.27 1.27)) (justify left) hide)
     )
@@
         (path "/3a719eb3-09ce-4343-8f6e-20cc0aaf5261/e5bb215a-09a7-47e9-9b6f-2807241074ff"
           (reference "C356") (unit 1)
+        )
+      )
+    )
+  )
+  (symbol (lib_id "power:PWR_FLAG") (at 152.4 38.1 0) (unit 1)
+    (in_bom yes) (on_board yes) (dnp no) (fields_autoplaced)
+    (property "Reference" "#FLG021" (at 152.4 36.195 0)
+      (effects (font (size 1.27 1.27)) hide)
+    )
+    (property "Value" "PWR_FLAG" (at 152.4 33.02 0)
+      (effects (font (size 1.27 1.27)))
+    )
+    (property "Footprint" "" (at 152.4 38.1 0)
+      (effects (font (size 1.27 1.27)) hide)
+    )
+    (property "Datasheet" "~" (at 152.4 38.1 0)
+      (effects (font (size 1.27 1.27)) hide)
+    )
+    (pin "1")
+    (instances
+      (project "AMS-board-2024"
+        (path "/3a719eb3-09ce-4343-8f6e-20cc0aaf5261/e5bb215a-09a7-47e9-9b6f-2807241074ff"
+          (reference "#FLG021") (unit 1)
         )
       )
@@
       (effects (font (size 1.27 1.27) italic) (justify left) hide)
     )
-    (property "Datasheet" "chrome-extension://efaidnbmnnnibpcajpcglclefindmkaj/https://www.panjit.com.tw/upload/datasheet/2N7002K-AU.pdf" (at 193.04 251.46 0)
+    (property "Datasheet" "https://www.panjit.com.tw/upload/datasheet/2N7002K-AU.pdf" (at 193.04 251.46 0)
       (effects (font (size 1.27 1.27)) (justify left) hide)
     )
