File: AMS-board-2024/power.kicad_sch (KiCad schematic)
At the start: 65 parts, among them Q109 DMT6007LFGQ, Q110 BSS308PE, Q111 2N7002K-AU, Q112 2N7002K-AU, Q113 DMT6007LFGQ, Q114 2N7002K-AU, U18 UCC12040, U19 AP74700QW6-7, U20 VOMA617A, U21 LM5060, U22 LMR33630APCQRNXRQ1

Commit message: チップ抵抗、チップコンデンササイズ修正
Parts:
- C346, C349, C350, C359, C360, C361, C362, C365, C366: footprint Capacitor_SMD:C_0603_1608Metric -> Capacitor_SMD:C_0402_1005Metric
- C367, C368: footprint Capacitor_SMD:C_0805_2012Metric -> Capacitor_SMD:C_1206_3216Metric
- R634, R636, R637, R638, R639, R640, R641, R643, R644, R645, R646, R647, R648, R649, R650, R651, R652, R653: footprint Resistor_SMD:R_0603_1608Metric -> Resistor_SMD:R_0402_1005Metric
Changed lines of the file:
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@@
       (effects (font (size 1.27 1.27)) (justify left))
     )
-    (property "Footprint" "Resistor_SMD:R_0603_1608Metric" (at 292.862 146.05 90)
+    (property "Footprint" "Resistor_SMD:R_0402_1005Metric" (at 292.862 146.05 90)
       (effects (font (size 1.27 1.27)) hide)
     )
@@
       (effects (font (size 1.27 1.27)) (justify right))
     )
-    (property "Footprint" "Resistor_SMD:R_0603_1608Metric" (at 173.228 228.6 90)
+    (property "Footprint" "Resistor_SMD:R_0402_1005Metric" (at 173.228 228.6 90)
       (effects (font (size 1.27 1.27)) hide)
     )
@@
       (effects (font (size 1.27 1.27)) (justify left))
     )
-    (property "Footprint" "Resistor_SMD:R_0603_1608Metric" (at 239.522 44.45 90)
+    (property "Footprint" "Resistor_SMD:R_0402_1005Metric" (at 239.522 44.45 90)
       (effects (font (size 1.27 1.27)) hide)
     )
@@
       (effects (font (size 1.27 1.27)) (justify left))
     )
-    (property "Footprint" "Capacitor_SMD:C_0603_1608Metric" (at 267.6652 78.74 0)
+    (property "Footprint" "Capacitor_SMD:C_0402_1005Metric" (at 267.6652 78.74 0)
       (effects (font (size 1.27 1.27)) hide)
     )
@@
       (effects (font (size 1.27 1.27)) (justify left))
     )
-    (property "Footprint" "Capacitor_SMD:C_0805_2012Metric" (at 318.4652 137.16 0)
+    (property "Footprint" "Capacitor_SMD:C_1206_3216Metric" (at 318.4652 137.16 0)
       (effects (font (size 1.27 1.27)) hide)
     )
@@
       (effects (font (size 1.27 1.27)) (justify left))
     )
-    (property "Footprint" "Resistor_SMD:R_0603_1608Metric" (at 201.422 171.45 90)
+    (property "Footprint" "Resistor_SMD:R_0402_1005Metric" (at 201.422 171.45 90)
       (effects (font (size 1.27 1.27)) hide)
     )
@@
       (effects (font (size 1.27 1.27)) (justify left))
     )
-    (property "Footprint" "Capacitor_SMD:C_0805_2012Metric" (at 331.1652 137.16 0)
+    (property "Footprint" "Capacitor_SMD:C_1206_3216Metric" (at 331.1652 137.16 0)
       (effects (font (size 1.27 1.27)) hide)
     )
@@
       (effects (font (size 1.27 1.27)) (justify left))
     )
-    (property "Footprint" "Resistor_SMD:R_0603_1608Metric" (at 188.722 69.85 90)
+    (property "Footprint" "Resistor_SMD:R_0402_1005Metric" (at 188.722 69.85 90)
       (effects (font (size 1.27 1.27)) hide)
     )
@@
       (effects (font (size 1.27 1.27)) (justify left))
     )
-    (property "Footprint" "Resistor_SMD:R_0603_1608Metric" (at 176.022 146.05 90)
+    (property "Footprint" "Resistor_SMD:R_0402_1005Metric" (at 176.022 146.05 90)
       (effects (font (size 1.27 1.27)) hide)
     )
@@
       (effects (font (size 1.27 1.27)))
     )
-    (property "Footprint" "Resistor_SMD:R_0603_1608Metric" (at 328.93 160.528 90)
+    (property "Footprint" "Resistor_SMD:R_0402_1005Metric" (at 328.93 160.528 90)
       (effects (font (size 1.27 1.27)) hide)
     )
@@
       (effects (font (size 1.27 1.27)) (justify left))
     )
-    (property "Footprint" "Resistor_SMD:R_0603_1608Metric" (at 214.122 57.15 90)
+    (property "Footprint" "Resistor_SMD:R_0402_1005Metric" (at 214.122 57.15 90)
       (effects (font (size 1.27 1.27)) hide)
     )
@@
       (effects (font (size 1.27 1.27)))
     )
-    (property "Footprint" "Resistor_SMD:R_0603_1608Metric" (at 171.45 249.428 90)
+    (property "Footprint" "Resistor_SMD:R_0402_1005Metric" (at 171.45 249.428 90)
       (effects (font (size 1.27 1.27)) hide)
     )
@@
       (effects (font (size 1.27 1.27)) (justify left))
     )
-    (property "Footprint" "Capacitor_SMD:C_0603_1608Metric" (at 305.7652 137.16 0)
+    (property "Footprint" "Capacitor_SMD:C_0402_1005Metric" (at 305.7652 137.16 0)
       (effects (font (size 1.27 1.27)) hide)
     )
@@
       (effects (font (size 1.27 1.27)) (justify right))
     )
-    (property "Footprint" "Capacitor_SMD:C_0603_1608Metric" (at 62.5348 218.44 0)
+    (property "Footprint" "Capacitor_SMD:C_0402_1005Metric" (at 62.5348 218.44 0)
       (effects (font (size 1.27 1.27)) hide)
     )
@@
       (effects (font (size 1.27 1.27)) (justify left))
     )
-    (property "Footprint" "Capacitor_SMD:C_0603_1608Metric" (at 110.1852 66.04 0)
+    (property "Footprint" "Capacitor_SMD:C_0402_1005Metric" (at 110.1852 66.04 0)
       (effects (font (size 1.27 1.27)) hide)
     )
@@
       (effects (font (size 1.27 1.27)))
     )
-    (property "Footprint" "Resistor_SMD:R_0603_1608Metric" (at 158.75 160.528 90)
+    (property "Footprint" "Resistor_SMD:R_0402_1005Metric" (at 158.75 160.528 90)
       (effects (font (size 1.27 1.27)) hide)
     )
@@
       (effects (font (size 1.27 1.27)) (justify left))
     )
-    (property "Footprint" "Capacitor_SMD:C_0603_1608Metric" (at 282.9052 134.62 0)
+    (property "Footprint" "Capacitor_SMD:C_0402_1005Metric" (at 282.9052 134.62 0)
       (effects (font (size 1.27 1.27)) hide)
     )
@@
       (effects (font (size 1.27 1.27)) (justify left))
     )
-    (property "Footprint" "Resistor_SMD:R_0603_1608Metric" (at 188.722 222.25 90)
+    (property "Footprint" "Resistor_SMD:R_0402_1005Metric" (at 188.722 222.25 90)
       (effects (font (size 1.27 1.27)) hide)
     )
@@
       (effects (font (size 1.27 1.27)) (justify left))
     )
-    (property "Footprint" "Resistor_SMD:R_0603_1608Metric" (at 150.622 222.25 90)
+    (property "Footprint" "Resistor_SMD:R_0402_1005Metric" (at 150.622 222.25 90)
       (effects (font (size 1.27 1.27)) hide)
     )
@@
       (effects (font (size 1.27 1.27)) (justify left))
     )
-    (property "Footprint" "Resistor_SMD:R_0603_1608Metric" (at 292.862 133.35 90)
+    (property "Footprint" "Resistor_SMD:R_0402_1005Metric" (at 292.862 133.35 90)
       (effects (font (size 1.27 1.27)) hide)
     )
@@
       (effects (font (size 1.27 1.27)) (justify right))
     )
-    (property "Footprint" "Capacitor_SMD:C_0603_1608Metric" (at 126.0348 218.44 0)
+    (property "Footprint" "Capacitor_SMD:C_0402_1005Metric" (at 126.0348 218.44 0)
       (effects (font (size 1.27 1.27)) hide)
     )
@@
       (effects (font (size 1.27 1.27)) (justify left))
     )
-    (property "Footprint" "Resistor_SMD:R_0603_1608Metric" (at 214.122 69.85 90)
+    (property "Footprint" "Resistor_SMD:R_0402_1005Metric" (at 214.122 69.85 90)
       (effects (font (size 1.27 1.27)) hide)
     )
@@
       (effects (font (size 1.27 1.27)) (justify left))
     )
-    (property "Footprint" "Capacitor_SMD:C_0603_1608Metric" (at 229.5652 137.16 0)
+    (property "Footprint" "Capacitor_SMD:C_0402_1005Metric" (at 229.5652 137.16 0)
       (effects (font (size 1.27 1.27)) hide)
     )
@@
       (effects (font (size 1.27 1.27)) (justify left))
     )
-    (property "Footprint" "Resistor_SMD:R_0603_1608Metric" (at 341.122 133.35 90)
+    (property "Footprint" "Resistor_SMD:R_0402_1005Metric" (at 341.122 133.35 90)
       (effects (font (size 1.27 1.27)) hide)
     )
@@
       (effects (font (size 1.27 1.27)) (justify left))
     )
-    (property "Footprint" "Capacitor_SMD:C_0603_1608Metric" (at 252.4252 149.86 0)
+    (property "Footprint" "Capacitor_SMD:C_0402_1005Metric" (at 252.4252 149.86 0)
       (effects (font (size 1.27 1.27)) hide)
     )
@@
       (effects (font (size 1.27 1.27)))
     )
-    (property "Footprint" "Capacitor_SMD:C_0603_1608Metric" (at 237.49 59.9948 0)
+    (property "Footprint" "Capacitor_SMD:C_0402_1005Metric" (at 237.49 59.9948 0)
       (effects (font (size 1.27 1.27)) hide)
     )
@@
       (effects (font (size 1.27 1.27)) (justify left))
     )
-    (property "Footprint" "Resistor_SMD:R_0603_1608Metric" (at 74.422 222.25 90)
+    (property "Footprint" "Resistor_SMD:R_0402_1005Metric" (at 74.422 222.25 90)
       (effects (font (size 1.27 1.27)) hide)
     )
@@
       (effects (font (size 1.27 1.27)))
     )
-    (property "Footprint" "Resistor_SMD:R_0603_1608Metric" (at 246.38 141.478 90)
+    (property "Footprint" "Resistor_SMD:R_0402_1005Metric" (at 246.38 141.478 90)
       (effects (font (size 1.27 1.27)) hide)
     )
@@
       (effects (font (size 1.27 1.27)) (justify left))
     )
-    (property "Footprint" "Resistor_SMD:R_0603_1608Metric" (at 214.122 44.45 90)
-      (effects (font (size 1.27 1.27)) hide)
-    )
+    (property "Footprint" "Resistor_SMD:R_0402_1005Metric" (at 214.122 44.45 90)
+      (effects (font (size 1.27 1.27)) hide)
+    )

Commit message: アノテーションし直し、
Parts:
- renumbered C345 to C329, C346 to C330, C347 to C331, C348 to C332, C349 to C333, C350 to C334, C353 to C335, C351 to C336, C352 to C337, C354 to C338, C355 to C339, C356 to C340, C357 to C341, C358 to C342, C360 to C343, C359 to C344, C361 to C345, C362 to C346, C363 to C347, C365 to C348, C364 to C349, C366 to C350, C367 to C351, C368 to C352, D203 to D171, D204 to D172, D205 to D173, D206 to D174, D207 to D175, D208 to D176, D209 to D177, R633 to R601, R634 to R602, R635 to R603, R636 to R604, R637 to R605, R638 to R606, R639 to R607, R641 to R608, R642 to R609, R640 to R610, R643 to R611, R647 to R612, R644 to R613, R645 to R614, R646 to R615, R648 to R616, R649 to R617, R650 to R618, R651 to R619, R652 to R620, R653 to R621
