File: AMS-board-2024/power.kicad_sch (KiCad schematic)
At the start: 65 parts, among them Q109 DMT6007LFGQ, Q110 BSS308PE, Q111 2N7002K-AU, Q112 2N7002K-AU, Q113 DMT6007LFGQ, Q114 2N7002K-AU, U18 UCC12040, U19 AP74700QW6-7, U20 VOMA617A, U21 LM5060, U22 LMR33630APCQRNXRQ1

Commit message: 絶縁パルストランス数削減
Parts:
- renumbered L28 to L21
Changed lines of the file:
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@@
   (symbol (lib_id "ProjectEV:L_EXLA1V06") (at 288.29 127 90) (unit 1)
     (in_bom yes) (on_board yes) (dnp no)
-    (property "Reference" "L28" (at 288.29 121.92 90)
+    (property "Reference" "L21" (at 288.29 121.92 90)
       (effects (font (size 1.27 1.27)))
     )
@@
       (project "AMS-board-2024"
         (path "/3a719eb3-09ce-4343-8f6e-20cc0aaf5261/e5bb215a-09a7-47e9-9b6f-2807241074ff"
-          (reference "L28") (unit 1)
+          (reference "L21") (unit 1)
         )
       )

Commit message: LEDの配線修正
Connections:
- net PWRIN-: now also D171.2 (A), D172.1 (K); no longer R601.2
- net at C331.1, C333.1, D173.2 (A2)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: now also R601.1; no longer D171.1 (K), D172.2 (A)
- new net: D171.1 (K), D172.2 (A), R601.2
Other:
- moved on the sheet: D171, D172, R601

Commit message: DCDC入力コンデンサ追加
Parts:
- added C380: 22u, Capacitor_SMD:C_1206_3216Metric, symbol Device:C
- added C381: 0.1u, Capacitor_SMD:C_0402_1005Metric, symbol Device:C
Connections:
- net PWRIN-: now also C380.2, C381.2
- net PWROUT+: now also C380.1, C381.1
- net at C348.1, L21.1, U22.12 (SW): now also U22.3 (NC)
Other:
- moved on the sheet: C341, C342, C343, D175, Q111, R605, R608, R612, U20

Commit message: DCDC ENABLE周辺回路修正
Parts:
- removed R612: 100k, Resistor_SMD:R_0402_1005Metric, symbol Device:R
- removed U20: VOMA617A, ProjectEV:Package_SOP-4_4.57x4.92mm_P2.54mm_VOMA617A, symbol ProjectEV:Isolator_VOMA617A
- R608: value 2.2k -> 10k
Connections:
- net S11_DCDC_EN: now also Q111.3 (D), R608.2
Other:
- moved on the sheet: D175, Q111, R605, R608

Commit message: 抵抗修正
3.3k -> 3k (1608)
15k -> 100k (1005, プルアップ/ダウン), 5.1k (1005, LED用)
Parts:
- R601: value 15k -> 5.1k; footprint Resistor_SMD:R_0603_1608Metric -> Resistor_SMD:R_0402_1005Metric
- R608: value 10k -> 100k
Changed lines of the file:
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@@
       (effects (font (size 1.27 1.27)) (justify left))
     )
-    (property "Value" "10k" (at 167.64 147.32 0)
+    (property "Value" "100k" (at 167.64 147.32 0)
       (effects (font (size 1.27 1.27)) (justify left))
     )
@@
       (effects (font (size 1.27 1.27)) (justify left))
     )
-    (property "Value" "15k" (at 66.04 45.72 0)
-      (effects (font (size 1.27 1.27)) (justify left))
-    )
-    (property "Footprint" "Resistor_SMD:R_0603_1608Metric" (at 61.722 44.45 90)
-      (effects (font (size 1.27 1.27)) hide)
-    )
+    (property "Value" "5.1k" (at 66.04 45.72 0)
+      (effects (font (size 1.27 1.27)) (justify left))
+    )
+    (property "Footprint" "Resistor_SMD:R_0402_1005Metric" (at 61.722 44.45 90)
+      (effects (font (size 1.27 1.27)) hide)
+    )

Commit message: アノテーションし直し
Parts:
- renumbered C329 to C338, C330 to C339, C331 to C340, C332 to C341, C333 to C342, C334 to C343, C335 to C344, C336 to C345, C337 to C346, C338 to C347, C339 to C348, C380 to C349, C341 to C350, C340 to C351, C342 to C352, C343 to C353, C381 to C354, C344 to C355, C345 to C356, C346 to C357, C347 to C358, C348 to C359, C349 to C360, C350 to C361, C351 to C362, C352 to C363, D175 to D174, D174 to D175, L21 to L17, Q111 to Q110, Q110 to Q111, R605 to R604, R604 to R605, R608 to R606, R606 to R607, R607 to R608, R613 to R612, R614 to R613, R615 to R614, R616 to R615, R617 to R616, R618 to R617, R619 to R618, R620 to R619, R621 to R620, U21 to U20, U22 to U21
