File: AMS-board-2024/battery-stack-monitor.kicad_sch (KiCad schematic)
At the start: 8 parts, among them U23 LM25180-Q1, U24 LTC2949

Commit message: 絶縁電源作成
Parts:
- added C370: C, symbol Device:C
- added L28: YA8779-BLD, ProjectEV:Transformer_YA8779-BLD, symbol ProjectEV:Transformer_YA8779
- added R652, R653, R654, R655: R, symbol Device:R
Connections:
- net at U23.1 (SW): now also D210.2 (A), L28.4, R652.1
- net at U23.2 (FB): now also R652.2
- net VIN+: now reaches U23.3 (VIN)
- net VIN+: now also C368.1, D211.2 (A), L28.1, R655.1
- net VIN-: now reaches U23.4 (EN/UVLO)
- net VIN-: now also C368.2, U23.8 (GND), U23.9 (DAP), C370.2, R654.2, R655.2
- net at U23.5 (SS/BIAS): now also C370.1
- net at U23.6 (TC): now also R653.2
- net at U23.7 (RSET): now also R653.1, R654.1
- net at C369.1: now also D212.1 (K), D213.1 (K)
- net GNDA: now reaches C369.2
- net GNDA: now also D213.2 (A), L28.5, L28.6
- net at D211.1 (K): now also D210.1 (K)
- net at D212.2 (A): now also L28.7, L28.8
Other:
- moved on the sheet: C369, D210, D211, D212, D213, U23

Commit message: 電源部分完成
定数チェック必要
Parts:
- added C371: 1000p, Capacitor_SMD:C_0402_1005Metric, symbol Device:C
- added C372: 1u, Capacitor_SMD:C_0603_1608Metric, symbol Device:C
- added D214: LED, LED_SMD:LED_0603_1608Metric, symbol Device:LED
- added Q115: 2N7002K-AU, ProjectEV:Package_SOT-23_2N7002K-AU, symbol ProjectEV:Transistor_2N7002K-AU
- added R656: 2.4M, Resistor_SMD:R_0603_1608Metric, symbol Device:R
- added R657: 750k, Resistor_SMD:R_0603_1608Metric, symbol Device:R
- added R658: 100k, Resistor_SMD:R_0603_1608Metric, symbol Device:R
- added R659, R660: 5.1k, Resistor_SMD:R_0603_1608Metric, symbol Device:R
- added R661: 25.5k, Resistor_SMD:R_0603_1608Metric, symbol Device:R
- added U25: NCV8711BMTW500TBG, ProjectEV:Package_WDFN-6-1EP_2x2mm_P0.5mm_EP0.95x1.65mm_NCV8711BMTW500TBG, symbol ProjectEV:Regulator_NCV8711BMTW500TBG
- C370: value C -> 0.047u; footprint (none) -> Capacitor_SMD:C_0603_1608Metric
- R652: value R -> 150k; footprint (none) -> Resistor_SMD:R_0603_1608Metric
- R653: value R -> 180k; footprint (none) -> Resistor_SMD:R_0603_1608Metric
- R654: value R -> 12.1k; footprint (none) -> Resistor_SMD:R_0603_1608Metric
- R655: value R -> 137k; footprint (none) -> Resistor_SMD:R_0603_1608Metric
Connections:
- net GNDA: now also C372.2, Q115.2 (S), R657.2, U25.3 (GND), U25.7 (EP)
- net VIN-: now also R661.1; no longer C370.2, R654.2, U23.8 (GND), U23.9 (DAP)
- net +7V: now reaches C369.1, D212.1 (K), D213.1 (K)
- net +7V: now also U25.4 (EN), U25.6 (IN)
- new net: C371.2, R656.2, R657.1, U25.2 (ADJ)
- new net: R658.2, R660.1, U25.5 (PG)
- new net: Q115.1 (G), R660.2
- new net: C370.2, R654.2, R661.2, U23.8 (GND), U23.9 (DAP)
- new net: D214.1 (K), Q115.3 (D)
- new net: D214.2 (A), R659.2
- new net +5VD: C371.1, C372.1, R656.1, R658.1, R659.1, U25.1 (OUT)

Commit message: 回路追加、ラベル修正
Parts:
- added C263 (x4), C335: 0.1u, Capacitor_SMD:C_0603_1608Metric, symbol Device:C
- added C306, C310: 10n, Capacitor_SMD:C_0603_1608Metric, symbol Device:C
- added C367 (x7): 1u, Capacitor_SMD:C_0603_1608Metric, symbol Device:C
- added FL15: DLW43SH101XK2, ProjectEV:CommonModeChoke_DLW43SH101, symbol ProjectEV:CommonModeChoke_DLW43SH101
- added H1, H2: MountingHole_Pad, symbol Mechanical:MountingHole_Pad
- added R557, R559: 1k, Resistor_SMD:R_0603_1608Metric, symbol Device:R
- added R560, R561: 60.4, Resistor_SMD:R_0603_1608Metric, symbol Device:R
- added R563, R564: 294, Resistor_SMD:R_0603_1608Metric, symbol Device:R
- added R670: SH8518F600BHEP, ProjectEV:ShuntRegistor_SH8518F600BHEP, symbol ProjectEV:ShuntRegistor_SH8518F600BHEP
- added R671, R672: 5.1k, Resistor_SMD:R_0603_1608Metric, symbol Device:R
- added U15: NV24C16SNVLT3G, ProjectEV:Package_TSOP-5_NV24C16SNVLT3G, symbol ProjectEV:Memory_NV24C16SNVLT3G
Connections:
- net +5VD: now also U24.19 (AVCC), U24.20 (DVCC), C367.1, C367.1
- net GNDA: now also U24.17 (DGND), U24.18 (AGND), U24.26 (IOVCC), U24.49 (EP), C263.1, C263.1, C263.1, C263.1, C306.1, C310.1, C335.2, C367.2, C367.2, C367.2, C367.2, C367.2, R559.1, U15.2 (VSS)
- net at U24.14 (SCL): now also R672.2, U15.1 (SCL)
- net at U24.15 (SDA): now also R671.2, U15.3 (SDA)
- net S12_BYP1: now reaches U24.16 (BYP1)
- net S12_BYP1: now also C335.1, C367.1, R671.1, R672.1, U15.4 (VCC)
- net at U24.25 (BYP2): now also C367.1
- net at U24.27 (SDI(VCMP)): now also R557.1, R559.2
- net at U24.28 (SDO(IBIAS)): now also R557.2
- net at U24.29 (SCK(IP)): now also FL15.4, R560.2
- net at U24.30 (CSB(IM)): now also FL15.1, R561.1
- net at U24.35 (VREF): now also C367.1
- net S12_I_{SENSE}_P: now reaches U24.38 (I2P)
- net S12_I_{SENSE}_P: now also U24.45 (I1P), R670.3
- net at U24.39 (CF2P): now also C263.2, C367.2
- net at U24.40 (CF2M): now also C263.2, C367.1
- net S12_I_{SENSE}_N: now reaches U24.41 (I2M)
- net S12_I_{SENSE}_N: now also U24.42 (I1M), R670.4
- net at U24.43 (CF1M): now also C263.2, C367.1
- net at U24.44 (CF1P): now also C263.2, C367.2
- net +7V renamed S12_+7V
- new net: C310.2, R563.1, R564.2
- new net: C306.2, R560.1, R561.2
- new net S12_Shunt_N: H2.1, R670.2
- new net S12_Shunt_P: H1.1, R670.1
- new net isoSPI_N: FL15.2, R564.1
- new net isoSPI_P: FL15.3, R563.2
- no-connect marks 0 -> 1
Other:
- moved on the sheet: U24

Commit message: Battery Stack Monitor完成
チェック未済
Parts:
- added C388, C389, C390: 0.1u, Capacitor_SMD:C_0603_1608Metric, symbol Device:C
- added Q116, Q117, Q118: STD7ANM60N, ProjectEV:Package_TO-252_STD7ANM60N, symbol ProjectEV:Transistor_STD7ANM60N
- added R673, R675, R678: 2M, Resistor_SMD:R_0603_1608Metric, symbol Device:R
- added R674, R676, R677: 20k, Resistor_SMD:R_0603_1608Metric, symbol Device:R
- added R679: 10k, Resistor_SMD:R_0603_1608Metric, symbol Device:R
- added R680: TMP6131QDYARQ1, ProjectEV:Package_SOD-523_TMP6131QDYARQ1, symbol ProjectEV:Sensor_TMP6131QDYARQ1
- renumbered C306 to C374, C310 to C375, C367 to C376, C367 to C377, C367 to C378, C367 to C379, C367 to C380, C367 to C381, C367 to C382, C263 to C383, C263 to C384, C263 to C385, C263 to C386, C335 to C387, FL15 to FL18, R557 to R664, R559 to R665, R560 to R666, R561 to R667, R563 to R668, R564 to R669, U15 to U26
Connections:
- net S12_I_{SENSE}_N is gone; now on net GNDA: R670.4, U24.41 (I2M), U24.42 (I1M)
- net GNDA: now also U24.47 (VBATM), C388.2, C389.2, C390.2, R674.2, R676.2, R680.1 (-)
- net at U24.1 (V1): now also R679.1, R680.2 (+)
- net at U24.11 (V10): now also Q117.1 (G)
- net at U24.12 (V11): now also Q118.1 (G)
- net at U24.2 (V2): now also C388.1, Q117.3 (S), R676.1
- net at U24.3 (V3): now also C389.1, Q118.3 (S), R677.2
- net S12_VREF: now reaches C380.1, U24.35 (VREF)
- net S12_VREF: now also R677.1, R679.2
- net S12_VBATP: now reaches U24.48 (VBATP)
- net S12_VBATP: now also C390.1, Q116.3 (S), R674.1
- net at U24.9 (V8): now also Q116.1 (G)
- net isoSPI_N renamed I_N
- net isoSPI_P renamed I_P
- new net: Q118.2 (D), R678.2
- new net: Q117.2 (D), R675.1
- new net: Q116.2 (D), R673.1
- new net V_{BAT}+: R673.2
- new net V_{LOAD}+: R675.2
- new net V_{LOAD}-: R678.1
- no-connect marks 1 -> 6
Other:
- note added: "Low Side Current Sensing"
- note added: "S12_I_{SENSE}_N"
- moved on the sheet: C374, C375, C376, C377, C378, C379, C380, C381, C382, C383, C384, C385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

Commit message: 追加回路
電源電圧変更、水晶振動子追加
Parts:
- removed D212: SS3040HE-AU_R1_000A1, ProjectEV:D_SOD-123HE_SS3040HE, symbol ProjectEV:D_SS3040HE
- removed D213: HPZR-C7V6-QX, ProjectEV:D_SOD-123W_HPZR-Cxxx-QX, symbol ProjectEV:D_HPZR-C7V6-QX
- removed H1, H2: MountingHole_Pad, symbol Mechanical:MountingHole_Pad
- removed L28: YA8779-BLD, ProjectEV:Transformer_YA8779-BLD, symbol ProjectEV:Transformer_YA8779
- added C391: 0.1u, Capacitor_SMD:C_0603_1608Metric, symbol Device:C
- added C392, C393: 18p, Capacitor_SMD:C_0402_1005Metric, symbol Device:C
- added D212: DFLS1100Q-7, ProjectEV:D_PowerDI-123_DFLS1100, symbol ProjectEV:D_DFLS1100
- added D213: BZT52H-C16, ProjectEV:D_SOD-123F_BZT52H-xxx, symbol ProjectEV:D_BZT52H-C16
- added L28: YA8916-BLD, ProjectEV:Transformer_YA8916-BLD, symbol ProjectEV:Transformer_YA8916
- added Y2: ABLS-4.000MHZ-K4T, ProjectEV:Crystal_ABLS, symbol ProjectEV:Crystal_ABLS-4.000MHZ-K4T
- C369: value 100u -> 22u
- C372: value 1u -> 10u
- R657: value 750k -> 267k
Connections:
- net GNDA: now also C391.2, C392.1, C393.1, D213.2 (A), L28.7
- net VIN+: now also L28.1
- net at U24.33 (CLKI): now also C392.2, Y2.1
- net at U24.34 (CLKO): now also C393.2, Y2.2
- net at D210.2 (A), R652.1, U23.1 (SW): now also L28.4
- net +5VD renamed +12VA
- net +12VA: now also C391.1
- net S12_+7V renamed S12_+15V
- net S12_+15V: now also D212.1 (K), D213.1 (K)
- net S12_Shunt_N renamed Shunt_N
- net S12_Shunt_P renamed Shunt_P
- new net: D212.2 (A), L28.8
- now unconnected: U24.21 (DNC), U24.22 (DNC), U24.23 (DNC), U24.24 (DNC), U24.31 (DNC), U24.32 (DNC), U24.36 (DNC), U24.37 (DNC), U24.46 (DNC), U24.6 (DNC)
- no-connect marks 6 -> 9
Other:
- note added: "MAX 0.2 A"
- moved on the sheet: C372, D214, Q115, R658, R659, R660

Commit message: アノテーションし直し
Parts:
- renumbered C368 to C369, C390 to C371, C393 to C372, C392 to C373, C377 to C374, C376 to C375, C379 to C376, C378 to C377, C380 to C378, C369 to C379, C383 to C380, C384 to C382, C385 to C383, C382 to C384, C386 to C385, C389 to C386, C388 to C387, C371 to C388, C374 to C389, C391 to C390, C372 to C391, C375 to C392, C387 to C393, D211 to D210, D210 to D211, L28 to L29, Q118 to Q115, Q117 to Q116, Q115 to Q117, Q116 to Q118, R655 to R654, R661 to R655, R652 to R656, R653 to R657, R654 to R658, R670 to R659, R656 to R660, R657 to R661, R664 to R662, R677 to R663, R678 to R664, R675 to R668, R676 to R669, R658 to R670, R660 to R671, R659 to R672, R668 to R675, R669 to R676, R679 to R677, R680 to R678, R671 to R679, R672 to R680

Commit message: 階層シート内の電源シンボル修正
階層シート内で電源シンボルをなるべく使わないようにする
修正途中
Connections:
- net GNDA renamed V_{BAT}-
Other:
- moved on the sheet: C369, C370, C371, C372, C373, C374, C375, C376, C377, C378, C379, C380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

Commit message: ラベル修正とテキスト等の追加
階層シート内の電源シンボルをまとめて階層ラベルとして上層に出し、上層のシートで電源シンボルに接続
Connections:
- net +12VA renamed S12_+12V
- net V_{BAT}+ renamed V_{ACC}+
- net V_{BAT}- renamed V_{ACC}-
Other:
- note added: "ISOLATION"
- moved on the sheet: Q115, R663, R664
