File: AMS-board-2024/battery-stack-monitor.kicad_sch (KiCad schematic)
At the start: 68 parts, among them Q115 STD7ANM60N, Q116 STD7ANM60N, Q117 2N7002K-AU, Q118 STD7ANM60N, U23 LM25180-Q1, U24 LTC2949, U25 NCV8711BMTW500TBG, U26 NV24C16SNVLT3G, Y2 ABLS-4.000MHZ-K4T

Commit message: チップ抵抗、チップコンデンササイズ修正
Parts:
- C370, C371, C374, C375, C376, C377, C378, C380, C381, C382, C383, C384, C385, C386, C387, C389, C390, C392, C393: footprint Capacitor_SMD:C_0603_1608Metric -> Capacitor_SMD:C_0402_1005Metric
- R654, R655, R656, R657, R658, R660, R661, R662, R665, R670, R671, R672, R677, R679, R680: footprint Resistor_SMD:R_0603_1608Metric -> Resistor_SMD:R_0402_1005Metric
Changed lines of the file:
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@@
       (effects (font (size 1.27 1.27)))
     )
-    (property "Footprint" "Capacitor_SMD:C_0603_1608Metric" (at 209.55 130.5052 0)
+    (property "Footprint" "Capacitor_SMD:C_0402_1005Metric" (at 209.55 130.5052 0)
       (effects (font (size 1.27 1.27)) hide)
     )
@@
       (effects (font (size 1.27 1.27)))
     )
-    (property "Footprint" "Capacitor_SMD:C_0603_1608Metric" (at 167.64 145.7452 0)
+    (property "Footprint" "Capacitor_SMD:C_0402_1005Metric" (at 167.64 145.7452 0)
       (effects (font (size 1.27 1.27)) hide)
     )
@@
       (effects (font (size 1.27 1.27)))
     )
-    (property "Footprint" "Capacitor_SMD:C_0603_1608Metric" (at 393.7 148.8948 0)
+    (property "Footprint" "Capacitor_SMD:C_0402_1005Metric" (at 393.7 148.8948 0)
       (effects (font (size 1.27 1.27)) hide)
     )
@@
       (effects (font (size 1.27 1.27)) (justify left))
     )
-    (property "Footprint" "Resistor_SMD:R_0603_1608Metric" (at 264.922 57.15 90)
+    (property "Footprint" "Resistor_SMD:R_0402_1005Metric" (at 264.922 57.15 90)
       (effects (font (size 1.27 1.27)) hide)
     )
@@
       (effects (font (size 1.27 1.27)) (justify right))
     )
-    (property "Footprint" "Resistor_SMD:R_0603_1608Metric" (at 357.378 171.45 90)
+    (property "Footprint" "Resistor_SMD:R_0402_1005Metric" (at 357.378 171.45 90)
       (effects (font (size 1.27 1.27)) hide)
     )
@@
       (effects (font (size 1.27 1.27)) (justify left))
     )
-    (property "Footprint" "Capacitor_SMD:C_0603_1608Metric" (at 72.0852 93.98 0)
+    (property "Footprint" "Capacitor_SMD:C_0402_1005Metric" (at 72.0852 93.98 0)
       (effects (font (size 1.27 1.27)) hide)
     )
@@
       (effects (font (size 1.27 1.27)) (justify left))
     )
-    (property "Footprint" "Capacitor_SMD:C_0603_1608Metric" (at 244.8052 177.8 0)
+    (property "Footprint" "Capacitor_SMD:C_0402_1005Metric" (at 244.8052 177.8 0)
       (effects (font (size 1.27 1.27)) hide)
     )
@@
       (effects (font (size 1.27 1.27)) (justify left))
     )
-    (property "Footprint" "Resistor_SMD:R_0603_1608Metric" (at 353.822 151.13 90)
+    (property "Footprint" "Resistor_SMD:R_0402_1005Metric" (at 353.822 151.13 90)
       (effects (font (size 1.27 1.27)) hide)
     )
@@
       (effects (font (size 1.27 1.27)))
     )
-    (property "Footprint" "Capacitor_SMD:C_0603_1608Metric" (at 189.23 130.5052 0)
+    (property "Footprint" "Capacitor_SMD:C_0402_1005Metric" (at 189.23 130.5052 0)
       (effects (font (size 1.27 1.27)) hide)
     )
@@
       (effects (font (size 1.27 1.27)) (justify left))
     )
-    (property "Footprint" "Capacitor_SMD:C_0603_1608Metric" (at 232.1052 180.34 0)
+    (property "Footprint" "Capacitor_SMD:C_0402_1005Metric" (at 232.1052 180.34 0)
       (effects (font (size 1.27 1.27)) hide)
     )
@@
       (effects (font (size 1.27 1.27)) (justify left))
     )
-    (property "Footprint" "Resistor_SMD:R_0603_1608Metric" (at 366.522 151.13 90)
+    (property "Footprint" "Resistor_SMD:R_0402_1005Metric" (at 366.522 151.13 90)
       (effects (font (size 1.27 1.27)) hide)
     )
@@
       (effects (font (size 1.27 1.27)))
     )
-    (property "Footprint" "Capacitor_SMD:C_0603_1608Metric" (at 264.16 126.0348 0)
+    (property "Footprint" "Capacitor_SMD:C_0402_1005Metric" (at 264.16 126.0348 0)
       (effects (font (size 1.27 1.27)) hide)
     )
@@
       (effects (font (size 1.27 1.27)) (justify left))
     )
-    (property "Footprint" "Capacitor_SMD:C_0603_1608Metric" (at 160.9852 184.15 0)
+    (property "Footprint" "Capacitor_SMD:C_0402_1005Metric" (at 160.9852 184.15 0)
       (effects (font (size 1.27 1.27)) hide)
     )
@@
       (effects (font (size 1.27 1.27)) (justify left))
     )
-    (property "Footprint" "Resistor_SMD:R_0603_1608Metric" (at 61.722 82.55 90)
+    (property "Footprint" "Resistor_SMD:R_0402_1005Metric" (at 61.722 82.55 90)
       (effects (font (size 1.27 1.27)) hide)
     )
@@
       (effects (font (size 1.27 1.27)))
     )
-    (property "Footprint" "Capacitor_SMD:C_0603_1608Metric" (at 314.96 126.0348 0)
+    (property "Footprint" "Capacitor_SMD:C_0402_1005Metric" (at 314.96 126.0348 0)
       (effects (font (size 1.27 1.27)) hide)
     )
@@
       (effects (font (size 1.27 1.27)))
     )
-    (property "Footprint" "Capacitor_SMD:C_0603_1608Metric" (at 167.64 160.9852 0)
+    (property "Footprint" "Capacitor_SMD:C_0402_1005Metric" (at 167.64 160.9852 0)
       (effects (font (size 1.27 1.27)) hide)
     )
@@
       (effects (font (size 1.27 1.27)) (justify left))
     )
-    (property "Footprint" "Resistor_SMD:R_0603_1608Metric" (at 61.722 69.85 90)
+    (property "Footprint" "Resistor_SMD:R_0402_1005Metric" (at 61.722 69.85 90)
       (effects (font (size 1.27 1.27)) hide)
     )
@@
       (effects (font (size 1.27 1.27)) (justify left))
     )
-    (property "Footprint" "Resistor_SMD:R_0603_1608Metric" (at 99.822 68.58 90)
+    (property "Footprint" "Resistor_SMD:R_0402_1005Metric" (at 99.822 68.58 90)
       (effects (font (size 1.27 1.27)) hide)
     )
@@
       (effects (font (size 1.27 1.27)) (justify left))
     )
-    (property "Footprint" "Resistor_SMD:R_0603_1608Metric" (at 112.522 83.82 90)
+    (property "Footprint" "Resistor_SMD:R_0402_1005Metric" (at 112.522 83.82 90)
       (effects (font (size 1.27 1.27)) hide)
     )
@@
       (effects (font (size 1.27 1.27)))
     )
-    (property "Footprint" "Capacitor_SMD:C_0603_1608Metric" (at 167.64 140.6652 0)
+    (property "Footprint" "Capacitor_SMD:C_0402_1005Metric" (at 167.64 140.6652 0)
       (effects (font (size 1.27 1.27)) hide)
     )
@@
       (effects (font (size 1.27 1.27)))
     )
-    (property "Footprint" "Resistor_SMD:R_0603_1608Metric" (at 247.65 148.082 90)
+    (property "Footprint" "Resistor_SMD:R_0402_1005Metric" (at 247.65 148.082 90)
       (effects (font (size 1.27 1.27)) hide)
     )
@@
       (effects (font (size 1.27 1.27)) (justify left))
     )
-    (property "Footprint" "Resistor_SMD:R_0603_1608Metric" (at 264.922 44.45 90)
+    (property "Footprint" "Resistor_SMD:R_0402_1005Metric" (at 264.922 44.45 90)
       (effects (font (size 1.27 1.27)) hide)
     )
@@
       (effects (font (size 1.27 1.27)) (justify left))
     )
-    (property "Footprint" "Capacitor_SMD:C_0603_1608Metric" (at 199.0852 121.92 0)
+    (property "Footprint" "Capacitor_SMD:C_0402_1005Metric" (at 199.0852 121.92 0)
       (effects (font (size 1.27 1.27)) hide)
     )
@@
       (effects (font (size 1.27 1.27)))
     )
-    (property "Footprint" "Resistor_SMD:R_0603_1608Metric" (at 260.35 148.082 90)
+    (property "Footprint" "Resistor_SMD:R_0402_1005Metric" (at 260.35 148.082 90)
       (effects (font (size 1.27 1.27)) hide)
     )
@@
       (effects (font (size 1.27 1.27)) (justify left))
     )
-    (property "Footprint" "Capacitor_SMD:C_0603_1608Metric" (at 209.2452 121.92 0)
+    (property "Footprint" "Capacitor_SMD:C_0402_1005Metric" (at 209.2452 121.92 0)
       (effects (font (size 1.27 1.27)) hide)
     )
@@
       (effects (font (size 1.27 1.27)) (justify left))
     )
-    (property "Footprint" "Capacitor_SMD:C_0603_1608Metric" (at 242.2652 48.26 0)
+    (property "Footprint" "Capacitor_SMD:C_0402_1005Metric" (at 242.2652 48.26 0)
       (effects (font (size 1.27 1.27)) hide)
     )
@@
       (effects (font (size 1.27 1.27)) (justify left))
     )
-    (property "Footprint" "Resistor_SMD:R_0603_1608Metric" (at 214.122 44.45 90)
+    (property "Footprint" "Resistor_SMD:R_0402_1005Metric" (at 214.122 44.45 90)
       (effects (font (size 1.27 1.27)) hide)
     )
@@
       (effects (font (size 1.27 1.27)) (justify left))
     )
-    (property "Footprint" "Resistor_SMD:R_0603_1608Metric" (at 99.822 83.82 90)
+    (property "Footprint" "Resistor_SMD:R_0402_1005Metric" (at 99.822 83.82 90)
       (effects (font (size 1.27 1.27)) hide)
     )
@@
       (effects (font (size 1.27 1.27)) (justify left))
     )
-    (property "Footprint" "Resistor_SMD:R_0603_1608Metric" (at 277.622 44.45 90)
+    (property "Footprint" "Resistor_SMD:R_0402_1005Metric" (at 277.622 44.45 90)
       (effects (font (size 1.27 1.27)) hide)
     )
@@
       (effects (font (size 1.27 1.27)) (justify left))
     )
-    (property "Footprint" "Resistor_SMD:R_0603_1608Metric" (at 214.122 57.15 90)
+    (property "Footprint" "Resistor_SMD:R_0402_1005Metric" (at 214.122 57.15 90)
       (effects (font (size 1.27 1.27)) hide)
     )
@@
       (effects (font (size 1.27 1.27)))
     )
-    (property "Footprint" "Capacitor_SMD:C_0603_1608Metric" (at 167.64 176.2252 0)
+    (property "Footprint" "Capacitor_SMD:C_0402_1005Metric" (at 167.64 176.2252 0)
       (effects (font (size 1.27 1.27)) hide)
     )
@@
       (effects (font (size 1.27 1.27)))
     )
-    (property "Footprint" "Capacitor_SMD:C_0603_1608Metric" (at 167.64 168.6052 0)
+    (property "Footprint" "Capacitor_SMD:C_0402_1005Metric" (at 167.64 168.6052 0)
       (effects (font (size 1.27 1.27)) hide)
     )
@@
       (effects (font (size 1.27 1.27)) (justify left))
     )
-    (property "Footprint" "Capacitor_SMD:C_0603_1608Metric" (at 219.4052 121.92 0)
+    (property "Footprint" "Capacitor_SMD:C_0402_1005Metric" (at 219.4052 121.92 0)
       (effects (font (size 1.27 1.27)) hide)
     )
@@
       (effects (font (size 1.27 1.27)) (justify left))
     )
-    (property "Footprint" "Capacitor_SMD:C_0603_1608Metric" (at 188.9252 121.92 0)
-      (effects (font (size 1.27 1.27)) hide)
-    )
+    (property "Footprint" "Capacitor_SMD:C_0402_1005Metric" (at 188.9252 121.92 0)
+      (effects (font (size 1.27 1.27)) hide)
+    )

Commit message: アノテーションし直し、
Parts:
- renumbered C369 to C353, C370 to C354, C379 to C355, C371 to C356, C372 to C357, C373 to C358, C374 to C359, C375 to C360, C376 to C361, C377 to C362, C378 to C363, C380 to C364, C381 to C365, C382 to C366, C383 to C367, C384 to C368, C385 to C369, C388 to C370, C386 to C371, C390 to C372, C387 to C373, C391 to C374, C389 to C375, C392 to C376, C393 to C377, D210 to D178, D211 to D179, D212 to D180, D213 to D181, D214 to D182, Q117 to Q116, Q116 to Q117, R654 to R622, R655 to R623, R656 to R624, R657 to R625, R658 to R626, R659 to R627, R660 to R628, R661 to R629, R662 to R630, R663 to R631, R664 to R632, R665 to R633, R670 to R634, R671 to R635, R666 to R636, R667 to R637, R672 to R638, R668 to R639, R669 to R640, R675 to R641, R676 to R642, R673 to R643, R674 to R644, R679 to R645, R677 to R646, R678 to R647, R680 to R648, U25 to U24, U24 to U25

Commit message: 絶縁パルストランス数削減
Parts:
- renumbered L29 to L22
Changed lines of the file:
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@@
   (symbol (lib_id "ProjectEV:Transformer_YA8916") (at 127 49.53 0) (unit 1)
     (in_bom yes) (on_board yes) (dnp no) (fields_autoplaced)
-    (property "Reference" "L29" (at 127 36.83 0)
+    (property "Reference" "L22" (at 127 36.83 0)
       (effects (font (size 1.27 1.27)))
     )
@@
       (project "AMS-board-2024"
         (path "/3a719eb3-09ce-4343-8f6e-20cc0aaf5261/2a544a11-bc7a-441e-95e4-66a5a426d897"
-          (reference "L29") (unit 1)
+          (reference "L22") (unit 1)
         )
       )

Commit message: フライバックDCDCの配線が間違っていたので修正
Connections:
- net VIN-: now also C354.2, R623.2, R626.2, U23.8 (GND), U23.9 (DAP); no longer R622.2, R623.1, U23.4 (EN/UVLO)
- new net: R622.2, R623.1, U23.4 (EN/UVLO)
Changed lines of the file:
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@@
   (junction (at 218.44 129.54) (diameter 0) (color 0 0 0 0)
   )
-  (junction (at 50.8 76.2) (diameter 0) (color 0 0 0 0)
-  )
   (junction (at 76.2 63.5) (diameter 0) (color 0 0 0 0)
   )
@@
   (junction (at 187.96 129.54) (diameter 0) (color 0 0 0 0)
   )
+  (junction (at 50.8 96.52) (diameter 0) (color 0 0 0 0)
+  )
   (junction (at 317.5 114.3) (diameter 0) (color 0 0 0 0)
   )
@@
   )
   (junction (at 215.9 38.1) (diameter 0) (color 0 0 0 0)
+  )
+  (junction (at 63.5 96.52) (diameter 0) (color 0 0 0 0)
   )
   (junction (at 355.6 160.02) (diameter 0) (color 0 0 0 0)
@@
     (stroke (width 0) (type default))
   )
-  (wire (pts (xy 50.8 76.2) (xy 38.1 76.2))
+  (wire (pts (xy 50.8 96.52) (xy 38.1 96.52))
     (stroke (width 0) (type default))
   )
@@
     (stroke (width 0) (type default))
   )
+  (wire (pts (xy 50.8 96.52) (xy 63.5 96.52))
+    (stroke (width 0) (type default))
+  )
   (wire (pts (xy 215.9 48.26) (xy 215.9 53.34))
     (stroke (width 0) (type default))
@@
     (stroke (width 0) (type default))
   )
-  (wire (pts (xy 50.8 73.66) (xy 50.8 76.2))
-    (stroke (width 0) (type default))
-  )
   (wire (pts (xy 355.6 177.8) (xy 279.4 177.8))
     (stroke (width 0) (type default))
@@
     (stroke (width 0) (type default))
   )
+  (wire (pts (xy 50.8 73.66) (xy 50.8 96.52))
+    (stroke (width 0) (type default))
+  )
   (wire (pts (xy 170.18 88.9) (xy 185.42 88.9))
     (stroke (width 0) (type default))
@@
   )
   (wire (pts (xy 330.2 190.5) (xy 330.2 193.04))
-    (stroke (width 0) (type default))
-  )
-  (wire (pts (xy 50.8 76.2) (xy 63.5 76.2))
     (stroke (width 0) (type default))
   )
@@
     (effects (font (size 1.27 1.27)) (justify left))
   )
-  (hierarchical_label "VIN-" (shape input) (at 38.1 76.2 180) (fields_autoplaced)
+  (hierarchical_label "VIN-" (shape input) (at 38.1 96.52 180) (fields_autoplaced)
     (effects (font (size 1.27 1.27)) (justify right))
   )

Commit message: リニアレギュレータの入力にコンデンサを追加
Parts:
- added C378: 0.1u, Capacitor_SMD:C_0402_1005Metric, symbol Device:C
- added C379: 1u, Capacitor_SMD:C_0402_1005Metric, symbol Device:C
Connections:
- net S12_+15V: now also C378.1, C379.1
- net V_{ACC}-: now also C378.2, C379.2
Other:
- moved on the sheet: C370, C372, C374, D182, Q116, R628, R629, R634, R635, R638, U24

Commit message: 2M Ohmsのチップ抵抗のサイズを3216に変更
Parts:
- R632, R639, R643: footprint Resistor_SMD:R_0603_1608Metric -> Resistor_SMD:R_1206_3216Metric
Changed lines of the file:
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@@
       (effects (font (size 1.27 1.27)) (justify right))
     )
-    (property "Footprint" "Resistor_SMD:R_0603_1608Metric" (at 255.778 222.25 90)
+    (property "Footprint" "Resistor_SMD:R_1206_3216Metric" (at 255.778 222.25 90)
       (effects (font (size 1.27 1.27)) hide)
     )
@@
       (effects (font (size 1.27 1.27)) (justify right))
     )
-    (property "Footprint" "Resistor_SMD:R_0603_1608Metric" (at 293.878 196.85 90)
+    (property "Footprint" "Resistor_SMD:R_1206_3216Metric" (at 293.878 196.85 90)
       (effects (font (size 1.27 1.27)) hide)
     )
@@
       (effects (font (size 1.27 1.27)) (justify right))
     )
-    (property "Footprint" "Resistor_SMD:R_0603_1608Metric" (at 331.978 196.85 90)
-      (effects (font (size 1.27 1.27)) hide)
-    )
+    (property "Footprint" "Resistor_SMD:R_1206_3216Metric" (at 331.978 196.85 90)
+      (effects (font (size 1.27 1.27)) hide)
+    )

Commit message: VACC-とS12_ISENSE_Nを0 Ohmsで接続
Parts:
- added R612: 0, Resistor_SMD:R_0603_1608Metric, symbol Device:R
Connections:
- net V_{ACC}-: now also R612.1; no longer C364.1, C366.1, C367.1, C369.1, R627.4, U25.26 (IOVCC), U25.41 (I2M), U25.42 (I1M)
- new net S12_I_{SENSE}_N: C364.1, C366.1, C367.1, C369.1, R612.2, R627.4, U25.26 (IOVCC), U25.41 (I2M), U25.42 (I1M)
Other:
- note removed: "S12_I_{SENSE}_N"
Changed lines of the file:
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@@
     (stroke (width 0) (type default))
   )
-  (wire (pts (xy 241.3 99.06) (xy 241.3 76.2))
+  (wire (pts (xy 241.3 99.06) (xy 241.3 86.36))
     (stroke (width 0) (type default))
   )
@@
   )
   (wire (pts (xy 368.3 154.94) (xy 368.3 157.48))
+    (stroke (width 0) (type default))
+  )
+  (wire (pts (xy 241.3 78.74) (xy 241.3 76.2))
     (stroke (width 0) (type default))
   )
@@
     (effects (font (size 2.54 2.54)) (justify left bottom))
   )
-  (text "S12_I_{SENSE}_N" (at 208.28 99.06 0)
+  (text "Low Side Current Sensing" (at 180.34 80.01 0)
     (effects (font (size 1.27 1.27)) (justify left bottom))
   )
-  (text "Low Side Current Sensing" (at 180.34 80.01 0)
+  (label "S12_I_{SENSE}_N" (at 208.28 99.06 0) (fields_autoplaced)
     (effects (font (size 1.27 1.27)) (justify left bottom))
   )
@@
         )
       )
+    )
+  )
+  (symbol (lib_id "Device:R") (at 241.3 82.55 0) (unit 1)
+    (in_bom yes) (on_board yes) (dnp no) (fields_autoplaced)
+    (property "Reference" "R612" (at 243.84 81.28 0)
+      (effects (font (size 1.27 1.27)) (justify left))
+    )
+    (property "Value" "0" (at 243.84 83.82 0)
+      (effects (font (size 1.27 1.27)) (justify left))
+    )
+    (property "Footprint" "Resistor_SMD:R_0603_1608Metric" (at 239.522 82.55 90)
+      (effects (font (size 1.27 1.27)) hide)
+    )
+    (property "Datasheet" "~" (at 241.3 82.55 0)
+      (effects (font (size 1.27 1.27)) hide)
+    )
+    (pin "1")
+    (pin "2")
+    (instances
+      (project "AMS-board-2024"
+        (path "/3a719eb3-09ce-4343-8f6e-20cc0aaf5261/2a544a11-bc7a-441e-95e4-66a5a426d897"
+          (reference "R612") (unit 1)
+        )
+      )

Commit message: サーミスタのマイナス側をシャント抵抗に接続
Connections:
- net S12_I_{SENSE}_N: now also R647.1 (-)
- net V_{ACC}-: no longer R647.1 (-)
Other:
- moved on the sheet: R646, R647
Changed lines of the file:
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@@
   (junction (at 165.1 167.64) (diameter 0) (color 0 0 0 0)
   )
-  (junction (at 355.6 241.3) (diameter 0) (color 0 0 0 0)
-  )
   (junction (at 177.8 142.24) (diameter 0) (color 0 0 0 0)
   )
@@
   (junction (at 218.44 109.22) (diameter 0) (color 0 0 0 0)
   )
-  (junction (at 355.6 177.8) (diameter 0) (color 0 0 0 0)
+  (junction (at 330.2 177.8) (diameter 0) (color 0 0 0 0)
   )
   (junction (at 203.2 200.66) (diameter 0) (color 0 0 0 0)
@@
     (stroke (width 0) (type default))
   )
-  (wire (pts (xy 383.54 241.3) (xy 355.6 241.3))
+  (wire (pts (xy 330.2 241.3) (xy 383.54 241.3))
     (stroke (width 0) (type default))
   )
@@
     (stroke (width 0) (type default))
   )
-  (wire (pts (xy 353.06 165.1) (xy 355.6 165.1))
+  (wire (pts (xy 327.66 165.1) (xy 330.2 165.1))
     (stroke (width 0) (type default))
   )
@@
     (stroke (width 0) (type default))
   )
-  (wire (pts (xy 330.2 241.3) (xy 355.6 241.3))
-    (stroke (width 0) (type default))
-  )
   (wire (pts (xy 165.1 167.64) (xy 167.64 167.64))
     (stroke (width 0) (type default))
@@
     (stroke (width 0) (type default))
   )
-  (wire (pts (xy 355.6 177.8) (xy 279.4 177.8))
+  (wire (pts (xy 330.2 177.8) (xy 279.4 177.8))
     (stroke (width 0) (type default))
   )
@@
     (stroke (width 0) (type default))
   )
-  (wire (pts (xy 355.6 189.23) (xy 355.6 241.3))
-    (stroke (width 0) (type default))
-  )
   (wire (pts (xy 292.1 190.5) (xy 292.1 193.04))
     (stroke (width 0) (type default))
@@
     (stroke (width 0) (type default))
   )
+  (wire (pts (xy 354.33 177.8) (xy 355.6 177.8))
+    (stroke (width 0) (type default))
+  )
   (wire (pts (xy 177.8 152.4) (xy 177.8 160.02))
     (stroke (width 0) (type default))
@@
     (stroke (width 0) (type default))
   )
-  (wire (pts (xy 355.6 175.26) (xy 355.6 177.8))
+  (wire (pts (xy 330.2 175.26) (xy 330.2 177.8))
     (stroke (width 0) (type default))
   )
@@
     (stroke (width 0) (type default))
   )
-  (wire (pts (xy 355.6 177.8) (xy 355.6 179.07))
-    (stroke (width 0) (type default))
-  )
   (wire (pts (xy 198.12 91.44) (xy 198.12 93.98))
     (stroke (width 0) (type default))
   )
+  (wire (pts (xy 330.2 177.8) (xy 344.17 177.8))
+    (stroke (width 0) (type default))
+  )
   (wire (pts (xy 205.74 198.12) (xy 205.74 200.66))
     (stroke (width 0) (type default))
@@
     (stroke (width 0) (type default))
   )
-  (wire (pts (xy 355.6 165.1) (xy 355.6 167.64))
+  (wire (pts (xy 330.2 165.1) (xy 330.2 167.64))
     (stroke (width 0) (type default))
   )
@@
     (effects (font (size 1.27 1.27)) (justify left bottom))
   )
-  (global_label "S12_VREF" (shape input) (at 353.06 165.1 180) (fields_autoplaced)
+  (label "S12_I_{SENSE}_N" (at 355.6 177.8 0) (fields_autoplaced)
+    (effects (font (size 1.27 1.27)) (justify left bottom))
+  )
+  (global_label "S12_VREF" (shape input) (at 327.66 165.1 180) (fields_autoplaced)
     (effects (font (size 1.27 1.27)) (justify right))
-    (property "Intersheetrefs" "${INTERSHEET_REFS}" (at 340.8825 165.1 0)
+    (property "Intersheetrefs" "${INTERSHEET_REFS}" (at 315.4825 165.1 0)
       (effects (font (size 1.27 1.27)) (justify right) hide)
     )
@@
     )
   )
-  (symbol (lib_id "Device:R") (at 355.6 171.45 180) (unit 1)
-    (in_bom yes) (on_board yes) (dnp no) (fields_autoplaced)
-    (property "Reference" "R646" (at 358.14 170.18 0)
+  (symbol (lib_id "Device:R") (at 330.2 171.45 180) (unit 1)
+    (in_bom yes) (on_board yes) (dnp no) (fields_autoplaced)
+    (property "Reference" "R646" (at 332.74 170.18 0)
       (effects (font (size 1.27 1.27)) (justify right))
     )
-    (property "Value" "10k" (at 358.14 172.72 0)
+    (property "Value" "10k" (at 332.74 172.72 0)
       (effects (font (size 1.27 1.27)) (justify right))
     )
-    (property "Footprint" "Resistor_SMD:R_0402_1005Metric" (at 357.378 171.45 90)
-      (effects (font (size 1.27 1.27)) hide)
-    )
-    (property "Datasheet" "~" (at 355.6 171.45 0)
+    (property "Footprint" "Resistor_SMD:R_0402_1005Metric" (at 331.978 171.45 90)
+      (effects (font (size 1.27 1.27)) hide)
+    )
+    (property "Datasheet" "~" (at 330.2 171.45 0)
       (effects (font (size 1.27 1.27)) hide)
     )
@@
     )
   )
-  (symbol (lib_id "ProjectEV:Sensor_TMP6131QDYARQ1") (at 355.6 184.15 0) (unit 1)
-    (in_bom yes) (on_board yes) (dnp no) (fields_autoplaced)
-    (property "Reference" "R647" (at 358.14 182.88 0)
-      (effects (font (size 1.27 1.27)) (justify left))
-    )
-    (property "Value" "TMP6131QDYARQ1" (at 358.14 185.42 0)
-      (effects (font (size 1.27 1.27)) (justify left))
-    )
-    (property "Footprint" "ProjectEV:Package_SOD-523_TMP6131QDYARQ1" (at 355.6 184.15 0)
-      (effects (font (size 1.27 1.27)) hide)
-    )
-    (property "Datasheet" "https://www.ti.com/lit/ds/symlink/tmp61-q1.pdf" (at 355.6 195.58 0)
-      (effects (font (size 1.27 1.27)) hide)
-    )
+  (symbol (lib_id "ProjectEV:Sensor_TMP6131QDYARQ1") (at 349.25 177.8 90) (unit 1)
+    (in_bom yes) (on_board yes) (dnp no) (fields_autoplaced)
+    (property "Reference" "R647" (at 349.25 171.45 90)
+      (effects (font (size 1.27 1.27)))
+    )
+    (property "Value" "TMP6131QDYARQ1" (at 349.25 173.99 90)
+      (effects (font (size 1.27 1.27)))
+    )
+    (property "Footprint" "ProjectEV:Package_SOD-523_TMP6131QDYARQ1" (at 349.25 177.8 0)
+      (effects (font (size 1.27 1.27)) hide)
+    )
+    (property "Datasheet" "https://www.ti.com/lit/ds/symlink/tmp61-q1.pdf" (at 360.68 177.8 0)
+      (effects (font (size 1.27 1.27)) hide)
+    )
