File: AMS-board-2024/battery-stack-monitor.kicad_sch (KiCad schematic)
At the start: 71 parts, among them Q115 STD7ANM60N, Q116 2N7002K-AU, Q117 STD7ANM60N, Q118 STD7ANM60N, U23 LM25180-Q1, U24 NCV8711BMTW500TBG, U25 LTC2949, U26 NV24C16SNVLT3G, Y2 ABLS-4.000MHZ-K4T

Commit message: 修正
Connections:
- net S12_I_{SENSE}_N: no longer C364.1, C366.1, C367.1, C369.1
- net V_{ACC}-: now also C364.1, C366.1, C367.1, C369.1
Changed lines of the file:
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@@
   (junction (at 177.8 139.7) (diameter 0) (color 0 0 0 0)
   )
-  (junction (at 220.98 109.22) (diameter 0) (color 0 0 0 0)
-  )
   (junction (at 241.3 38.1) (diameter 0) (color 0 0 0 0)
   )
@@
   (junction (at 254 203.2) (diameter 0) (color 0 0 0 0)
   )
+  (junction (at 218.44 109.22) (diameter 0) (color 0 0 0 0)
+  )
   (junction (at 134.62 190.5) (diameter 0) (color 0 0 0 0)
   )
@@
   (junction (at 355.6 160.02) (diameter 0) (color 0 0 0 0)
   )
-  (junction (at 218.44 109.22) (diameter 0) (color 0 0 0 0)
-  )
   (junction (at 330.2 177.8) (diameter 0) (color 0 0 0 0)
   )
@@
   )
   (junction (at 292.1 241.3) (diameter 0) (color 0 0 0 0)
+  )
+  (junction (at 254 109.22) (diameter 0) (color 0 0 0 0)
   )
   (junction (at 134.62 203.2) (diameter 0) (color 0 0 0 0)
@@
     (stroke (width 0) (type default))
   )
-  (wire (pts (xy 218.44 109.22) (xy 220.98 109.22))
-    (stroke (width 0) (type default))
-  )
   (wire (pts (xy 200.66 93.98) (xy 200.66 99.06))
     (stroke (width 0) (type default))
@@
     (stroke (width 0) (type default))
   )
+  (wire (pts (xy 218.44 109.22) (xy 254 109.22))
+    (stroke (width 0) (type default))
+  )
   (wire (pts (xy 217.17 129.54) (xy 218.44 129.54))
     (stroke (width 0) (type default))
@@
     (stroke (width 0) (type default))
   )
+  (wire (pts (xy 254 109.22) (xy 254 127))
+    (stroke (width 0) (type default))
+  )
   (wire (pts (xy 228.6 38.1) (xy 241.3 38.1))
     (stroke (width 0) (type default))
@@
     (stroke (width 0) (type default))
   )
-  (wire (pts (xy 220.98 99.06) (xy 220.98 109.22))
+  (wire (pts (xy 220.98 99.06) (xy 220.98 132.08))
     (stroke (width 0) (type default))
   )
@@
     (stroke (width 0) (type default))
   )
-  (wire (pts (xy 220.98 109.22) (xy 220.98 132.08))
-    (stroke (width 0) (type default))
-  )
   (wire (pts (xy 152.4 38.1) (xy 152.4 40.64))
     (stroke (width 0) (type default))
@@
     (stroke (width 0) (type default))
   )
-  (wire (pts (xy 254 76.2) (xy 254 127))
-    (stroke (width 0) (type default))
-  )
+  (wire (pts (xy 254 76.2) (xy 254 109.22))
+    (stroke (width 0) (type default))
+  )

Commit message: 修正
Connections:
- net S12_I_{SENSE}_N: no longer U25.26 (IOVCC)
- net V_{ACC}-: now also U25.26 (IOVCC)
Changed lines of the file:
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@@
   (junction (at 228.6 48.26) (diameter 0) (color 0 0 0 0)
   )
-  (junction (at 228.6 99.06) (diameter 0) (color 0 0 0 0)
-  )
   (junction (at 228.6 63.5) (diameter 0) (color 0 0 0 0)
   )
@@
   )
   (junction (at 266.7 38.1) (diameter 0) (color 0 0 0 0)
+  )
+  (junction (at 254 142.24) (diameter 0) (color 0 0 0 0)
   )
   (junction (at 317.5 127) (diameter 0) (color 0 0 0 0)
@@
     (stroke (width 0) (type default))
   )
-  (wire (pts (xy 228.6 99.06) (xy 241.3 99.06))
-    (stroke (width 0) (type default))
-  )
   (wire (pts (xy 231.14 170.18) (xy 226.06 170.18))
     (stroke (width 0) (type default))
@@
     (stroke (width 0) (type default))
   )
-  (wire (pts (xy 226.06 142.24) (xy 228.6 142.24))
-    (stroke (width 0) (type default))
-  )
   (wire (pts (xy 330.2 215.9) (xy 332.74 215.9))
     (stroke (width 0) (type default))
@@
     (stroke (width 0) (type default))
   )
-  (wire (pts (xy 220.98 99.06) (xy 228.6 99.06))
+  (wire (pts (xy 220.98 99.06) (xy 241.3 99.06))
     (stroke (width 0) (type default))
   )
@@
     (stroke (width 0) (type default))
   )
-  (wire (pts (xy 228.6 99.06) (xy 228.6 142.24))
-    (stroke (width 0) (type default))
-  )
   (wire (pts (xy 76.2 38.1) (xy 76.2 63.5))
     (stroke (width 0) (type default))
@@
     (stroke (width 0) (type default))
   )
+  (wire (pts (xy 226.06 142.24) (xy 254 142.24))
+    (stroke (width 0) (type default))
+  )

Commit message: アノテーションし直し
Parts:
- renumbered C353 to C364, C354 to C365, C355 to C366, C356 to C367, C357 to C368, C358 to C369, C359 to C370, C360 to C371, C361 to C372, C362 to C373, C363 to C374, C364 to C375, C379 to C376, C365 to C377, C366 to C378, C378 to C379, C367 to C380, C368 to C381, C369 to C382, C371 to C383, C370 to C384, C373 to C385, C372 to C386, C375 to C387, C374 to C388, C376 to C389, C377 to C390, L22 to L18, R622 to R621, R623 to R622, R624 to R623, R625 to R624, R626 to R625, R627 to R626, R628 to R627, R629 to R628, R612 to R629, R636 to R634, R637 to R635, R634 to R636, R635 to R637, R646 to R643, R643 to R644, R644 to R645, R647 to R646, R645 to R647, U23 to U22, U25 to U23, U26 to U25
